File: AUDIO.sch (KiCad schematic (older format))
At the start: 54 parts, among them J206 Conn_02x06, J207 Conn_02x03, U207 WM8731-Audio, U208 TPS79533, Y203 12.288MHz

Commit message: add cached symbols to local library
Parts:
- TRS204, TRS205, TRS206: symbol Connector:AudioJack4_Switch-Connector -> OTTOdiy_SMD-library:AudioJack4_Switch-Connector-Connector
- U207: symbol Audio:WM8731-Audio -> OTTOdiy_SMD-library:WM8731-Audio-Audio
- U208: symbol Regulator_Linear:TPS79533 -> OTTOdiy_SMD-library:TPS79533-Regulator_Linear
Changed lines of the file:
@@
 EESchema Schematic File Version 4
-LIBS:OTTOdiy_SMD-cache
 EELAYER 30 0
 EELAYER END
@@
 	5000 3150 5200 3150
 $Comp
-L Audio:WM8731-Audio U207
+L OTTOdiy_SMD-library:WM8731-Audio-Audio U207
 U 1 1 5DEEB139
 P 3700 2000
@@
 $EndComp
 $Comp
-L Connector:AudioJack4_Switch-Connector TRS206
+L OTTOdiy_SMD-library:AudioJack4_Switch-Connector-Connector TRS206
 U 1 1 5DF17A71
 P 10350 2950
@@
 $EndComp
 $Comp
-L Connector:AudioJack4_Switch-Connector TRS204
+L OTTOdiy_SMD-library:AudioJack4_Switch-Connector-Connector TRS204
 U 1 1 5DF1C677
 P 10350 1050
@@
 $EndComp
 $Comp
-L Connector:AudioJack4_Switch-Connector TRS205
+L OTTOdiy_SMD-library:AudioJack4_Switch-Connector-Connector TRS205
 U 1 1 5DF1DA7D
 P 10350 2000
@@
 $EndComp
 $Comp
-L Regulator_Linear:TPS79533 U208
+L OTTOdiy_SMD-library:TPS79533-Regulator_Linear U208
 U 1 1 5E2DC32B
 P 4950 6750

Commit message: PWR entry, ESD, JTAG, PU/PDs modified. Review pass 1
Parts:
- added D? (x6): 5V, symbol Device:D_TVS_ALT
Connections:
- wire segments 195 -> 214
Changed lines of the file:
@@
 Text Label 8950 2950 0    50   ~ 0
 HP_OUT_R
-Wire Wire Line
-	8950 2950 10000 2950
-Wire Wire Line
-	8950 3150 10000 3150
 NoConn ~ 10000 950
 Wire Wire Line
@@
 Text Label 8950 1050 0    50   ~ 0
 LINE_IN_R
-Wire Wire Line
-	8950 1250 10000 1250
-Wire Wire Line
-	8950 1050 10000 1050
 NoConn ~ 10000 1350
 NoConn ~ 10000 1150
@@
 LINE_OUT_R
 NoConn ~ 10000 1700
-Wire Wire Line
-	8950 2200 10000 2200
-Wire Wire Line
-	8950 2000 10000 2000
 Wire Wire Line
 	9900 1800 10000 1800
@@
 I2S_DOUT*
 $Comp
-L power:GNDA #PWR?
+L power:GNDA #PWR0101
 U 1 1 5DF89554
 P 3500 6250
-F 0 "#PWR?" H 3500 6000 50  0001 C CNN
+F 0 "#PWR0101" H 3500 6000 50  0001 C CNN
 F 1 "GNDA" V 3505 6122 50  0000 R CNN
 F 2 "" H 3500 6250 50  0001 C CNN
@@
 AR Path="/5D186267/5D1201D8/5DB14620/5DF89B24" Ref="#PWR?"  Part="1"
 AR Path="/5D186267/5D1201D8/5D12037D/5DF89B24" Ref="#PWR?"  Part="1"
-AR Path="/5C4408C6/5DF89B24" Ref="#PWR?"  Part="1"
-F 0 "#PWR?" H 3600 6000 50  0001 C CNN
+AR Path="/5C4408C6/5DF89B24" Ref="#PWR0102"  Part="1"
+F 0 "#PWR0102" H 3600 6000 50  0001 C CNN
 F 1 "GND" V 3605 6122 50  0000 R CNN
 F 2 "" H 3600 6250 50  0001 C CNN
@@
 Wire Wire Line
 	3500 6250 3600 6250
+$Comp
+L Device:D_TVS_ALT D?
+U 1 1 5E6966BE
+P 8400 1500
+F 0 "D?" V 8354 1579 50  0000 L CNN
+F 1 "5V" V 8445 1579 50  0000 L CNN
+F 2 "" H 8400 1500 50  0001 C CNN
+F 3 "~" H 8400 1500 50  0001 C CNN
+	1    8400 1500
+	0    1    1    0
+$EndComp
+$Comp
+L Device:D_TVS_ALT D?
+U 1 1 5E69A1DF
+P 7800 1500
+F 0 "D?" V 7754 1579 50  0000 L CNN
+F 1 "5V" V 7845 1579 50  0000 L CNN
+F 2 "" H 7800 1500 50  0001 C CNN
+F 3 "~" H 7800 1500 50  0001 C CNN
+	1    7800 1500
+	0    1    1    0
+$EndComp
+$Comp
+L Device:D_TVS_ALT D?
+U 1 1 5E69B188
+P 7800 2400
+F 0 "D?" V 7754 2479 50  0000 L CNN
+F 1 "5V" V 7845 2479 50  0000 L CNN
+F 2 "" H 7800 2400 50  0001 C CNN
+F 3 "~" H 7800 2400 50  0001 C CNN
+	1    7800 2400
+	0    1    1    0
+$EndComp
+$Comp
+L Device:D_TVS_ALT D?
+U 1 1 5E69BAA0
+P 8400 2400
+F 0 "D?" V 8354 2479 50  0000 L CNN
+F 1 "5V" V 8445 2479 50  0000 L CNN
+F 2 "" H 8400 2400 50  0001 C CNN
+F 3 "~" H 8400 2400 50  0001 C CNN
+	1    8400 2400
+	0    1    1    0
+$EndComp
+$Comp
+L Device:D_TVS_ALT D?
+U 1 1 5E69D8F4
+P 8350 3350
+F 0 "D?" V 8304 3429 50  0000 L CNN
+F 1 "5V" V 8395 3429 50  0000 L CNN
+F 2 "" H 8350 3350 50  0001 C CNN
+F 3 "~" H 8350 3350 50  0001 C CNN
+	1    8350 3350
+	0    1    1    0
+$EndComp
+$Comp
+L Device:D_TVS_ALT D?
+U 1 1 5E69E1BB
+P 7800 3350
+F 0 "D?" V 7754 3429 50  0000 L CNN
+F 1 "5V" V 7845 3429 50  0000 L CNN
+F 2 "" H 7800 3350 50  0001 C CNN
+F 3 "~" H 7800 3350 50  0001 C CNN
+	1    7800 3350
+	0    1    1    0
+$EndComp
+Wire Wire Line
+	7800 1050 7800 1350
+Wire Wire Line
+	7800 1050 10000 1050
+Wire Wire Line
+	8400 1350 8400 1250
+Wire Wire Line
+	8400 1250 10000 1250
+Wire Wire Line
+	7800 2000 7800 2250
+Wire Wire Line
+	7800 2000 10000 2000
+Wire Wire Line
+	8400 2200 8400 2250
+Wire Wire Line
+	8400 2200 10000 2200
+Wire Wire Line
+	7800 2950 7800 3200
+Wire Wire Line
+	7800 2950 10000 2950
+$Comp
+L power:GNDA #PWR?
+U 1 1 5E6EB4B6
+P 8400 1700
+F 0 "#PWR?" H 8400 1450 50  0001 C CNN
+F 1 "GNDA" H 8405 1527 50  0000 C CNN
+F 2 "" H 8400 1700 50  0001 C CNN
+F 3 "" H 8400 1700 50  0001 C CNN
+	1    8400 1700
+	1    0    0    -1
+$EndComp
+$Comp
+L power:GNDA #PWR?
+U 1 1 5E760195
+P 7800 1700
+F 0 "#PWR?" H 7800 1450 50  0001 C CNN
+F 1 "GNDA" H 7805 1527 50  0000 C CNN
+F 2 "" H 7800 1700 50  0001 C CNN
+F 3 "" H 7800 1700 50  0001 C CNN
+	1    7800 1700
+	1    0    0    -1
+$EndComp
+$Comp
+L power:GNDA #PWR?
+U 1 1 5E7604A1
+P 7800 2600
+F 0 "#PWR?" H 7800 2350 50  0001 C CNN
+F 1 "GNDA" H 7805 2427 50  0000 C CNN
+F 2 "" H 7800 2600 50  0001 C CNN
+F 3 "" H 7800 2600 50  0001 C CNN
+	1    7800 2600
+	1    0    0    -1
+$EndComp
+$Comp
+L power:GNDA #PWR?
+U 1 1 5E76073E
+P 8400 2600
+F 0 "#PWR?" H 8400 2350 50  0001 C CNN
+F 1 "GNDA" H 8405 2427 50  0000 C CNN
+F 2 "" H 8400 2600 50  0001 C CNN
+F 3 "" H 8400 2600 50  0001 C CNN
+	1    8400 2600
+	1    0    0    -1
+$EndComp
+$Comp
+L power:GNDA #PWR?
+U 1 1 5E760B0D
+P 8350 3550
+F 0 "#PWR?" H 8350 3300 50  0001 C CNN
+F 1 "GNDA" H 8355 3377 50  0000 C CNN
+F 2 "" H 8350 3550 50  0001 C CNN
+F 3 "" H 8350 3550 50  0001 C CNN
+	1    8350 3550
+	1    0    0    -1
+$EndComp
+$Comp
+L power:GNDA #PWR?
+U 1 1 5E7610A7
+P 7800 3550
+F 0 "#PWR?" H 7800 3300 50  0001 C CNN
+F 1 "GNDA" H 7805 3377 50  0000 C CNN
+F 2 "" H 7800 3550 50  0001 C CNN
+F 3 "" H 7800 3550 50  0001 C CNN
+	1    7800 3550
+	1    0    0    -1
+$EndComp
+Wire Wire Line
+	8350 3150 8350 3200
+Wire Wire Line
+	8350 3150 10000 3150
+Wire Wire Line
+	8350 3500 8350 3550
+Wire Wire Line
+	7800 3500 7800 3550
+Wire Wire Line
+	8400 2550 8400 2600
+Wire Wire Line
+	7800 2550 7800 2600
+Wire Wire Line
+	7800 1650 7800 1700
+Wire Wire Line
+	8400 1650 8400 1700
+Wire Wire Line
+	7800 1050 7600 1050
+Connection ~ 7800 1050
+Connection ~ 8400 1250
+Wire Wire Line
+	8200 1250 8400 1250
+Wire Wire Line
+	7800 2000 7600 2000
+Connection ~ 7800 2000
+Wire Wire Line
+	8400 2200 8200 2200
+Connection ~ 8400 2200
+Wire Wire Line
+	7800 2950 7600 2950
+Connection ~ 7800 2950
+Wire Wire Line
+	8350 3150 8200 3150
+Connection ~ 8350 3150
+Wire Wire Line
+	1200 2300 750  2300
 $EndSCHEMATC
