File: KiCad/MCU.sch (KiCad schematic (older format))
At the start: 47 parts, among them J202 Conn_02x03, J203 Conn_02x05, J204 Conn_02x05, J205 Conn_02x04, SW201 SW_Push, SW202 SW_DIP_x02, U201 TPS79533, U7 STM32F407VGTx, Y201 8MHz, Y202 32.768kHz

Commit message: roll in changes from Bastian
Parts:
- removed C?: 1000pF, symbol Device:C
- removed J?: Conn_ARM_JTAG_SWD_20, symbol Connector:Conn_ARM_JTAG_SWD_20
- added C?: 100nF, Capacitor_SMD:C_0805_2012Metric_Pad1.15x1.40mm_HandSolder_marked, symbol Device:C
- added J?: Conn_ARM_JTAG_SWD_10, symbol Connector:Conn_ARM_JTAG_SWD_10
- R?: value 10k -> 40.2k
Connections:
- net labels added: (F427)_SAI1_FS_A, (F427)_SAI1_MCLK_A, (F427)_SAI1_SCK_A, (F427)_SAI1_SD_A, (F427)_SAI1_SD_B, +3V3A_MCU
- net labels removed: ICP_SWCLK, ICP_SWDIO
- wire segments 305 -> 313
- no-connect marks 6 -> 2

Commit message: added buck/boost power supply for 5V rail
Connections:
- net labels added: 5V_REG_IOUT, PWR_PWM_SYNC
- wire segments 313 -> 315
Changed lines of the file:
@@
 AR Path="/5DDA96E4" Ref="U7"  Part="1"
 AR Path="/5C4320DF/5DDA96E4" Ref="U202"  Part="1"
-F 0 "U202" H 8150 4061 50  0000 C CNN
-F 1 "STM32F407VGTx" H 8750 4050 50  0000 C CNN
+F 0 "U202" H 8750 4100 50  0000 C CNN
+F 1 "STM32F407VGTx" H 8950 4000 50  0000 C CNN
 F 2 "Package_QFP:LQFP-100_14x14mm_P0.5mm" H 7450 4350 50  0001 R CNN
 F 3 "http://www.st.com/st-web-ui/static/active/en/resource/technical/document/datasheet/DM00037051.pdf" H 8150 6950 50  0001 C CNN
@@
 Wire Wire Line
 	5850 6850 6950 6850
+Wire Wire Line
+	6950 8750 6650 8750
+Wire Wire Line
+	9350 8150 10000 8150
+Text GLabel 10000 8150 2    50   Input ~ 0
+5V_REG_IOUT
+Text GLabel 6650 8750 0    50   Input ~ 0
+PWR_PWM_SYNC
 $EndSCHEMATC

Commit message: added power switching and extra pulls for programming lines
Parts:
- removed C208, C209: 10µF, Capacitor_SMD:C_0805_2012Metric_Pad1.15x1.40mm_HandSolder, symbol Device:C
- removed C76: 100nF, Capacitor_SMD:C_0805_2012Metric_Pad1.15x1.40mm_HandSolder_marked, symbol Device:C
- removed R?: 0, symbol Device:R
- removed R?: 100k, symbol Device:R
- removed U201: TPS79533, Package_TO_SOT_SMD:SOT-223-6, symbol OTTOdiy_SMD-library:TPS79533-Regulator_Linear
- added R? (x3): 10k, symbol Device:R
Connections:
- net labels added: ICP_SWCLK, ICP_SWDIO
- net labels removed: +5V_MCU
- wire segments 315 -> 308

Commit message: connected unconnected signals and MIDI to spare MCU UART
Parts:
- gave numbers to parts that had none: 8
Connections:
- net labels added: 5V_PWM_SYNC, HP_SENSE, MIDI_IN, MIDI_OUT, PI_PWR_EN
- net labels removed: MAIN_POWER, PWR_PWM_SYNC
- wire segments 308 -> 306
Changed lines of the file:
@@
 I2C_SDA
 Wire Wire Line
-	13850 8850 15000 8850
-Text GLabel 13850 8850 0    50   Output ~ 0
-MAIN_POWER
-Wire Wire Line
 	10200 5650 9350 5650
 Wire Wire Line
 	10200 5750 9350 5750
-Text GLabel 14600 8550 2    50   Output ~ 0
+Text GLabel 5850 7750 0    50   Input ~ 0
 BL_PWM
 Wire Wire Line
-	14600 8550 13850 8550
-Wire Wire Line
 	10500 8850 9350 8850
-Wire Wire Line
-	15000 8700 13850 8700
 Text Label 10500 6450 2    50   ~ 0
 BOOT1
@@
 Wire Wire Line
 	6950 3950 7050 3950
-Text GLabel 15100 9450 2    50   Input ~ 0
+Text GLabel 9900 4550 2    50   Input ~ 0
 PWR_BUTTON
 Wire Wire Line
-	14600 9000 13850 9000
-Wire Wire Line
-	15100 9450 13850 9450
-Wire Wire Line
-	14600 9150 13850 9150
-Wire Wire Line
-	14600 9300 13850 9300
+	9900 4550 9350 4550
 Text Label 7650 3950 2    50   ~ 0
 VBAT
@@
 Text Label 10200 5750 2    50   ~ 0
 USBD_P
-Text Label 15000 8700 2    50   ~ 0
+Text Label 12040 8750 2    50   ~ 0
 BRIGHTNESS
 Text Label 10500 8850 2    50   ~ 0
@@
 	10000 7350 9350 7350
 Wire Wire Line
-	10500 9150 9350 9150
-Wire Wire Line
 	9350 6050 10500 6050
-Wire Wire Line
-	10500 8950 9350 8950
-Wire Wire Line
-	9350 9050 10500 9050
 Text Label 10500 6050 2    50   ~ 0
 SPI_CS_MCU_LED
-Text Label 10500 8950 2    50   ~ 0
-SPI_SCLK_MCU
-Text Label 10500 9050 2    50   ~ 0
-SPI_MISO_MCU
-Text Label 10500 9150 2    50   ~ 0
-SPI_MOSI_MCU
 Wire Wire Line
 	10500 6750 9350 6750
@@
 SPI_MISO_MCU
 Text Label 10500 6750 2    50   ~ 0
-SPI_MOSI_MCU
-Wire Wire Line
-	10500 7750 9350 7750
-Wire Wire Line
-	10500 7550 9350 7550
-Wire Wire Line
-	9350 7650 10500 7650
-Text Label 10500 7450 2    50   ~ 0
-SPI_CS_MCU_LED
-Text Label 10500 7550 2    50   ~ 0
-SPI_SCLK_MCU
-Text Label 10500 7650 2    50   ~ 0
-SPI_MISO_MCU
-Text Label 10500 7750 2    50   ~ 0
 SPI_MOSI_MCU
 Connection ~ 11150 3450
@@
 Wire Notes Line
 	3400 10950 750  10950
-Text GLabel 14600 9000 2    50   BiDi ~ 0
+Text GLabel 5930 8050 0    50   BiDi ~ 0
 TRIGGER1
-Text GLabel 14600 9150 2    50   BiDi ~ 0
+Text GLabel 5930 8150 0    50   BiDi ~ 0
 TRIGGER2
-Text GLabel 14600 9300 2    50   BiDi ~ 0
+Text GLabel 5930 8250 0    50   BiDi ~ 0
 TRIGGER3
 $Comp
@@
 	14350 5550 14350 5750
 $Comp
-L power:GND #PWR?
+L power:GND #PWR0103
 U 1 1 5E0C5791
 P 14350 7050
-F 0 "#PWR?" H 14350 6800 50  0001 C CNN
+F 0 "#PWR0103" H 14350 6800 50  0001 C CNN
 F 1 "GND" H 14355 6877 50  0000 C CNN
 F 2 "" H 14350 7050 50  0001 C CNN
@@
 	6850 4300 6850 4550
 $Comp
-L Device:R R?
+L Device:R R8
 U 1 1 5E39B322
 P 11750 8050
-F 0 "R?" V 11957 8050 50  0000 C CNN
+F 0 "R8" V 11957 8050 50  0000 C CNN
 F 1 "40.2k" V 11866 8050 50  0000 C CNN
 F 2 "" V 11680 8050 50  0001 C CNN
@@
 $EndComp
 $Comp
-L Device:R R?
+L Device:R R5
 U 1 1 5E39D1BD
 P 11300 8250
-F 0 "R?" H 11370 8296 50  0000 L CNN
+F 0 "R5" H 11370 8296 50  0000 L CNN
 F 1 "10k" H 11370 8205 50  0000 L CNN
 F 2 "" V 11230 8250 50  0001 C CNN
@@
 	11300 8400 11300 8450
 $Comp
-L Device:Ferrite_Bead FB?
+L Device:Ferrite_Bead FB1
 U 1 1 5E433262
 P 6500 3200
-F 0 "FB?" V 6226 3200 50  0000 C CNN
+F 0 "FB1" V 6226 3200 50  0000 C CNN
 F 1 "1kΩ@100Mhz" V 6317 3200 50  0000 C CNN
 F 2 "" V 6430 3200 50  0001 C CNN
@@
 $EndComp
 $Comp
-L Connector:Conn_ARM_JTAG_SWD_10 J?
+L Connector:Conn_ARM_JTAG_SWD_10 J1
 U 1 1 5DEBF301
 P 14350 6350
-F 0 "J?" H 13906 6396 50  0000 R CNN
+F 0 "J1" H 13906 6396 50  0000 R CNN
 F 1 "Conn_ARM_JTAG_SWD_10" H 13906 6305 50  0000 R CNN
 F 2 "" H 14350 6350 50  0001 C CNN
@@
 $EndComp
 $Comp
-L power:GND #PWR?
+L power:GND #PWR0104
 U 1 1 5DF55D36
 P 14550 7050
-F 0 "#PWR?" H 14550 6800 50  0001 C CNN
+F 0 "#PWR0104" H 14550 6800 50  0001 C CNN
 F 1 "GND" H 14555 6877 50  0000 C CNN
 F 2 "" H 14550 7050 50  0001 C CNN
@@
 NoConn ~ 13850 6550
 $Comp
-L Device:C C?
+L Device:C C57
 U 1 1 5E00B522
 P 10800 8250
-AR Path="/5C4320DF/5E00B522" Ref="C?"  Part="1"
+AR Path="/5C4320DF/5E00B522" Ref="C57"  Part="1"
 AR Path="/5C4320DF/5DB999B7/5E00B522" Ref="C?"  Part="1"
-F 0 "C?" H 10685 8204 50  0000 R CNN
+F 0 "C57" H 10685 8204 50  0000 R CNN
 F 1 "100nF" H 10685 8295 50  0000 R CNN
 F 2 "Capacitor_SMD:C_0805_2012Metric_Pad1.15x1.40mm_HandSolder_marked" H 10838 8100 50  0001 C CNN
@@
 $EndComp
 $Comp
-L power:GND #PWR?
+L power:GND #PWR0105
 U 1 1 5E00C6D9
 P 11300 8450
-AR Path="/5C4320DF/5E00C6D9" Ref="#PWR?"  Part="1"
+AR Path="/5C4320DF/5E00C6D9" Ref="#PWR0105"  Part="1"
 AR Path="/5C4320DF/5DB999B7/5E00C6D9" Ref="#PWR?"  Part="1"
-F 0 "#PWR?" H 11300 8200 50  0001 C CNN
+F 0 "#PWR0105" H 11300 8200 50  0001 C CNN
 F 1 "GND" H 11305 8277 50  0000 C CNN
 F 2 "" H 11300 8450 50  0001 C CNN
@@
 $EndComp
 $Comp
-L power:GND #PWR?
+L power:GND #PWR0106
 U 1 1 5E00D36E
 P 10800 8450
-AR Path="/5C4320DF/5E00D36E" Ref="#PWR?"  Part="1"
+AR Path="/5C4320DF/5E00D36E" Ref="#PWR0106"  Part="1"
 AR Path="/5C4320DF/5DB999B7/5E00D36E" Ref="#PWR?"  Part="1"
-F 0 "#PWR?" H 10800 8200 50  0001 C CNN
+F 0 "#PWR0106" H 10800 8200 50  0001 C CNN
 F 1 "GND" H 10805 8277 50  0000 C CNN
 F 2 "" H 10800 8450 50  0001 C CNN
@@
 Connection ~ 10800 8050
 $Comp
-L power:GND #PWR?
+L power:GND #PWR0107
 U 1 1 5E27FCD0
 P 8350 10150
-AR Path="/5C4320DF/5E27FCD0" Ref="#PWR?"  Part="1"
+AR Path="/5C4320DF/5E27FCD0" Ref="#PWR0107"  Part="1"
 AR Path="/5C4320DF/5DB999B7/5E27FCD0" Ref="#PWR?"  Part="1"
-F 0 "#PWR?" H 8350 9900 50  0001 C CNN
+F 0 "#PWR0107" H 8350 9900 50  0001 C CNN
 F 1 "GND" H 8355 9977 50  0000 C CNN
 F 2 "" H 8350 10150 50  0001 C CNN
@@
 	5850 6850 6950 6850
 Wire Wire Line
-	6950 8750 6650 8750
-Wire Wire Line
 	9350 8150 10000 8150
 Text GLabel 10000 8150 2    50   Input ~ 0
 5V_REG_IOUT
-Text GLabel 6650 8750 0    50   Input ~ 0
-PWR_PWM_SYNC
-Wire Wire Line
-	9350 7450 10500 7450
+Text GLabel 6080 7650 0    50   Input ~ 0
+5V_PWM_SYNC
 Text GLabel 12200 5850 2    50   Input ~ 0
 ICP_SWDIO
@@
 	13500 6050 13850 6050
 $Comp
-L Device:R R?
+L Device:R R4
 U 1 1 5E181DA6
 P 6100 4000
-F 0 "R?" H 6170 4045 50  0000 L CNN
+F 0 "R4" H 6170 4045 50  0000 L CNN
 F 1 "10k" H 6170 3955 50  0000 L CNN
 F 2 "" V 6030 4000 50  0001 C CNN
@@
 	6100 4300 6850 4300
 $Comp
-L Device:R R?
+L Device:R R6
 U 1 1 5E183D37
 P 11500 5600
-F 0 "R?" H 11570 5645 50  0000 L CNN
+F 0 "R6" H 11570 5645 50  0000 L CNN
 F 1 "10k" H 11570 5555 50  0000 L CNN
 F 2 "" V 11430 5600 50  0001 C CNN
@@
 $EndComp
 $Comp
-L Device:R R?
+L Device:R R7
 U 1 1 5E185281
 P 11600 6200
-F 0 "R?" H 11670 6245 50  0000 L CNN
+F 0 "R7" H 11670 6245 50  0000 L CNN
 F 1 "10k" H 11670 6155 50  0000 L CNN
 F 2 "" V 11530 6200 50  0001 C CNN
@@
 	11600 5950 12100 5950
 $Comp
-L power:GND #PWR?
+L power:GND #PWR0108
 U 1 1 5E18676D
 P 11600 6450
-F 0 "#PWR?" H 11600 6200 50  0001 C CNN
+F 0 "#PWR0108" H 11600 6200 50  0001 C CNN
 F 1 "GND" H 11605 6277 50  0000 C CNN
 F 2 "" H 11600 6450 50  0001 C CNN
@@
 Wire Wire Line
 	11500 5300 11500 5450
+Wire Wire Line
+	5850 7750 6950 7750
+Wire Wire Line
+	9350 8250 10600 8250
+Wire Wire Line
+	10600 8250 10600 8750
+Wire Wire Line
+	10600 8750 12040 8750
+Wire Wire Line
+	6080 7650 6950 7650
+Wire Wire Line
+	5960 7950 6950 7950
+Wire Wire Line
+	5930 8150 6950 8150
+Wire Wire Line
+	5930 8050 6950 8050
+Wire Wire Line
+	5930 8250 6950 8250
+Text GLabel 5960 7950 0    50   Input ~ 0
+PI_PWR_EN
+Text GLabel 5940 8350 0    50   Input ~ 0
+HP_SENSE
+Wire Wire Line
+	5940 8350 6950 8350
+Text GLabel 10280 5450 2    50   Output ~ 0
+MIDI_OUT
+Text GLabel 10280 5550 2    50   Input ~ 0
+MIDI_IN
+Wire Wire Line
+	9350 5450 10280 5450
+Wire Wire Line
+	9350 5550 10280 5550
 $EndSCHEMATC

Commit message: add all resistor part numbers and create footprint library
Parts:
- R202, R205, R206, R207: value 2k2 -> 2.2k; EstimatedCost(USD) (none) -> $.001525; MPN (none) -> RC0805FR-072K2L; Manufacturer (none) -> Yageo
- R203, R204: EstimatedCost(USD) (none) -> $.001675; MPN (none) -> RC0805FR-0710KL; Manufacturer (none) -> Yageo
- R4, R6, R7: value 10k -> 6.8k; footprint (none) -> Resistor_SMD:R_0805_2012Metric_Pad1.15x1.40mm_HandSolder; EstimatedCost(USD) (none) -> $.003576; MPN (none) -> RC0805FR-076K8L; Manufacturer (none) -> Yageo
- R5: footprint (none) -> Resistor_SMD:R_0805_2012Metric_Pad1.15x1.40mm_HandSolder; EstimatedCost(USD) (none) -> $.001675; MPN (none) -> RC0805FR-0710KL; Manufacturer (none) -> Yageo
- R8: footprint (none) -> Resistor_SMD:R_0805_2012Metric_Pad1.15x1.40mm_HandSolder; EstimatedCost(USD) (none) -> $.001774; MPN (none) -> RC0805FR-0740K2L; Manufacturer (none) -> Yageo
Changed lines of the file:
@@
 P 14950 1100
 F 0 "R202" V 14743 1100 50  0000 C CNN
-F 1 "2k2" V 14834 1100 50  0000 C CNN
+F 1 "2.2k" V 14834 1100 50  0000 C CNN
 F 2 "Resistor_SMD:R_0805_2012Metric_Pad1.15x1.40mm_HandSolder" V 14880 1100 50  0001 C CNN
-F 3 "~" H 14950 1100 50  0001 C CNN
+F 3 "https://datasheet.lcsc.com/szlcsc/YAGEO-RC0805FR-072K2L_C114561.pdf" H 14950 1100 50  0001 C CNN
+F 4 "$.001525" H 14950 1100 50  0001 C CNN "EstimatedCost(USD)"
+F 5 "RC0805FR-072K2L" H 14950 1100 50  0001 C CNN "MPN"
+F 6 "Yageo" H 14950 1100 50  0001 C CNN "Manufacturer"
 	1    14950 1100
 	0    1    1    0
@@
 P 14950 1450
 F 0 "R205" V 14743 1450 50  0000 C CNN
-F 1 "2k2" V 14834 1450 50  0000 C CNN
+F 1 "2.2k" V 14834 1450 50  0000 C CNN
 F 2 "Resistor_SMD:R_0805_2012Metric_Pad1.15x1.40mm_HandSolder" V 14880 1450 50  0001 C CNN
-F 3 "~" H 14950 1450 50  0001 C CNN
+F 3 "https://datasheet.lcsc.com/szlcsc/YAGEO-RC0805FR-072K2L_C114561.pdf" H 14950 1450 50  0001 C CNN
+F 4 "$.001525" H 14950 1450 50  0001 C CNN "EstimatedCost(USD)"
+F 5 "RC0805FR-072K2L" H 14950 1450 50  0001 C CNN "MPN"
+F 6 "Yageo" H 14950 1450 50  0001 C CNN "Manufacturer"
 	1    14950 1450
 	0    1    1    0
@@
 F 1 "10k" H 6880 1495 50  0000 R CNN
 F 2 "Resistor_SMD:R_0805_2012Metric_Pad1.15x1.40mm_HandSolder" V 6880 1450 50  0001 C CNN
-F 3 "~" H 6950 1450 50  0001 C CNN
+F 3 "https://datasheet.lcsc.com/szlcsc/YAGEO-RC0805FR-0710KL_C84376.pdf" H 6950 1450 50  0001 C CNN
+F 4 "$.001675" H 6950 1450 50  0001 C CNN "EstimatedCost(USD)"
+F 5 "RC0805FR-0710KL" H 6950 1450 50  0001 C CNN "MPN"
+F 6 "Yageo" H 6950 1450 50  0001 C CNN "Manufacturer"
 	1    6950 1450
 	-1   0    0    1
@@
 F 1 "10k" H 6530 1495 50  0000 R CNN
 F 2 "Resistor_SMD:R_0805_2012Metric_Pad1.15x1.40mm_HandSolder" V 6530 1450 50  0001 C CNN
-F 3 "~" H 6600 1450 50  0001 C CNN
+F 3 "https://datasheet.lcsc.com/szlcsc/YAGEO-RC0805FR-0710KL_C84376.pdf" H 6600 1450 50  0001 C CNN
+F 4 "$.001675" H 6600 1450 50  0001 C CNN "EstimatedCost(USD)"
+F 5 "RC0805FR-0710KL" H 6600 1450 50  0001 C CNN "MPN"
+F 6 "Yageo" H 6600 1450 50  0001 C CNN "Manufacturer"
 	1    6600 1450
 	-1   0    0    1
@@
 AR Path="/5C4320DF/5C4AB597/5E83B2BF" Ref="R?"  Part="1"
 F 0 "R206" V 15157 1800 50  0000 C CNN
-F 1 "2k2" V 15066 1800 50  0000 C CNN
+F 1 "2.2k" V 15066 1800 50  0000 C CNN
 F 2 "Resistor_SMD:R_0805_2012Metric_Pad1.15x1.40mm_HandSolder" V 14880 1800 50  0001 C CNN
-F 3 "~" H 14950 1800 50  0001 C CNN
+F 3 "https://datasheet.lcsc.com/szlcsc/YAGEO-RC0805FR-072K2L_C114561.pdf" H 14950 1800 50  0001 C CNN
+F 4 "$.001525" H 14950 1800 50  0001 C CNN "EstimatedCost(USD)"
+F 5 "RC0805FR-072K2L" H 14950 1800 50  0001 C CNN "MPN"
+F 6 "Yageo" H 14950 1800 50  0001 C CNN "Manufacturer"
 	1    14950 1800
 	0    -1   -1   0
@@
 AR Path="/5C4320DF/5C4AB597/5E83B2C5" Ref="R?"  Part="1"
 F 0 "R207" V 14743 2150 50  0000 C CNN
-F 1 "2k2" V 14834 2150 50  0000 C CNN
+F 1 "2.2k" V 14834 2150 50  0000 C CNN
 F 2 "Resistor_SMD:R_0805_2012Metric_Pad1.15x1.40mm_HandSolder" V 14880 2150 50  0001 C CNN
-F 3 "~" H 14950 2150 50  0001 C CNN
+F 3 "https://datasheet.lcsc.com/szlcsc/YAGEO-RC0805FR-072K2L_C114561.pdf" H 14950 2150 50  0001 C CNN
+F 4 "$.001525" H 14950 2150 50  0001 C CNN "EstimatedCost(USD)"
+F 5 "RC0805FR-072K2L" H 14950 2150 50  0001 C CNN "MPN"
+F 6 "Yageo" H 14950 2150 50  0001 C CNN "Manufacturer"
 	1    14950 2150
 	0    1    1    0
@@
 F 0 "R8" V 11957 8050 50  0000 C CNN
 F 1 "40.2k" V 11866 8050 50  0000 C CNN
-F 2 "" V 11680 8050 50  0001 C CNN
-F 3 "~" H 11750 8050 50  0001 C CNN
+F 2 "Resistor_SMD:R_0805_2012Metric_Pad1.15x1.40mm_HandSolder" V 11680 8050 50  0001 C CNN
+F 3 "https://datasheet.lcsc.com/szlcsc/YAGEO-RC0805FR-0740K2L_C273827.pdf" H 11750 8050 50  0001 C CNN
+F 4 "RC0805FR-0740K2L" H 11750 8050 50  0001 C CNN "MPN"
+F 5 "$.001774" H 11750 8050 50  0001 C CNN "EstimatedCost(USD)"
+F 6 "Yageo" H 11750 8050 50  0001 C CNN "Manufacturer"
 	1    11750 8050
 	0    -1   -1   0
@@
 F 0 "R5" H 11370 8296 50  0000 L CNN
 F 1 "10k" H 11370 8205 50  0000 L CNN
-F 2 "" V 11230 8250 50  0001 C CNN
-F 3 "~" H 11300 8250 50  0001 C CNN
+F 2 "Resistor_SMD:R_0805_2012Metric_Pad1.15x1.40mm_HandSolder" V 11230 8250 50  0001 C CNN
+F 3 "https://datasheet.lcsc.com/szlcsc/YAGEO-RC0805FR-0710KL_C84376.pdf" H 11300 8250 50  0001 C CNN
+F 4 "$.001675" H 11300 8250 50  0001 C CNN "EstimatedCost(USD)"
+F 5 "RC0805FR-0710KL" H 11300 8250 50  0001 C CNN "MPN"
+F 6 "Yageo" H 11300 8250 50  0001 C CNN "Manufacturer"
 	1    11300 8250
 	1    0    0    -1
@@
 P 6100 4000
 F 0 "R4" H 6170 4045 50  0000 L CNN
-F 1 "10k" H 6170 3955 50  0000 L CNN
-F 2 "" V 6030 4000 50  0001 C CNN
-F 3 "~" H 6100 4000 50  0001 C CNN
+F 1 "6.8k" H 6170 3955 50  0000 L CNN
+F 2 "Resistor_SMD:R_0805_2012Metric_Pad1.15x1.40mm_HandSolder" V 6030 4000 50  0001 C CNN
+F 3 "https://datasheet.lcsc.com/szlcsc/YAGEO-RC0805FR-076K8L_C114550.pdf" H 6100 4000 50  0001 C CNN
+F 4 "$.003576" H 6100 4000 50  0001 C CNN "EstimatedCost(USD)"
+F 5 "RC0805FR-076K8L" H 6100 4000 50  0001 C CNN "MPN"
+F 6 "Yageo" H 6100 4000 50  0001 C CNN "Manufacturer"
 	1    6100 4000
 	1    0    0    -1
@@
 P 11500 5600
 F 0 "R6" H 11570 5645 50  0000 L CNN
-F 1 "10k" H 11570 5555 50  0000 L CNN
-F 2 "" V 11430 5600 50  0001 C CNN
-F 3 "~" H 11500 5600 50  0001 C CNN
+F 1 "6.8k" H 11570 5555 50  0000 L CNN
+F 2 "Resistor_SMD:R_0805_2012Metric_Pad1.15x1.40mm_HandSolder" V 11430 5600 50  0001 C CNN
+F 3 "https://datasheet.lcsc.com/szlcsc/YAGEO-RC0805FR-076K8L_C114550.pdf" H 11500 5600 50  0001 C CNN
+F 4 "$.003576" H 11500 5600 50  0001 C CNN "EstimatedCost(USD)"
+F 5 "RC0805FR-076K8L" H 11500 5600 50  0001 C CNN "MPN"
+F 6 "Yageo" H 11500 5600 50  0001 C CNN "Manufacturer"
 	1    11500 5600
 	1    0    0    -1
@@
 P 11600 6200
 F 0 "R7" H 11670 6245 50  0000 L CNN
-F 1 "10k" H 11670 6155 50  0000 L CNN
-F 2 "" V 11530 6200 50  0001 C CNN
-F 3 "~" H 11600 6200 50  0001 C CNN
+F 1 "6.8k" H 11670 6155 50  0000 L CNN
+F 2 "Resistor_SMD:R_0805_2012Metric_Pad1.15x1.40mm_HandSolder" V 11530 6200 50  0001 C CNN
+F 3 "https://datasheet.lcsc.com/szlcsc/YAGEO-RC0805FR-076K8L_C114550.pdf" H 11600 6200 50  0001 C CNN
+F 4 "$.003576" H 11600 6200 50  0001 C CNN "EstimatedCost(USD)"
+F 5 "RC0805FR-076K8L" H 11600 6200 50  0001 C CNN "MPN"
+F 6 "Yageo" H 11600 6200 50  0001 C CNN "Manufacturer"
 	1    11600 6200
 	1    0    0    -1

Commit message: added part numbers for capacitors and crystals
Parts:
- removed C206, C207: 12.5pF, Capacitor_SMD:C_0805_2012Metric_Pad1.15x1.40mm_HandSolder, symbol Device:C
- added C96, C97: 15pF, Capacitor_SMD:C_0805_2012Metric_Pad1.15x1.40mm_HandSolder, symbol Device:C
- BT201: footprint Battery:QJ1220-2SMT -> OTTO_Footprints_Lib:QJ1220-2SMT; EstimatedCost(USD) (none) -> $0.186364; MPN (none) -> CR1220-2; Manufacturer (none) -> Q&J
- C204, C205: value 20pF -> 30pF
- C211: value 4.7µF -> 4.7uF
- C218, C219, C223: value 1µF -> 1uF
- C221, C222: value 2.2µF -> 2.2uF
- C226: value 10µF -> 10uF
- C48, C49, C50, C51, C52, C53, C54, C55, C56, C57: footprint Capacitor_SMD:C_0805_2012Metric_Pad1.15x1.40mm_HandSolder_marked -> Capacitor_SMD:C_0805_2012Metric_Pad1.15x1.40mm_HandSolder; EstimatedCost(USD) (none) -> $0.017724; MPN (none) -> CL21B104JBCNNNC; Manufacturer (none) -> Samsung Electro-Mechanics
- Y201: footprint Crystal:Crystal_HC49-U_Vertical -> Crystal:Crystal_SMD_HC49-SD_HandSoldering; EstimatedCost(USD) (none) -> $0.075854; MPN (none) -> X49SM8MSD2SC; Manufacturer (none) -> Yangxing Tech
- Y202: footprint Crystal:Crystal_DS26_D2.0mm_L6.0mm_Horizontal -> Crystal:Crystal_SMD_SeikoEpson_MC306-4Pin_8.0x3.2mm_HandSoldering; EstimatedCost(USD) (none) -> $0.237879; MPN (none) -> Q13MC3061000300; Manufacturer (none) -> Seiko Epson
