File: KiCad/MCU.sch (KiCad schematic (older format))
At the start: 44 parts, among them J1 Conn_ARM_JTAG_SWD_10, J202 Conn_02x03, J203 Conn_02x05, J204 Conn_02x05, J205 Conn_02x04, SW201 SW_Push, SW202 SW_DIP_x02, U7 STM32F407VGTx, Y201 8MHz, Y202 32.768kHz

Commit message: more part numbers added: audio caps
Parts:
- C204, C205: EstimatedCost(USD) (none) -> $0.005588; MPN (none) -> CC0805JRNPO9BN300; Manufacturer (none) -> Yageo
- C211: EstimatedCost(USD) (none) -> $0.031439; MPN (none) -> CL21B475KAFNNNE; Manufacturer (none) -> Samsung Electro-Mechanics
- C218, C219, C223: EstimatedCost(USD) (none) -> $0.067176; MPN (none) -> CL21B105KBFVPNE; Manufacturer (none) -> Samsung Electro-Mechanics
- C221, C222: EstimatedCost(USD) (none) -> $0.01848; MPN (none) -> CL21B225KAFNNNE; Manufacturer (none) -> Samsung Electro-Mechanics
- C226: EstimatedCost(USD) (none) -> $0.041113; MPN (none) -> CL21B106KOQNNNE; Manufacturer (none) -> Samsung Electro-Mechanics
- C96, C97: EstimatedCost(USD) (none) -> $0.00985; MPN (none) -> CL21C150JBANNNC; Manufacturer (none) -> Samsung Electro-Mechanics
Changed lines of the file:
@@
 F 1 "4.7uF" H 8265 3155 50  0000 L CNN
 F 2 "Capacitor_SMD:C_0805_2012Metric_Pad1.15x1.40mm_HandSolder" H 8188 3050 50  0001 C CNN
-F 3 "~" H 8150 3200 50  0001 C CNN
+F 3 "https://datasheet.lcsc.com/szlcsc/Samsung-Electro-Mechanics-CL21B475KAFNNNE_C98195.pdf" H 8150 3200 50  0001 C CNN
+F 4 "$0.031439" H 8150 3200 50  0001 C CNN "EstimatedCost(USD)"
+F 5 "CL21B475KAFNNNE" H 8150 3200 50  0001 C CNN "MPN"
+F 6 "Samsung Electro-Mechanics" H 8150 3200 50  0001 C CNN "Manufacturer"
 	1    8150 3200
 	1    0    0    -1
@@
 F 1 "1uF" H 10285 3745 50  0000 R CNN
 F 2 "Capacitor_SMD:C_0805_2012Metric_Pad1.15x1.40mm_HandSolder" H 10438 3550 50  0001 C CNN
-F 3 "~" H 10400 3700 50  0001 C CNN
+F 3 "https://datasheet.lcsc.com/szlcsc/Samsung-Electro-Mechanics-CL21B105KBFVPNE_C307362.pdf" H 10400 3700 50  0001 C CNN
+F 4 "$0.067176" H 10400 3700 50  0001 C CNN "EstimatedCost(USD)"
+F 5 "CL21B105KBFVPNE" H 10400 3700 50  0001 C CNN "MPN"
+F 6 "Samsung Electro-Mechanics" H 10400 3700 50  0001 C CNN "Manufacturer"
 	1    10400 3700
 	-1   0    0    1
@@
 F 1 "30pF" H 11365 1305 50  0000 L CNN
 F 2 "Capacitor_SMD:C_0805_2012Metric_Pad1.15x1.40mm_HandSolder" H 11288 1200 50  0001 C CNN
-F 3 "~" H 11250 1350 50  0001 C CNN
+F 3 "https://datasheet.lcsc.com/szlcsc/YAGEO-CC0805JRNPO9BN300_C107114.pdf" H 11250 1350 50  0001 C CNN
+F 4 "$0.005588" H 11250 1350 50  0001 C CNN "EstimatedCost(USD)"
+F 5 "CC0805JRNPO9BN300" H 11250 1350 50  0001 C CNN "MPN"
+F 6 "Yageo" H 11250 1350 50  0001 C CNN "Manufacturer"
 	1    11250 1350
 	1    0    0    -1
@@
 F 1 "30pF" H 10865 1305 50  0000 L CNN
 F 2 "Capacitor_SMD:C_0805_2012Metric_Pad1.15x1.40mm_HandSolder" H 10788 1200 50  0001 C CNN
-F 3 "~" H 10750 1350 50  0001 C CNN
+F 3 "https://datasheet.lcsc.com/szlcsc/YAGEO-CC0805JRNPO9BN300_C107114.pdf" H 10750 1350 50  0001 C CNN
+F 4 "$0.005588" H 10750 1350 50  0001 C CNN "EstimatedCost(USD)"
+F 5 "CC0805JRNPO9BN300" H 10750 1350 50  0001 C CNN "MPN"
+F 6 "Yageo" H 10750 1350 50  0001 C CNN "Manufacturer"
 	1    10750 1350
 	1    0    0    -1
@@
 F 1 "2.2uF" V 6339 4950 50  0000 C CNN
 F 2 "Capacitor_SMD:C_0805_2012Metric_Pad1.15x1.40mm_HandSolder" H 6538 4800 50  0001 C CNN
-F 3 "~" H 6500 4950 50  0001 C CNN
+F 3 "https://datasheet.lcsc.com/szlcsc/Samsung-Electro-Mechanics-CL21B225KAFNNNE_C19110.pdf" H 6500 4950 50  0001 C CNN
+F 4 "$0.01848" H 6500 4950 50  0001 C CNN "EstimatedCost(USD)"
+F 5 "CL21B225KAFNNNE" H 6500 4950 50  0001 C CNN "MPN"
+F 6 "Samsung Electro-Mechanics" H 6500 4950 50  0001 C CNN "Manufacturer"
 	1    6500 4950
 	0    1    1    0
@@
 F 1 "2.2uF" V 6751 5250 50  0000 C CNN
 F 2 "Capacitor_SMD:C_0805_2012Metric_Pad1.15x1.40mm_HandSolder" H 6538 5100 50  0001 C CNN
-F 3 "~" H 6500 5250 50  0001 C CNN
+F 3 "https://datasheet.lcsc.com/szlcsc/Samsung-Electro-Mechanics-CL21B225KAFNNNE_C19110.pdf" H 6500 5250 50  0001 C CNN
+F 4 "$0.01848" H 6500 5250 50  0001 C CNN "EstimatedCost(USD)"
+F 5 "CL21B225KAFNNNE" H 6500 5250 50  0001 C CNN "MPN"
+F 6 "Samsung Electro-Mechanics" H 6500 5250 50  0001 C CNN "Manufacturer"
 	1    6500 5250
 	0    1    1    0
@@
 F 1 "1uF" H 5235 5345 50  0000 R CNN
 F 2 "Capacitor_SMD:C_0805_2012Metric_Pad1.15x1.40mm_HandSolder" H 5388 5150 50  0001 C CNN
-F 3 "~" H 5350 5300 50  0001 C CNN
+F 3 "https://datasheet.lcsc.com/szlcsc/Samsung-Electro-Mechanics-CL21B105KBFVPNE_C307362.pdf" H 5350 5300 50  0001 C CNN
+F 4 "$0.067176" H 5350 5300 50  0001 C CNN "EstimatedCost(USD)"
+F 5 "CL21B105KBFVPNE" H 5350 5300 50  0001 C CNN "MPN"
+F 6 "Samsung Electro-Mechanics" H 5350 5300 50  0001 C CNN "Manufacturer"
 	1    5350 5300
 	-1   0    0    1
@@
 F 1 "10uF" V 1889 6700 50  0000 C CNN
 F 2 "Capacitor_SMD:C_0805_2012Metric_Pad1.15x1.40mm_HandSolder" H 2088 6550 50  0001 C CNN
-F 3 "~" H 2050 6700 50  0001 C CNN
+F 3 "https://datasheet.lcsc.com/szlcsc/Samsung-Electro-Mechanics-CL21B106KOQNNNE_C95841.pdf" H 2050 6700 50  0001 C CNN
+F 4 "$0.041113" H 2050 6700 50  0001 C CNN "EstimatedCost(USD)"
+F 5 "CL21B106KOQNNNE" H 2050 6700 50  0001 C CNN "MPN"
+F 6 "Samsung Electro-Mechanics" H 2050 6700 50  0001 C CNN "Manufacturer"
 	1    2050 6700
 	0    1    1    0
@@
 F 1 "1uF" H 7635 3745 50  0000 R CNN
 F 2 "Capacitor_SMD:C_0805_2012Metric_Pad1.15x1.40mm_HandSolder" H 7788 3550 50  0001 C CNN
-F 3 "~" H 7750 3700 50  0001 C CNN
+F 3 "https://datasheet.lcsc.com/szlcsc/Samsung-Electro-Mechanics-CL21B105KBFVPNE_C307362.pdf" H 7750 3700 50  0001 C CNN
+F 4 "$0.067176" H 7750 3700 50  0001 C CNN "EstimatedCost(USD)"
+F 5 "CL21B105KBFVPNE" H 7750 3700 50  0001 C CNN "MPN"
+F 6 "Samsung Electro-Mechanics" H 7750 3700 50  0001 C CNN "Manufacturer"
 	1    7750 3700
 	1    0    0    -1
@@
 F 1 "15pF" H 12765 1305 50  0000 L CNN
 F 2 "Capacitor_SMD:C_0805_2012Metric_Pad1.15x1.40mm_HandSolder" H 12688 1200 50  0001 C CNN
-F 3 "~" H 12650 1350 50  0001 C CNN
+F 3 "https://datasheet.lcsc.com/szlcsc/Samsung-Electro-Mechanics-CL21C150JBANNNC_C1794.pdf" H 12650 1350 50  0001 C CNN
+F 4 "$0.00985" H 12650 1350 50  0001 C CNN "EstimatedCost(USD)"
+F 5 "CL21C150JBANNNC" H 12650 1350 50  0001 C CNN "MPN"
+F 6 "Samsung Electro-Mechanics" H 12650 1350 50  0001 C CNN "Manufacturer"
 	1    12650 1350
 	1    0    0    -1
@@
 F 1 "15pF" H 13265 1305 50  0000 L CNN
 F 2 "Capacitor_SMD:C_0805_2012Metric_Pad1.15x1.40mm_HandSolder" H 13188 1200 50  0001 C CNN
-F 3 "~" H 13150 1350 50  0001 C CNN
+F 3 "https://datasheet.lcsc.com/szlcsc/Samsung-Electro-Mechanics-CL21C150JBANNNC_C1794.pdf" H 13150 1350 50  0001 C CNN
+F 4 "$0.00985" H 13150 1350 50  0001 C CNN "EstimatedCost(USD)"
+F 5 "CL21C150JBANNNC" H 13150 1350 50  0001 C CNN "MPN"
+F 6 "Samsung Electro-Mechanics" H 13150 1350 50  0001 C CNN "Manufacturer"
 	1    13150 1350
 	1    0    0    -1

Commit message: add more part numbers, samtec connector footprint
Parts:
- FB1: footprint (none) -> Capacitor_SMD:C_0805_2012Metric_Pad1.15x1.40mm_HandSolder; EstimatedCost(USD) (none) -> $0.079339; MPN (none) -> MPZ2012S102ATD25; Manufacturer (none) -> TDK
- J1: footprint (none) -> OTTO_Footprints_Lib:FTSH-105-01-X-DV-K; EstimatedCost(USD) (none) -> $2.30; MPN (none) -> FTSH-105-01-F-DV-K-A-P; Manufacturer (none) -> Samtec
Connections:
- net labels added: DC_IN
- net labels removed: +5V_IN
Other:
- note added: "This connector can be useful to expand the features of the OTTO. \nNormally, DC_IN and +5V_MCU are connected via jumpers, \nbut with an expansion board, you could add a battery with char-\nging circuit to the board. \nPWR_BUTTON is routed here in case the battery IC needs it to \npower up.\nThen there's a connector to program the MCU in case the \nRaspberry Pi has problems doing this.\nI2C and th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"
- note removed: "This connector can be useful to expand the features of the OTTO. \nNormally, the +5V_IN and +5V_MCU are connected via jumpers, \nbut with an expansion board, you could add a battery with char-\nging circuit to the board. \nPWR_BUTTON is routed here in case the battery IC needs it to \npower up.\nThen there's a connector to program the MCU in case the \nRaspberry Pi has problems doing this.\nI2C a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"
Changed lines of the file:
@@
 	900  7850 1800 7850
 Text GLabel 2500 7100 2    50   Input ~ 0
-+5V_IN
+DC_IN
 Text GLabel 1600 7100 0    50   Input ~ 0
-+5V_IN
+DC_IN
 Text GLabel 1450 7600 0    50   Input ~ 0
 PWR_BUTTON
@@
 EXP_GPIO_2_ADC
 Text GLabel 12050 8050 2    50   Input ~ 0
-+5V_IN
+DC_IN
 Text Label 900  8700 0    50   ~ 0
 EXP_GPIO_3_PWM
@@
 	1500 7650 1800 7650
 Text Notes 800  10900 0    50   ~ 0
-This connector can be useful to expand the features of the OTTO. \nNormally, the +5V_IN and +5V_MCU are connected via jumpers, \nbut with an expansion board, you could add a battery with char-\nging circuit to the board. \nPWR_BUTTON is routed here in case the battery IC needs it to \npower up.\nThen there's a connector to program the MCU in case the \nRaspberry Pi has problems doing this.\nI2C and the other connections can be used for the charging \ncircuit, too. (ADC for battery level, PWM for status LEDs)\nThe last bit is for a CV/Gate I/O.
+This connector can be useful to expand the features of the OTTO. \nNormally, DC_IN and +5V_MCU are connected via jumpers, \nbut with an expansion board, you could add a battery with char-\nging circuit to the board. \nPWR_BUTTON is routed here in case the battery IC needs it to \npower up.\nThen there's a connector to program the MCU in case the \nRaspberry Pi has problems doing this.\nI2C and the other connections can be used for the charging \ncircuit, too. (ADC for battery level, PWM for status LEDs)\nThe last bit is for a CV/Gate I/O.
 Wire Notes Line
 	750  10950 750  6300
@@
 F 0 "FB1" V 6226 3200 50  0000 C CNN
 F 1 "1kΩ@100Mhz" V 6317 3200 50  0000 C CNN
-F 2 "" V 6430 3200 50  0001 C CNN
-F 3 "~" H 6500 3200 50  0001 C CNN
+F 2 "Capacitor_SMD:C_0805_2012Metric_Pad1.15x1.40mm_HandSolder" V 6430 3200 50  0001 C CNN
+F 3 "https://datasheet.lcsc.com/szlcsc/TDK-MPZ2012S102ATD25_C80983.pdf" H 6500 3200 50  0001 C CNN
+F 4 "$0.079339" H 6500 3200 50  0001 C CNN "EstimatedCost(USD)"
+F 5 "MPZ2012S102ATD25" H 6500 3200 50  0001 C CNN "MPN"
+F 6 "TDK" H 6500 3200 50  0001 C CNN "Manufacturer"
 	1    6500 3200
 	0    1    1    0
@@
 F 0 "J1" H 13906 6396 50  0000 R CNN
 F 1 "Conn_ARM_JTAG_SWD_10" H 13906 6305 50  0000 R CNN
-F 2 "" H 14350 6350 50  0001 C CNN
-F 3 "http://infocenter.arm.com/help/topic/com.arm.doc.ddi0314h/DDI0314H_coresight_components_trm.pdf" V 14000 5100 50  0001 C CNN
+F 2 "OTTO_Footprints_Lib:FTSH-105-01-X-DV-K" H 14350 6350 50  0001 C CNN
+F 3 "http://suddendocs.samtec.com/catalog_english/ftsh_smt.pdf" V 14000 5100 50  0001 C CNN
+F 4 "$2.30" H 14350 6350 50  0001 C CNN "EstimatedCost(USD)"
+F 5 "FTSH-105-01-F-DV-K-A-P" H 14350 6350 50  0001 C CNN "MPN"
+F 6 "Samtec" H 14350 6350 50  0001 C CNN "Manufacturer"
 	1    14350 6350
 	-1   0    0    -1
