File: KiCad/MCU.sch (KiCad schematic (older format))
At the start: 44 parts, among them J1 Conn_ARM_JTAG_SWD_10, J202 Conn_02x03, J203 Conn_02x05, J204 Conn_02x05, J205 Conn_02x04, SW201 SW_Push, SW202 SW_DIP_x02, U7 STM32F407VGTx, Y201 8MHz, Y202 32.768kHz

Commit message: add switch and encoder parts. BM Complete. Footprints complete.
Parts:
- FB1: footprint Capacitor_SMD:C_0805_2012Metric_Pad1.15x1.40mm_HandSolder -> Inductor_SMD:L_0805_2012Metric_Pad1.15x1.40mm_HandSolder
- J202, J203, J204, J205: AssemblyOption (none) -> DNP; EstimatedCost(USD) (none) -> $0.00; MPN (none) -> N/A; Manufacturer (none) -> N/A
- SW201: value SW_Push -> 6x6x5mm; EstimatedCost(USD) (none) -> $0.038303; MPN (none) -> K2-6639DP-C4SW-04; Manufacturer (none) -> Korean Hroparts Elec
- SW202: footprint Button_Switch_THT:XKB_DSIC02LH-P -> OTTO_Footprints_Lib:SW_DIP_SPSTx02_Slide_HRO_EP-02KS; EstimatedCost(USD) (none) -> $0.636364; MPN (none) -> EP-02KS; Manufacturer (none) -> Korean Hroparts Elec
- U7: EstimatedCost(USD) (none) -> $6.469697; MPN (none) -> STM32F407VGT6; Manufacturer (none) -> STMicroelectronics
Changed lines of the file:
@@
 F 0 "SW202" H 7350 1567 50  0000 C CNN
 F 1 "SW_DIP_x02" H 7350 1476 50  0000 C CNN
-F 2 "Button_Switch_THT:XKB_DSIC02LH-P" H 7350 1200 50  0001 C CNN
-F 3 "~" H 7350 1200 50  0001 C CNN
+F 2 "OTTO_Footprints_Lib:SW_DIP_SPSTx02_Slide_HRO_EP-02KS" H 7350 1200 50  0001 C CNN
+F 3 "https://datasheet.lcsc.com/szlcsc/Korean-Hroparts-Elec-EP-02KS_C129087.pdf" H 7350 1200 50  0001 C CNN
+F 4 "$0.636364" H 7350 1200 12700 0001 C CNN "EstimatedCost(USD)"
+F 5 "EP-02KS" H 7350 1200 12700 0001 C CNN "MPN"
+F 6 "Korean Hroparts Elec" H 7350 1200 12700 0001 C CNN "Manufacturer"
 	1    7350 1200
 	1    0    0    -1
@@
 AR Path="/5C4320DF/5DC4F71A" Ref="SW201"  Part="1"
 F 0 "SW201" H 9350 1385 50  0000 C CNN
-F 1 "SW_Push" H 9350 1294 50  0000 C CNN
+F 1 "6x6x5mm" H 9350 1294 50  0000 C CNN
 F 2 "Button_Switch_THT:SW_PUSH_6mm_H5mm" H 9350 1300 50  0001 C CNN
-F 3 "~" H 9350 1300 50  0001 C CNN
+F 3 "https://datasheet.lcsc.com/szlcsc/Korean-Hroparts-Elec-K2-6639DP-C4SW-04_C223746.pdf" H 9350 1300 50  0001 C CNN
+F 4 "$0.038303" H 9350 1100 12700 0001 C CNN "EstimatedCost(USD)"
+F 5 "K2-6639DP-C4SW-04" H 9350 1100 12700 0001 C CNN "MPN"
+F 6 "Korean Hroparts Elec" H 9350 1100 12700 0001 C CNN "Manufacturer"
 	1    9350 1100
 	1    0    0    -1
@@
 F 2 "Package_QFP:LQFP-100_14x14mm_P0.5mm" H 7450 4350 50  0001 R CNN
 F 3 "http://www.st.com/st-web-ui/static/active/en/resource/technical/document/datasheet/DM00037051.pdf" H 8150 6950 50  0001 C CNN
+F 4 "$6.469697" H 8150 6950 12700 0001 C CNN "EstimatedCost(USD)"
+F 5 "STM32F407VGT6" H 8150 6950 12700 0001 C CNN "MPN"
+F 6 "STMicroelectronics" H 8150 6950 12700 0001 C CNN "Manufacturer"
 	1    8150 6950
 	1    0    0    -1
@@
 F 1 "Conn_02x05" H 2050 8176 50  0000 C CNN
 F 2 "Connector_PinHeader_2.54mm:PinHeader_2x05_P2.54mm_Vertical" H 2000 7850 50  0001 C CNN
-F 3 "~" H 2000 7850 50  0001 C CNN
+F 3 "N/A" H 2000 7850 50  0001 C CNN
+F 4 "DNP" H 2000 7850 12700 0001 C CNN "AssemblyOption"
+F 5 "$0.00" H 2000 7850 12700 0001 C CNN "EstimatedCost(USD)"
+F 6 "N/A" H 2000 7850 12700 0001 C CNN "MPN"
+F 7 "N/A" H 2000 7850 12700 0001 C CNN "Manufacturer"
 	1    2000 7850
 	1    0    0    -1
@@
 F 1 "Conn_02x05" H 2050 8926 50  0000 C CNN
 F 2 "Connector_PinHeader_2.54mm:PinHeader_2x05_P2.54mm_Vertical" H 2000 8600 50  0001 C CNN
-F 3 "~" H 2000 8600 50  0001 C CNN
+F 3 "N/A" H 2000 8600 50  0001 C CNN
+F 4 "DNP" H 2000 8600 12700 0001 C CNN "AssemblyOption"
+F 5 "$0.00" H 2000 8600 12700 0001 C CNN "EstimatedCost(USD)"
+F 6 "N/A" H 2000 8600 12700 0001 C CNN "MPN"
+F 7 "N/A" H 2000 8600 12700 0001 C CNN "Manufacturer"
 	1    2000 8600
 	1    0    0    -1
@@
 F 1 "Conn_02x03" H 2050 7426 50  0000 C CNN
 F 2 "Connector_PinHeader_2.54mm:PinHeader_2x03_P2.54mm_Vertical" H 2000 7200 50  0001 C CNN
-F 3 "~" H 2000 7200 50  0001 C CNN
+F 3 "N/A" H 2000 7200 50  0001 C CNN
+F 4 "DNP" H 2000 7200 12700 0001 C CNN "AssemblyOption"
+F 5 "$0.00" H 2000 7200 12700 0001 C CNN "EstimatedCost(USD)"
+F 6 "N/A" H 2000 7200 12700 0001 C CNN "MPN"
+F 7 "N/A" H 2000 7200 12700 0001 C CNN "Manufacturer"
 	1    2000 7200
 	1    0    0    -1
@@
 F 1 "Conn_02x04" H 2050 9476 50  0000 C CNN
 F 2 "Connector_PinHeader_2.54mm:PinHeader_2x04_P2.54mm_Vertical" H 2000 9250 50  0001 C CNN
-F 3 "~" H 2000 9250 50  0001 C CNN
+F 3 "N/A" H 2000 9250 50  0001 C CNN
+F 4 "DNP" H 2000 9250 12700 0001 C CNN "AssemblyOption"
+F 5 "$0.00" H 2000 9250 12700 0001 C CNN "EstimatedCost(USD)"
+F 6 "N/A" H 2000 9250 12700 0001 C CNN "MPN"
+F 7 "N/A" H 2000 9250 12700 0001 C CNN "Manufacturer"
 	1    2000 9250
 	1    0    0    -1
@@
 F 0 "FB1" V 6226 3200 50  0000 C CNN
 F 1 "1kΩ@100Mhz" V 6317 3200 50  0000 C CNN
-F 2 "Capacitor_SMD:C_0805_2012Metric_Pad1.15x1.40mm_HandSolder" V 6430 3200 50  0001 C CNN
+F 2 "Inductor_SMD:L_0805_2012Metric_Pad1.15x1.40mm_HandSolder" V 6430 3200 50  0001 C CNN
 F 3 "https://datasheet.lcsc.com/szlcsc/TDK-MPZ2012S102ATD25_C80983.pdf" H 6500 3200 50  0001 C CNN
 F 4 "$0.079339" H 6500 3200 50  0001 C CNN "EstimatedCost(USD)"

Commit message: add BOM scripts, fix schematic hierarchy
Parts:
- added TP10: TestPoint, TestPoint:TestPoint_Keystone_5000-5004_Miniature, symbol Connector:TestPoint
- BT201: value CR1220 -> CR1220 HOLDER; EstimatedCost(USD) $0.186364 -> (none); UnitCost(USD) (none) -> $0.186364
- C204, C205: EstimatedCost(USD) $0.005588 -> (none); UnitCost(USD) (none) -> $0.005588
- C211: EstimatedCost(USD) $0.031439 -> (none); UnitCost(USD) (none) -> $0.031439
- C218, C219, C223: EstimatedCost(USD) $0.067176 -> (none); UnitCost(USD) (none) -> $0.067176
- C221, C222: EstimatedCost(USD) $0.01848 -> (none); UnitCost(USD) (none) -> $0.01848
- C226: AssemblyOption (none) -> DNP; EstimatedCost(USD) $0.041113 -> (none); UnitCost(USD) (none) -> $0.041113
- C48, C49, C50, C51, C52, C53, C54, C55, C56, C57: EstimatedCost(USD) $0.017724 -> (none); UnitCost(USD) (none) -> $0.017724
- C96, C97: EstimatedCost(USD) $0.00985 -> (none); UnitCost(USD) (none) -> $0.00985
- FB1: EstimatedCost(USD) $0.079339 -> (none); UnitCost(USD) (none) -> $0.079339
- J1: EstimatedCost(USD) $2.30 -> (none); UnitCost(USD) (none) -> $2.30
- J202, J203, J204, J205: EstimatedCost(USD) $0.00 -> (none); UnitCost(USD) (none) -> $0.00
- R202, R205, R206, R207: EstimatedCost(USD) $.001525 -> (none); UnitCost(USD) (none) -> $.001525
- R203, R204, R5: EstimatedCost(USD) $.001675 -> (none); UnitCost(USD) (none) -> $.001675
- R4, R6, R7: value 6.8k -> 10k; EstimatedCost(USD) $.003576 -> (none); MPN RC0805FR-076K8L -> RC0805FR-0710KL; UnitCost(USD) (none) -> $.001675
- R8: EstimatedCost(USD) $.001774 -> (none); UnitCost(USD) (none) -> $.001774
- SW201: EstimatedCost(USD) $0.038303 -> (none); UnitCost(USD) (none) -> $0.038303
- SW202: EstimatedCost(USD) $0.636364 -> (none); UnitCost(USD) (none) -> $0.636364
- U7: EstimatedCost(USD) $6.469697 -> (none); UnitCost(USD) (none) -> $6.469697
- Y201: EstimatedCost(USD) $0.075854 -> (none); UnitCost(USD) (none) -> $0.075854
- Y202: EstimatedCost(USD) $0.237879 -> (none); UnitCost(USD) (none) -> $0.237879
Connections:
- net labels added: LED_PWR_EN
- net labels removed: BL_PWM
- wire segments 306 -> 303
- no-connect marks 2 -> 40

Commit message: Add power switch and other misc nice to haves
Connections:
- net labels added: +5V_PI, +5V_REG, +5V_USB, LI_SENSE, LO_SENSE
- wire segments 303 -> 312
- no-connect marks 40 -> 33

Commit message: Fixes for external battery board and Routing started
Parts:
- removed J202: Conn_02x03, Connector_PinHeader_2.54mm:PinHeader_2x03_P2.54mm_Vertical, symbol Connector_Generic:Conn_02x03_Odd_Even
- added J202: Conn_02x04, Connector_PinHeader_2.54mm:PinHeader_2x04_P2.54mm_Vertical, symbol Connector_Generic:Conn_02x04_Odd_Even
Connections:
- net labels added: 5V_RUN, BARREL_IN, BATT_IN, GPIO16_RASPI, GPIO17_RASPI, GPIO26_RASPI, GPIO27_RASPI
- net labels removed: +5V_PI, +5V_REG
- wire segments 312 -> 324
- no-connect marks 33 -> 28
Other:
- note added: "This connector can be useful to expand the features of the OTTO. \nWith an expansion board, you could add a battery with char-\nging circuit to the board. \nPWR_BUTTON is routed here in case the battery IC needs it to \npower up.\nI2C and the other connections can be used for the charging \ncircuit, too. (ADC for battery level, PWM for status LEDs)\nThe last bit is for a CV/Gate I/O."
- note removed: "This connector can be useful to expand the features of the OTTO. \nNormally, DC_IN and +5V_MCU are connected via jumpers, \nbut with an expansion board, you could add a battery with char-\nging circuit to the board. \nPWR_BUTTON is routed here in case the battery IC needs it to \npower up.\nThen there's a connector to program the MCU in case the \nRaspberry Pi has problems doing this.\nI2C and th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"

Commit message: Add SP3T style DP3T footprint and some schematic labels
Parts:
- added TP? (x2): TestPoint, TestPoint:TestPoint_Keystone_5000-5004_Miniature, symbol Connector:TestPoint
Changed lines of the file:
@@
 $Descr A3 16535 11693
 encoding utf-8
-Sheet 2 7
+Sheet 4 7
 Title "OTTOdiy"
 Date "2020-01-10"
@@
 EndData
 $EndBitmap
-Text HLabel 10000 7650 2    50   Input ~ 0
+Text HLabel 10000 7650 2    50   BiDi ~ 0
 GPIO26_RASPI
-Text HLabel 10000 7750 2    50   Input ~ 0
+Text HLabel 10000 7750 2    50   BiDi ~ 0
 GPIO27_RASPI
-Text HLabel 10000 7550 2    50   Input ~ 0
+Text HLabel 10000 7550 2    50   BiDi ~ 0
 GPIO17_RASPI
-Text HLabel 10000 7450 2    50   Input ~ 0
+Text HLabel 10000 7450 2    50   BiDi ~ 0
 GPIO16_RASPI
 Wire Wire Line
@@
 Text Label 1200 7200 0    50   ~ 0
 +5V_USB
+$Comp
+L Connector:TestPoint TP?
+U 1 1 5ED2EDF0
+P 10000 6550
+F 0 "TP?" V 10000 6750 50  0000 L CNN
+F 1 "TestPoint" V 10000 6950 50  0000 L CNN
+F 2 "TestPoint:TestPoint_Keystone_5000-5004_Miniature" H 10200 6550 50  0001 C CNN
+F 3 "N/A" H 10200 6550 50  0001 C CNN
+F 4 "DNP" H 10000 6550 50  0001 C CNN "AssemblyOption"
+F 5 "N/A" H 10000 6550 50  0001 C CNN "MPN"
+F 6 "N/A" H 10000 6550 50  0001 C CNN "Manufacturer"
+F 7 "$0.00" H 10000 6550 50  0001 C CNN "UnitCost(USD)"
+	1    10000 6550
+	0    1    1    0
+$EndComp
+$Comp
+L Connector:TestPoint TP?
+U 1 1 5ED2F541
+P 10000 6650
+F 0 "TP?" V 10000 6850 50  0000 L CNN
+F 1 "TestPoint" V 10000 7050 50  0000 L CNN
+F 2 "TestPoint:TestPoint_Keystone_5000-5004_Miniature" H 10200 6650 50  0001 C CNN
+F 3 "N/A" H 10200 6650 50  0001 C CNN
+F 4 "DNP" H 10000 6650 50  0001 C CNN "AssemblyOption"
+F 5 "N/A" H 10000 6650 50  0001 C CNN "MPN"
+F 6 "N/A" H 10000 6650 50  0001 C CNN "Manufacturer"
+F 7 "$0.00" H 10000 6650 50  0001 C CNN "UnitCost(USD)"
+	1    10000 6650
+	0    1    1    0
+$EndComp
 $EndSCHEMATC

Commit message: fix electrical rules check errors
Parts:
- added TP18: TestPoint, TestPoint:TestPoint_Keystone_5000-5004_Miniature, symbol Connector:TestPoint
- gave numbers to parts that had none: 2
Connections:
- wire segments 324 -> 327
Changed lines of the file:
@@
 (F427)_SAI1_SD_B
 Wire Wire Line
-	5850 6450 6950 6450
+	5850 6450 6000 6450
 Wire Wire Line
 	5850 6550 6950 6550
@@
 +5V_USB
 $Comp
-L Connector:TestPoint TP?
+L Connector:TestPoint TP16
 U 1 1 5ED2EDF0
 P 10000 6550
-F 0 "TP?" V 10000 6750 50  0000 L CNN
+F 0 "TP16" V 10000 6750 50  0000 L CNN
 F 1 "TestPoint" V 10000 6950 50  0000 L CNN
 F 2 "TestPoint:TestPoint_Keystone_5000-5004_Miniature" H 10200 6550 50  0001 C CNN
@@
 $EndComp
 $Comp
-L Connector:TestPoint TP?
+L Connector:TestPoint TP17
 U 1 1 5ED2F541
 P 10000 6650
-F 0 "TP?" V 10000 6850 50  0000 L CNN
+F 0 "TP17" V 10000 6850 50  0000 L CNN
 F 1 "TestPoint" V 10000 7050 50  0000 L CNN
 F 2 "TestPoint:TestPoint_Keystone_5000-5004_Miniature" H 10200 6650 50  0001 C CNN
@@
 	0    1    1    0
 $EndComp
+$Comp
+L Connector:TestPoint TP18
+U 1 1 5EE1F8D3
+P 5850 6250
+F 0 "TP18" V 5804 6438 50  0000 L CNN
+F 1 "TestPoint" V 5895 6438 50  0000 L CNN
+F 2 "TestPoint:TestPoint_Keystone_5000-5004_Miniature" H 6050 6250 50  0001 C CNN
+F 3 "N/A" H 6050 6250 50  0001 C CNN
+F 4 "DNP" H 5850 6250 50  0001 C CNN "AssemblyOption"
+F 5 "N/A" H 5850 6250 50  0001 C CNN "MPN"
+F 6 "N/A" H 5850 6250 50  0001 C CNN "Manufacturer"
+F 7 "$0.00" H 5850 6250 50  0001 C CNN "UnitCost(USD)"
+	1    5850 6250
+	0    -1   1    0
+$EndComp
+Wire Wire Line
+	5850 6250 6000 6250
+Wire Wire Line
+	6000 6250 6000 6450
+Connection ~ 6000 6450
+Wire Wire Line
+	6000 6450 6950 6450
 $EndSCHEMATC

Commit message: routed buck boost supply
Parts:
- added R25: 10k, Resistor_SMD:R_0805_2012Metric_Pad1.15x1.40mm_HandSolder, symbol Device:R
- R202, R205: AssemblyOption (none) -> DNP
- R203, R204, R4, R6, R7: value 10k -> 47k; MPN RC0805FR-0710KL -> RC0805FR-0747KL; UnitCost(USD) $.001675 -> $.004358
- SW201: MPN K2-6639DP-C4SW-04 -> K2-1102DP-C4SW-04; UnitCost(USD) $0.038303 -> $0.034447
Connections:
- net labels added: DC_IN_DIV_5, GPIO0_RASPI, GPIO1_RASPI, PWM1_GPIO13_RASPI
- net labels removed: GPIO16_RASPI, GPIO17_RASPI, GPIO26_RASPI, GPIO27_RASPI, HP_SENSE, LI_SENSE, LO_SENSE
- wire segments 327 -> 324
- no-connect marks 28 -> 32

Commit message: routed 3v3 and power switches
Parts:
- added D?: RED LED, LED_SMD:LED_0805_2012Metric_Pad1.15x1.40mm_HandSolder, symbol Device:LED_ALT
- added R?: 330, Resistor_SMD:R_0805_2012Metric_Pad1.15x1.40mm_HandSolder, symbol Device:R
Connections:
- wire segments 324 -> 327
- no-connect marks 32 -> 31
Changed lines of the file:
@@
 NoConn ~ 6950 7350
 NoConn ~ 6950 7450
-NoConn ~ 6950 7550
 NoConn ~ 6950 7750
 Wire Wire Line
@@
 NoConn ~ 9350 7650
 NoConn ~ 9350 7750
+$Comp
+L Device:LED_ALT D?
+U 1 1 5E4D3D7B
+P 5400 7550
+F 0 "D?" H 5393 7295 50  0000 C CNN
+F 1 "RED LED" H 5393 7386 50  0000 C CNN
+F 2 "LED_SMD:LED_0805_2012Metric_Pad1.15x1.40mm_HandSolder" H 5400 7550 50  0001 C CNN
+F 3 "https://datasheet.lcsc.com/szlcsc/Everlight-Elec-17-21SURC-S530-A3-TR8_C72037.pdf" H 5400 7550 50  0001 C CNN
+F 4 "17-21SURC/S530-A3/TR8" H 5400 7550 50  0001 C CNN "MPN"
+F 5 "Everlight Elec" H 5400 7550 50  0001 C CNN "Manufacturer"
+F 6 "$0.017818" H 5400 7550 50  0001 C CNN "UnitCost(USD)"
+	1    5400 7550
+	-1   0    0    1
+$EndComp
+Text GLabel 5150 7550 0    50   Input ~ 0
++3V3_MCU
+Wire Wire Line
+	5150 7550 5250 7550
+$Comp
+L Device:R R?
+U 1 1 5E4F922A
+P 5800 7550
+F 0 "R?" V 5593 7550 50  0000 C CNN
+F 1 "330" V 5684 7550 50  0000 C CNN
+F 2 "Resistor_SMD:R_0805_2012Metric_Pad1.15x1.40mm_HandSolder" V 5730 7550 50  0001 C CNN
+F 3 "https://datasheet.lcsc.com/szlcsc/YAGEO-RC0805FR-07330RL_C105878.pdf" H 5800 7550 50  0001 C CNN
+F 4 "RC0805FR-07330RL" H 5800 7550 50  0001 C CNN "MPN"
+F 5 "Yageo" H 5800 7550 50  0001 C CNN "Manufacturer"
+F 6 "$.001575" H 5800 7550 50  0001 C CNN "UnitCost(USD)"
+	1    5800 7550
+	0    1    1    0
+$EndComp
+Wire Wire Line
+	5550 7550 5650 7550
+Wire Wire Line
+	5950 7550 6950 7550
 $EndSCHEMATC
