File: KiCad/MCU.sch (KiCad schematic (older format))
At the start: 51 parts, among them J1 Conn_ARM_JTAG_SWD_10, J202 Conn_02x04, J203 Conn_02x05, J204 Conn_02x05, J205 Conn_02x04, SW201 6x6x5mm, SW202 SW_DIP_x02, U7 STM32F407VGTx, Y201 8MHz, Y202 32.768kHz

Commit message: add fault/status LED to MCU
Parts:
- gave numbers to parts that had none: 2
Changed lines of the file:
@@
 NoConn ~ 9350 7750
 $Comp
-L Device:LED_ALT D?
+L Device:LED_ALT D57
 U 1 1 5E4D3D7B
 P 5400 7550
-F 0 "D?" H 5393 7295 50  0000 C CNN
+F 0 "D57" H 5393 7295 50  0000 C CNN
 F 1 "RED LED" H 5393 7386 50  0000 C CNN
 F 2 "LED_SMD:LED_0805_2012Metric_Pad1.15x1.40mm_HandSolder" H 5400 7550 50  0001 C CNN
@@
 	5150 7550 5250 7550
 $Comp
-L Device:R R?
+L Device:R R28
 U 1 1 5E4F922A
 P 5800 7550
-F 0 "R?" V 5593 7550 50  0000 C CNN
+F 0 "R28" V 5593 7550 50  0000 C CNN
 F 1 "330" V 5684 7550 50  0000 C CNN
 F 2 "Resistor_SMD:R_0805_2012Metric_Pad1.15x1.40mm_HandSolder" V 5730 7550 50  0001 C CNN

Commit message: routed mcu decoupling
Parts:
- removed C223: 1uF, Capacitor_SMD:C_0805_2012Metric_Pad1.15x1.40mm_HandSolder, symbol Device:C
- removed C56: 100nF, Capacitor_SMD:C_0805_2012Metric_Pad1.15x1.40mm_HandSolder, symbol Device:C
- removed Y202: 32.768kHz, Crystal:Crystal_SMD_SeikoEpson_MC306-4Pin_8.0x3.2mm_HandSoldering, symbol Device:Crystal
- added Y202: 32.768kHz, Crystal:Crystal_SMD_SeikoEpson_MC306-4Pin_8.0x3.2mm_HandSoldering, symbol Device:Crystal_GND23
Connections:
- net labels added: STATUS_LED
- wire segments 327 -> 326
Changed lines of the file:
@@
-$Comp
-L Device:Crystal Y?
-U 1 1 5DC4F680
-P 12900 1100
-AR Path="/5C4320DF/5DB999B7/5DC4F680" Ref="Y?"  Part="1"
-AR Path="/5C4320DF/5DC4F680" Ref="Y202"  Part="1"
-F 0 "Y202" H 12900 1368 50  0000 C CNN
-F 1 "32.768kHz" H 12900 1277 50  0000 C CNN
-F 2 "Crystal:Crystal_SMD_SeikoEpson_MC306-4Pin_8.0x3.2mm_HandSoldering" H 12900 1100 50  0001 C CNN
-F 3 "https://datasheet.lcsc.com/szlcsc/Seiko-Epson-Q13MC3061000300_C16320.pdf" H 12900 1100 50  0001 C CNN
-F 4 "$0.237879" H 12900 1100 12700 0001 C CNN "UnitCost(USD)"
-F 5 "Q13MC3061000300" H 12900 1100 12700 0001 C CNN "MPN"
-F 6 "Seiko Epson" H 12900 1100 12700 0001 C CNN "Manufacturer"
-	1    12900 1100
-	-1   0    0    -1
-$EndComp
 $Comp
 L Device:Crystal Y?
@@
 $EndComp
 Wire Wire Line
-	13150 1200 13150 1100
-Wire Wire Line
-	13150 1100 13050 1100
-Wire Wire Line
-	12750 1100 12650 1100
-Wire Wire Line
-	12650 1100 12650 1200
+	13250 1300 13250 1100
+Wire Wire Line
+	13250 1100 13050 1100
+Wire Wire Line
+	12750 1100 12550 1100
+Wire Wire Line
+	12550 1100 12550 1300
 Wire Wire Line
 	11250 1200 11250 1100
@@
 Wire Wire Line
 	11000 1600 11250 1600
-$Comp
-L power:GND #PWR0209
-U 1 1 5DC4F6B8
-P 12900 1700
-AR Path="/5C4320DF/5DC4F6B8" Ref="#PWR0209"  Part="1"
-AR Path="/5C4320DF/5DB999B7/5DC4F6B8" Ref="#PWR?"  Part="1"
-F 0 "#PWR0209" H 12900 1450 50  0001 C CNN
-F 1 "GND" H 12905 1527 50  0000 C CNN
-F 2 "" H 12900 1700 50  0001 C CNN
-F 3 "" H 12900 1700 50  0001 C CNN
-	1    12900 1700
-	1    0    0    -1
-$EndComp
-Wire Wire Line
-	12650 1500 12650 1600
-Wire Wire Line
-	12650 1600 12900 1600
-Wire Wire Line
-	13150 1600 13150 1500
-Wire Wire Line
-	12900 1700 12900 1600
-Connection ~ 12900 1600
-Wire Wire Line
-	12900 1600 13150 1600
-Text Label 12250 1100 0    50   ~ 0
+Wire Wire Line
+	12550 1600 12550 1800
+Wire Wire Line
+	12550 1800 12900 1800
+Connection ~ 12900 1800
+Wire Wire Line
+	12900 1800 13000 1800
+Text Label 12150 1100 0    50   ~ 0
 OSC32_IN
-Text Label 13650 1100 2    50   ~ 0
+Text Label 13850 1100 2    50   ~ 0
 OSC32_OUT
 Wire Wire Line
-	13650 1100 13150 1100
-Connection ~ 13150 1100
-Wire Wire Line
-	12250 1100 12650 1100
-Connection ~ 12650 1100
+	13850 1100 13250 1100
+Connection ~ 13250 1100
+Wire Wire Line
+	12150 1100 12550 1100
+Connection ~ 12550 1100
 Text Label 10350 1100 0    50   ~ 0
 OSC_IN
@@
 Wire Wire Line
 	6250 5250 6250 4950
-Wire Wire Line
-	6250 4950 5850 4950
 Wire Wire Line
 	6250 4950 6350 4950
@@
 Text Label 14350 1800 0    50   ~ 0
 I2C2_SCL
-$Comp
-L Device:C C223
-U 1 1 5E3EF6FE
-P 5350 5300
-AR Path="/5C4320DF/5E3EF6FE" Ref="C223"  Part="1"
-AR Path="/5C4320DF/5DB999B7/5E3EF6FE" Ref="C?"  Part="1"
-F 0 "C223" H 5235 5254 50  0000 R CNN
-F 1 "1uF" H 5235 5345 50  0000 R CNN
-F 2 "Capacitor_SMD:C_0805_2012Metric_Pad1.15x1.40mm_HandSolder" H 5388 5150 50  0001 C CNN
-F 3 "https://datasheet.lcsc.com/szlcsc/Samsung-Electro-Mechanics-CL21B105KBFVPNE_C307362.pdf" H 5350 5300 50  0001 C CNN
-F 4 "$0.067176" H 5350 5300 50  0001 C CNN "UnitCost(USD)"
-F 5 "CL21B105KBFVPNE" H 5350 5300 50  0001 C CNN "MPN"
-F 6 "Samsung Electro-Mechanics" H 5350 5300 50  0001 C CNN "Manufacturer"
-	1    5350 5300
-	-1   0    0    1
-$EndComp
-$Comp
-L Device:C C56
-U 1 1 5E3EF704
-P 5850 5300
-AR Path="/5C4320DF/5E3EF704" Ref="C56"  Part="1"
-AR Path="/5C4320DF/5DB999B7/5E3EF704" Ref="C?"  Part="1"
-F 0 "C56" H 5735 5254 50  0000 R CNN
-F 1 "100nF" H 5735 5345 50  0000 R CNN
-F 2 "Capacitor_SMD:C_0805_2012Metric_Pad1.15x1.40mm_HandSolder" H 5888 5150 50  0001 C CNN
-F 3 "https://datasheet.lcsc.com/szlcsc/Samsung-Electro-Mechanics-CL21B104JBCNNNC_C62912.pdf" H 5850 5300 50  0001 C CNN
-F 4 "$0.017724" H 5850 5300 12700 0001 C CNN "UnitCost(USD)"
-F 5 "CL21B104JBCNNNC" H 5850 5300 12700 0001 C CNN "MPN"
-F 6 "Samsung Electro-Mechanics" H 5850 5300 12700 0001 C CNN "Manufacturer"
-	1    5850 5300
-	-1   0    0    1
-$EndComp
 Wire Wire Line
 	6950 5150 6850 5150
 Wire Wire Line
 	6850 5150 6850 5650
-Wire Wire Line
-	6850 5650 5850 5650
-Wire Wire Line
-	5350 5650 5350 5450
-Wire Wire Line
-	5850 5150 5850 4950
-Connection ~ 5850 4950
-Wire Wire Line
-	5850 4950 5350 4950
-Wire Wire Line
-	5350 5150 5350 4950
-Connection ~ 5350 4950
-Wire Wire Line
-	5350 4950 5250 4950
-Wire Wire Line
-	5850 5450 5850 5650
-Connection ~ 5850 5650
-Wire Wire Line
-	5850 5650 5350 5650
 Wire Wire Line
 	15100 1800 15200 1800
@@
 	11200 8050 11650 8050
 Wire Wire Line
-	5350 5650 5150 5650
-Connection ~ 5350 5650
-Wire Wire Line
 	8650 3450 9150 3450
 Wire Wire Line
@@
 Text GLabel 6050 3200 0    50   Input ~ 0
 +3V3_MCU
-Text GLabel 5150 5650 0    50   Input ~ 0
+Text GLabel 5850 5650 0    50   Input ~ 0
 +3V3A_MCU
 Wire Wire Line
@@
 L Device:C C96
 U 1 1 5E1FEFB6
-P 12650 1350
+P 12550 1450
 AR Path="/5C4320DF/5E1FEFB6" Ref="C96"  Part="1"
 AR Path="/5C4320DF/5DB999B7/5E1FEFB6" Ref="C?"  Part="1"
-F 0 "C96" H 12765 1396 50  0000 L CNN
-F 1 "15pF" H 12765 1305 50  0000 L CNN
-F 2 "Capacitor_SMD:C_0805_2012Metric_Pad1.15x1.40mm_HandSolder" H 12688 1200 50  0001 C CNN
-F 3 "https://datasheet.lcsc.com/szlcsc/Samsung-Electro-Mechanics-CL21C150JBANNNC_C1794.pdf" H 12650 1350 50  0001 C CNN
-F 4 "$0.00985" H 12650 1350 50  0001 C CNN "UnitCost(USD)"
-F 5 "CL21C150JBANNNC" H 12650 1350 50  0001 C CNN "MPN"
-F 6 "Samsung Electro-Mechanics" H 12650 1350 50  0001 C CNN "Manufacturer"
-	1    12650 1350
+F 0 "C96" H 12665 1496 50  0000 L CNN
+F 1 "15pF" H 12665 1405 50  0000 L CNN
+F 2 "Capacitor_SMD:C_0805_2012Metric_Pad1.15x1.40mm_HandSolder" H 12588 1300 50  0001 C CNN
+F 3 "https://datasheet.lcsc.com/szlcsc/Samsung-Electro-Mechanics-CL21C150JBANNNC_C1794.pdf" H 12550 1450 50  0001 C CNN
+F 4 "$0.00985" H 12550 1450 50  0001 C CNN "UnitCost(USD)"
+F 5 "CL21C150JBANNNC" H 12550 1450 50  0001 C CNN "MPN"
+F 6 "Samsung Electro-Mechanics" H 12550 1450 50  0001 C CNN "Manufacturer"
+	1    12550 1450
 	1    0    0    -1
 $EndComp
@@
 L Device:C C97
 U 1 1 5E2015EC
-P 13150 1350
+P 13250 1450
 AR Path="/5C4320DF/5E2015EC" Ref="C97"  Part="1"
 AR Path="/5C4320DF/5DB999B7/5E2015EC" Ref="C?"  Part="1"
-F 0 "C97" H 13265 1396 50  0000 L CNN
-F 1 "15pF" H 13265 1305 50  0000 L CNN
-F 2 "Capacitor_SMD:C_0805_2012Metric_Pad1.15x1.40mm_HandSolder" H 13188 1200 50  0001 C CNN
-F 3 "https://datasheet.lcsc.com/szlcsc/Samsung-Electro-Mechanics-CL21C150JBANNNC_C1794.pdf" H 13150 1350 50  0001 C CNN
-F 4 "$0.00985" H 13150 1350 50  0001 C CNN "UnitCost(USD)"
-F 5 "CL21C150JBANNNC" H 13150 1350 50  0001 C CNN "MPN"
-F 6 "Samsung Electro-Mechanics" H 13150 1350 50  0001 C CNN "Manufacturer"
-	1    13150 1350
+F 0 "C97" H 13365 1496 50  0000 L CNN
+F 1 "15pF" H 13365 1405 50  0000 L CNN
+F 2 "Capacitor_SMD:C_0805_2012Metric_Pad1.15x1.40mm_HandSolder" H 13288 1300 50  0001 C CNN
+F 3 "https://datasheet.lcsc.com/szlcsc/Samsung-Electro-Mechanics-CL21C150JBANNNC_C1794.pdf" H 13250 1450 50  0001 C CNN
+F 4 "$0.00985" H 13250 1450 50  0001 C CNN "UnitCost(USD)"
+F 5 "CL21C150JBANNNC" H 13250 1450 50  0001 C CNN "MPN"
+F 6 "Samsung Electro-Mechanics" H 13250 1450 50  0001 C CNN "Manufacturer"
+	1    13250 1450
 	1    0    0    -1
 $EndComp
@@
 Wire Wire Line
 	5950 7550 6950 7550
+$Comp
+L Device:Crystal_GND23 Y202
+U 1 1 5E2B8B30
+P 12900 1100
+F 0 "Y202" H 12900 1481 50  0000 C CNN
+F 1 "32.768kHz" H 12900 1390 50  0000 C CNN
+F 2 "Crystal:Crystal_SMD_SeikoEpson_MC306-4Pin_8.0x3.2mm_HandSoldering" H 12900 1100 50  0001 C CNN
+F 3 "https://datasheet.lcsc.com/szlcsc/Seiko-Epson-Q13MC3061000300_C16320.pdf" H 12900 1100 50  0001 C CNN
+F 4 "Q13MC3061000300" H 12900 1100 50  0001 C CNN "MPN"
+F 5 "Seiko Epson" H 12900 1100 50  0001 C CNN "Manufacturer"
+F 6 "$0.237879" H 12900 1100 50  0001 C CNN "UnitCost(USD)"
+	1    12900 1100
+	1    0    0    -1
+$EndComp
+$Comp
+L power:GND #PWR0209
+U 1 1 5DC4F6B8
+P 13250 1950
+AR Path="/5C4320DF/5DC4F6B8" Ref="#PWR0209"  Part="1"
+AR Path="/5C4320DF/5DB999B7/5DC4F6B8" Ref="#PWR?"  Part="1"
+F 0 "#PWR0209" H 13250 1700 50  0001 C CNN
+F 1 "GND" H 13255 1777 50  0000 C CNN
+F 2 "" H 13250 1950 50  0001 C CNN
+F 3 "" H 13250 1950 50  0001 C CNN
+	1    13250 1950
+	1    0    0    -1
+$EndComp
+Wire Wire Line
+	12900 1300 12900 1800
+Wire Wire Line
+	12900 900  12900 850
+Wire Wire Line
+	12900 850  13100 850
+Wire Wire Line
+	13100 850  13100 1350
+Wire Wire Line
+	13100 1350 13000 1350
+Wire Wire Line
+	13000 1350 13000 1800
+Connection ~ 13000 1800
+Wire Wire Line
+	13000 1800 13250 1800
+Wire Wire Line
+	13250 1800 13250 1600
+Wire Wire Line
+	13250 1800 13250 1950
+Connection ~ 13250 1800
+Wire Wire Line
+	5850 5650 6850 5650
+Wire Wire Line
+	5250 4950 6250 4950
+Text Label 6050 7550 0    50   ~ 0
+STATUS_LED
 $EndSCHEMATC

Commit message: fix peripheral connections and route more critical components
Parts:
- added C56: 100nF, Capacitor_SMD:C_0805_2012Metric_Pad1.15x1.40mm_HandSolder, symbol Device:C
- added R29, R30: 10k, Resistor_SMD:R_0805_2012Metric_Pad1.15x1.40mm_HandSolder, symbol Device:R
- added TP1: TestPoint, TestPoint:TestPoint_Keystone_5000-5004_Miniature, symbol Connector:TestPoint
Connections:
- net labels added: +3V3_RASPI, 3V3_RASPI_DIV_2, MCU_PC8
- wire segments 326 -> 336
- no-connect marks 31 -> 28
Other:
- note added: "3V3_RASPI Voltage Divider to ADC"
- note added: "DC_IN Voltage Divider to ADC"
- note added: "Standard 10-pin ARM SWD Interface"

Commit message: routed audio
Parts:
- removed R25: 10k, Resistor_SMD:R_0805_2012Metric_Pad1.15x1.40mm_HandSolder, symbol Device:R
- removed TP10: TestPoint, TestPoint:TestPoint_Keystone_5000-5004_Miniature, symbol Connector:TestPoint
- removed Y202: 32.768kHz, Crystal:Crystal_SMD_SeikoEpson_MC306-4Pin_8.0x3.2mm_HandSoldering, symbol Device:Crystal_GND23
- added Y202: 32.768kHz, OTTO_Footprints_Lib:Crystal_SMD_3215-2Pin_3.2x1.5mm_HandSoldering, symbol Device:Crystal
- Y201: value 8MHz -> 25MHz; footprint Crystal:Crystal_SMD_HC49-SD_HandSoldering -> Crystal:Crystal_SMD_5032-2Pin_5.0x3.2mm_HandSoldering; MPN X49SM8MSD2SC -> X503225MSB2GI; UnitCost(USD) $0.075854 -> $0.171212
Connections:
- net labels removed: TAMPER_RTC
- wire segments 336 -> 349
- no-connect marks 28 -> 6

Commit message: Placement of all components
Parts:
- R6, R7: value 47k -> 10k; AssemblyOption (none) -> DNP; MPN RC0805FR-0747KL -> RC0805FR-0710KL; UnitCost(USD) $.004358 -> $.001675
Changed lines of the file:
@@
 Wire Wire Line
 	6100 4300 6850 4300
-$Comp
-L Device:R R6
-U 1 1 5E183D37
-P 11500 5600
-F 0 "R6" H 11570 5645 50  0000 L CNN
-F 1 "47k" H 11570 5555 50  0000 L CNN
-F 2 "Resistor_SMD:R_0805_2012Metric_Pad1.15x1.40mm_HandSolder" V 11430 5600 50  0001 C CNN
-F 3 "https://datasheet.lcsc.com/szlcsc/YAGEO-RC0805FR-0747KL_C126351.pdf" H 11500 5600 50  0001 C CNN
-F 4 "$.004358" H 11500 5600 50  0001 C CNN "UnitCost(USD)"
-F 5 "RC0805FR-0747KL" H 11500 5600 50  0001 C CNN "MPN"
-F 6 "Yageo" H 11500 5600 50  0001 C CNN "Manufacturer"
-	1    11500 5600
-	1    0    0    -1
-$EndComp
-$Comp
-L Device:R R7
-U 1 1 5E185281
-P 11500 6200
-F 0 "R7" H 11570 6245 50  0000 L CNN
-F 1 "47k" H 11570 6155 50  0000 L CNN
-F 2 "Resistor_SMD:R_0805_2012Metric_Pad1.15x1.40mm_HandSolder" V 11430 6200 50  0001 C CNN
-F 3 "https://datasheet.lcsc.com/szlcsc/YAGEO-RC0805FR-0747KL_C126351.pdf" H 11500 6200 50  0001 C CNN
-F 4 "$.004358" H 11500 6200 50  0001 C CNN "UnitCost(USD)"
-F 5 "RC0805FR-0747KL" H 11500 6200 50  0001 C CNN "MPN"
-F 6 "Yageo" H 11500 6200 50  0001 C CNN "Manufacturer"
-	1    11500 6200
-	1    0    0    -1
-$EndComp
 Wire Wire Line
 	9350 5850 11500 5850
@@
 Wire Wire Line
 	6050 9050 6950 9050
+$Comp
+L Device:R R6
+U 1 1 5E372364
+P 11500 5600
+F 0 "R6" H 11570 5646 50  0000 L CNN
+F 1 "10k" H 11570 5555 50  0000 L CNN
+F 2 "Resistor_SMD:R_0805_2012Metric_Pad1.15x1.40mm_HandSolder" V 11430 5600 50  0001 C CNN
+F 3 "https://datasheet.lcsc.com/szlcsc/YAGEO-RC0805FR-0710KL_C84376.pdf" H 11500 5600 50  0001 C CNN
+F 4 "$.001675" H 11500 5600 50  0001 C CNN "UnitCost(USD)"
+F 5 "RC0805FR-0710KL" H 11500 5600 50  0001 C CNN "MPN"
+F 6 "Yageo" H 11500 5600 50  0001 C CNN "Manufacturer"
+F 7 "DNP" V 11500 5600 50  0000 C CNN "AssemblyOption"
+	1    11500 5600
+	1    0    0    -1
+$EndComp
+$Comp
+L Device:R R7
+U 1 1 5E372D75
+P 11500 6200
+F 0 "R7" H 11570 6246 50  0000 L CNN
+F 1 "10k" H 11570 6155 50  0000 L CNN
+F 2 "Resistor_SMD:R_0805_2012Metric_Pad1.15x1.40mm_HandSolder" V 11430 6200 50  0001 C CNN
+F 3 "https://datasheet.lcsc.com/szlcsc/YAGEO-RC0805FR-0710KL_C84376.pdf" H 11500 6200 50  0001 C CNN
+F 4 "$.001675" H 11500 6200 50  0001 C CNN "UnitCost(USD)"
+F 5 "RC0805FR-0710KL" H 11500 6200 50  0001 C CNN "MPN"
+F 6 "Yageo" H 11500 6200 50  0001 C CNN "Manufacturer"
+F 7 "DNP" V 11500 6200 50  0000 C CNN "AssemblyOption"
+	1    11500 6200
+	1    0    0    -1
+$EndComp
 $EndSCHEMATC

Commit message: change mcu reset button and route more stuff
Parts:
- SW201: value 6x6x5mm -> 5.2x5.2x1.5mm; footprint Button_Switch_THT:SW_PUSH_6mm_H5mm -> OTTO_Footprints_Lib:SW_SPST_5.2x5.2x1.5mm; MPN K2-1102DP-C4SW-04 -> K2-1187SQ-A4SW-06; UnitCost(USD) $0.034447 -> $0.0467
Changed lines of the file:
@@
 F 6 "Korean Hroparts Elec" H 7350 1200 12700 0001 C CNN "Manufacturer"
 	1    7350 1200
-	1    0    0    -1
+	-1   0    0    -1
 $EndComp
 Text Label 6250 1100 0    50   ~ 0
@@
 AR Path="/5C4320DF/5DC4F71A" Ref="SW201"  Part="1"
 F 0 "SW201" H 9350 1385 50  0000 C CNN
-F 1 "6x6x5mm" H 9350 1294 50  0000 C CNN
-F 2 "Button_Switch_THT:SW_PUSH_6mm_H5mm" H 9350 1300 50  0001 C CNN
-F 3 "https://datasheet.lcsc.com/szlcsc/Korean-Hroparts-Elec-K2-1102DP-C4SW-04_C110153.pdf" H 9350 1300 50  0001 C CNN
-F 4 "$0.034447" H 9350 1100 12700 0001 C CNN "UnitCost(USD)"
-F 5 "K2-1102DP-C4SW-04" H 9350 1100 12700 0001 C CNN "MPN"
+F 1 "5.2x5.2x1.5mm" H 9350 1294 50  0000 C CNN
+F 2 "OTTO_Footprints_Lib:SW_SPST_5.2x5.2x1.5mm" H 9350 1300 50  0001 C CNN
+F 3 "https://datasheet.lcsc.com/szlcsc/Korean-Hroparts-Elec-K2-1187SQ-A4SW-06_C92584.pdf" H 9350 1300 50  0001 C CNN
+F 4 "$0.0467" H 9350 1100 12700 0001 C CNN "UnitCost(USD)"
+F 5 "K2-1187SQ-A4SW-06" H 9350 1100 12700 0001 C CNN "MPN"
 F 6 "Korean Hroparts Elec" H 9350 1100 12700 0001 C CNN "Manufacturer"
 	1    9350 1100

Commit message: Add and route 7 extra buttons/LEDs
Connections:
- net labels added: COL_8
- wire segments 349 -> 351
- no-connect marks 6 -> 5
Changed lines of the file:
@@
 Text Label 2700 2600 2    50   ~ 0
 SPI_MOSI_MCU
-$Sheet
-S 750  3050 1000 2650
-U 5C971830
-F0 "KEYS+ENCODERS" 50
-F1 "KEYS+ENCODERS.sch" 50
-F2 "ROW_1" I R 1750 3150 50
-F3 "ROW_2" I R 1750 3250 50
-F4 "ROW_3" I R 1750 3350 50
-F5 "ROW_4" I R 1750 3450 50
-F6 "ROW_5" I R 1750 3550 50
-F7 "ROW_6" I R 1750 3650 50
-F8 "ROW_7" I R 1750 3750 50
-F9 "COL_1" I R 1750 4000 50
-F10 "COL_2" I R 1750 4100 50
-F11 "COL_3" I R 1750 4200 50
-F12 "COL_4" I R 1750 4300 50
-F13 "COL_5" I R 1750 4400 50
-F14 "COL_6" I R 1750 4500 50
-F15 "ROW_8" I R 1750 3850 50
-F16 "ENC_A_1" I R 1750 4750 50
-F17 "ENC_B_1" I R 1750 4850 50
-F18 "ENC_A_2" I R 1750 5000 50
-F19 "ENC_B_2" I R 1750 5100 50
-F20 "ENC_A_3" I R 1750 5250 50
-F21 "ENC_A_4" I R 1750 5500 50
-F22 "ENC_B_4" I R 1750 5600 50
-F23 "ENC_B_3" I R 1750 5350 50
-F24 "COL_7" I R 1750 4600 50
-$EndSheet
 Text Label 2700 3150 2    50   ~ 0
 ROW_1
@@
 NoConn ~ 9350 9150
 NoConn ~ 9350 9050
-NoConn ~ 9350 8950
 Text Label 10000 8650 2    50   ~ 0
 5V_PWM_SYNC
@@
 COL_7
 Wire Wire Line
+	2700 5700 1750 5700
+Wire Wire Line
+	1750 4850 2700 4850
+Text Label 2700 4850 2    50   ~ 0
+ENC_A_1
+Wire Wire Line
 	2700 5600 1750 5600
 Wire Wire Line
-	1750 4750 2700 4750
-Text Label 2700 4750 2    50   ~ 0
-ENC_A_1
-Wire Wire Line
-	2700 5500 1750 5500
-Wire Wire Line
-	1750 5350 2700 5350
-Wire Wire Line
-	2700 5250 1750 5250
-Wire Wire Line
-	1750 5100 2700 5100
-Wire Wire Line
-	2700 5000 1750 5000
-Wire Wire Line
-	1750 4850 2700 4850
+	1750 5450 2700 5450
+Wire Wire Line
+	2700 5350 1750 5350
+Wire Wire Line
+	1750 5200 2700 5200
+Wire Wire Line
+	2700 5100 1750 5100
+Wire Wire Line
+	1750 4950 2700 4950
+Text Label 2700 5700 2    50   ~ 0
+ENC_B_4
 Text Label 2700 5600 2    50   ~ 0
-ENC_B_4
-Text Label 2700 5500 2    50   ~ 0
 ENC_A_4
+Text Label 2700 5450 2    50   ~ 0
+ENC_B_3
 Text Label 2700 5350 2    50   ~ 0
-ENC_B_3
-Text Label 2700 5250 2    50   ~ 0
 ENC_A_3
+Text Label 2700 5200 2    50   ~ 0
+ENC_B_2
 Text Label 2700 5100 2    50   ~ 0
-ENC_B_2
-Text Label 2700 5000 2    50   ~ 0
 ENC_A_2
-Text Label 2700 4850 2    50   ~ 0
+Text Label 2700 4950 2    50   ~ 0
 ENC_B_1
 Wire Wire Line
@@
 	1    0    0    -1
 $EndComp
+$Sheet
+S 750  3050 1000 2700
+U 5C971830
+F0 "KEYS+ENCODERS" 50
+F1 "KEYS+ENCODERS.sch" 50
+F2 "ROW_1" I R 1750 3150 50
+F3 "ROW_2" I R 1750 3250 50
+F4 "ROW_3" I R 1750 3350 50
+F5 "ROW_4" I R 1750 3450 50
+F6 "ROW_5" I R 1750 3550 50
+F7 "ROW_6" I R 1750 3650 50
+F8 "ROW_7" I R 1750 3750 50
+F9 "COL_1" I R 1750 4000 50
+F10 "COL_2" I R 1750 4100 50
+F11 "COL_3" I R 1750 4200 50
+F12 "COL_4" I R 1750 4300 50
+F13 "COL_5" I R 1750 4400 50
+F14 "COL_6" I R 1750 4500 50
+F15 "ROW_8" I R 1750 3850 50
+F16 "ENC_A_1" I R 1750 4850 50
+F17 "ENC_B_1" I R 1750 4950 50
+F18 "ENC_A_2" I R 1750 5100 50
+F19 "ENC_B_2" I R 1750 5200 50
+F20 "ENC_A_3" I R 1750 5350 50
+F21 "ENC_A_4" I R 1750 5600 50
+F22 "ENC_B_4" I R 1750 5700 50
+F23 "ENC_B_3" I R 1750 5450 50
+F24 "COL_7" I R 1750 4600 50
+F25 "COL_8" I R 1750 4700 50
+$EndSheet
+Text Label 2700 4700 2    50   ~ 0
+COL_8
+Wire Wire Line
+	2700 4700 1750 4700
+Text Label 10000 8950 2    50   ~ 0
+COL_8
+Wire Wire Line
+	10000 8950 9350 8950
 $EndSCHEMATC

Commit message: cleaned up audio area, added board version pin
Connections:
- wire segments 351 -> 352
- no-connect marks 5 -> 4
Other:
- note added: "PC2 is reserved to find out the board \nversion with a specified voltage"
Changed lines of the file:
@@
 	0    1    1    0
 $EndComp
-NoConn ~ 9350 9150
-NoConn ~ 9350 9050
 Text Label 10000 8650 2    50   ~ 0
 5V_PWM_SYNC
@@
 Text Label 10000 8050 2    50   ~ 0
 ROW_6
-Text Label 10000 8150 2    50   ~ 0
+Text Label 10000 9150 2    50   ~ 0
 ROW_7
 Text Label 10000 8250 2    50   ~ 0
@@
 	9350 8050 10000 8050
 Wire Wire Line
-	10000 8150 9350 8150
+	10000 9150 9350 9150
 Wire Wire Line
 	9350 8250 10000 8250
@@
 Wire Wire Line
 	10000 8950 9350 8950
+$Comp
+L power:GND #PWR0147
+U 1 1 5E5EA3D1
+P 10100 8150
+F 0 "#PWR0147" H 10100 7900 50  0001 C CNN
+F 1 "GND" V 10105 8022 50  0000 R CNN
+F 2 "" H 10100 8150 50  0001 C CNN
+F 3 "" H 10100 8150 50  0001 C CNN
+	1    10100 8150
+	0    -1   -1   0
+$EndComp
+Wire Wire Line
+	10100 8150 9350 8150
+Text Notes 10450 8150 0    50   ~ 0
+PC2 is reserved to find out the board \nversion with a specified voltage
+NoConn ~ 9350 9050
 $EndSCHEMATC
