File: KiCad/PERIPHERALS.sch (KiCad schematic (older format))
At the start: 18 parts, among them CN201 1x4 MALE 1.5mm, CN202 1x4 MALE 1.5mm, Q1 IRF9321PbF, SW203 ALPS SKHH angled, U204 USB6B1

Commit message: roll in changes from Bastian
Parts:
- D?: Manufacturer (none) -> Littelfuse; Part Number (none) -> SMAJ12CA
Changed lines of the file:
@@
 F 2 "" H 1450 1250 50  0001 C CNN
 F 3 "~" H 1450 1250 50  0001 C CNN
+F 4 "SMAJ12CA" V 1450 1250 50  0001 C CNN "Part Number"
+F 5 "Littelfuse" V 1450 1250 50  0001 C CNN "Manufacturer"
 	1    1450 1250
 	0    1    1    0

Commit message: added buck/boost power supply for 5V rail
Parts:
- added C? (x3): 0.1uF, symbol Device:C
- added C?: 10uF, symbol Device:C
- added C?: 1uF, symbol Device:C
- added C?: 100pF, symbol Device:C
- added C?: 22pF, symbol Device:C
- added C?: 680pF, symbol Device:C
- added C?: 47pF, symbol Device:C
- added C?: 47uF, symbol Device:C
- added L?: 4.7uH, symbol Device:L
- added R?: 42.2k, symbol Device:R
- added R?: 33k, symbol Device:R
- added R?: 845k, symbol Device:R
- added R? (x2): 100k, symbol Device:R
- added R?: 158k, symbol Device:R
- added R?: 10k, symbol Device:R
- added U?: LTC3112_TSSOP20_A, TSSOP-20_FE/CA, symbol OTTOdiy_SMD-library:LTC3112_TSSOP20_A
Connections:
- net labels added: 5V_REG, 5V_REG_IOUT, PWR_PWM_SYNC
- wire segments 66 -> 149

Commit message: added power switching and extra pulls for programming lines
Parts:
- removed Q1: IRF9321PbF, Package_SO:SOIC-8_3.9x4.9mm_P1.27mm, symbol OTTOdiy_SMD-library:Q_PMOS_SSSGDDDD-Device
- removed R210: 100k, Resistor_SMD:R_0805_2012Metric_Pad1.15x1.40mm_HandSolder, symbol Device:R
- added C?: 10nF, Capacitor_SMD:C_0805_2012Metric_Pad1.15x1.40mm_HandSolder_marked, symbol Device:C
- added C? (x3): 470uF, Capacitor_SMD:C_0805_2012Metric_Pad1.15x1.40mm_HandSolder_marked, symbol Device:C
- added C?: 4.7uF, Capacitor_SMD:C_0805_2012Metric_Pad1.15x1.40mm_HandSolder_marked, symbol Device:C
- added C?: 10uF, Capacitor_SMD:C_0805_2012Metric_Pad1.15x1.40mm_HandSolder_marked, symbol Device:C
- added C?: 15pF, Capacitor_SMD:C_0805_2012Metric_Pad1.15x1.40mm_HandSolder_marked, symbol Device:C
- added L?: 2.2uH, symbol Device:L
- added R?: 100k, symbol Device:R
- added R?: 0, symbol Device:R
- added R?: 40.2k, symbol Device:R
- added R?: 182k, symbol Device:R
- added U?: TPS22918_SOT23-6_A, Package_TO_SOT_SMD:SOT-23-6, symbol OTTOdiy_SMD-library:TPS22918_SOT23-6_A
- added U?: TLV62568_SOT-23-5_A, Package_TO_SOT_SMD:SOT-23-5, symbol OTTOdiy_SMD-library:TLV62568_SOT-23-5_A
Connections:
- net labels added: +5V_PI, +5V_REG, PI_PWR_EN
- net labels removed: +5V_MAIN, +5V_MCU, 5V_REG, MAIN_POWER
- wire segments 149 -> 194
Other:
- note removed: "Connected via Jumpers \non the Expansion Header"

Commit message: connected unconnected signals and MIDI to spare MCU UART
Parts:
- removed C?: 10nF, Capacitor_SMD:C_0805_2012Metric_Pad1.15x1.40mm_HandSolder_marked, symbol Device:C
- removed R?: 100k, symbol Device:R
- removed R?: 0, symbol Device:R
- removed U?: TPS22918_SOT23-6_A, Package_TO_SOT_SMD:SOT-23-6, symbol OTTOdiy_SMD-library:TPS22918_SOT23-6_A
- added C87: 10nF, Capacitor_SMD:C_0805_2012Metric_Pad1.15x1.40mm_HandSolder_marked, symbol Device:C
- added R16: 100k, symbol Device:R
- added R17: 0, symbol Device:R
- added U5: TPS22918_SOT23-6_A, Package_TO_SOT_SMD:SOT-23-6, symbol OTTOdiy_SMD-library:TPS22918_SOT23-6_A
- gave numbers to parts that had none: 33
Connections:
- net labels added: 5V_PWM_SYNC
- net labels removed: PWR_PWM_SYNC

Commit message: add all resistor part numbers and create footprint library
Parts:
- D48: MPN (none) -> SMAJ12CA; Part Number SMAJ12CA -> (none)
- PHOTO201: EstimatedCost(USD) (none) -> $0.22; MPN (none) -> ALS-PDIC243-3B; Manufacturer (none) -> Everlight Elec
- R13, R14, R15, R16: footprint (none) -> Resistor_SMD:R_0805_2012Metric_Pad1.15x1.40mm_HandSolder; EstimatedCost(USD) (none) -> $.00169; MPN (none) -> RC0805FR-07100KL; Manufacturer (none) -> Yageo
- R17: footprint (none) -> Resistor_SMD:R_0805_2012Metric_Pad1.15x1.40mm_HandSolder; EstimatedCost(USD) (none) -> $.001203; MPN (none) -> RC0805JR-070RL; Manufacturer (none) -> Yageo
- R18: footprint (none) -> Resistor_SMD:R_0805_2012Metric_Pad1.15x1.40mm_HandSolder; EstimatedCost(USD) (none) -> $.010229; MPN (none) -> CR0805-FX-1823ELF; Manufacturer (none) -> Bourns
- R19: footprint (none) -> Resistor_SMD:R_0805_2012Metric_Pad1.15x1.40mm_HandSolder; EstimatedCost(USD) (none) -> $.001774; MPN (none) -> RC0805FR-0740K2L; Manufacturer (none) -> Yageo
- R20: footprint (none) -> Resistor_SMD:R_0805_2012Metric_Pad1.15x1.40mm_HandSolder; EstimatedCost(USD) (none) -> $.004141; MPN (none) -> RK73H2ATTD4222F; Manufacturer (none) -> KOA Speer Elec
- R21: footprint (none) -> Resistor_SMD:R_0805_2012Metric_Pad1.15x1.40mm_HandSolder; EstimatedCost(USD) (none) -> $.001703; MPN (none) -> RC0805FR-0733KL; Manufacturer (none) -> Yageo
- R211: EstimatedCost(USD) (none) -> $.001675; MPN (none) -> RC0805FR-0710KL; Manufacturer (none) -> Yageo
- R22: footprint (none) -> Resistor_SMD:R_0805_2012Metric_Pad1.15x1.40mm_HandSolder; EstimatedCost(USD) (none) -> $.009826; MPN (none) -> ERJ6ENF8453V; Manufacturer (none) -> Panasonic
- R23: footprint (none) -> Resistor_SMD:R_0805_2012Metric_Pad1.15x1.40mm_HandSolder; EstimatedCost(USD) (none) -> $.010537; MPN (none) -> CR0805-FX-1583ELF; Manufacturer (none) -> Bourns
- R24: footprint (none) -> Resistor_SMD:R_0805_2012Metric_Pad1.15x1.40mm_HandSolder; EstimatedCost(USD) (none) -> $.001675; MPN (none) -> RC0805FR-0710KL; Manufacturer (none) -> Yageo
- U3: footprint TSSOP-20_FE/CA -> OTTO_Footprints_Lib:TSSOP-20_FE_CA; MPN (none) -> LTC3112EFE-TRPBF; Manufacturer (none) -> Analog Devices; Part Number LTC3112EFE-TRPBF -> (none)
- U4: Manufacturer (none) -> Texas Instruments
Changed lines of the file:
@@
 F 1 "ALS-PDIC243-3B" H 2441 5055 50  0000 L CNN
 F 2 "OptoDevice:ALS-PDIC243-3B" H 2450 5200 50  0001 C CNN
-F 3 "~" H 2250 5100 50  0001 C CNN
+F 3 "https://datasheet.lcsc.com/szlcsc/1810281710_Everlight-Elec-ALS-PDIC243-3B_C141718.pdf" H 2250 5100 50  0001 C CNN
+F 4 "$0.22" H 2250 5100 50  0001 C CNN "EstimatedCost(USD)"
+F 5 "ALS-PDIC243-3B" H 2250 5100 50  0001 C CNN "MPN"
+F 6 "Everlight Elec" H 2250 5100 50  0001 C CNN "Manufacturer"
 	1    2250 5100
 	1    0    0    -1
@@
 F 1 "10k" H 2870 5605 50  0000 L CNN
 F 2 "Resistor_SMD:R_0805_2012Metric_Pad1.15x1.40mm_HandSolder" V 2730 5650 50  0001 C CNN
-F 3 "~" H 2800 5650 50  0001 C CNN
+F 3 "https://datasheet.lcsc.com/szlcsc/YAGEO-RC0805FR-0710KL_C84376.pdf" H 2800 5650 50  0001 C CNN
+F 4 "$.001675" H 2800 5650 50  0001 C CNN "EstimatedCost(USD)"
+F 5 "RC0805FR-0710KL" H 2800 5650 50  0001 C CNN "MPN"
+F 6 "Yageo" H 2800 5650 50  0001 C CNN "Manufacturer"
 	1    2800 5650
 	1    0    0    -1
@@
 F 2 "" H 3000 2200 50  0001 C CNN
 F 3 "~" H 3000 2200 50  0001 C CNN
-F 4 "SMAJ12CA" V 3000 2200 50  0001 C CNN "Part Number"
-F 5 "Littelfuse" V 3000 2200 50  0001 C CNN "Manufacturer"
+F 4 "Littelfuse" V 3000 2200 50  0001 C CNN "Manufacturer"
+F 5 "SMAJ12CA" H 3000 2200 50  0001 C CNN "MPN"
 	1    3000 2200
 	0    1    1    0
@@
 F 0 "R13" H 3720 2496 50  0000 L CNN
 F 1 "100k" H 3720 2405 50  0000 L CNN
-F 2 "" V 3580 2450 50  0001 C CNN
-F 3 "~" H 3650 2450 50  0001 C CNN
+F 2 "Resistor_SMD:R_0805_2012Metric_Pad1.15x1.40mm_HandSolder" V 3580 2450 50  0001 C CNN
+F 3 "https://datasheet.lcsc.com/szlcsc/YAGEO-RC0805FR-07100KL_C96346.pdf" H 3650 2450 50  0001 C CNN
+F 4 "$.00169" H 3650 2450 50  0001 C CNN "EstimatedCost(USD)"
+F 5 "RC0805FR-07100KL" H 3650 2450 50  0001 C CNN "MPN"
+F 6 "Yageo" H 3650 2450 50  0001 C CNN "Manufacturer"
 	1    3650 2450
 	1    0    0    -1
@@
 F 0 "U3" H 9250 4350 60  0000 C CNN
 F 1 "LTC3112_TSSOP20_A" H 10400 4350 60  0000 C CNN
-F 2 "TSSOP-20_FE/CA" H 10350 1650 50  0001 L BNN
+F 2 "OTTO_Footprints_Lib:TSSOP-20_FE_CA" H 10350 1650 50  0001 L BNN
 F 3 "" H 10050 3300 60  0001 C CNN
-F 4 "LTC3112EFE-TRPBF" H 10350 1750 50  0001 L BNN "Part Number"
+F 4 "LTC3112EFE-TRPBF" H 10050 3300 50  0001 C CNN "MPN"
+F 5 "Analog Devices" H 10050 3300 50  0001 C CNN "Manufacturer"
 	1    10050 3300
 	1    0    0    -1
@@
 F 0 "R20" H 12020 4196 50  0000 L CNN
 F 1 "42.2k" H 12020 4105 50  0000 L CNN
-F 2 "" V 11880 4150 50  0001 C CNN
-F 3 "~" H 11950 4150 50  0001 C CNN
+F 2 "Resistor_SMD:R_0805_2012Metric_Pad1.15x1.40mm_HandSolder" V 11880 4150 50  0001 C CNN
+F 3 "https://datasheet.lcsc.com/szlcsc/1901151033_KOA-Speer-Elec-RK73H2ATTD4222F_C317446.pdf" H 11950 4150 50  0001 C CNN
+F 4 "$.004141" H 11950 4150 50  0001 C CNN "EstimatedCost(USD)"
+F 5 "RK73H2ATTD4222F" H 11950 4150 50  0001 C CNN "MPN"
+F 6 "KOA Speer Elec" H 11950 4150 50  0001 C CNN "Manufacturer"
 	1    11950 4150
 	1    0    0    -1
@@
 F 0 "R21" V 11993 3300 50  0000 C CNN
 F 1 "33k" V 12084 3300 50  0000 C CNN
-F 2 "" V 12130 3300 50  0001 C CNN
-F 3 "~" H 12200 3300 50  0001 C CNN
+F 2 "Resistor_SMD:R_0805_2012Metric_Pad1.15x1.40mm_HandSolder" V 12130 3300 50  0001 C CNN
+F 3 "https://datasheet.lcsc.com/szlcsc/YAGEO-RC0805FR-0733KL_C141696.pdf" H 12200 3300 50  0001 C CNN
+F 4 "$.001703" H 12200 3300 50  0001 C CNN "EstimatedCost(USD)"
+F 5 "RC0805FR-0733KL" H 12200 3300 50  0001 C CNN "MPN"
+F 6 "Yageo" H 12200 3300 50  0001 C CNN "Manufacturer"
 	1    12200 3300
 	0    1    1    0
@@
 F 0 "R22" H 12720 3346 50  0000 L CNN
 F 1 "845k" H 12720 3255 50  0000 L CNN
-F 2 "" V 12580 3300 50  0001 C CNN
-F 3 "~" H 12650 3300 50  0001 C CNN
+F 2 "Resistor_SMD:R_0805_2012Metric_Pad1.15x1.40mm_HandSolder" V 12580 3300 50  0001 C CNN
+F 3 "https://datasheet.lcsc.com/szlcsc/1910291303_PANASONIC-ERJ6ENF8453V_C416871.pdf" H 12650 3300 50  0001 C CNN
+F 4 "$.009826" H 12650 3300 50  0001 C CNN "EstimatedCost(USD)"
+F 5 "ERJ6ENF8453V" H 12650 3300 50  0001 C CNN "MPN"
+F 6 "Panasonic" H 12650 3300 50  0001 C CNN "Manufacturer"
 	1    12650 3300
 	1    0    0    -1
@@
 F 0 "R23" H 12720 4196 50  0000 L CNN
 F 1 "158k" H 12720 4105 50  0000 L CNN
-F 2 "" V 12580 4150 50  0001 C CNN
-F 3 "~" H 12650 4150 50  0001 C CNN
+F 2 "Resistor_SMD:R_0805_2012Metric_Pad1.15x1.40mm_HandSolder" V 12580 4150 50  0001 C CNN
+F 3 "https://datasheet.lcsc.com/szlcsc/1812131302_BOURNS-CR0805-FX-1583ELF_C203773.pdf" H 12650 4150 50  0001 C CNN
+F 4 "$.010537" H 12650 4150 50  0001 C CNN "EstimatedCost(USD)"
+F 5 "CR0805-FX-1583ELF" H 12650 4150 50  0001 C CNN "MPN"
+F 6 "Bourns" H 12650 4150 50  0001 C CNN "Manufacturer"
 	1    12650 4150
 	1    0    0    -1
@@
 F 0 "R24" H 13120 3696 50  0000 L CNN
 F 1 "10k" H 13120 3605 50  0000 L CNN
-F 2 "" V 12980 3650 50  0001 C CNN
-F 3 "~" H 13050 3650 50  0001 C CNN
+F 2 "Resistor_SMD:R_0805_2012Metric_Pad1.15x1.40mm_HandSolder" V 12980 3650 50  0001 C CNN
+F 3 "https://datasheet.lcsc.com/szlcsc/YAGEO-RC0805FR-0710KL_C84376.pdf" H 13050 3650 50  0001 C CNN
+F 4 "$.001675" H 13050 3650 50  0001 C CNN "EstimatedCost(USD)"
+F 5 "RC0805FR-0710KL" H 13050 3650 50  0001 C CNN "MPN"
+F 6 "Yageo" H 13050 3650 50  0001 C CNN "Manufacturer"
 	1    13050 3650
 	1    0    0    -1
@@
 F 0 "R16" H 9570 9096 50  0000 L CNN
 F 1 "100k" H 9570 9005 50  0000 L CNN
-F 2 "" V 9430 9050 50  0001 C CNN
-F 3 "~" H 9500 9050 50  0001 C CNN
+F 2 "Resistor_SMD:R_0805_2012Metric_Pad1.15x1.40mm_HandSolder" V 9430 9050 50  0001 C CNN
+F 3 "https://datasheet.lcsc.com/szlcsc/YAGEO-RC0805FR-07100KL_C96346.pdf" H 9500 9050 50  0001 C CNN
+F 4 "$.00169" H 9500 9050 50  0001 C CNN "EstimatedCost(USD)"
+F 5 "RC0805FR-07100KL" H 9500 9050 50  0001 C CNN "MPN"
+F 6 "Yageo" H 9500 9050 50  0001 C CNN "Manufacturer"
 	1    9500 9050
 	1    0    0    -1
@@
 F 0 "R17" V 10594 8050 50  0000 C CNN
 F 1 "0" V 10685 8050 50  0000 C CNN
-F 2 "" V 10730 8050 50  0001 C CNN
-F 3 "~" H 10800 8050 50  0001 C CNN
+F 2 "Resistor_SMD:R_0805_2012Metric_Pad1.15x1.40mm_HandSolder" V 10730 8050 50  0001 C CNN
+F 3 "https://datasheet.lcsc.com/szlcsc/YAGEO-RC0805JR-070RL_C96345.pdf" H 10800 8050 50  0001 C CNN
+F 4 "$.001203" H 10800 8050 50  0001 C CNN "EstimatedCost(USD)"
+F 5 "RC0805JR-070RL" H 10800 8050 50  0001 C CNN "MPN"
+F 6 "Yageo" H 10800 8050 50  0001 C CNN "Manufacturer"
 	1    10800 8050
 	0    1    1    0
@@
 F 3 "http://www.ti.com/lit/ds/symlink/tlv62568.pdf" H 9800 6150 50  0001 C CNN
 F 4 "TLV62568DBVR" H 10450 5350 50  0001 C CNN "MPN"
+F 5 "Texas Instruments" H 10050 5700 50  0001 C CNN "Manufacturer"
 	1    10050 5700
 	1    0    0    -1
@@
 F 0 "R19" H 11770 6846 50  0000 L CNN
 F 1 "40.2k" H 11770 6755 50  0000 L CNN
-F 2 "" V 11630 6800 50  0001 C CNN
-F 3 "~" H 11700 6800 50  0001 C CNN
+F 2 "Resistor_SMD:R_0805_2012Metric_Pad1.15x1.40mm_HandSolder" V 11630 6800 50  0001 C CNN
+F 3 "https://datasheet.lcsc.com/szlcsc/YAGEO-RC0805FR-0740K2L_C273827.pdf" H 11700 6800 50  0001 C CNN
+F 4 "RC0805FR-0740K2L" H 11700 6800 50  0001 C CNN "MPN"
+F 5 "$.001774" H 11700 6800 50  0001 C CNN "EstimatedCost(USD)"
+F 6 "Yageo" H 11700 6800 50  0001 C CNN "Manufacturer"
 	1    11700 6800
 	1    0    0    -1
@@
 F 0 "R18" H 11770 6096 50  0000 L CNN
 F 1 "182k" H 11770 6005 50  0000 L CNN
-F 2 "" V 11630 6050 50  0001 C CNN
-F 3 "~" H 11700 6050 50  0001 C CNN
+F 2 "Resistor_SMD:R_0805_2012Metric_Pad1.15x1.40mm_HandSolder" V 11630 6050 50  0001 C CNN
+F 3 "https://datasheet.lcsc.com/szlcsc/1812131302_BOURNS-CR0805-FX-1823ELF_C203816.pdf" H 11700 6050 50  0001 C CNN
+F 4 "$.010229" H 11700 6050 50  0001 C CNN "EstimatedCost(USD)"
+F 5 "CR0805-FX-1823ELF" H 11700 6050 50  0001 C CNN "MPN"
+F 6 "Bourns" H 11700 6050 50  0001 C CNN "Manufacturer"
 	1    11700 6050
 	1    0    0    -1
@@
 F 0 "R14" H 7970 4396 50  0000 L CNN
 F 1 "100k" H 7970 4305 50  0000 L CNN
-F 2 "" V 7830 4350 50  0001 C CNN
-F 3 "~" H 7900 4350 50  0001 C CNN
+F 2 "Resistor_SMD:R_0805_2012Metric_Pad1.15x1.40mm_HandSolder" V 7830 4350 50  0001 C CNN
+F 3 "https://datasheet.lcsc.com/szlcsc/YAGEO-RC0805FR-07100KL_C96346.pdf" H 7900 4350 50  0001 C CNN
+F 4 "$.00169" H 7900 4350 50  0001 C CNN "EstimatedCost(USD)"
+F 5 "RC0805FR-07100KL" H 7900 4350 50  0001 C CNN "MPN"
+F 6 "Yageo" H 7900 4350 50  0001 C CNN "Manufacturer"
 	1    7900 4350
 	1    0    0    -1
@@
 F 0 "R15" H 8370 3496 50  0000 L CNN
 F 1 "100k" H 8370 3405 50  0000 L CNN
-F 2 "" V 8230 3450 50  0001 C CNN
-F 3 "~" H 8300 3450 50  0001 C CNN
+F 2 "Resistor_SMD:R_0805_2012Metric_Pad1.15x1.40mm_HandSolder" V 8230 3450 50  0001 C CNN
+F 3 "https://datasheet.lcsc.com/szlcsc/YAGEO-RC0805FR-07100KL_C96346.pdf" H 8300 3450 50  0001 C CNN
+F 4 "$.00169" H 8300 3450 50  0001 C CNN "EstimatedCost(USD)"
+F 5 "RC0805FR-07100KL" H 8300 3450 50  0001 C CNN "MPN"
+F 6 "Yageo" H 8300 3450 50  0001 C CNN "Manufacturer"
 	1    8300 3450
 	1    0    0    -1

Commit message: added part numbers for capacitors and crystals
Parts:
- removed C79, C81, C84: 470uF, Capacitor_SMD:C_0805_2012Metric_Pad1.15x1.40mm_HandSolder_marked, symbol Device:C
- added C79, C81, C84: 470uF, Capacitor_SMD:C_Elec_6.3x7.7, symbol Device:CP
- C232: value 10µF -> 10uF
- C58, C59: footprint Capacitor_SMD:C_0805_2012Metric_Pad1.15x1.40mm_HandSolder_marked -> Capacitor_SMD:C_0805_2012Metric_Pad1.15x1.40mm_HandSolder; EstimatedCost(USD) (none) -> $0.017724; MPN (none) -> CL21B104JBCNNNC; Manufacturer (none) -> Samsung Electro-Mechanics
- C80, C85, C92, C94: footprint (none) -> Capacitor_SMD:C_0805_2012Metric_Pad1.15x1.40mm_HandSolder
- C82, C83, C91: value 0.1uF -> 100nF; footprint (none) -> Capacitor_SMD:C_0805_2012Metric_Pad1.15x1.40mm_HandSolder; EstimatedCost(USD) (none) -> $0.017724; MPN (none) -> CL21B104JBCNNNC; Manufacturer (none) -> Samsung Electro-Mechanics
- C86, C88, C93: footprint Capacitor_SMD:C_0805_2012Metric_Pad1.15x1.40mm_HandSolder_marked -> Capacitor_SMD:C_0805_2012Metric_Pad1.15x1.40mm_HandSolder
- C87: footprint Capacitor_SMD:C_0805_2012Metric_Pad1.15x1.40mm_HandSolder_marked -> Capacitor_SMD:C_0805_2012Metric_Pad1.15x1.40mm_HandSolder; EstimatedCost(USD) (none) -> $0.007546; MPN (none) -> CL21B103KBCNNNC; Manufacturer (none) -> Samsung Electro-Mechanics
- C89: footprint (none) -> Capacitor_SMD:C_0805_2012Metric_Pad1.15x1.40mm_HandSolder; EstimatedCost(USD) (none) -> $0.009476; MPN (none) -> CL21C220JBANNNC; Manufacturer (none) -> Samsung Electro-Mechanics
- C90: value 100pF -> 100nF; footprint (none) -> Capacitor_SMD:C_0805_2012Metric_Pad1.15x1.40mm_HandSolder; EstimatedCost(USD) (none) -> $0.017724; MPN (none) -> CL21B104JBCNNNC; Manufacturer (none) -> Samsung Electro-Mechanics
- C95: footprint (none) -> Capacitor_SMD:C_1206_3216Metric_Pad1.42x1.75mm_HandSolder; EstimatedCost(USD) (none) -> $0.390909; MPN (none) -> GRM31CR61E476ME44L; Manufacturer (none) -> Murata Electronics
- DISPLAY201: AssemblyOption (none) -> DNP

Commit message: more part numbers added: audio caps
Parts:
- C232, C80, C88: EstimatedCost(USD) (none) -> $0.041113; MPN (none) -> CL21B106KOQNNNE; Manufacturer (none) -> Samsung Electro-Mechanics
- C85: EstimatedCost(USD) (none) -> $0.067176; MPN (none) -> CL21B105KBFVPNE; Manufacturer (none) -> Samsung Electro-Mechanics
- C86: EstimatedCost(USD) (none) -> $0.031439; MPN (none) -> CL21B475KAFNNNE; Manufacturer (none) -> Samsung Electro-Mechanics
- C92: EstimatedCost(USD) (none) -> $0.008589; MPN (none) -> CC0805JRNPO9BN681; Manufacturer (none) -> Yageo
- C93: EstimatedCost(USD) (none) -> $0.00985; MPN (none) -> CL21C150JBANNNC; Manufacturer (none) -> Samsung Electro-Mechanics
- C94: EstimatedCost(USD) (none) -> $0.022222; MPN (none) -> CC0805JRNPO9BN470; Manufacturer (none) -> Yageo
Changed lines of the file:
@@
 F 1 "10uF" H 3315 6755 50  0000 L CNN
 F 2 "Capacitor_SMD:C_0805_2012Metric_Pad1.15x1.40mm_HandSolder" H 3238 6650 50  0001 C CNN
-F 3 "~" H 3200 6800 50  0001 C CNN
+F 3 "https://datasheet.lcsc.com/szlcsc/Samsung-Electro-Mechanics-CL21B106KOQNNNE_C95841.pdf" H 3200 6800 50  0001 C CNN
+F 4 "$0.041113" H 3200 6800 50  0001 C CNN "EstimatedCost(USD)"
+F 5 "CL21B106KOQNNNE" H 3200 6800 50  0001 C CNN "MPN"
+F 6 "Samsung Electro-Mechanics" H 3200 6800 50  0001 C CNN "Manufacturer"
 	1    3200 6800
 	1    0    0    -1
@@
 F 1 "680pF" V 11639 3300 50  0000 C CNN
 F 2 "Capacitor_SMD:C_0805_2012Metric_Pad1.15x1.40mm_HandSolder" H 11838 3150 50  0001 C CNN
-F 3 "~" H 11800 3300 50  0001 C CNN
+F 3 "https://datasheet.lcsc.com/szlcsc/YAGEO-CC0805JRNPO9BN681_C107121.pdf" H 11800 3300 50  0001 C CNN
+F 4 "$0.008589" H 11800 3300 50  0001 C CNN "EstimatedCost(USD)"
+F 5 "CC0805JRNPO9BN681" H 11800 3300 50  0001 C CNN "MPN"
+F 6 "Yageo" H 11800 3300 50  0001 C CNN "Manufacturer"
 	1    11800 3300
 	0    1    1    0
@@
 F 1 "47pF" H 13165 3205 50  0000 L CNN
 F 2 "Capacitor_SMD:C_0805_2012Metric_Pad1.15x1.40mm_HandSolder" H 13088 3100 50  0001 C CNN
-F 3 "~" H 13050 3250 50  0001 C CNN
+F 3 "https://datasheet.lcsc.com/szlcsc/YAGEO-CC0805JRNPO9BN470_C107118.pdf" H 13050 3250 50  0001 C CNN
+F 4 "$0.022222" H 13050 3250 50  0001 C CNN "EstimatedCost(USD)"
+F 5 "CC0805JRNPO9BN470" H 13050 3250 50  0001 C CNN "MPN"
+F 6 "Yageo" H 13050 3250 50  0001 C CNN "Manufacturer"
 	1    13050 3250
 	1    0    0    -1
@@
 F 1 "4.7uF" H 8965 5855 50  0000 L CNN
 F 2 "Capacitor_SMD:C_0805_2012Metric_Pad1.15x1.40mm_HandSolder" H 8888 5750 50  0001 C CNN
-F 3 "~" H 8850 5900 50  0001 C CNN
+F 3 "https://datasheet.lcsc.com/szlcsc/Samsung-Electro-Mechanics-CL21B475KAFNNNE_C98195.pdf" H 8850 5900 50  0001 C CNN
+F 4 "$0.031439" H 8850 5900 50  0001 C CNN "EstimatedCost(USD)"
+F 5 "CL21B475KAFNNNE" H 8850 5900 50  0001 C CNN "MPN"
+F 6 "Samsung Electro-Mechanics" H 8850 5900 50  0001 C CNN "Manufacturer"
 	1    8850 5900
 	1    0    0    -1
@@
 F 1 "10uF" H 11315 5855 50  0000 L CNN
 F 2 "Capacitor_SMD:C_0805_2012Metric_Pad1.15x1.40mm_HandSolder" H 11238 5750 50  0001 C CNN
-F 3 "~" H 11200 5900 50  0001 C CNN
+F 3 "https://datasheet.lcsc.com/szlcsc/Samsung-Electro-Mechanics-CL21B106KOQNNNE_C95841.pdf" H 11200 5900 50  0001 C CNN
+F 4 "$0.041113" H 11200 5900 50  0001 C CNN "EstimatedCost(USD)"
+F 5 "CL21B106KOQNNNE" H 11200 5900 50  0001 C CNN "MPN"
+F 6 "Samsung Electro-Mechanics" H 11200 5900 50  0001 C CNN "Manufacturer"
 	1    11200 5900
 	1    0    0    -1
@@
 F 1 "15pF" H 12265 6005 50  0000 L CNN
 F 2 "Capacitor_SMD:C_0805_2012Metric_Pad1.15x1.40mm_HandSolder" H 12188 5900 50  0001 C CNN
-F 3 "~" H 12150 6050 50  0001 C CNN
+F 3 "https://datasheet.lcsc.com/szlcsc/Samsung-Electro-Mechanics-CL21C150JBANNNC_C1794.pdf" H 12150 6050 50  0001 C CNN
+F 4 "$0.00985" H 12150 6050 50  0001 C CNN "EstimatedCost(USD)"
+F 5 "CL21C150JBANNNC" H 12150 6050 50  0001 C CNN "MPN"
+F 6 "Samsung Electro-Mechanics" H 12150 6050 50  0001 C CNN "Manufacturer"
 	1    12150 6050
 	1    0    0    -1
@@
 F 1 "10uF" H 7965 3305 50  0000 L CNN
 F 2 "Capacitor_SMD:C_0805_2012Metric_Pad1.15x1.40mm_HandSolder" H 7888 3200 50  0001 C CNN
-F 3 "~" H 7850 3350 50  0001 C CNN
+F 3 "https://datasheet.lcsc.com/szlcsc/Samsung-Electro-Mechanics-CL21B106KOQNNNE_C95841.pdf" H 7850 3350 50  0001 C CNN
+F 4 "$0.041113" H 7850 3350 50  0001 C CNN "EstimatedCost(USD)"
+F 5 "CL21B106KOQNNNE" H 7850 3350 50  0001 C CNN "MPN"
+F 6 "Samsung Electro-Mechanics" H 7850 3350 50  0001 C CNN "Manufacturer"
 	1    7850 3350
 	1    0    0    -1
@@
 F 1 "1uF" H 8815 3405 50  0000 L CNN
 F 2 "Capacitor_SMD:C_0805_2012Metric_Pad1.15x1.40mm_HandSolder" H 8738 3300 50  0001 C CNN
-F 3 "~" H 8700 3450 50  0001 C CNN
+F 3 "https://datasheet.lcsc.com/szlcsc/Samsung-Electro-Mechanics-CL21B105KBFVPNE_C307362.pdf" H 8700 3450 50  0001 C CNN
+F 4 "$0.067176" H 8700 3450 50  0001 C CNN "EstimatedCost(USD)"
+F 5 "CL21B105KBFVPNE" H 8700 3450 50  0001 C CNN "MPN"
+F 6 "Samsung Electro-Mechanics" H 8700 3450 50  0001 C CNN "Manufacturer"
 	1    8700 3450
 	1    0    0    -1
