File: KiCad/PERIPHERALS.sch (KiCad schematic (older format))
At the start: 49 parts, among them CN201 1x4 MALE 1.25mm, CN202 1x4 MALE 1.25mm, Q1 IRF9321PbF, SW203 ALPS SKHH angled, U204 USB6B1, U3 LTC3112_TSSOP20_A, U4 TLV62568_SOT-23-5_A, U5 TPS22918_SOT23-6_A

Commit message: add switch and encoder parts. BM Complete. Footprints complete.
Parts:
- L1: footprint (none) -> OTTO_Footprints_Lib:L_7.3x6.6_H3; EstimatedCost(USD) (none) -> $0.078246; MPN (none) -> MCS0630-4R7MN2; Manufacturer (none) -> PSA(Prosperity Dielectrics)
- L2: footprint (none) -> OTTO_Footprints_Lib:L_7.3x6.6_H3; EstimatedCost(USD) (none) -> $0.078246; MPN (none) -> MCS0630-2R2MN2; Manufacturer (none) -> PSA(Prosperity Dielectrics)
- PHOTO201: footprint OptoDevice:ALS-PDIC243-3B -> OTTO_Footprints_Lib:ALS-PDIC243-3B
- Q1: value IRF9321PbF -> AO4485; EstimatedCost(USD) (none) -> $0.284848; MPN (none) -> AO4485; Manufacturer (none) -> Alpha & Omega Semicon
- SW203: value ALPS SKHH angled -> 6x6x5.85mm (RA); EstimatedCost(USD) (none) -> $0.134848; MPN (none) -> SKHHLWA010; Manufacturer (none) -> ALPS Electric
- U204: EstimatedCost(USD) (none) -> $0.689394; MPN (none) -> USB6B1; Manufacturer (none) -> STMicroelectronics
- U3: EstimatedCost(USD) (none) -> $4.06; MPN LTC3112EFE-TRPBF -> LTC3112EFE#PBF
- U4: EstimatedCost(USD) (none) -> $0.083576
- U5: EstimatedCost(USD) (none) -> $0.228788; MPN (none) -> TPS22918DBVR; Manufacturer (none) -> Texas Instruments
- USB201: footprint Spatz:USB_B -> OTTO_Footprints_Lib:USB_B; EstimatedCost(USD) (none) -> $0.40303; MPN (none) -> 292304-1; Manufacturer (none) -> TE Connectivity
Changed lines of the file:
@@
 F 0 "PHOTO201" H 2441 5146 50  0000 L CNN
 F 1 "ALS-PDIC243-3B" H 2441 5055 50  0000 L CNN
-F 2 "OptoDevice:ALS-PDIC243-3B" H 2450 5200 50  0001 C CNN
+F 2 "OTTO_Footprints_Lib:ALS-PDIC243-3B" H 2450 5200 50  0001 C CNN
 F 3 "https://datasheet.lcsc.com/szlcsc/1810281710_Everlight-Elec-ALS-PDIC243-3B_C141718.pdf" H 2250 5100 50  0001 C CNN
 F 4 "$0.22" H 2250 5100 50  0001 C CNN "EstimatedCost(USD)"
@@
 F 0 "USB201" H 2605 4017 50  0000 C CNN
 F 1 "USB_B" H 2605 3926 50  0000 C CNN
-F 2 "Spatz:USB_B" H 2700 3500 50  0001 C CNN
-F 3 " ~" H 2700 3500 50  0001 C CNN
+F 2 "OTTO_Footprints_Lib:USB_B" H 2700 3500 50  0001 C CNN
+F 3 "https://datasheet.lcsc.com/szlcsc/TE-Connectivity-292304-1_C86462.pdf" H 2700 3500 50  0001 C CNN
+F 4 "$0.40303" H 2550 3550 12700 0001 C CNN "EstimatedCost(USD)"
+F 5 "292304-1" H 2550 3550 12700 0001 C CNN "MPN"
+F 6 "TE Connectivity" H 2550 3550 12700 0001 C CNN "Manufacturer"
 	1    2550 3550
 	1    0    0    -1
@@
 AR Path="/5C4320DF/5C4AB597/5D34A785" Ref="SW203"  Part="1"
 F 0 "SW203" H 4000 5735 50  0000 C CNN
-F 1 "ALPS SKHH angled" H 4000 5644 50  0000 C CNN
+F 1 "6x6x5.85mm (RA)" H 4000 5644 50  0000 C CNN
 F 2 "Button_Switch_THT:SW_Tactile_SKHH_Angled" H 4000 5650 50  0001 C CNN
-F 3 "" H 4000 5650 50  0001 C CNN
+F 3 "https://datasheet.lcsc.com/szlcsc/ALPS-Electric-SKHHLWA010_C125050.pdf" H 4000 5650 50  0001 C CNN
+F 4 "$0.134848" H 4000 5450 12700 0001 C CNN "EstimatedCost(USD)"
+F 5 "SKHHLWA010" H 4000 5450 12700 0001 C CNN "MPN"
+F 6 "ALPS Electric" H 4000 5450 12700 0001 C CNN "Manufacturer"
 	1    4000 5450
 	-1   0    0    -1
@@
 AR Path="/5C4320DF/5C4AB597/5E314238" Ref="Q1"  Part="1"
 F 0 "Q1" V 3993 1950 50  0000 C CNN
-F 1 "IRF9321PbF" V 3902 1950 50  0000 C CNN
+F 1 "AO4485" V 3902 1950 50  0000 C CNN
 F 2 "Package_SO:SOIC-8_3.9x4.9mm_P1.27mm" H 3850 2050 50  0001 C CNN
-F 3 "~" H 3650 1950 50  0001 C CNN
+F 3 "https://datasheet.lcsc.com/szlcsc/Alpha-Omega-Semicon-AOS-AO4485_C51499.pdf" H 3650 1950 50  0001 C CNN
+F 4 "$0.284848" H 3650 1950 12700 0001 C CNN "EstimatedCost(USD)"
+F 5 "AO4485" H 3650 1950 12700 0001 C CNN "MPN"
+F 6 "Alpha & Omega Semicon" H 3650 1950 12700 0001 C CNN "Manufacturer"
 	1    3650 1950
 	0    -1   -1   0
@@
 F 2 "OTTO_Footprints_Lib:TSSOP-20_FE_CA" H 10350 1650 50  0001 L BNN
 F 3 "https://www.analog.com/media/en/technical-documentation/data-sheets/3112fd.pdf" H 10050 3300 60  0001 C CNN
-F 4 "LTC3112EFE-TRPBF" H 10050 3300 50  0001 C CNN "MPN"
+F 4 "LTC3112EFE#PBF" H 10050 3300 50  0001 C CNN "MPN"
 F 5 "Analog Devices" H 10050 3300 50  0001 C CNN "Manufacturer"
+F 6 "$4.06" H 10050 3300 12700 0001 C CNN "EstimatedCost(USD)"
 	1    10050 3300
 	1    0    0    -1
@@
 F 0 "L1" V 9869 1850 50  0000 C CNN
 F 1 "4.7uH" V 9960 1850 50  0000 C CNN
-F 2 "" H 10050 1850 50  0001 C CNN
-F 3 "~" H 10050 1850 50  0001 C CNN
+F 2 "OTTO_Footprints_Lib:L_7.3x6.6_H3" H 10050 1850 50  0001 C CNN
+F 3 "https://datasheet.lcsc.com/szlcsc/1904111131_Prosperity-Dielectrics-MCS0630-4R7MN2_C385253.pdf" H 10050 1850 50  0001 C CNN
+F 4 "$0.078246" H 10050 1850 12700 0001 C CNN "EstimatedCost(USD)"
+F 5 "MCS0630-4R7MN2" H 10050 1850 12700 0001 C CNN "MPN"
+F 6 "PSA(Prosperity Dielectrics)" H 10050 1850 12700 0001 C CNN "Manufacturer"
 	1    10050 1850
 	0    1    1    0
@@
 F 2 "Package_TO_SOT_SMD:SOT-23-6" H 10050 8350 50  0001 C CNN
 F 3 "http://www.ti.com/lit/ds/symlink/tps22918.pdf" H 10100 7150 50  0001 C CNN
+F 4 "$0.228788" H 10050 7850 12700 0001 C CNN "EstimatedCost(USD)"
+F 5 "TPS22918DBVR" H 10050 7850 12700 0001 C CNN "MPN"
+F 6 "Texas Instruments" H 10050 7850 12700 0001 C CNN "Manufacturer"
 	1    10050 7850
 	1    0    0    -1
@@
 F 4 "TLV62568DBVR" H 10450 5350 50  0001 C CNN "MPN"
 F 5 "Texas Instruments" H 10050 5700 50  0001 C CNN "Manufacturer"
+F 6 "$0.083576" H 10050 5700 12700 0001 C CNN "EstimatedCost(USD)"
 	1    10050 5700
 	1    0    0    -1
@@
 F 0 "L2" V 11089 5600 50  0000 C CNN
 F 1 "2.2uH" V 10998 5600 50  0000 C CNN
-F 2 "" H 10900 5600 50  0001 C CNN
-F 3 "~" H 10900 5600 50  0001 C CNN
+F 2 "OTTO_Footprints_Lib:L_7.3x6.6_H3" H 10900 5600 50  0001 C CNN
+F 3 "https://datasheet.lcsc.com/szlcsc/1904111131_Prosperity-Dielectrics-MCS0630-2R2MN2_C385252.pdf" H 10900 5600 50  0001 C CNN
+F 4 "$0.078246" H 10900 5600 12700 0001 C CNN "EstimatedCost(USD)"
+F 5 "MCS0630-2R2MN2" H 10900 5600 12700 0001 C CNN "MPN"
+F 6 "PSA(Prosperity Dielectrics)" H 10900 5600 12700 0001 C CNN "Manufacturer"
 	1    10900 5600
 	0    -1   -1   0
@@
 F 2 "Package_SO:SOIC-8_3.9x4.9mm_P1.27mm" H 3950 3650 50  0001 C CNN
 F 3 "http://www.st.com/content/ccc/resource/technical/document/datasheet/3e/ec/b2/54/b2/76/47/90/CD00001361.pdf/files/CD00001361.pdf/jcr:content/translations/en.CD00001361.pdf" H 3000 3550 50  0001 C CNN
+F 4 "$0.689394" H 3950 3650 12700 0001 C CNN "EstimatedCost(USD)"
+F 5 "USB6B1" H 3950 3650 12700 0001 C CNN "MPN"
+F 6 "STMicroelectronics" H 3950 3650 12700 0001 C CNN "Manufacturer"
 	1    3950 3650
 	-1   0    0    -1

Commit message: add BOM scripts, fix schematic hierarchy
Parts:
- added C76: 47uF, Capacitor_SMD:C_1206_3216Metric_Pad1.42x1.75mm_HandSolder, symbol Device:C
- added C77: 10nF, Capacitor_SMD:C_0805_2012Metric_Pad1.15x1.40mm_HandSolder, symbol Device:C
- added R10: 100k, Resistor_SMD:R_0805_2012Metric_Pad1.15x1.40mm_HandSolder, symbol Device:R
- added R12: 0, Resistor_SMD:R_0805_2012Metric_Pad1.15x1.40mm_HandSolder, symbol Device:R
- added SW48: SW_DIP_x02, OTTO_Footprints_Lib:SW_DIP_SPSTx02_Slide_HRO_EP-02KS, symbol Switch:SW_DIP_x02
- added U2: TPS22918_SOT23-6_A, Package_TO_SOT_SMD:SOT-23-6, symbol OTTOdiy_SMD-library:TPS22918_SOT23-6_A
- C232, C80, C88: EstimatedCost(USD) $0.041113 -> (none); UnitCost(USD) (none) -> $0.041113
- C58, C59, C82, C83, C90, C91: EstimatedCost(USD) $0.017724 -> (none); UnitCost(USD) (none) -> $0.017724
- C79, C81, C84: EstimatedCost(USD) $0.03996 -> (none); UnitCost(USD) (none) -> $0.03996
- C85: EstimatedCost(USD) $0.067176 -> (none); UnitCost(USD) (none) -> $0.067176
- C86: EstimatedCost(USD) $0.031439 -> (none); UnitCost(USD) (none) -> $0.031439
- C87: EstimatedCost(USD) $0.007546 -> (none); UnitCost(USD) (none) -> $0.007546
- C89: EstimatedCost(USD) $0.009476 -> (none); UnitCost(USD) (none) -> $0.009476
- C92: EstimatedCost(USD) $0.008589 -> (none); UnitCost(USD) (none) -> $0.008589
- C93: EstimatedCost(USD) $0.00985 -> (none); UnitCost(USD) (none) -> $0.00985
- C94: EstimatedCost(USD) $0.022222 -> (none); UnitCost(USD) (none) -> $0.022222
- C95: EstimatedCost(USD) $0.390909 -> (none); UnitCost(USD) (none) -> $0.390909
- CN201, CN202: value 1x4 MALE 1.25mm -> 1x4 MALE Molex PicoBlade; EstimatedCost(USD) $0.156061 -> (none); UnitCost(USD) (none) -> $0.156061
- D48: value 15V -> 15V BI TVS; EstimatedCost(USD) $0.029539 -> (none); UnitCost(USD) (none) -> $0.029539
- D49: value 15V -> 15V ZENER; EstimatedCost(USD) $0.010021 -> (none); UnitCost(USD) (none) -> $0.010021
- DC201: value Barrel_Jack_Switch_2.0mmID_6.5mmOD -> Barrel Jack, 2.0mmID, 6.5mmOD; EstimatedCost(USD) $0.034374 -> (none); UnitCost(USD) (none) -> $0.034374
- DISPLAY201: value 2.8INCH_IPS_SPI -> 2.8 Inch IPS Display, SPI Interface; EstimatedCost(USD) $8.68 -> (none); UnitCost(USD) (none) -> $8.68
- L1, L2: EstimatedCost(USD) $0.078246 -> (none); UnitCost(USD) (none) -> $0.078246
- PHOTO201: EstimatedCost(USD) $0.22 -> (none); UnitCost(USD) (none) -> $0.22
- Q1: EstimatedCost(USD) $0.284848 -> (none); UnitCost(USD) (none) -> $0.284848
- R13, R14, R15, R16: EstimatedCost(USD) $.00169 -> (none); UnitCost(USD) (none) -> $.00169
- R17: EstimatedCost(USD) $.001203 -> (none); UnitCost(USD) (none) -> $.001203
- R18: EstimatedCost(USD) $.010229 -> (none); UnitCost(USD) (none) -> $.010229
- R19: EstimatedCost(USD) $.001774 -> (none); UnitCost(USD) (none) -> $.001774
- R20: EstimatedCost(USD) $.004141 -> (none); UnitCost(USD) (none) -> $.004141
- R21: EstimatedCost(USD) $.001703 -> (none); UnitCost(USD) (none) -> $.001703
- R211, R24: EstimatedCost(USD) $.001675 -> (none); UnitCost(USD) (none) -> $.001675
- R22: EstimatedCost(USD) $.009826 -> (none); UnitCost(USD) (none) -> $.009826
- R23: EstimatedCost(USD) $.010537 -> (none); UnitCost(USD) (none) -> $.010537
- SW203: EstimatedCost(USD) $0.134848 -> (none); UnitCost(USD) (none) -> $0.134848
- U204: EstimatedCost(USD) $0.689394 -> (none); UnitCost(USD) (none) -> $0.689394
- U3: EstimatedCost(USD) $4.06 -> (none); UnitCost(USD) (none) -> $4.06
- U4: EstimatedCost(USD) $0.083576 -> (none); UnitCost(USD) (none) -> $0.083576
- U5: EstimatedCost(USD) $0.228788 -> (none); UnitCost(USD) (none) -> $0.228788
- USB201: EstimatedCost(USD) $0.40303 -> (none); UnitCost(USD) (none) -> $0.40303
Connections:
- net labels added: +5V_LEDS, LED_PWR_EN
- wire segments 196 -> 227
Other:
- note added: "Power Override\n"

Commit message: Add power switch and other misc nice to haves
Parts:
- added SW49: SW_SPDT, Button_Switch_SMD:SW_SPDT_CK-JS102011SAQN, symbol Switch:SW_SPDT
Connections:
- net labels added: +3V3A_MCU, +5V_USB, BARREL_IN
- wire segments 227 -> 239
Other:
- note added: "Power Select\n"

Commit message: Fixes for external battery board and Routing started
Parts:
- removed SW49: SW_SPDT, Button_Switch_SMD:SW_SPDT_CK-JS102011SAQN, symbol Switch:SW_SPDT
- added SW49: SW_SP3T (DP3T Parallel), OTTO_Footprints_Lib:SW_SP3T_CK-JS203011JCQN, symbol Switch:SW_SP3T
Connections:
- net labels added: +5V_RASPI, 5V_RUN, BATT_IN
- net labels removed: +5V_PI
- wire segments 239 -> 245
Changed lines of the file:
@@
 Connection ~ 12800 6350
 Text GLabel 13250 6350 2    50   Output ~ 0
-+5V_PI
++5V_RASPI
 Wire Wire Line
 	8800 6350 9350 6350
@@
 L power:GND #PWR0137
 U 1 1 5DFD152B
-P 8350 3550
-F 0 "#PWR0137" H 8350 3300 50  0001 C CNN
-F 1 "GND" H 8355 3377 50  0000 C CNN
-F 2 "" H 8350 3550 50  0001 C CNN
-F 3 "" H 8350 3550 50  0001 C CNN
-	1    8350 3550
+P 8550 3550
+F 0 "#PWR0137" H 8550 3300 50  0001 C CNN
+F 1 "GND" H 8555 3377 50  0000 C CNN
+F 2 "" H 8550 3550 50  0001 C CNN
+F 3 "" H 8550 3550 50  0001 C CNN
+	1    8550 3550
 	1    0    0    -1
 $EndComp
@@
 L Device:C C82
 U 1 1 5DFCE5AF
-P 8350 3300
-F 0 "C82" H 8465 3346 50  0000 L CNN
-F 1 "100nF" H 8465 3255 50  0000 L CNN
-F 2 "Capacitor_SMD:C_0805_2012Metric_Pad1.15x1.40mm_HandSolder" H 8388 3150 50  0001 C CNN
-F 3 "https://datasheet.lcsc.com/szlcsc/Samsung-Electro-Mechanics-CL21B104JBCNNNC_C62912.pdf" H 8350 3300 50  0001 C CNN
-F 4 "$0.017724" H 8350 3300 12700 0001 C CNN "UnitCost(USD)"
-F 5 "CL21B104JBCNNNC" H 8350 3300 12700 0001 C CNN "MPN"
-F 6 "Samsung Electro-Mechanics" H 8350 3300 12700 0001 C CNN "Manufacturer"
-	1    8350 3300
+P 8550 3300
+F 0 "C82" H 8665 3346 50  0000 L CNN
+F 1 "100nF" H 8665 3255 50  0000 L CNN
+F 2 "Capacitor_SMD:C_0805_2012Metric_Pad1.15x1.40mm_HandSolder" H 8588 3150 50  0001 C CNN
+F 3 "https://datasheet.lcsc.com/szlcsc/Samsung-Electro-Mechanics-CL21B104JBCNNNC_C62912.pdf" H 8550 3300 50  0001 C CNN
+F 4 "$0.017724" H 8550 3300 12700 0001 C CNN "UnitCost(USD)"
+F 5 "CL21B104JBCNNNC" H 8550 3300 12700 0001 C CNN "MPN"
+F 6 "Samsung Electro-Mechanics" H 8550 3300 12700 0001 C CNN "Manufacturer"
+	1    8550 3300
 	1    0    0    -1
 $EndComp
@@
 	7950 3550 7950 3450
 Wire Wire Line
-	8350 3550 8350 3450
-Wire Wire Line
-	8350 3050 8350 3150
+	8550 3550 8550 3450
 Wire Wire Line
 	8350 1950 7900 1950
@@
 	8350 3050 8350 2550
 Wire Wire Line
-	8950 3050 8350 3050
+	8950 3050 8550 3050
 Wire Wire Line
 	7900 2450 7900 2500
@@
 Text GLabel 2650 7150 0    50   Input ~ 0
 BL_PWM
-$Comp
-L Switch:SW_SPDT SW49
-U 1 1 5E20BC7B
-P 6700 1950
-F 0 "SW49" H 6700 1625 50  0000 C CNN
-F 1 "SW_SPDT" H 6700 1716 50  0000 C CNN
-F 2 "Button_Switch_SMD:SW_SPDT_CK-JS102011SAQN" H 6700 1950 50  0001 C CNN
-F 3 "https://datasheet.lcsc.com/szlcsc/1810301448_XKB-Enterprise-SS-12D11L5_C319010.pdf" H 6700 1950 50  0001 C CNN
-F 4 "SS-12D11L5" H 6700 1950 50  0001 C CNN "MPN"
-F 5 "XKB Enterprise" H 6700 1950 50  0001 C CNN "Manufacturer"
-F 6 "$0.290909" H 6700 1950 50  0001 C CNN "UnitCost(USD)"
-	1    6700 1950
-	-1   0    0    1
-$EndComp
 Wire Wire Line
 	6900 1950 7500 1950
@@
 	7500 1950 7900 1950
 Wire Wire Line
-	3950 1850 6500 1850
+	3950 1850 5500 1850
 Wire Wire Line
 	3650 3950 3650 3300
@@
 Text Notes 6450 2250 0    50   ~ 0
 Power Select\n
-Text HLabel 5650 3300 2    50   Input ~ 0
+Text HLabel 5650 3300 2    50   Output ~ 0
 +5V_USB
 Wire Wire Line
@@
 EndData
 $EndBitmap
+Text HLabel 5650 1600 2    50   Output ~ 0
+BARREL_IN
+Wire Wire Line
+	5650 1600 5500 1600
+Wire Wire Line
+	5500 1600 5500 1850
+Connection ~ 5500 1850
+Wire Wire Line
+	5500 1850 6500 1850
+$Comp
+L Switch:SW_SP3T SW49
+U 1 1 5E4CE77D
+P 6700 1950
+F 0 "SW49" H 6700 2233 50  0000 C CNN
+F 1 "SW_SP3T (DP3T Parallel)" H 6700 2142 50  0000 C CNN
+F 2 "OTTO_Footprints_Lib:SW_SP3T_CK-JS203011JCQN" H 6075 2125 50  0001 C CNN
+F 3 "https://datasheet.lcsc.com/szlcsc/C-K-JS203011JCQN_C221669.pdf" H 6075 2125 50  0001 C CNN
+F 4 "JS203011JCQN" H 6700 1950 50  0001 C CNN "MPN"
+F 5 "C&K" H 6700 1950 50  0001 C CNN "Manufacturer"
+F 6 "$0.586364" H 6700 1950 50  0001 C CNN "UnitCost(USD)"
+	1    6700 1950
+	-1   0    0    -1
+$EndComp
+Wire Wire Line
+	6500 1950 6350 1950
+Text HLabel 6350 1950 0    50   Input ~ 0
+BATT_IN
+Text HLabel 7500 3050 0    50   Input ~ 0
+5V_RUN
+Wire Wire Line
+	7500 3050 8350 3050
+Wire Wire Line
+	8550 3150 8550 3050
+Connection ~ 8550 3050
+Wire Wire Line
+	8550 3050 8350 3050
 $EndSCHEMATC

Commit message: routed buck boost supply
Connections:
- net labels added: SW1, SW2, USBD_N_CON, USBD_P_CON
- net labels removed: USBD__N, USBD__P

Commit message: routed 3v3 and power switches
Connections:
- net labels added: 3V3_SW, 5V_SW1, 5V_SW2, BARL
- net labels removed: SW1, SW2
Changed lines of the file:
@@
 L Device:C C91
 U 1 1 5DF7BA4E
-P 11600 1450
-F 0 "C91" H 11715 1496 50  0000 L CNN
-F 1 "100nF" H 11715 1405 50  0000 L CNN
-F 2 "Capacitor_SMD:C_0805_2012Metric_Pad1.15x1.40mm_HandSolder" H 11638 1300 50  0001 C CNN
-F 3 "https://datasheet.lcsc.com/szlcsc/Samsung-Electro-Mechanics-CL21B104JBCNNNC_C62912.pdf" H 11600 1450 50  0001 C CNN
-F 4 "$0.017724" H 11600 1450 12700 0001 C CNN "UnitCost(USD)"
-F 5 "CL21B104JBCNNNC" H 11600 1450 12700 0001 C CNN "MPN"
-F 6 "Samsung Electro-Mechanics" H 11600 1450 12700 0001 C CNN "Manufacturer"
-	1    11600 1450
-	1    0    0    -1
-$EndComp
-Wire Wire Line
-	11600 1300 11600 1100
-Wire Wire Line
-	11600 1100 11350 1100
+P 11750 1450
+F 0 "C91" H 11865 1496 50  0000 L CNN
+F 1 "100nF" H 11865 1405 50  0000 L CNN
+F 2 "Capacitor_SMD:C_0805_2012Metric_Pad1.15x1.40mm_HandSolder" H 11788 1300 50  0001 C CNN
+F 3 "https://datasheet.lcsc.com/szlcsc/Samsung-Electro-Mechanics-CL21B104JBCNNNC_C62912.pdf" H 11750 1450 50  0001 C CNN
+F 4 "$0.017724" H 11750 1450 12700 0001 C CNN "UnitCost(USD)"
+F 5 "CL21B104JBCNNNC" H 11750 1450 12700 0001 C CNN "MPN"
+F 6 "Samsung Electro-Mechanics" H 11750 1450 12700 0001 C CNN "Manufacturer"
+	1    11750 1450
+	1    0    0    -1
+$EndComp
+Wire Wire Line
+	11750 1300 11750 1100
+Wire Wire Line
+	11750 1100 11350 1100
 Connection ~ 11350 1100
 Wire Wire Line
 	11350 1100 11350 1450
 Wire Wire Line
-	11600 1600 11600 1750
-Wire Wire Line
-	11600 1750 11250 1750
+	11750 1600 11750 1750
+Wire Wire Line
+	11750 1750 11250 1750
 Wire Wire Line
 	11250 1550 11350 1550
@@
 +5V_REG
 Text Label 8700 1100 2    50   ~ 0
-SW1
-Text Label 11400 1100 0    50   ~ 0
-SW2
+5V_SW1
+Text Label 11450 1100 0    50   ~ 0
+5V_SW2
+Text Label 11150 4500 0    50   ~ 0
+3V3_SW
+Text Label 3100 1850 0    50   ~ 0
+BARL
 $EndSCHEMATC

Commit message: fix peripheral connections and route more critical components
Changed lines of the file:
@@
 +5V_REG
 Text GLabel 7450 8050 0    50   Input ~ 0
-+5V_REG
++3V3_MCU
 Text GLabel 10150 8200 0    50   Input ~ 0
 +5V_REG
