File: KiCad/PERIPHERALS.sch (KiCad schematic (older format))
At the start: 56 parts, among them CN201 1x4 MALE Molex PicoBlade, CN202 1x4 MALE Molex PicoBlade, Q1 AO4485, SW203 6x6x5.85mm (RA), SW48 SW_DIP_x02, SW49 SW_SP3T (DP3T Parallel), U2 TPS22918_SOT23-6_A, U204 USB6B1, U3 LTC3112_TSSOP20_A, U4 TLV62568_SOT-23-5_A, U5 TPS22918_SOT23-6_A

Commit message: routed audio
Parts:
- added R31, R32: 10k, Resistor_SMD:R_0805_2012Metric_Pad1.15x1.40mm_HandSolder, symbol Device:R
Connections:
- net labels added: USBCON_N, USBCON_P
- net labels removed: USBD_N_CON, USBD_P_CON
- wire segments 245 -> 247
Changed lines of the file:
@@
 	2550 4650 2550 4750
 Text Label 3350 4150 2    50   ~ 0
-USBD_P_CON
+USBCON_P
 Text Label 3350 4250 2    50   ~ 0
-USBD_N_CON
+USBCON_N
 Wire Wire Line
 	2850 4250 3350 4250
@@
 Wire Wire Line
 	8800 4500 9550 4500
-Text GLabel 9150 7150 0    50   Input ~ 0
+Text GLabel 8650 7150 0    50   Input ~ 0
 PI_PWR_EN
 $Comp
@@
 Text HLabel 7500 2850 0    50   Input ~ 0
 5V_PWM_SYNC
-Text HLabel 9150 9000 0    50   Input ~ 0
+Text HLabel 8650 9000 0    50   Input ~ 0
 LED_PWR_EN
 Text HLabel 14250 3800 2    50   Output ~ 0
@@
 Text Label 3100 1850 0    50   ~ 0
 BARL
+$Comp
+L Device:R R31
+U 1 1 5E6739EA
+P 9000 7150
+F 0 "R31" V 9115 7150 50  0000 C CNN
+F 1 "10k" V 9206 7150 50  0000 C CNN
+F 2 "Resistor_SMD:R_0805_2012Metric_Pad1.15x1.40mm_HandSolder" V 8930 7150 50  0001 C CNN
+F 3 "https://datasheet.lcsc.com/szlcsc/YAGEO-RC0805FR-0710KL_C84376.pdf" H 9000 7150 50  0001 C CNN
+F 4 "$.001675" H 9000 7150 50  0001 C CNN "UnitCost(USD)"
+F 5 "RC0805FR-0710KL" H 9000 7150 50  0001 C CNN "MPN"
+F 6 "Yageo" H 9000 7150 50  0001 C CNN "Manufacturer"
+	1    9000 7150
+	0    1    1    0
+$EndComp
+$Comp
+L Device:R R32
+U 1 1 5E674E79
+P 9000 9000
+F 0 "R32" V 9115 9000 50  0000 C CNN
+F 1 "10k" V 9206 9000 50  0000 C CNN
+F 2 "Resistor_SMD:R_0805_2012Metric_Pad1.15x1.40mm_HandSolder" V 8930 9000 50  0001 C CNN
+F 3 "https://datasheet.lcsc.com/szlcsc/YAGEO-RC0805FR-0710KL_C84376.pdf" H 9000 9000 50  0001 C CNN
+F 4 "$.001675" H 9000 9000 50  0001 C CNN "UnitCost(USD)"
+F 5 "RC0805FR-0710KL" H 9000 9000 50  0001 C CNN "MPN"
+F 6 "Yageo" H 9000 9000 50  0001 C CNN "Manufacturer"
+	1    9000 9000
+	0    1    1    0
+$EndComp
+Wire Wire Line
+	8650 9000 8850 9000
+Wire Wire Line
+	8650 7150 8850 7150
 $EndSCHEMATC

Commit message: change mcu reset button and route more stuff
Parts:
- L1: footprint OTTO_Footprints_Lib:L_7.3x6.6_H3 -> OTTO_Footprints_Lib:L_5.75x5.2_H3; MPN MCS0630-4R7MN2 -> MS0530-4R7M; Manufacturer PSA(Prosperity Dielectrics) -> COILMX; UnitCost(USD) $0.078246 -> $0.19697
- L2: footprint OTTO_Footprints_Lib:L_7.3x6.6_H3 -> OTTO_Footprints_Lib:L_4.75x4.2_H2; MPN MCS0630-2R2MN2 -> MS0420-2R2M; Manufacturer PSA(Prosperity Dielectrics) -> COILMX; UnitCost(USD) $0.078246 -> $0.231818
Changed lines of the file:
@@
 F 0 "L1" V 9919 950 50  0000 C CNN
 F 1 "4.7uH" V 10010 950 50  0000 C CNN
-F 2 "OTTO_Footprints_Lib:L_7.3x6.6_H3" H 10100 950 50  0001 C CNN
-F 3 "https://datasheet.lcsc.com/szlcsc/1904111131_Prosperity-Dielectrics-MCS0630-4R7MN2_C385253.pdf" H 10100 950 50  0001 C CNN
-F 4 "$0.078246" H 10100 950 12700 0001 C CNN "UnitCost(USD)"
-F 5 "MCS0630-4R7MN2" H 10100 950 12700 0001 C CNN "MPN"
-F 6 "PSA(Prosperity Dielectrics)" H 10100 950 12700 0001 C CNN "Manufacturer"
+F 2 "OTTO_Footprints_Lib:L_5.75x5.2_H3" H 10100 950 50  0001 C CNN
+F 3 "https://datasheet.lcsc.com/szlcsc/1910211209_COILMX-MS0530-4R7M_C380165.pdf" H 10100 950 50  0001 C CNN
+F 4 "$0.19697" H 10100 950 12700 0001 C CNN "UnitCost(USD)"
+F 5 "MS0530-4R7M" H 10100 950 12700 0001 C CNN "MPN"
+F 6 "COILMX" H 10100 950 12700 0001 C CNN "Manufacturer"
 	1    10100 950
 	0    1    1    0
@@
 F 0 "L2" V 11789 4500 50  0000 C CNN
 F 1 "2.2uH" V 11698 4500 50  0000 C CNN
-F 2 "OTTO_Footprints_Lib:L_7.3x6.6_H3" H 11600 4500 50  0001 C CNN
-F 3 "https://datasheet.lcsc.com/szlcsc/1904111131_Prosperity-Dielectrics-MCS0630-2R2MN2_C385252.pdf" H 11600 4500 50  0001 C CNN
-F 4 "$0.078246" H 11600 4500 12700 0001 C CNN "UnitCost(USD)"
-F 5 "MCS0630-2R2MN2" H 11600 4500 12700 0001 C CNN "MPN"
-F 6 "PSA(Prosperity Dielectrics)" H 11600 4500 12700 0001 C CNN "Manufacturer"
+F 2 "OTTO_Footprints_Lib:L_4.75x4.2_H2" H 11600 4500 50  0001 C CNN
+F 3 "https://datasheet.lcsc.com/szlcsc/1910211209_COILMX-MS0420-2R2M_C380154.pdf" H 11600 4500 50  0001 C CNN
+F 4 "$0.231818" H 11600 4500 12700 0001 C CNN "UnitCost(USD)"
+F 5 "MS0420-2R2M" H 11600 4500 12700 0001 C CNN "MPN"
+F 6 "COILMX" H 11600 4500 12700 0001 C CNN "Manufacturer"
 	1    11600 4500
 	0    -1   -1   0

Commit message: completed board
Connections:
- net labels added: LED_PWR_EN_OVERRIDE, PI_PWR_EN_OVERRIDE
- net labels removed: +3V3A_MCU
Changed lines of the file:
@@
 USBD_N
 Text GLabel 2450 5300 2    50   Input ~ 0
-+3V3A_MCU
++3V3_MCU
 $Comp
 L Device:Q_Photo_NPN PHOTO201
@@
 	11250 7150 11250 7250
 Wire Wire Line
-	9150 7150 9400 7150
+	9150 7150 9500 7150
 Wire Wire Line
 	12300 6650 12400 6650
@@
 	11250 8400 11250 9000
 Wire Wire Line
-	9150 9000 9400 9000
+	9150 9000 9500 9000
 Connection ~ 11250 9000
 Wire Wire Line
@@
 +5V_LEDS
 Wire Wire Line
-	8400 8050 9400 8050
-Wire Wire Line
-	9400 8050 9400 7150
-Connection ~ 9400 7150
-Wire Wire Line
-	9400 7150 11250 7150
-Wire Wire Line
-	8400 8150 9400 8150
-Wire Wire Line
-	9400 8150 9400 9000
-Connection ~ 9400 9000
-Wire Wire Line
-	9400 9000 11250 9000
+	8400 8050 9500 8050
+Wire Wire Line
+	9500 8050 9500 7150
+Connection ~ 9500 7150
+Wire Wire Line
+	9500 7150 11250 7150
+Wire Wire Line
+	8400 8150 9500 8150
+Wire Wire Line
+	9500 8150 9500 9000
+Connection ~ 9500 9000
+Wire Wire Line
+	9500 9000 11250 9000
 Wire Wire Line
 	7800 8150 7700 8150
@@
 Wire Wire Line
 	8650 7150 8850 7150
+Text Label 8550 8050 0    50   ~ 0
+PI_PWR_EN_OVERRIDE
+Text Label 8550 8150 0    50   ~ 0
+LED_PWR_EN_OVERRIDE
 $EndSCHEMATC

Commit message: Extend board by 1mm to align ports
Parts:
- removed SW203: 6x6x5.85mm (RA), Button_Switch_THT:SW_Tactile_SKHH_Angled, symbol Switch:SW_Push
- added SW203: SW_DPDT_x2, OTTO_Footprints_Lib:SSAC120100, symbol Switch:SW_DPDT_x2
Connections:
- no-connect marks 3 -> 4
Changed lines of the file:
@@
 Wire Wire Line
 	2550 4550 2550 4650
-Wire Wire Line
-	3700 6200 3850 6200
-Wire Wire Line
-	4300 6200 4150 6200
-$Comp
-L Device:C C?
-U 1 1 5D34A773
-P 4000 6200
-AR Path="/5C4320DF/5C4AB60A/5D34A773" Ref="C?"  Part="1"
-AR Path="/5C4320DF/5C6CAC95/5D34A773" Ref="C?"  Part="1"
-AR Path="/5C4320DF/5C4AB597/5D34A773" Ref="C58"  Part="1"
-F 0 "C58" V 4160 6200 50  0000 C CNN
-F 1 "100nF" V 4251 6200 50  0000 C CNN
-F 2 "Capacitor_SMD:C_0805_2012Metric_Pad1.15x1.40mm_HandSolder" H 4038 6050 50  0001 C CNN
-F 3 "https://datasheet.lcsc.com/szlcsc/Samsung-Electro-Mechanics-CL21B104JBCNNNC_C62912.pdf" H 4000 6200 50  0001 C CNN
-F 4 "$0.017724" H 4000 6200 12700 0001 C CNN "UnitCost(USD)"
-F 5 "CL21B104JBCNNNC" H 4000 6200 12700 0001 C CNN "MPN"
-F 6 "Samsung Electro-Mechanics" H 4000 6200 12700 0001 C CNN "Manufacturer"
-	1    4000 6200
-	0    1    1    0
-$EndComp
-Text GLabel 4600 6050 2    50   Input ~ 0
+Text GLabel 4600 5950 2    50   Input ~ 0
 PWR_BUTTON
 Wire Wire Line
-	3700 6050 3700 6200
-Wire Wire Line
-	4300 6050 4300 6200
-$Comp
-L Switch:SW_Push SW?
-U 1 1 5D34A785
-P 4000 6050
-AR Path="/5C4320DF/5C6CAC95/5D34A785" Ref="SW?"  Part="1"
-AR Path="/5C4320DF/5C4AB597/5D34A785" Ref="SW203"  Part="1"
-F 0 "SW203" H 4000 6335 50  0000 C CNN
-F 1 "6x6x5.85mm (RA)" H 4000 6244 50  0000 C CNN
-F 2 "Button_Switch_THT:SW_Tactile_SKHH_Angled" H 4000 6250 50  0001 C CNN
-F 3 "https://datasheet.lcsc.com/szlcsc/ALPS-Electric-SKHHLWA010_C125050.pdf" H 4000 6250 50  0001 C CNN
-F 4 "$0.134848" H 4000 6050 12700 0001 C CNN "UnitCost(USD)"
-F 5 "SKHHLWA010" H 4000 6050 12700 0001 C CNN "MPN"
-F 6 "ALPS Electric" H 4000 6050 12700 0001 C CNN "Manufacturer"
-	1    4000 6050
-	-1   0    0    -1
-$EndComp
-Wire Wire Line
-	4200 6050 4300 6050
+	3700 6050 3700 6300
+Wire Wire Line
+	4300 5950 4300 6300
+Wire Wire Line
+	4200 5950 4300 5950
 $Comp
 L Connector:Barrel_Jack_Switch DC?
@@
 Wire Wire Line
 	3700 6050 3800 6050
-Connection ~ 4300 6050
-Wire Wire Line
-	4300 6050 4600 6050
+Connection ~ 4300 5950
+Wire Wire Line
+	4300 5950 4600 5950
 $Comp
 L power:GND #PWR?
@@
 Text Label 8550 8150 0    50   ~ 0
 LED_PWR_EN_OVERRIDE
+$Comp
+L Switch:SW_DPDT_x2 SW203
+U 1 1 5E67BD76
+P 4000 5950
+F 0 "SW203" H 4000 5625 50  0000 C CNN
+F 1 "SW_DPDT_x2" H 4000 5716 50  0000 C CNN
+F 2 "OTTO_Footprints_Lib:SSAC120100" H 4000 5950 50  0001 C CNN
+F 3 "~" H 4000 5950 50  0001 C CNN
+	1    4000 5950
+	-1   0    0    1
+$EndComp
+Wire Wire Line
+	3700 6300 3850 6300
+Wire Wire Line
+	4300 6300 4150 6300
+$Comp
+L Device:C C?
+U 1 1 5D34A773
+P 4000 6300
+AR Path="/5C4320DF/5C4AB60A/5D34A773" Ref="C?"  Part="1"
+AR Path="/5C4320DF/5C6CAC95/5D34A773" Ref="C?"  Part="1"
+AR Path="/5C4320DF/5C4AB597/5D34A773" Ref="C58"  Part="1"
+F 0 "C58" V 4160 6300 50  0000 C CNN
+F 1 "100nF" V 4251 6300 50  0000 C CNN
+F 2 "Capacitor_SMD:C_0805_2012Metric_Pad1.15x1.40mm_HandSolder" H 4038 6150 50  0001 C CNN
+F 3 "https://datasheet.lcsc.com/szlcsc/Samsung-Electro-Mechanics-CL21B104JBCNNNC_C62912.pdf" H 4000 6300 50  0001 C CNN
+F 4 "$0.017724" H 4000 6300 12700 0001 C CNN "UnitCost(USD)"
+F 5 "CL21B104JBCNNNC" H 4000 6300 12700 0001 C CNN "MPN"
+F 6 "Samsung Electro-Mechanics" H 4000 6300 12700 0001 C CNN "Manufacturer"
+	1    4000 6300
+	0    1    1    0
+$EndComp
+NoConn ~ 3800 5850
 $EndSCHEMATC

Commit message: More JLC part numbers added
Parts:
- removed C59: 100nF, Capacitor_SMD:C_0805_2012Metric_Pad1.15x1.40mm_HandSolder, symbol Device:C
- removed PHOTO201: ALS-PDIC243-3B, OTTO_Footprints_Lib:ALS-PDIC243-3B, symbol Device:Q_Photo_NPN
- removed R211: 10k, Resistor_SMD:R_0805_2012Metric_Pad1.15x1.40mm_HandSolder, symbol Device:R
- added CN203: Conn_01x05, Connector_PinSocket_2.54mm:PinSocket_1x06_P2.54mm_Vertical, symbol Connector_Generic:Conn_01x06
- C232, C80, C88: JLCASM (none) -> BASIC; LCSC PN (none) -> C15850; MPN CL21B106KOQNNNE -> CL21A106KAYNNNE; Manufacturer Samsung Electro-Mechanics -> (none); UnitCost(USD) $0.041113 -> Samsung Electro-Mechanics
- C58, C82, C83, C90, C91: JLCASM (none) -> BASIC; LCSC PN (none) -> C49678; MPN CL21B104JBCNNNC -> CC0805KRX7R9BB104; Manufacturer Samsung Electro-Mechanics -> (none); UnitCost(USD) $0.017724 -> Samsung Electro-Mechanics
- C76, C95: footprint Capacitor_SMD:C_1206_3216Metric_Pad1.42x1.75mm_HandSolder -> Capacitor_SMD:C_1206_3216Metric; JLCASM (none) -> EXT; LCSC PN (none) -> C68361; MPN GRM31CR61E476ME44L -> CL31A476MQHNNNE; Manufacturer Murata Electronics -> (none); UnitCost(USD) $0.390909 -> Murata Electronics
- C77, C87: JLCASM (none) -> BASIC; LCSC PN (none) -> C1710; MPN CL21B103KBCNNNC -> CL21B103KBANNNC; Manufacturer Samsung Electro-Mechanics -> (none); UnitCost(USD) $0.007546 -> Samsung Electro-Mechanics
- C79, C81, C84: footprint Capacitor_SMD:C_Elec_6.3x7.7 -> Capacitor_SMD:CP_Elec_6.3x7.7; JLCASM (none) -> DNP; LCSC PN (none) -> C134834; MPN RVT1A471M0607 -> VZH471M0JTR-0607; Manufacturer Honor Elec -> (none); UnitCost(USD) $0.03996 -> Honor Elec
- C85: JLCASM (none) -> BASIC; LCSC PN (none) -> C28323; MPN CL21B105KBFVPNE -> CL21B105KBFNNNE; Manufacturer Samsung Electro-Mechanics -> (none); UnitCost(USD) $0.067176 -> Samsung Electro-Mechanics
- C86: JLCASM (none) -> BASIC; LCSC PN (none) -> C1779; MPN CL21B475KAFNNNE -> CL21A475KAQNNNE; Manufacturer Samsung Electro-Mechanics -> (none); UnitCost(USD) $0.031439 -> Samsung Electro-Mechanics
- C89: JLCASM (none) -> BASIC; LCSC PN (none) -> C1804; Manufacturer Samsung Electro-Mechanics -> (none); UnitCost(USD) $0.009476 -> Samsung Electro-Mechanics
- C92: JLCASM (none) -> BASIC; LCSC PN (none) -> C53150; MPN CC0805JRNPO9BN681 -> CL21B681KBANNNC; Manufacturer Yageo -> (none); UnitCost(USD) $0.008589 -> Yageo
- C93: JLCASM (none) -> BASIC; LCSC PN (none) -> C1794; Manufacturer Samsung Electro-Mechanics -> (none); UnitCost(USD) $0.00985 -> Samsung Electro-Mechanics
- C94: JLCASM (none) -> BASIC; LCSC PN (none) -> C14857; MPN CC0805JRNPO9BN470 -> CL21C470JBANNNC; Manufacturer Yageo -> (none); UnitCost(USD) $0.022222 -> Yageo
- CN201, CN202: JLCASM (none) -> DNP; LCSC PN (none) -> C240847; Manufacturer Molex -> (none); UnitCost(USD) $0.156061 -> Molex
- D48: JLCASM (none) -> EXT; LCSC PN (none) -> C123803; Manufacturer MDD(Microdiode Electronics) -> (none); UnitCost(USD) $0.029539 -> MDD(Microdiode Electronics)
- D49: JLCASM (none) -> EXT; LCSC PN (none) -> C173427; Manufacturer MDD(Microdiode Electronics) -> (none); UnitCost(USD) $0.010021 -> MDD(Microdiode Electronics)
- DC201: JLCASM (none) -> DNP; LCSC PN (none) -> C16214; Manufacturer BOOMELE(Boom Precision Elec) -> (none); UnitCost(USD) $0.034374 -> BOOMELE(Boom Precision Elec)
- DISPLAY201: Manufacturer JR E-Shop -> (none); UnitCost(USD) $8.68 -> JR E-Shop
- L1: footprint OTTO_Footprints_Lib:L_5.75x5.2_H3 -> Inductor_SMD:L_Sunlord_MWSA0518_5.4x5.2mm; JLCASM (none) -> EXT; LCSC PN (none) -> C408410; MPN MS0530-4R7M -> MWSA0503S-4R7MT; Manufacturer COILMX -> (none); UnitCost(USD) $0.19697 -> COILMX
- L2: footprint OTTO_Footprints_Lib:L_4.75x4.2_H2 -> OTTO_Footprints_Lib:L_Sunlord_MWSA0518_5.4x5.2mm; JLCASM (none) -> EXT; LCSC PN (none) -> C408335; MPN MS0420-2R2M -> MWSA0402S-2R2MT; Manufacturer COILMX -> (none); UnitCost(USD) $0.231818 -> COILMX
- Q1: JLCASM (none) -> EXT; LCSC PN (none) -> C51499; Manufacturer Alpha & Omega Semicon -> (none); UnitCost(USD) $0.284848 -> Alpha & Omega Semicon
- R10, R13, R14, R15, R16: JLCASM (none) -> BASIC; LCSC PN (none) -> C17407; MPN RC0805FR-07100KL -> 0805W8F1003T5E; Manufacturer Yageo -> (none); UnitCost(USD) $.00169 -> Yageo
- R12, R17: footprint Resistor_SMD:R_0805_2012Metric_Pad1.15x1.40mm_HandSolder -> Resistor_SMD:R_1206_3216Metric; JLCASM (none) -> BASIC; LCSC PN (none) -> C25334; MPN RC0805JR-070RL -> 1206W4F100LT5E; Manufacturer Yageo -> (none); UnitCost(USD) $.001203 -> Yageo
- R18: Manufacturer Bourns -> (none); UnitCost(USD) $.010229 -> Bourns
- R19: JLCASM (none) -> BASIC; LCSC PN (none) -> C17678; MPN RC0805FR-0740K2L -> 0805W8F4022T5E; Manufacturer Yageo -> (none); UnitCost(USD) $.001774 -> Yageo
- R20: Manufacturer KOA Speer Elec -> (none); UnitCost(USD) $.004141 -> KOA Speer Elec
- R21: JLCASM (none) -> BASIC; LCSC PN (none) -> C17633; MPN RC0805FR-0733KL -> 0805W8F3302T5E; Manufacturer Yageo -> (none); UnitCost(USD) $.001703 -> Yageo
- R22: value 845k -> 270k; JLCASM (none) -> BASIC; LCSC PN (none) -> C17589; MPN ERJ6ENF8453V -> 0805W8F2703T5E; Manufacturer Panasonic -> (none); UnitCost(USD) $.009826 -> Panasonic
- R23: value 158k -> 51k; JLCASM (none) -> BASIC; LCSC PN (none) -> C17737; MPN CR0805-FX-1583ELF -> 0805W8F5102T5E; Manufacturer Bourns -> (none); UnitCost(USD) $.010537 -> Bourns
- R24, R31, R32: JLCASM (none) -> BASIC; LCSC PN (none) -> C17414; MPN RC0805FR-0710KL -> 0805W8F1002T5E; Manufacturer Yageo -> (none); UnitCost(USD) $.001675 -> Yageo
- SW203: JLCASM (none) -> DNP; LCSC PN (none) -> C202374; MPN (none) -> SSAC120100; UnitCost(USD) (none) -> ALPS Electric
- SW48: JLCASM (none) -> DNP; LCSC PN (none) -> C129087; Manufacturer Korean Hroparts Elec -> (none); UnitCost(USD) $0.636364 -> Korean Hroparts Elec
- SW49: JLCASM (none) -> DNP; LCSC PN (none) -> C221669; Manufacturer C&K -> (none); UnitCost(USD) $0.586364 -> C&K
- U2, U5: JLCASM (none) -> EXT; LCSC PN (none) -> C131941; Manufacturer Texas Instruments -> (none); UnitCost(USD) $0.228788 -> Texas Instruments
- U204: JLCASM (none) -> EXT; LCSC PN (none) -> C10508; Manufacturer STMicroelectronics -> (none); UnitCost(USD) $0.689394 -> STMicroelectronics
- U3: JLCASM (none) -> EXT; LCSC PN (none) -> C117291; Manufacturer Analog Devices -> (none); UnitCost(USD) $4.06 -> Analog Devices
- U4: JLCASM (none) -> EXT; LCSC PN (none) -> C163219; Manufacturer Texas Instruments -> (none); UnitCost(USD) $0.083576 -> Texas Instruments
- USB201: JLCASM (none) -> NO; LCSC PN (none) -> C86462; Manufacturer TE Connectivity -> (none); UnitCost(USD) $0.40303 -> TE Connectivity
Connections:
- net labels removed: BRIGHTNESS
- wire segments 247 -> 241

Commit message: Selected all LCSC parts. Check of part numbers complete
Parts:
- removed C93: 15pF, Capacitor_SMD:C_0805_2012Metric_Pad1.15x1.40mm_HandSolder, symbol Device:C
- removed R19: 40.2k, Resistor_SMD:R_0805_2012Metric_Pad1.15x1.40mm_HandSolder, symbol Device:R
- removed U4: TLV62568_SOT-23-5_A, Package_TO_SOT_SMD:SOT-23-5, symbol OTTOdiy_SMD-library:TLV62568_SOT-23-5_A
- added C59: 10uF, Capacitor_SMD:C_0805_2012Metric_Pad1.15x1.40mm_HandSolder, symbol Device:C
- added D54: 1N4148, Diode_SMD:D_SOD-323_HandSoldering, symbol Device:D
- added R9: 49.9k, Resistor_SMD:R_0805_2012Metric_Pad1.15x1.40mm_HandSolder, symbol Device:R
- added TP3: TestPoint, TestPoint:TestPoint_THTPad_D1.0mm_Drill0.5mm, symbol Connector:TestPoint
- added U4: MP2359, Package_TO_SOT_SMD:TSOT-23-6_HandSoldering, symbol OTTOdiy_SMD-library:MP2359
- C232, C58, C77, C80, C82, C83, C85, C87, C89, C90, C91: UnitCost(USD) Samsung Electro-Mechanics -> (none)
- C76, C95: UnitCost(USD) Murata Electronics -> (none)
- C79, C81, C84: LCSC PN C134834 -> C134834; UnitCost(USD) Honor Elec -> (none)
- C86: value 4.7uF -> 22nF; LCSC PN C1779 -> C1729; MPN CL21A475KAQNNNE -> CL21B223KBANNNC; UnitCost(USD) Samsung Electro-Mechanics -> (none)
- C88: value 10uF -> 22uF; LCSC PN C15850 -> C45783; MPN CL21A106KAYNNNE -> CL21A226MAQNNNE; UnitCost(USD) Samsung Electro-Mechanics -> (none)
- C92, C94, R10, R12, R13, R14, R15, R16, R17, R21, R24, R31, R32: UnitCost(USD) Yageo -> (none)
- CN201, CN202: UnitCost(USD) Molex -> (none)
- CN203: JLCASM (none) -> N/A; MPN (none) -> N/A
- D48, D49: UnitCost(USD) MDD(Microdiode Electronics) -> (none)
- DC201: UnitCost(USD) BOOMELE(Boom Precision Elec) -> (none)
- DISPLAY201: JLCASM (none) -> N/A; UnitCost(USD) JR E-Shop -> (none)
- L1: UnitCost(USD) COILMX -> (none)
- L2: value 2.2uH -> 4.7uH; footprint OTTO_Footprints_Lib:L_Sunlord_MWSA0518_5.4x5.2mm -> Inductor_SMD:L_Sunlord_MWSA0518_5.4x5.2mm; LCSC PN C408335 -> C408410; MPN MWSA0402S-2R2MT -> MWSA0503S-4R7MT; UnitCost(USD) COILMX -> (none)
- Q1: UnitCost(USD) Alpha & Omega Semicon -> (none)
- R18: value 182k -> 16k; JLCASM (none) -> BASIC; LCSC PN (none) -> C17490; MPN CR0805-FX-1823ELF -> 0805W8F1602T5E; UnitCost(USD) Bourns -> (none)
- R20: value 42.2k -> 22k; JLCASM (none) -> BASIC; LCSC PN (none) -> C17560; MPN RK73H2ATTD4222F -> 0805W8F2202T5E; UnitCost(USD) KOA Speer Elec -> (none)
- R22: UnitCost(USD) Panasonic -> (none)
- R23: UnitCost(USD) Bourns -> (none)
- SW203: UnitCost(USD) ALPS Electric -> (none)
- SW48: UnitCost(USD) Korean Hroparts Elec -> (none)
- SW49: UnitCost(USD) C&K -> (none)
- U2, U5: UnitCost(USD) Texas Instruments -> (none)
- U204: MPN USB6B1 -> USB6B1RL; UnitCost(USD) STMicroelectronics -> (none)
- U3: UnitCost(USD) Analog Devices -> (none)
- USB201: UnitCost(USD) TE Connectivity -> (none)
Connections:
- wire segments 241 -> 244
Other:
- note added: "IOUT sources 24uA for each 1A being pulled on VOUT.\nR20=22k means this output will be 528 mV/A"
