File: KiCad/PERIPHERALS.sch (KiCad schematic (older format))
At the start: 58 parts, among them CN201 1x4 MALE Molex PicoBlade, CN202 1x4 MALE Molex PicoBlade, CN203 Conn_01x05, Q1 AO4485, SW203 SW_DPDT_x2, SW48 SW_DIP_x02, SW49 SW_SP3T (DP3T Parallel), U2 TPS22918_SOT23-6_A, U204 USB6B1, U3 LTC3112_TSSOP20_A, U4 MP2359, U5 TPS22918_SOT23-6_A

Commit message: Finish selecting jlc parts
Parts:
- removed U204: USB6B1, Package_SO:SOIC-8_3.9x4.9mm_P1.27mm, symbol Power_Protection:USB6B1
- added U204: SRV05-4, Package_TO_SOT_SMD:SOT-23-6, symbol Power_Protection:SRV05-4
- C79, C81, C84: JLCASM DNP -> EXT; LCSC PN C134834 -> C134738; MPN VZH471M0JTR-0607 -> VE-471M0JTR-0607
- D48, D49, U3: JLCASM EXT -> EXTDNP
- Q1: value AO4485 -> AO4407A; JLCASM EXT -> BASIC; LCSC PN C51499 -> C16072; MPN AO4485 -> AO4407A
- R12, R17: footprint Resistor_SMD:R_1206_3216Metric -> Resistor_SMD:R_0805_2012Metric_Pad1.15x1.40mm_HandSolder; LCSC PN C25334 -> C17477; MPN 1206W4F100LT5E -> 0805W8F0000T5E
- USB201: JLCASM NO -> N/A
Connections:
- wire segments 244 -> 246
- no-connect marks 4 -> 6
Changed lines of the file:
@@
 Comment4 ""
 $EndDescr
-Text HLabel 4600 4250 2    50   Input ~ 0
+Text HLabel 3950 4200 2    50   Input ~ 0
 USBD_P
-Text HLabel 4600 4450 2    50   Input ~ 0
+Text HLabel 3950 4400 2    50   Input ~ 0
 USBD_N
 $Comp
@@
 F 5 "292304-1" H 2550 4150 12700 0001 C CNN "MPN"
 F 6 "" H 2550 4150 12700 0001 C CNN "Manufacturer"
-F 7 "NO" H 2550 4150 50  0001 C CNN "JLCASM"
+F 7 "N/A" H 2550 4150 50  0001 C CNN "JLCASM"
 F 8 "C86462" H 2550 4150 50  0001 C CNN "LCSC PN"
 	1    2550 4150
 	1    0    0    -1
 $EndComp
-Wire Wire Line
-	2550 4650 2550 4750
 Text Label 3350 4150 2    50   ~ 0
 USBCON_P
@@
 	2850 4250 3350 4250
 Wire Wire Line
-	2550 4750 3950 4750
-Wire Wire Line
 	2450 4550 2450 4650
 Wire Wire Line
 	2450 4650 2550 4650
-Connection ~ 2550 4650
-Wire Wire Line
-	2550 4550 2550 4650
 Text GLabel 4600 5950 2    50   Input ~ 0
 PWR_BUTTON
@@
 	2850 4150 3450 4150
 Wire Wire Line
-	3550 4450 3350 4450
+	4450 4450 3800 4450
 Wire Wire Line
 	3350 4450 3350 4250
@@
 AR Path="/5C4320DF/5C4AB597/5E314238" Ref="Q1"  Part="1"
 F 0 "Q1" V 3993 1950 50  0000 C CNN
-F 1 "AO4485" V 3902 1950 50  0000 C CNN
+F 1 "AO4407A" V 3902 1950 50  0000 C CNN
 F 2 "Package_SO:SOIC-8_3.9x4.9mm_P1.27mm" H 3850 2050 50  0001 C CNN
-F 3 "https://datasheet.lcsc.com/szlcsc/C51499.pdf" H 3650 1950 50  0001 C CNN
+F 3 "https://datasheet.lcsc.com/szlcsc/C16072.pdf" H 3650 1950 50  0001 C CNN
 F 4 "" H 3650 1950 12700 0001 C CNN "UnitCost(USD)"
-F 5 "AO4485" H 3650 1950 12700 0001 C CNN "MPN"
+F 5 "AO4407A" H 3650 1950 12700 0001 C CNN "MPN"
 F 6 "" H 3650 1950 12700 0001 C CNN "Manufacturer"
-F 7 "C51499" H 3650 1950 50  0001 C CNN "LCSC PN"
-F 8 "EXT" H 3650 1950 50  0001 C CNN "JLCASM"
+F 7 "C16072" H 3650 1950 50  0001 C CNN "LCSC PN"
+F 8 "BASIC" H 3650 1950 50  0001 C CNN "JLCASM"
 	1    3650 1950
 	0    -1   -1   0
@@
 F 5 "SMF15CA" H 3000 2200 50  0001 C CNN "MPN"
 F 6 "" H 3000 2200 50  0001 C CNN "UnitCost(USD)"
-F 7 "EXT" H 3000 2200 50  0001 C CNN "JLCASM"
+F 7 "EXTDNP" H 3000 2200 50  0001 C CNN "JLCASM"
 F 8 "C123803" H 3000 2200 50  0001 C CNN "LCSC PN"
 	1    3000 2200
@@
 F 6 "" H 3950 2050 50  0001 C CNN "Manufacturer"
 F 7 "C173427" H 3950 2050 50  0001 C CNN "LCSC PN"
-F 8 "EXT" H 3950 2050 50  0001 C CNN "JLCASM"
+F 8 "EXTDNP" H 3950 2050 50  0001 C CNN "JLCASM"
 	1    3950 2050
 	0    1    1    0
@@
 F 0 "R17" V 12344 6650 50  0000 C CNN
 F 1 "0" V 12435 6650 50  0000 C CNN
-F 2 "Resistor_SMD:R_1206_3216Metric" V 12480 6650 50  0001 C CNN
-F 3 "https://datasheet.lcsc.com/szlcsc/C25334.pdf" H 12550 6650 50  0001 C CNN
+F 2 "Resistor_SMD:R_0805_2012Metric_Pad1.15x1.40mm_HandSolder" V 12480 6650 50  0001 C CNN
+F 3 "https://datasheet.lcsc.com/szlcsc/C17477pdf" H 12550 6650 50  0001 C CNN
 F 4 "" H 12550 6650 50  0001 C CNN "UnitCost(USD)"
-F 5 "1206W4F100LT5E" H 12550 6650 50  0001 C CNN "MPN"
+F 5 "0805W8F0000T5E" H 12550 6650 50  0001 C CNN "MPN"
 F 6 "" H 12550 6650 50  0001 C CNN "Manufacturer"
 F 7 "BASIC" H 12550 6650 50  0001 C CNN "JLCASM"
-F 8 "C25334" H 12550 6650 50  0001 C CNN "LCSC PN"
+F 8 "C17477" H 12550 6650 50  0001 C CNN "LCSC PN"
 	1    12550 6650
 	0    1    1    0
@@
 	1    0    0    -1
 $EndComp
-Connection ~ 2550 4750
-Wire Wire Line
-	2550 4750 2550 4850
-Wire Wire Line
-	3950 4650 3950 4750
-$Comp
-L Power_Protection:USB6B1 U204
-U 1 1 5D2FDFC1
-P 3950 4350
-F 0 "U204" H 3700 4750 50  0000 C CNN
-F 1 "USB6B1" H 3700 4650 50  0000 C CNN
-F 2 "Package_SO:SOIC-8_3.9x4.9mm_P1.27mm" H 3950 4350 50  0001 C CNN
-F 3 "https://datasheet.lcsc.com/szlcsc/C10508.pdf" H 3000 4250 50  0001 C CNN
-F 4 "" H 3950 4350 12700 0001 C CNN "UnitCost(USD)"
-F 5 "USB6B1RL" H 3950 4350 12700 0001 C CNN "MPN"
-F 6 "" H 3950 4350 12700 0001 C CNN "Manufacturer"
-F 7 "EXT" H 3950 4350 50  0001 C CNN "JLCASM"
-F 8 "C10508" H 3950 4350 50  0001 C CNN "LCSC PN"
-	1    3950 4350
-	-1   0    0    -1
-$EndComp
 Wire Wire Line
 	2850 3950 3650 3950
@@
 F 3 "https://datasheet.lcsc.com/szlcsc/C134834.pdf" H 10350 6600 50  0001 C CNN
 F 4 "" H 10350 6600 12700 0001 C CNN "UnitCost(USD)"
-F 5 "VZH471M0JTR-0607" H 10350 6600 12700 0001 C CNN "MPN"
+F 5 "VE-471M0JTR-0607" H 10350 6600 12700 0001 C CNN "MPN"
 F 6 "" H 10350 6600 12700 0001 C CNN "Manufacturer"
-F 7 "DNP" H 10350 6600 50  0001 C CNN "JLCASM"
-F 8 "C134834" H 10350 6600 50  0001 C CNN "LCSC PN"
+F 7 "EXT" H 10350 6600 50  0001 C CNN "JLCASM"
+F 8 "C134738" H 10350 6600 50  0001 C CNN "LCSC PN"
 	1    10350 6600
 	1    0    0    -1
@@
 F 3 "https://datasheet.lcsc.com/szlcsc/C134834.pdf" H 9850 6600 50  0001 C CNN
 F 4 "" H 9850 6600 12700 0001 C CNN "UnitCost(USD)"
-F 5 "VZH471M0JTR-0607" H 9850 6600 12700 0001 C CNN "MPN"
+F 5 "VE-471M0JTR-0607" H 9850 6600 12700 0001 C CNN "MPN"
 F 6 "" H 9850 6600 12700 0001 C CNN "Manufacturer"
-F 7 "DNP" H 9850 6600 50  0001 C CNN "JLCASM"
-F 8 "C134834" H 9850 6600 50  0001 C CNN "LCSC PN"
+F 7 "EXT" H 9850 6600 50  0001 C CNN "JLCASM"
+F 8 "C134738" H 9850 6600 50  0001 C CNN "LCSC PN"
 	1    9850 6600
 	1    0    0    -1
@@
 F 3 "https://datasheet.lcsc.com/szlcsc/C134834.pdf" H 9350 6600 50  0001 C CNN
 F 4 "" H 9350 6600 12700 0001 C CNN "UnitCost(USD)"
-F 5 "VZH471M0JTR-0607" H 9350 6600 12700 0001 C CNN "MPN"
+F 5 "VE-471M0JTR-0607" H 9350 6600 12700 0001 C CNN "MPN"
 F 6 "" H 9350 6600 12700 0001 C CNN "Manufacturer"
-F 7 "DNP" H 9350 6600 50  0001 C CNN "JLCASM"
-F 8 "C134834" H 9350 6600 50  0001 C CNN "LCSC PN"
+F 7 "EXT" H 9350 6600 50  0001 C CNN "JLCASM"
+F 8 "C134738" H 9350 6600 50  0001 C CNN "LCSC PN"
 	1    9350 6600
 	1    0    0    -1
@@
 F 0 "R12" V 12344 8500 50  0000 C CNN
 F 1 "0" V 12435 8500 50  0000 C CNN
-F 2 "Resistor_SMD:R_1206_3216Metric" V 12480 8500 50  0001 C CNN
-F 3 "https://datasheet.lcsc.com/szlcsc/C25334.pdf" H 12550 8500 50  0001 C CNN
+F 2 "Resistor_SMD:R_0805_2012Metric_Pad1.15x1.40mm_HandSolder" V 12480 8500 50  0001 C CNN
+F 3 "https://datasheet.lcsc.com/szlcsc/C17477pdf" H 12550 8500 50  0001 C CNN
 F 4 "" H 12550 8500 50  0001 C CNN "UnitCost(USD)"
-F 5 "1206W4F100LT5E" H 12550 8500 50  0001 C CNN "MPN"
+F 5 "0805W8F0000T5E" H 12550 8500 50  0001 C CNN "MPN"
 F 6 "" H 12550 8500 50  0001 C CNN "Manufacturer"
 F 7 "BASIC" H 12550 8500 50  0001 C CNN "JLCASM"
-F 8 "C25334" H 12550 8500 50  0001 C CNN "LCSC PN"
+F 8 "C17477" H 12550 8500 50  0001 C CNN "LCSC PN"
 	1    12550 8500
 	0    1    1    0
@@
 	3950 1850 5500 1850
 Wire Wire Line
-	3650 3950 3650 3300
-Wire Wire Line
 	3650 3300 5500 3300
 Wire Wire Line
@@
 Wire Wire Line
 	5500 2050 6500 2050
-Connection ~ 3650 3950
-Wire Wire Line
-	3650 3950 3950 3950
 Text Label 4800 1850 0    50   ~ 0
 BARREL_IN
@@
 	3450 4150 3450 4250
 Wire Wire Line
-	3450 4250 3550 4250
-Wire Wire Line
-	3950 3950 3950 4050
-Wire Wire Line
-	4350 4250 4600 4250
-Wire Wire Line
-	4600 4450 4350 4450
+	3450 4250 3800 4250
 Text Notes 6450 2250 0    50   ~ 0
 Power Select\n
@@
 F 6 "" H 10100 2250 50  0001 C CNN "UnitCost(USD)"
 F 7 "C117291" H 10100 2250 50  0001 C CNN "LCSC PN"
-F 8 "EXT" H 10100 2250 50  0001 C CNN "JLCASM"
+F 8 "EXTDNP" H 10100 2250 50  0001 C CNN "JLCASM"
 	1    10100 2250
 	1    0    0    -1
@@
 Wire Wire Line
 	14700 3800 15150 3800
+$Comp
+L Power_Protection:SRV05-4 U204
+U 1 1 5EA94B2C
+P 4950 4350
+F 0 "U204" H 4950 5031 50  0000 C CNN
+F 1 "SRV05-4" H 4950 4940 50  0000 C CNN
+F 2 "Package_TO_SOT_SMD:SOT-23-6" H 5650 3900 50  0001 C CNN
+F 3 "http://www.onsemi.com/pub/Collateral/SRV05-4-D.PDF" H 4950 4350 50  0001 C CNN
+F 4 "BASIC" H 4950 4350 50  0001 C CNN "JLCASM"
+F 5 "C85364" H 4950 4350 50  0001 C CNN "LCSC PN"
+F 6 "SRV05-4-P-T7" H 4950 4350 50  0001 C CNN "MPN"
+	1    4950 4350
+	1    0    0    -1
+$EndComp
+Wire Wire Line
+	3950 4200 3800 4200
+Wire Wire Line
+	3800 4200 3800 4250
+Connection ~ 3800 4250
+Wire Wire Line
+	3800 4250 4450 4250
+Wire Wire Line
+	3950 4400 3800 4400
+Wire Wire Line
+	3800 4400 3800 4450
+Connection ~ 3800 4450
+Wire Wire Line
+	3800 4450 3350 4450
+Wire Wire Line
+	4950 3850 3650 3850
+Wire Wire Line
+	3650 3300 3650 3850
+Connection ~ 3650 3850
+Wire Wire Line
+	3650 3850 3650 3950
+Wire Wire Line
+	4950 4850 2550 4850
+Wire Wire Line
+	2550 4550 2550 4650
+Connection ~ 2550 4850
+Connection ~ 2550 4650
+Wire Wire Line
+	2550 4650 2550 4850
+NoConn ~ 5450 4250
+NoConn ~ 5450 4450
 $EndSCHEMATC

Commit message: Fix DAC footprint and other minor issues.
Parts:
- C79, C81, C84: footprint Capacitor_SMD:CP_Elec_6.3x7.7 -> OTTO_Footprints_Lib:CP_Elec_6.3x7.7
- Q1: footprint Package_SO:SOIC-8_3.9x4.9mm_P1.27mm -> OTTO_Footprints_Lib:SOIC-8_3.9x4.9mm_P1.27mm
- U2, U204, U5: footprint Package_TO_SOT_SMD:SOT-23-6 -> OTTO_Footprints_Lib:SOT-23-6
- U4: footprint Package_TO_SOT_SMD:TSOT-23-6_HandSoldering -> OTTO_Footprints_Lib:TSOT-23-6_HandSoldering
Changed lines of the file:
@@
 F 0 "Q1" V 3993 1950 50  0000 C CNN
 F 1 "AO4407A" V 3902 1950 50  0000 C CNN
-F 2 "Package_SO:SOIC-8_3.9x4.9mm_P1.27mm" H 3850 2050 50  0001 C CNN
+F 2 "OTTO_Footprints_Lib:SOIC-8_3.9x4.9mm_P1.27mm" H 3850 2050 50  0001 C CNN
 F 3 "https://datasheet.lcsc.com/szlcsc/C16072.pdf" H 3650 1950 50  0001 C CNN
 F 4 "" H 3650 1950 12700 0001 C CNN "UnitCost(USD)"
@@
 F 0 "U5" H 11800 6816 50  0000 C CNN
 F 1 "TPS22918_SOT23-6_A" H 11800 6725 50  0000 C CNN
-F 2 "Package_TO_SOT_SMD:SOT-23-6" H 11800 6950 50  0001 C CNN
+F 2 "OTTO_Footprints_Lib:SOT-23-6" H 11800 6950 50  0001 C CNN
 F 3 "https://datasheet.lcsc.com/szlcsc/C131941.pdf" H 11850 5750 50  0001 C CNN
 F 4 "" H 11800 6450 12700 0001 C CNN "UnitCost(USD)"
@@
 F 0 "C84" H 10468 6645 50  0000 L CNN
 F 1 "470uF" H 10468 6555 50  0000 L CNN
-F 2 "Capacitor_SMD:CP_Elec_6.3x7.7" H 10388 6450 50  0001 C CNN
+F 2 "OTTO_Footprints_Lib:CP_Elec_6.3x7.7" H 10388 6450 50  0001 C CNN
 F 3 "https://datasheet.lcsc.com/szlcsc/C134834.pdf" H 10350 6600 50  0001 C CNN
 F 4 "" H 10350 6600 12700 0001 C CNN "UnitCost(USD)"
@@
 F 0 "C81" H 9968 6645 50  0000 L CNN
 F 1 "470uF" H 9968 6555 50  0000 L CNN
-F 2 "Capacitor_SMD:CP_Elec_6.3x7.7" H 9888 6450 50  0001 C CNN
+F 2 "OTTO_Footprints_Lib:CP_Elec_6.3x7.7" H 9888 6450 50  0001 C CNN
 F 3 "https://datasheet.lcsc.com/szlcsc/C134834.pdf" H 9850 6600 50  0001 C CNN
 F 4 "" H 9850 6600 12700 0001 C CNN "UnitCost(USD)"
@@
 F 0 "C79" H 9468 6645 50  0000 L CNN
 F 1 "470uF" H 9468 6555 50  0000 L CNN
-F 2 "Capacitor_SMD:CP_Elec_6.3x7.7" H 9388 6450 50  0001 C CNN
+F 2 "OTTO_Footprints_Lib:CP_Elec_6.3x7.7" H 9388 6450 50  0001 C CNN
 F 3 "https://datasheet.lcsc.com/szlcsc/C134834.pdf" H 9350 6600 50  0001 C CNN
 F 4 "" H 9350 6600 12700 0001 C CNN "UnitCost(USD)"
@@
 F 0 "U2" H 11800 8666 50  0000 C CNN
 F 1 "TPS22918_SOT23-6_A" H 11800 8575 50  0000 C CNN
-F 2 "Package_TO_SOT_SMD:SOT-23-6" H 11800 8800 50  0001 C CNN
+F 2 "OTTO_Footprints_Lib:SOT-23-6" H 11800 8800 50  0001 C CNN
 F 3 "https://datasheet.lcsc.com/szlcsc/C131941.pdf" H 11850 7600 50  0001 C CNN
 F 4 "" H 11800 8300 12700 0001 C CNN "UnitCost(USD)"
@@
 F 0 "U4" H 10750 5065 50  0000 C CNN
 F 1 "MP2359" H 10750 4974 50  0000 C CNN
-F 2 "Package_TO_SOT_SMD:TSOT-23-6_HandSoldering" H 10800 5000 50  0001 C CNN
+F 2 "OTTO_Footprints_Lib:TSOT-23-6_HandSoldering" H 10800 5000 50  0001 C CNN
 F 3 "https://datasheet.lcsc.com/szlcsc/C14259.pdf" H 10800 5000 50  0001 C CNN
 F 4 "BASIC" H 10750 4650 50  0001 C CNN "JLCASM"
@@
 F 0 "U204" H 4950 5031 50  0000 C CNN
 F 1 "SRV05-4" H 4950 4940 50  0000 C CNN
-F 2 "Package_TO_SOT_SMD:SOT-23-6" H 5650 3900 50  0001 C CNN
+F 2 "OTTO_Footprints_Lib:SOT-23-6" H 5650 3900 50  0001 C CNN
 F 3 "http://www.onsemi.com/pub/Collateral/SRV05-4-D.PDF" H 4950 4350 50  0001 C CNN
 F 4 "BASIC" H 4950 4350 50  0001 C CNN "JLCASM"
