File: KiCad/AUDIO.sch (KiCad schematic (older format))
At the start: 60 parts, among them J206 Conn_02x06, J207 Conn_02x03, U207 WM8731-Audio, U208 TPS79533, Y203 12.288MHz

Commit message: roll in changes from Bastian
Parts:
- removed D? (x5): 5V, symbol Device:D_TVS_ALT
- added D? (x6): 5V, symbol Device:D_TVS_ALT
- added R235, R236, R237, R238: 33, Resistor_SMD:R_0805_2012Metric_Pad1.15x1.40mm_HandSolder, symbol Device:R
- D?: Manufacturer (none) -> Littelfuse; Part Number (none) -> SMA5.0CA
Connections:
- net labels added: (F427)_SAI1_FS_A, (F427)_SAI1_SCK_A, (F427)_SAI1_SD_A, (F427)_SAI1_SD_B, AMP_OUT_L, AMP_OUT_R
- wire segments 214 -> 217
- no-connect marks 55 -> 53

Commit message: added power switching and extra pulls for programming lines
Connections:
- net labels added: +5V_PI
- net labels removed: +5V_MAIN
- wire segments 217 -> 218
Changed lines of the file:
@@
-EESchema Schematic File Version 4
+EESchema Schematic File Version 5
 EELAYER 30 0
 EELAYER END
-$Descr A4 11693 8268
+$Descr A3 16535 11693
 encoding utf-8
 Sheet 7 7
@@
 Comment3 ""
 Comment4 ""
+Comment5 ""
+Comment6 ""
+Comment7 ""
+Comment8 ""
+Comment9 ""
 $EndDescr
 Wire Wire Line
@@
 	-1   0    0    -1
 $EndComp
-Text GLabel 4250 6850 0    50   Input ~ 0
-+5V_MAIN
+Text GLabel 4150 6750 0    50   Input ~ 0
++5V_PI
 Text GLabel 6150 6850 2    50   Input ~ 0
 +3V3_ANALOG
-Wire Wire Line
-	4250 6850 4350 6850
 Wire Wire Line
 	6150 6850 5550 6850
@@
 	1200 6050 1300 6050
 Text GLabel 10200 5100 2    50   Input ~ 0
-+5V_MAIN
++5V_PI
 $Comp
 L Device:C C?
@@
 L Device:C C267
 U 1 1 5E317C6C
-P 4350 7100
-F 0 "C267" H 4235 7054 50  0000 R CNN
-F 1 "10µF" H 4235 7145 50  0000 R CNN
-F 2 "Capacitor_SMD:C_0805_2012Metric_Pad1.15x1.40mm_HandSolder" H 4388 6950 50  0001 C CNN
-F 3 "~" H 4350 7100 50  0001 C CNN
-	1    4350 7100
+P 4250 7100
+F 0 "C267" H 4135 7054 50  0000 R CNN
+F 1 "10µF" H 4135 7145 50  0000 R CNN
+F 2 "Capacitor_SMD:C_0805_2012Metric_Pad1.15x1.40mm_HandSolder" H 4288 6950 50  0001 C CNN
+F 3 "~" H 4250 7100 50  0001 C CNN
+	1    4250 7100
 	-1   0    0    1
 $EndComp
@@
 Wire Wire Line
 	5550 6850 5550 6950
-Wire Wire Line
-	4450 6850 4350 6850
-Wire Wire Line
-	4350 6850 4350 6950
-Wire Wire Line
-	4450 6750 4350 6750
-Wire Wire Line
-	4350 6750 4350 6850
-Connection ~ 4350 6850
 Connection ~ 5550 6850
 Wire Wire Line
@@
 	4950 7350 4950 7450
 Wire Wire Line
-	4350 7250 4350 7350
-Wire Wire Line
-	4350 7350 4950 7350
+	4250 7250 4250 7350
+Wire Wire Line
+	4250 7350 4950 7350
 Wire Wire Line
 	6050 7350 6050 7250
@@
 Wire Wire Line
 	1700 7450 1600 7450
+Wire Wire Line
+	4150 6750 4250 6750
+Wire Wire Line
+	4250 6750 4250 6950
+Wire Wire Line
+	4250 6750 4350 6750
+Connection ~ 4250 6750
+Wire Wire Line
+	4450 6850 4350 6850
+Wire Wire Line
+	4350 6750 4350 6850
+Connection ~ 4350 6750
+Wire Wire Line
+	4350 6750 4450 6750
 $EndSCHEMATC

Commit message: connected unconnected signals and MIDI to spare MCU UART
Parts:
- gave numbers to parts that had none: 7
Connections:
- wire segments 218 -> 219

Commit message: add all resistor part numbers and create footprint library
Parts:
- D50, D51, D52, D53, D54, D55, D56: MPN (none) -> SMA5.0CA; Part Number SMA5.0CA -> (none)
- MK201: EstimatedCost(USD) (none) -> $.127273; MPN (none) -> GMI6050P-42db; Manufacturer (none) -> INGHAi
- R218, R219, R222, R224: EstimatedCost(USD) (none) -> $.001726; MPN (none) -> RC0805FR-075K1L; Manufacturer (none) -> Yageo
- R220, R223: EstimatedCost(USD) (none) -> $.001752; MPN (none) -> RC0805FR-07100RL; Manufacturer (none) -> Yageo
- R221, R225, R228, R229, R230: EstimatedCost(USD) (none) -> $.004358; MPN (none) -> RC0805FR-0747KL; Manufacturer (none) -> Yageo
- R226: EstimatedCost(USD) (none) -> $.001714; MPN (none) -> RC0805FR-07680RL; Manufacturer (none) -> Yageo
- R227: EstimatedCost(USD) (none) -> $.001575; MPN (none) -> RC0805FR-07330RL; Manufacturer (none) -> Yageo
- R231, R232, R233, R234, R235, R236, R237, R238: EstimatedCost(USD) (none) -> $.001685; MPN (none) -> RC0805FR-0733RL; Manufacturer (none) -> Yageo

Commit message: added part numbers for capacitors and crystals
Parts:
- C243, C246, C247, C250, C264: value 10µ -> 10uF
- C251, C253, C254, C255, C257: value 1µF (AUDIO) -> 1uF (AUDIO); footprint Capacitor_THT:C_Rect_L7.2mm_W5.0mm_P5.00mm_FKS2_FKP2_MKS2_MKP2 -> OTTO_Footprints_Lib:C_Rect_L7.2mm_W5.0mm_P5.00mm_FKS2_FKP2_MKS2_MKP2
- C252, C256, C259: value 220p (C0G) -> 220pF (C0G); footprint Capacitor_SMD:C_0805_2012Metric_Pad1.15x1.40mm_HandSolder -> Capacitor_SMD:C_1206_3216Metric_Pad1.42x1.75mm_HandSolder
- C258, C262: value 220µF -> 220uF
- C260, C261, C267, C268: value 10µF -> 10uF
- C70, C71, C72, C73, C74, C75: footprint Capacitor_SMD:C_0805_2012Metric_Pad1.15x1.40mm_HandSolder_marked -> Capacitor_SMD:C_0805_2012Metric_Pad1.15x1.40mm_HandSolder; EstimatedCost(USD) (none) -> $0.017724; MPN (none) -> CL21B104JBCNNNC; Manufacturer (none) -> Samsung Electro-Mechanics
- MK201: EstimatedCost(USD) $.127273 -> $0.127273
- Y203: footprint Crystal:Crystal_HC49-U_Vertical -> Crystal:Crystal_SMD_HC49-SD_HandSoldering; EstimatedCost(USD) (none) -> $0.084038; MPN (none) -> X49SM12288MSD2SC; Manufacturer (none) -> Yangxing Tech

Commit message: more part numbers added: audio caps
Parts:
- C243, C246, C247, C250, C260, C261, C264, C267, C268: EstimatedCost(USD) (none) -> $0.041113; MPN (none) -> CL21B106KOQNNNE; Manufacturer (none) -> Samsung Electro-Mechanics
- C251, C253, C254, C255, C257: EstimatedCost(USD) (none) -> $0.315152; MPN (none) -> MKS2C041001F00JSSD; Manufacturer (none) -> WIMA
- C252, C256, C259: footprint Capacitor_SMD:C_1206_3216Metric_Pad1.42x1.75mm_HandSolder -> Capacitor_SMD:C_0805_2012Metric_Pad1.15x1.40mm_HandSolder; EstimatedCost(USD) (none) -> $0.010055; MPN (none) -> CL21C221JBANNNC; Manufacturer (none) -> Samsung Electro-Mechanics
- C258, C262: EstimatedCost(USD) (none) -> $0.168182; MPN (none) -> UHE1V221MPD6; Manufacturer (none) -> Nichicon
- C265, C266: value 20pF -> 30pF; EstimatedCost(USD) (none) -> $0.005588; MPN (none) -> CC0805JRNPO9BN300; Manufacturer (none) -> Yageo
Connections:
- net labels removed: XTI, XTO
- wire segments 219 -> 209
Other:
- note removed: "Audio caps\n1µF: WIMA MKS2C041001F00JSSD\n220µF: Nichicon UHE1V221MPD6\n\nMicrophone:\nINGHAi GMI6050p"

Commit message: add more part numbers, samtec connector footprint
Parts:
- removed D50, D51, D52, D53, D54, D55, D56: 5V, symbol Device:D_TVS_ALT
- removed DUMMY202: FE-PI AUDIO Z V2, Spatz:Raspberry Pi Zero - (minus 1 hole), symbol Connector:Raspberry_Pi_2_3
- added D50, D51, D52, D53, D54, D55, D56: 6V, Package_TO_SOT_SMD:SOT-323_SC-70_Handsoldering, symbol OTTOdiy_SMD-library:D_TVS_SC70-3
Connections:
- no-connect marks 53 -> 13
Other:
- note removed: "Dummy for component alignment"

Commit message: add switch and encoder parts. BM Complete. Footprints complete.
Parts:
- J206: footprint Connector_Harwin:Harwin_M20-7810645_2x06_P2.54mm_Vertical_SolderHoles -> OTTO_Footprints_Lib:Harwin_M20-7810645_2x06_P2.54mm_Vertical_SolderHoles; EstimatedCost(USD) (none) -> $1.71; MPN (none) -> M20-7810645; Manufacturer (none) -> Harwin
- J207: footprint Connector_Harwin:Harwin_M20-7810345_2x03_P2.54mm_Vertical_SolderHoles -> OTTO_Footprints_Lib:Harwin_M20-7810345_2x03_P2.54mm_Vertical_SolderHoles; EstimatedCost(USD) (none) -> $0.92; MPN (none) -> M20-7810345; Manufacturer (none) -> Harwin
- MK201: footprint Sensor_Audio:INGHAi GMI6050p -> OTTO_Footprints_Lib:INGHAi_GMI6050p
- TRS204, TRS205, TRS206: footprint Spatz:3.5mm_jack_PJ-3930-8A -> OTTO_Footprints_Lib:3.5mm_jack_PJ-3930-8A; EstimatedCost(USD) (none) -> $0.456061; MPN (none) -> PJ-3930-8A; Manufacturer (none) -> Korean Hroparts Elec
- U207: value WM8731-Audio -> WM8731; EstimatedCost(USD) (none) -> $2.181818; MPN (none) -> WM8731SEDS/RV; Manufacturer (none) -> Cirrus Logic
- U208: EstimatedCost(USD) (none) -> $2.324242; MPN (none) -> TPS79533DCQR; Manufacturer (none) -> Texas Instruments
Changed lines of the file:
@@
 F 0 "TRS206" H 12170 4550 50  0000 R CNN
 F 1 "PJ-3930-8A" H 12170 4459 50  0000 R CNN
-F 2 "Spatz:3.5mm_jack_PJ-3930-8A" H 12550 4450 50  0001 C CNN
-F 3 "" H 12550 4450 50  0001 C CNN
+F 2 "OTTO_Footprints_Lib:3.5mm_jack_PJ-3930-8A" H 12550 4450 50  0001 C CNN
+F 3 "https://datasheet.lcsc.com/szlcsc/1911181432_Korean-Hroparts-Elec-PJ-3930-8A_C145811.pdf" H 12550 4450 50  0001 C CNN
+F 4 "$0.456061" H 12450 4450 12700 0001 C CNN "EstimatedCost(USD)"
+F 5 "PJ-3930-8A" H 12450 4450 12700 0001 C CNN "MPN"
+F 6 "Korean Hroparts Elec" H 12450 4450 12700 0001 C CNN "Manufacturer"
 	1    12450 4450
 	-1   0    0    -1
@@
 F 0 "TRS205" H 12170 3350 50  0000 R CNN
 F 1 "PJ-3930-8A" H 12170 3259 50  0000 R CNN
-F 2 "Spatz:3.5mm_jack_PJ-3930-8A" H 12550 3250 50  0001 C CNN
-F 3 "" H 12550 3250 50  0001 C CNN
+F 2 "OTTO_Footprints_Lib:3.5mm_jack_PJ-3930-8A" H 12550 3250 50  0001 C CNN
+F 3 "https://datasheet.lcsc.com/szlcsc/1911181432_Korean-Hroparts-Elec-PJ-3930-8A_C145811.pdf" H 12550 3250 50  0001 C CNN
+F 4 "$0.456061" H 12450 3250 12700 0001 C CNN "EstimatedCost(USD)"
+F 5 "PJ-3930-8A" H 12450 3250 12700 0001 C CNN "MPN"
+F 6 "Korean Hroparts Elec" H 12450 3250 12700 0001 C CNN "Manufacturer"
 	1    12450 3250
 	-1   0    0    -1
@@
 F 0 "MK201" V 11083 4150 50  0000 C CNN
 F 1 "Microphone" V 11174 4150 50  0000 C CNN
-F 2 "Sensor_Audio:INGHAi GMI6050p" V 11350 4250 50  0001 C CNN
+F 2 "OTTO_Footprints_Lib:INGHAi_GMI6050p" V 11350 4250 50  0001 C CNN
 F 3 "https://datasheet.lcsc.com/szlcsc/INGHAi-GMI6050P-42db_C233942.pdf" V 11350 4250 50  0001 C CNN
 F 4 "$0.127273" H 11350 4150 50  0001 C CNN "EstimatedCost(USD)"
@@
 F 1 "TPS79533" H 6250 8724 50  0000 C CNN
 F 2 "Package_TO_SOT_SMD:SOT-223-6" H 7000 8050 50  0001 C CNN
-F 3 "" H 7000 8050 50  0001 C CNN
+F 3 "http://www.ti.com/lit/ds/symlink/tps795.pdf" H 7000 8050 50  0001 C CNN
+F 4 "TPS79533DCQR" H 6250 8550 12700 0001 C CNN "MPN"
+F 5 "Texas Instruments" H 6250 8550 12700 0001 C CNN "Manufacturer"
+F 6 "$2.324242" H 6250 8550 12700 0001 C CNN "EstimatedCost(USD)"
 	1    6250 8550
 	1    0    0    -1
@@
 P 6350 2800
 F 0 "U207" H 6350 4065 50  0000 C CNN
-F 1 "WM8731-Audio" H 6350 3974 50  0000 C CNN
+F 1 "WM8731" H 6350 3974 50  0000 C CNN
 F 2 "Package_SO:TSSOP-28_4.4x9.7mm_P0.65mm" H 11300 1100 50  0001 L CNN
-F 3 "" H 11300 1100 50  0001 L CNN
+F 3 "https://statics.cirrus.com/pubs/proDatasheet/WM8731_v4.9.pdf" H 11300 1100 50  0001 L CNN
+F 4 "$2.181818" H 6350 2800 12700 0001 C CNN "EstimatedCost(USD)"
+F 5 "WM8731SEDS/RV" H 6350 2800 12700 0001 C CNN "MPN"
+F 6 "Cirrus Logic" H 6350 2800 12700 0001 C CNN "Manufacturer"
 	1    6350 2800
 	1    0    0    -1
@@
 F 0 "TRS204" H 12170 2400 50  0000 R CNN
 F 1 "PJ-3930-8A" H 12170 2309 50  0000 R CNN
-F 2 "Spatz:3.5mm_jack_PJ-3930-8A" H 12550 2300 50  0001 C CNN
-F 3 "" H 12550 2300 50  0001 C CNN
+F 2 "OTTO_Footprints_Lib:3.5mm_jack_PJ-3930-8A" H 12550 2300 50  0001 C CNN
+F 3 "https://datasheet.lcsc.com/szlcsc/1911181432_Korean-Hroparts-Elec-PJ-3930-8A_C145811.pdf" H 12550 2300 50  0001 C CNN
+F 4 "$0.456061" H 12450 2300 12700 0001 C CNN "EstimatedCost(USD)"
+F 5 "PJ-3930-8A" H 12450 2300 12700 0001 C CNN "MPN"
+F 6 "Korean Hroparts Elec" H 12450 2300 12700 0001 C CNN "Manufacturer"
 	1    12450 2300
 	-1   0    0    -1
@@
 F 0 "J207" H 11850 7617 50  0000 C CNN
 F 1 "Conn_02x03" H 11850 7526 50  0000 C CNN
-F 2 "Connector_Harwin:Harwin_M20-7810345_2x03_P2.54mm_Vertical_SolderHoles" H 11800 7300 50  0001 C CNN
-F 3 "~" H 11800 7300 50  0001 C CNN
+F 2 "OTTO_Footprints_Lib:Harwin_M20-7810345_2x03_P2.54mm_Vertical_SolderHoles" H 11800 7300 50  0001 C CNN
+F 3 "https://cdn.harwin.com/pdfs/Harwin_PC_Connectors_M20.pdf" H 11800 7300 50  0001 C CNN
+F 4 "$0.92" H 11800 7300 12700 0001 C CNN "EstimatedCost(USD)"
+F 5 "M20-7810345" H 11800 7300 12700 0001 C CNN "MPN"
+F 6 "Harwin" H 11800 7300 12700 0001 C CNN "Manufacturer"
 	1    11800 7300
 	1    0    0    -1
@@
 F 0 "J206" H 11850 6967 50  0000 C CNN
 F 1 "Conn_02x06" H 11850 6876 50  0000 C CNN
-F 2 "Connector_Harwin:Harwin_M20-7810645_2x06_P2.54mm_Vertical_SolderHoles" H 11800 6550 50  0001 C CNN
-F 3 "~" H 11800 6550 50  0001 C CNN
+F 2 "OTTO_Footprints_Lib:Harwin_M20-7810645_2x06_P2.54mm_Vertical_SolderHoles" H 11800 6550 50  0001 C CNN
+F 3 "https://cdn.harwin.com/pdfs/Harwin_PC_Connectors_M20.pdf" H 11800 6550 50  0001 C CNN
+F 4 "$1.71" H 11800 6550 12700 0001 C CNN "EstimatedCost(USD)"
+F 5 "M20-7810645" H 11800 6550 12700 0001 C CNN "MPN"
+F 6 "Harwin" H 11800 6550 12700 0001 C CNN "Manufacturer"
 	1    11800 6550
 	1    0    0    -1
