File: KiCad/AUDIO.sch (KiCad schematic (older format))
At the start: 64 parts, among them J206 Conn_02x06, J207 Conn_02x03, U207 WM8731, U208 TPS79533, Y203 12.288MHz

Commit message: add BOM scripts, fix schematic hierarchy
Parts:
- C243, C246, C247, C250, C260, C261, C264, C267, C268: EstimatedCost(USD) $0.041113 -> (none); UnitCost(USD) (none) -> $0.041113
- C251, C253, C254, C255, C257: EstimatedCost(USD) $0.315152 -> (none); UnitCost(USD) (none) -> $0.315152
- C252, C256, C259: EstimatedCost(USD) $0.010055 -> (none); UnitCost(USD) (none) -> $0.010055
- C258, C262: EstimatedCost(USD) $0.168182 -> (none); UnitCost(USD) (none) -> $0.168182
- C265, C266: EstimatedCost(USD) $0.005588 -> (none); UnitCost(USD) (none) -> $0.005588
- C70, C71, C72, C73, C74, C75: EstimatedCost(USD) $0.017724 -> (none); UnitCost(USD) (none) -> $0.017724
- D50, D51, D52, D53, D54, D55, D56: value 6V -> 6V BI TVS; EstimatedCost(USD) $0.159091 -> (none); UnitCost(USD) (none) -> $0.159091
- J206: EstimatedCost(USD) $1.71 -> (none); UnitCost(USD) (none) -> $1.71
- J207: EstimatedCost(USD) $0.92 -> (none); UnitCost(USD) (none) -> $0.92
- MK201: EstimatedCost(USD) $0.127273 -> (none); UnitCost(USD) (none) -> $0.127273
- R218, R219, R222, R224: EstimatedCost(USD) $.001726 -> (none); UnitCost(USD) (none) -> $.001726
- R220, R223: EstimatedCost(USD) $.001752 -> (none); UnitCost(USD) (none) -> $.001752
- R221, R225, R228, R229, R230: EstimatedCost(USD) $.004358 -> (none); UnitCost(USD) (none) -> $.004358
- R226: EstimatedCost(USD) $.001714 -> (none); UnitCost(USD) (none) -> $.001714
- R227: EstimatedCost(USD) $.001575 -> (none); UnitCost(USD) (none) -> $.001575
- R231, R232, R233, R234, R235, R236, R237, R238: EstimatedCost(USD) $.001685 -> (none); UnitCost(USD) (none) -> $.001685
- TRS204, TRS205, TRS206: EstimatedCost(USD) $0.456061 -> (none); UnitCost(USD) (none) -> $0.456061
- U207: EstimatedCost(USD) $2.181818 -> (none); UnitCost(USD) (none) -> $2.181818
- U208: EstimatedCost(USD) $2.324242 -> (none); UnitCost(USD) (none) -> $2.324242
- Y203: EstimatedCost(USD) $0.084038 -> (none); UnitCost(USD) (none) -> $0.084038

Commit message: Add power switch and other misc nice to haves
Parts:
- added J2, J3: JST 2-pin SH, Connector_JST:JST_SH_SM02B-SRSS-TB_1x02-1MP_P1.00mm_Horizontal, symbol Connector_Generic_MountingPin:Conn_01x02_MountingPin
- added TP11, TP12, TP13, TP14, TP15: TestPoint, TestPoint:TestPoint_Keystone_5000-5004_Miniature, symbol Connector:TestPoint
- R235, R236, R237, R238: AssemblyOption (none) -> DNP
Connections:
- net labels added: LI_SENSE, LO_SENSE
- wire segments 209 -> 228
- no-connect marks 13 -> 12

Commit message: Fixes for external battery board and Routing started
Connections:
- net labels added: +5V_RASPI
- net labels removed: +5V_PI
Changed lines of the file:
@@
 $EndComp
 Text GLabel 5450 8550 0    50   Input ~ 0
-+5V_PI
++5V_RASPI
 Text GLabel 7450 8650 2    50   Input ~ 0
 +3V3_ANALOG
@@
 $EndComp
 Text GLabel 12300 6750 2    50   Input ~ 0
-+5V_PI
++5V_RASPI
 Text GLabel 11400 6850 0    50   BiDi ~ 0
 I2C_SDA

Commit message: Add SP3T style DP3T footprint and some schematic labels
Other:
- note added: "Pi-Compatible External Codec Interface\nHeader is split for more PCB space"
- note removed: "split audio header\nfor more PCB space"

Commit message: routed buck boost supply
Parts:
- removed J2, J3: JST 2-pin SH, Connector_JST:JST_SH_SM02B-SRSS-TB_1x02-1MP_P1.00mm_Horizontal, symbol Connector_Generic_MountingPin:Conn_01x02_MountingPin
- removed TP11, TP12, TP13, TP14: TestPoint, TestPoint:TestPoint_Keystone_5000-5004_Miniature, symbol Connector:TestPoint
- added J2: Conn_02x04, Connector_PinHeader_2.54mm:PinHeader_2x04_P2.54mm_Vertical, symbol Connector_Generic:Conn_02x04_Odd_Even
- added R26: 100k, Resistor_SMD:R_0805_2012Metric_Pad1.15x1.40mm_HandSolder, symbol Device:R
- C258, C262: footprint Capacitor_THT:CP_Radial_D10.0mm_P5.00mm -> Capacitor_THT:CP_Radial_D6.3mm_P2.50mm; MPN UHE1V221MPD6 -> UHE1A221MED; UnitCost(USD) $0.168182 -> $0.116756
- C260, C261, J206, J207: AssemblyOption (none) -> DNP
Connections:
- net labels added: +5V_REG, AMP_ENABLE
- wire segments 228 -> 225
- no-connect marks 12 -> 10
Other:
- note added: "Header for external amplifier board."

Commit message: routed audio
Parts:
- Y203: footprint Crystal:Crystal_SMD_HC49-SD_HandSoldering -> Crystal:Crystal_SMD_5032-2Pin_5.0x3.2mm_HandSoldering; MPN X49SM12288MSD2SC -> 6I12288F20UCG; Manufacturer Yangxing Tech -> SJK(SHENZHEN CRYSTAL TECH); UnitCost(USD) $0.084038 -> $0.192424
Changed lines of the file:
@@
 F 0 "Y203" H 5650 6818 50  0000 C CNN
 F 1 "12.288MHz" H 5650 6727 50  0000 C CNN
-F 2 "Crystal:Crystal_SMD_HC49-SD_HandSoldering" H 5650 6550 50  0001 C CNN
-F 3 "https://datasheet.lcsc.com/szlcsc/Yangxing-Tech-X49SM12288MSD2SC_C11240.pdf" H 5650 6550 50  0001 C CNN
-F 4 "$0.084038" H 5650 6550 12700 0001 C CNN "UnitCost(USD)"
-F 5 "X49SM12288MSD2SC" H 5650 6550 12700 0001 C CNN "MPN"
-F 6 "Yangxing Tech" H 5650 6550 12700 0001 C CNN "Manufacturer"
+F 2 "Crystal:Crystal_SMD_5032-2Pin_5.0x3.2mm_HandSoldering" H 5650 6550 50  0001 C CNN
+F 3 "https://datasheet.lcsc.com/szlcsc/SHENZHEN-CRYSTAL-TECH-6I12288F20UCG_C251589.pdf" H 5650 6550 50  0001 C CNN
+F 4 "$0.192424" H 5650 6550 12700 0001 C CNN "UnitCost(USD)"
+F 5 "6I12288F20UCG" H 5650 6550 12700 0001 C CNN "MPN"
+F 6 "SJK(SHENZHEN CRYSTAL TECH)" H 5650 6550 12700 0001 C CNN "Manufacturer"
 	1    5650 6550
 	1    0    0    -1
@@
 F 6 "Littelfuse" H 11650 4100 50  0001 C CNN "Manufacturer"
 	1    11650 4100
-	1    0    0    -1
+	-1   0    0    -1
 $EndComp
 $Comp
@@
 F 6 "Littelfuse" H 11650 4500 50  0001 C CNN "Manufacturer"
 	1    11650 4500
-	1    0    0    -1
-$EndComp
-$Comp
+	-1   0    0    -1
+$EndComp
+$Comp

Commit message: add analog ground layout
Parts:
- added NT1: Net-Tie_2, OTTO_Footprints_Lib:NetTie-2_Pad5.0mm, symbol Device:Net-Tie_2
Connections:
- wire segments 225 -> 224
Changed lines of the file:
@@
 Wire Wire Line
 	7850 8250 7250 8250
-$Comp
-L power:GND #PWR?
-U 1 1 5E376CBF
-P 6750 8850
-AR Path="/5C4320DF/5E376CBF" Ref="#PWR?"  Part="1"
-AR Path="/5C4320DF/5DB999B7/5E376CBF" Ref="#PWR?"  Part="1"
-AR Path="/5C4408C6/5E376CBF" Ref="#PWR0256"  Part="1"
-F 0 "#PWR0256" H 6750 8600 50  0001 C CNN
-F 1 "GND" H 6755 8677 50  0000 C CNN
-F 2 "" H 6750 8850 50  0001 C CNN
-F 3 "" H 6750 8850 50  0001 C CNN
-	1    6750 8850
-	1    0    0    -1
-$EndComp
 Text Label 5600 5050 0    50   ~ 0
 I2S_LRCLK*
@@
 L power:GNDA #PWR0101
 U 1 1 5DF89554
-P 6700 6750
-F 0 "#PWR0101" H 6700 6500 50  0001 C CNN
-F 1 "GNDA" V 6705 6622 50  0000 R CNN
-F 2 "" H 6700 6750 50  0001 C CNN
-F 3 "" H 6700 6750 50  0001 C CNN
-	1    6700 6750
+P 6700 7000
+F 0 "#PWR0101" H 6700 6750 50  0001 C CNN
+F 1 "GNDA" V 6705 6872 50  0000 R CNN
+F 2 "" H 6700 7000 50  0001 C CNN
+F 3 "" H 6700 7000 50  0001 C CNN
+	1    6700 7000
 	0    1    1    0
 $EndComp
@@
 $Comp
 L power:GND #PWR?
-U 1 1 5E13F046
-P 7350 8850
-AR Path="/5C4320DF/5E13F046" Ref="#PWR?"  Part="1"
-AR Path="/5C4320DF/5DB999B7/5E13F046" Ref="#PWR?"  Part="1"
-AR Path="/5C4408C6/5E13F046" Ref="#PWR014"  Part="1"
-F 0 "#PWR014" H 7350 8600 50  0001 C CNN
-F 1 "GND" H 7355 8677 50  0000 C CNN
-F 2 "" H 7350 8850 50  0001 C CNN
-F 3 "" H 7350 8850 50  0001 C CNN
-	1    7350 8850
-	1    0    0    -1
-$EndComp
-$Comp
-L power:GND #PWR?
-U 1 1 5E13FBC2
-P 7850 8850
-AR Path="/5C4320DF/5E13FBC2" Ref="#PWR?"  Part="1"
-AR Path="/5C4320DF/5DB999B7/5E13FBC2" Ref="#PWR?"  Part="1"
-AR Path="/5C4408C6/5E13FBC2" Ref="#PWR015"  Part="1"
-F 0 "#PWR015" H 7850 8600 50  0001 C CNN
-F 1 "GND" H 7855 8677 50  0000 C CNN
-F 2 "" H 7850 8850 50  0001 C CNN
-F 3 "" H 7850 8850 50  0001 C CNN
-	1    7850 8850
-	1    0    0    -1
-$EndComp
-$Comp
-L power:GND #PWR?
 U 1 1 5E14054A
 P 5950 7100
@@
 L power:GND #PWR?
 U 1 1 5DF89B24
-P 6850 6750
+P 6900 7000
 AR Path="/5D186267/5D1201D8/5DB14620/5DF89B24" Ref="#PWR?"  Part="1"
 AR Path="/5D186267/5D1201D8/5D12037D/5DF89B24" Ref="#PWR?"  Part="1"
 AR Path="/5C4408C6/5DF89B24" Ref="#PWR0102"  Part="1"
-F 0 "#PWR0102" H 6850 6500 50  0001 C CNN
-F 1 "GND" V 6855 6622 50  0000 R CNN
-F 2 "" H 6850 6750 50  0001 C CNN
-F 3 "" H 6850 6750 50  0001 C CNN
-	1    6850 6750
+F 0 "#PWR0102" H 6900 6750 50  0001 C CNN
+F 1 "GND" V 6905 6872 50  0000 R CNN
+F 2 "" H 6900 7000 50  0001 C CNN
+F 3 "" H 6900 7000 50  0001 C CNN
+	1    6900 7000
 	0    -1   -1   0
-$EndComp
-Wire Wire Line
-	6700 6750 6850 6750
-$Comp
-L power:GND #PWR?
-U 1 1 5E13E31F
-P 6050 8850
-AR Path="/5C4320DF/5E13E31F" Ref="#PWR?"  Part="1"
-AR Path="/5C4320DF/5DB999B7/5E13E31F" Ref="#PWR?"  Part="1"
-AR Path="/5C4408C6/5E13E31F" Ref="#PWR013"  Part="1"
-F 0 "#PWR013" H 6050 8600 50  0001 C CNN
-F 1 "GND" H 6055 8677 50  0000 C CNN
-F 2 "" H 6050 8850 50  0001 C CNN
-F 3 "" H 6050 8850 50  0001 C CNN
-	1    6050 8850
-	1    0    0    -1
 $EndComp
 Wire Wire Line
@@
 Text GLabel 2600 10250 2    50   Output ~ 0
 (F427)_SAI1_SD_B
+$Comp
+L Device:Net-Tie_2 NT1
+U 1 1 5E3E65E9
+P 6800 7000
+F 0 "NT1" H 6800 7181 50  0000 C CNN
+F 1 "Net-Tie_2" H 6800 7090 50  0000 C CNN
+F 2 "OTTO_Footprints_Lib:NetTie-2_Pad5.0mm" H 6800 7000 50  0001 C CNN
+F 3 "N/A" H 6800 7000 50  0001 C CNN
+F 4 "DNP" H 6800 7000 50  0001 C CNN "AssemblyOption"
+F 5 "N/A" H 6800 7000 50  0001 C CNN "MPN"
+F 6 "N/A" H 6800 7000 50  0001 C CNN "Manufacturer"
+F 7 "$0.00" H 6800 7000 50  0001 C CNN "UnitCost(USD)"
+	1    6800 7000
+	1    0    0    -1
+$EndComp
+$Comp
+L power:GNDA #PWR0112
+U 1 1 5E45FDC2
+P 7850 8850
+F 0 "#PWR0112" H 7850 8600 50  0001 C CNN
+F 1 "GNDA" H 7855 8677 50  0000 C CNN
+F 2 "" H 7850 8850 50  0001 C CNN
+F 3 "" H 7850 8850 50  0001 C CNN
+	1    7850 8850
+	1    0    0    -1
+$EndComp
+$Comp
+L power:GNDA #PWR0113
+U 1 1 5E460570
+P 7350 8850
+F 0 "#PWR0113" H 7350 8600 50  0001 C CNN
+F 1 "GNDA" H 7355 8677 50  0000 C CNN
+F 2 "" H 7350 8850 50  0001 C CNN
+F 3 "" H 7350 8850 50  0001 C CNN
+	1    7350 8850
+	1    0    0    -1
+$EndComp
+$Comp
+L power:GNDA #PWR0114
+U 1 1 5E460972
+P 6750 8850
+F 0 "#PWR0114" H 6750 8600 50  0001 C CNN
+F 1 "GNDA" H 6755 8677 50  0000 C CNN
+F 2 "" H 6750 8850 50  0001 C CNN
+F 3 "" H 6750 8850 50  0001 C CNN
+	1    6750 8850
+	1    0    0    -1
+$EndComp
+$Comp
+L power:GNDA #PWR0115
+U 1 1 5E460CA8
+P 6050 8850
+F 0 "#PWR0115" H 6050 8600 50  0001 C CNN
+F 1 "GNDA" H 6055 8677 50  0000 C CNN
+F 2 "" H 6050 8850 50  0001 C CNN
+F 3 "" H 6050 8850 50  0001 C CNN
+	1    6050 8850
+	1    0    0    -1
+$EndComp
 $EndSCHEMATC
