File: KiCad/AUDIO.sch (KiCad schematic (older format))
At the start: 66 parts, among them J2 Conn_02x04, J206 Conn_02x06, J207 Conn_02x03, U207 WM8731, U208 AMS1117-3.3, Y203 12.288MHz

Commit message: Fix DAC footprint and other minor issues.
Parts:
- C267, C268: symbol Device:C -> Device:CP
- D50, D51, D52, D53, D55, D56: symbol OTTOdiy_SMD-library:D_TVS_SC70-3 -> Device:D_TVS
- U207: footprint Package_SO:TSSOP-28_4.4x9.7mm_P0.65mm -> OTTO_Footprints_Lib:SSOP-28_5.3x10.2mm_P0.65mm
- U208: footprint Package_TO_SOT_SMD:SOT-223-3_TabPin2 -> OTTO_Footprints_Lib:SOT-223-3_TabPin2
Changed lines of the file:
@@
 	6500 10300 6600 10300
 Wire Wire Line
-	11850 3300 13550 3300
-Wire Wire Line
-	11850 4500 13550 4500
+	11800 3300 13550 3300
+Wire Wire Line
+	11800 4500 13550 4500
 Wire Wire Line
 	3530 3050 3030 3050
 Wire Wire Line
-	11350 2350 11450 2350
-Wire Wire Line
-	11350 2550 11450 2550
-Wire Wire Line
-	11850 3500 13550 3500
-Wire Wire Line
-	11350 3300 11450 3300
-Wire Wire Line
-	11450 3500 11350 3500
-Wire Wire Line
-	11350 4700 11450 4700
-Wire Wire Line
-	11450 4500 11350 4500
-Wire Wire Line
-	11850 4700 13550 4700
+	11350 2350 11500 2350
+Wire Wire Line
+	11350 2550 11500 2550
+Wire Wire Line
+	11800 3500 13550 3500
+Wire Wire Line
+	11350 3300 11500 3300
+Wire Wire Line
+	11500 3500 11350 3500
+Wire Wire Line
+	11350 4700 11500 4700
+Wire Wire Line
+	11500 4500 11350 4500
+Wire Wire Line
+	11800 4700 13550 4700
 Wire Wire Line
 	4840 4450 4840 4650
@@
 Connection ~ 8150 2250
 Wire Wire Line
-	11850 2550 13550 2550
-Wire Wire Line
-	11850 2350 13550 2350
+	11800 2550 13550 2550
+Wire Wire Line
+	11800 2350 13550 2350
 Wire Wire Line
 	13450 2150 13550 2150
@@
 F 0 "U207" H 6800 4015 50  0000 C CNN
 F 1 "WM8731" H 6800 3924 50  0000 C CNN
-F 2 "Package_SO:TSSOP-28_4.4x9.7mm_P0.65mm" H 11750 1050 50  0001 L CNN
+F 2 "OTTO_Footprints_Lib:SSOP-28_5.3x10.2mm_P0.65mm" H 11750 1050 50  0001 L CNN
 F 3 "https://datasheet.lcsc.com/szlcsc/C323837.pdf" H 11750 1050 50  0001 L CNN
 F 4 "" H 6800 2750 12700 0001 C CNN "UnitCost(USD)"
@@
 $EndComp
 $Comp
-L OTTOdiy_SMD-library:D_TVS_SC70-3 D51
+L Device:D_TVS D51
 U 1 1 5E18B6FE
 P 11650 2550
@@
 $EndComp
 $Comp
-L OTTOdiy_SMD-library:D_TVS_SC70-3 D53
+L Device:D_TVS D53
 U 1 1 5E18BB75
 P 11650 3500
@@
 $EndComp
 $Comp
-L OTTOdiy_SMD-library:D_TVS_SC70-3 D56
+L Device:D_TVS D56
 U 1 1 5E18C14B
 P 11650 4700
@@
 $EndComp
 $Comp
-L OTTOdiy_SMD-library:D_TVS_SC70-3 D55
+L Device:D_TVS D55
 U 1 1 5E18C478
 P 11650 4500
@@
 $EndComp
 $Comp
-L OTTOdiy_SMD-library:D_TVS_SC70-3 D52
+L Device:D_TVS D52
 U 1 1 5E18C65B
 P 11650 3300
@@
 $EndComp
 $Comp
-L OTTOdiy_SMD-library:D_TVS_SC70-3 D50
+L Device:D_TVS D50
 U 1 1 5E18CB14
 P 11650 2350
@@
 F 0 "U208" H 6450 8592 50  0000 C CNN
 F 1 "AMS1117-3.3" H 6450 8501 50  0000 C CNN
-F 2 "Package_TO_SOT_SMD:SOT-223-3_TabPin2" H 6450 8550 50  0001 C CNN
+F 2 "OTTO_Footprints_Lib:SOT-223-3_TabPin2" H 6450 8550 50  0001 C CNN
 F 3 "http://www.advanced-monolithic.com/pdf/ds1117.pdf" H 6550 8100 50  0001 C CNN
 F 4 "BASIC" H 6450 8350 50  0001 C CNN "JLCASM"
@@
 $EndComp
 $Comp
-L Device:C C268
+L Device:CP C268
 U 1 1 5E2DCBC4
 P 6900 8600
@@
 F 8 "C7171" H 6900 8600 50  0001 C CNN "LCSC PN"
 	1    6900 8600
-	-1   0    0    1
-$EndComp
-$Comp
-L Device:C C267
+	-1   0    0    -1
+$EndComp
+$Comp
+L Device:CP C267
 U 1 1 5ECC00DF
 P 5850 8600

Commit message: Fix crystal symbols & Fix audio caps
Parts:
- Y203: symbol Device:Crystal -> Device:Crystal_GND24
Connections:
- wire segments 215 -> 218
Changed lines of the file:
@@
 encoding utf-8
 Sheet 2 7
-Title "OTTOdiy"
-Date "2020-01-10"
-Rev "1.0"
+Title "OTTO beta"
+Date "2020-05-25"
+Rev "0.1.0"
 Comp "https://github.com/otto-project"
-Comment1 "Design by Bastian \"Spatz\" Mohing and Steven \"adorbs\" Hang"
-Comment2 ""
+Comment1 ""
+Comment2 "Design by Bastian \"Spatz\" Mohing, Steven \"adorbs\" Hang,\\nand Bitfield Audio"
 Comment3 ""
 Comment4 ""
@@
 F 8 "C225866" H 7950 4650 50  0001 C CNN "LCSC PN"
 	1    7950 4650
-	0    1    1    0
+	0    -1   1    0
 $EndComp
 $Comp
@@
 F 8 "C225866" H 7950 5250 50  0001 C CNN "LCSC PN"
 	1    7950 5250
-	0    1    1    0
+	0    -1   1    0
 $EndComp
 $Comp
@@
 $EndComp
 $Comp
-L Device:Crystal Y?
+L Device:Crystal_GND24 Y?
 U 1 1 5DF55A7F
 P 5650 6550
@@
 	1    0    0    -1
 $EndComp
+$Comp
+L power:GND #PWR?
+U 1 1 5EEBDC1D
+P 5650 7100
+AR Path="/5C4320DF/5EEBDC1D" Ref="#PWR?"  Part="1"
+AR Path="/5C4320DF/5DB999B7/5EEBDC1D" Ref="#PWR?"  Part="1"
+AR Path="/5C4408C6/5EEBDC1D" Ref="#PWR?"  Part="1"
+F 0 "#PWR?" H 5650 6850 50  0001 C CNN
+F 1 "GND" H 5655 6927 50  0000 C CNN
+F 2 "" H 5650 7100 50  0001 C CNN
+F 3 "" H 5650 7100 50  0001 C CNN
+	1    5650 7100
+	1    0    0    -1
+$EndComp
+Wire Wire Line
+	5650 7100 5650 6750
+$Comp
+L power:GND #PWR?
+U 1 1 5EECD1C8
+P 5150 6250
+F 0 "#PWR?" H 5150 6000 50  0001 C CNN
+F 1 "GND" V 5155 6122 50  0000 R CNN
+F 2 "" H 5150 6250 50  0001 C CNN
+F 3 "" H 5150 6250 50  0001 C CNN
+	1    5150 6250
+	0    1    1    0
+$EndComp
+Wire Wire Line
+	5150 6250 5650 6250
+Wire Wire Line
+	5650 6250 5650 6350
 $EndSCHEMATC

Commit message: Screen backlight control (+more)
Connections:
- net labels added: RPI_UART_RX, RPI_UART_TX
- net labels removed: MIDI_IN, MIDI_OUT
Changed lines of the file:
@@
 Text Label 14250 8550 2    50   ~ 0
 I2S_BCLK*
-Text GLabel 13500 8450 2    50   Output ~ 0
-MIDI_IN
-Text GLabel 13500 8350 2    50   Input ~ 0
-MIDI_OUT
 $Comp
 L power:GND #PWR0251
@@
 	11850 7200 14350 7200
 Wire Wire Line
-	13500 8350 13300 8350
-Wire Wire Line
-	13500 8450 13300 8450
-Wire Wire Line
 	12800 8450 12600 8450
 Wire Wire Line
@@
 Wire Wire Line
 	5650 6250 5650 6350
+Text GLabel 13500 8350 2    50   Input ~ 0
+RPI_UART_TX
+Wire Wire Line
+	13500 8350 13300 8350
+Text GLabel 13500 8450 2    50   Input ~ 0
+RPI_UART_RX
+Wire Wire Line
+	13300 8450 13500 8450
 $EndSCHEMATC

Commit message: Add HEX spacers and fix AUX LED pinouts
Parts:
- C258, C262: footprint Capacitor_THT:CP_Radial_D6.3mm_P2.50mm -> Capacitor_SMD:CP_Elec_6.3x4.5; JLCASM DNP -> EXT; LCSC PN C225866 -> C250096; MPN UPW1A221MED1TD -> OVZ221M0JTR-0604
Changed lines of the file:
@@
 	6900 8450 6900 8350
+$Comp
+L power:GND #PWR?
+U 1 1 5EEBDC1D
+P 5650 7100
+AR Path="/5C4320DF/5EEBDC1D" Ref="#PWR?"  Part="1"
+AR Path="/5C4320DF/5DB999B7/5EEBDC1D" Ref="#PWR?"  Part="1"
+AR Path="/5C4408C6/5EEBDC1D" Ref="#PWR0109"  Part="1"
+F 0 "#PWR0109" H 5650 6850 50  0001 C CNN
+F 1 "GND" H 5655 6927 50  0000 C CNN
+F 2 "" H 5650 7100 50  0001 C CNN
+F 3 "" H 5650 7100 50  0001 C CNN
+	1    5650 7100
+	1    0    0    -1
+$EndComp
+Wire Wire Line
+	5650 7100 5650 6750
+$Comp
+L power:GND #PWR0111
+U 1 1 5EECD1C8
+P 5150 6250
+F 0 "#PWR0111" H 5150 6000 50  0001 C CNN
+F 1 "GND" V 5155 6122 50  0000 R CNN
+F 2 "" H 5150 6250 50  0001 C CNN
+F 3 "" H 5150 6250 50  0001 C CNN
+	1    5150 6250
+	0    1    1    0
+$EndComp
+Wire Wire Line
+	5150 6250 5650 6250
+Wire Wire Line
+	5650 6250 5650 6350
+Text GLabel 13500 8350 2    50   Input ~ 0
+RPI_UART_TX
+Wire Wire Line
+	13500 8350 13300 8350
+Text GLabel 13500 8450 2    50   Input ~ 0
+RPI_UART_RX
+Wire Wire Line
+	13300 8450 13500 8450
 $Comp
 L Device:C C72
@@
 F 0 "C258" V 7695 4650 50  0000 C CNN
 F 1 "220uF" V 7786 4650 50  0000 C CNN
-F 2 "Capacitor_THT:CP_Radial_D6.3mm_P2.50mm" H 7988 4500 50  0001 C CNN
-F 3 "https://datasheet.lcsc.com/szlcsc/C225866.pdf" H 7950 4650 50  0001 C CNN
+F 2 "Capacitor_SMD:CP_Elec_6.3x4.5" H 7988 4500 50  0001 C CNN
+F 3 "https://datasheet.lcsc.com/szlcsc/C250096.pdf" H 7950 4650 50  0001 C CNN
 F 4 "" H 7950 4650 50  0001 C CNN "UnitCost(USD)"
-F 5 "UPW1A221MED1TD" V 8100 4650 50  0000 C CNN "MPN"
+F 5 "OVZ221M0JTR-0604" V 8100 4650 50  0000 C CNN "MPN"
 F 6 "" H 7950 4650 50  0001 C CNN "Manufacturer"
-F 7 "DNP" H 7950 4650 50  0001 C CNN "JLCASM"
-F 8 "C225866" H 7950 4650 50  0001 C CNN "LCSC PN"
+F 7 "EXT" H 7950 4650 50  0001 C CNN "JLCASM"
+F 8 "C250096" H 7950 4650 50  0001 C CNN "LCSC PN"
 	1    7950 4650
 	0    -1   1    0
@@
 F 0 "C262" V 7695 5250 50  0000 C CNN
 F 1 "220uF" V 7786 5250 50  0000 C CNN
-F 2 "Capacitor_THT:CP_Radial_D6.3mm_P2.50mm" H 7988 5100 50  0001 C CNN
-F 3 "https://datasheet.lcsc.com/szlcsc/C225866.pdf" H 7950 5250 50  0001 C CNN
+F 2 "Capacitor_SMD:CP_Elec_6.3x4.5" H 7988 5100 50  0001 C CNN
+F 3 "https://datasheet.lcsc.com/szlcsc/C250096.pdf" H 7950 5250 50  0001 C CNN
 F 4 "" H 7950 5250 50  0001 C CNN "UnitCost(USD)"
-F 5 "UPW1A221MED1TD" V 8100 5250 50  0000 C CNN "MPN"
+F 5 "OVZ221M0JTR-0604" V 8100 5250 50  0000 C CNN "MPN"
 F 6 "" H 7950 5250 50  0001 C CNN "Manufacturer"
-F 7 "DNP" H 7950 5250 50  0001 C CNN "JLCASM"
-F 8 "C225866" H 7950 5250 50  0001 C CNN "LCSC PN"
+F 7 "EXT" H 7950 5250 50  0001 C CNN "JLCASM"
+F 8 "C250096" H 7950 5250 50  0001 C CNN "LCSC PN"
 	1    7950 5250
 	0    -1   1    0
@@
 F 8 "C123791" H 11650 4500 50  0001 C CNN "LCSC PN"
 	1    11650 4500
-	-1   0    0    -1
+	1    0    0    -1
 $EndComp
 $Comp
@@
 F 1 "AMS1117-3.3" H 6450 8501 50  0000 C CNN
 F 2 "OTTO_Footprints_Lib:SOT-223-3_TabPin2" H 6450 8550 50  0001 C CNN
-F 3 "http://www.advanced-monolithic.com/pdf/ds1117.pdf" H 6550 8100 50  0001 C CNN
+F 3 "https://datasheet.lcsc.com/szlcsc/C6186.pdf" H 6550 8100 50  0001 C CNN
 F 4 "BASIC" H 6450 8350 50  0001 C CNN "JLCASM"
 F 5 "C6186" H 6450 8350 50  0001 C CNN "LCSC PN"
@@
 	1    0    0    -1
 $EndComp
-$Comp
-L power:GND #PWR?
-U 1 1 5EEBDC1D
-P 5650 7100
-AR Path="/5C4320DF/5EEBDC1D" Ref="#PWR?"  Part="1"
-AR Path="/5C4320DF/5DB999B7/5EEBDC1D" Ref="#PWR?"  Part="1"
-AR Path="/5C4408C6/5EEBDC1D" Ref="#PWR0109"  Part="1"
-F 0 "#PWR0109" H 5650 6850 50  0001 C CNN
-F 1 "GND" H 5655 6927 50  0000 C CNN
-F 2 "" H 5650 7100 50  0001 C CNN
-F 3 "" H 5650 7100 50  0001 C CNN
-	1    5650 7100
-	1    0    0    -1
-$EndComp
-Wire Wire Line
-	5650 7100 5650 6750
-$Comp
-L power:GND #PWR0111
-U 1 1 5EECD1C8
-P 5150 6250
-F 0 "#PWR0111" H 5150 6000 50  0001 C CNN
-F 1 "GND" V 5155 6122 50  0000 R CNN
-F 2 "" H 5150 6250 50  0001 C CNN
-F 3 "" H 5150 6250 50  0001 C CNN
-	1    5150 6250
-	0    1    1    0
-$EndComp
-Wire Wire Line
-	5150 6250 5650 6250
-Wire Wire Line
-	5650 6250 5650 6350
-Text GLabel 13500 8350 2    50   Input ~ 0
-RPI_UART_TX
-Wire Wire Line
-	13500 8350 13300 8350
-Text GLabel 13500 8450 2    50   Input ~ 0
-RPI_UART_RX
-Wire Wire Line
-	13300 8450 13500 8450
 $EndSCHEMATC

Commit message: Replace inductors with larger part that is available at jlc
Parts:
- J2, J206, J207, NT1, TP15: AssemblyOption DNP -> (none)
Changed lines of the file:
@@
 F 5 "M20-7810345" H 13000 9100 12700 0001 C CNN "MPN"
 F 6 "" H 13000 9100 12700 0001 C CNN "Manufacturer"
-F 7 "DNP" H 13050 8900 50  0000 C CNN "AssemblyOption"
+F 7 "" H 13050 8900 50  0000 C CNN "AssemblyOption"
 F 8 "N/A" H 13000 9100 50  0001 C CNN "JLCASM"
 	1    13000 9100
@@
 F 5 "M20-7810645" H 13000 8250 12700 0001 C CNN "MPN"
 F 6 "" H 13000 8250 12700 0001 C CNN "Manufacturer"
-F 7 "DNP" H 13050 7850 50  0000 C CNN "AssemblyOption"
+F 7 "" H 13050 7850 50  0000 C CNN "AssemblyOption"
 F 8 "N/A" H 13000 8250 50  0001 C CNN "JLCASM"
 	1    13000 8250
@@
 F 2 "Connector_PinHeader_2.54mm:PinHeader_2x04_P2.54mm_Vertical" H 10150 8150 50  0001 C CNN
 F 3 "" H 10150 8150 50  0001 C CNN
-F 4 "DNP" H 10150 8150 50  0001 C CNN "AssemblyOption"
+F 4 "" H 10150 8150 50  0001 C CNN "AssemblyOption"
 F 5 "N/A" H 10150 8150 50  0001 C CNN "MPN"
 F 6 "" H 10150 8150 50  0001 C CNN "Manufacturer"
@@
 F 2 "OTTO_Footprints_Lib:NetTie-2_Pad5.0mm" H 6800 7000 50  0001 C CNN
 F 3 "" H 6800 7000 50  0001 C CNN
-F 4 "DNP" H 6800 7000 50  0001 C CNN "AssemblyOption"
+F 4 "" H 6800 7000 50  0001 C CNN "AssemblyOption"
 F 5 "N/A" H 6800 7000 50  0001 C CNN "MPN"
 F 6 "" H 6800 7000 50  0001 C CNN "Manufacturer"
@@
 F 2 "TestPoint:TestPoint_THTPad_D1.0mm_Drill0.5mm" H 8650 5900 50  0001 C CNN
 F 3 "" H 8650 5900 50  0001 C CNN
-F 4 "DNP" H 8450 5900 50  0001 C CNN "AssemblyOption"
+F 4 "" H 8450 5900 50  0001 C CNN "AssemblyOption"
 F 5 "N/A" H 8450 5900 50  0001 C CNN "MPN"
 F 6 "" H 8450 5900 50  0001 C CNN "Manufacturer"

Commit message: Main board v0.1.0 as ordered
Parts:
- C258, C262: footprint Capacitor_SMD:CP_Elec_6.3x4.5 -> OTTO_Footprints_Lib:CP_Elec_6.3x4.5
- C267, C268: footprint Capacitor_Tantalum_SMD:CP_EIA-3216-18_Kemet-A_Pad1.58x1.35mm_HandSolder -> OTTO_Footprints_Lib:CP_EIA-3216-18_Kemet-A_Pad1.58x1.35mm_HandSolder
Changed lines of the file:
@@
-$Comp
-L Device:CP C?
-U 1 1 5DF0ABC4
-P 7950 4650
-AR Path="/5C4320DF/5DB999B7/5DF0ABC4" Ref="C?"  Part="1"
-AR Path="/5C4320DF/5DF0ABC4" Ref="C?"  Part="1"
-AR Path="/5C4408C6/5DF0ABC4" Ref="C258"  Part="1"
-F 0 "C258" V 7695 4650 50  0000 C CNN
-F 1 "220uF" V 7786 4650 50  0000 C CNN
-F 2 "Capacitor_SMD:CP_Elec_6.3x4.5" H 7988 4500 50  0001 C CNN
-F 3 "https://datasheet.lcsc.com/szlcsc/C250096.pdf" H 7950 4650 50  0001 C CNN
-F 4 "" H 7950 4650 50  0001 C CNN "UnitCost(USD)"
-F 5 "OVZ221M0JTR-0604" V 8100 4650 50  0000 C CNN "MPN"
-F 6 "" H 7950 4650 50  0001 C CNN "Manufacturer"
-F 7 "EXT" H 7950 4650 50  0001 C CNN "JLCASM"
-F 8 "C250096" H 7950 4650 50  0001 C CNN "LCSC PN"
-	1    7950 4650
-	0    -1   1    0
-$EndComp
 $Comp
 L Device:CP C?
@@
 F 0 "C262" V 7695 5250 50  0000 C CNN
 F 1 "220uF" V 7786 5250 50  0000 C CNN
-F 2 "Capacitor_SMD:CP_Elec_6.3x4.5" H 7988 5100 50  0001 C CNN
+F 2 "OTTO_Footprints_Lib:CP_Elec_6.3x4.5" H 7988 5100 50  0001 C CNN
 F 3 "https://datasheet.lcsc.com/szlcsc/C250096.pdf" H 7950 5250 50  0001 C CNN
 F 4 "" H 7950 5250 50  0001 C CNN "UnitCost(USD)"
@@
 F 0 "C268" H 6785 8554 50  0000 R CNN
 F 1 "10uf Tantalum" H 6785 8645 50  0000 R CNN
-F 2 "Capacitor_Tantalum_SMD:CP_EIA-3216-18_Kemet-A_Pad1.58x1.35mm_HandSolder" H 6938 8450 50  0001 C CNN
+F 2 "OTTO_Footprints_Lib:CP_EIA-3216-18_Kemet-A_Pad1.58x1.35mm_HandSolder" H 6938 8450 50  0001 C CNN
 F 3 "https://datasheet.lcsc.com/szlcsc/C7171.pdf" H 6900 8600 50  0001 C CNN
 F 4 "" H 6900 8600 50  0001 C CNN "UnitCost(USD)"
@@
 F 0 "C267" H 5735 8554 50  0000 R CNN
 F 1 "10uf Tantalum" H 5735 8645 50  0000 R CNN
-F 2 "Capacitor_Tantalum_SMD:CP_EIA-3216-18_Kemet-A_Pad1.58x1.35mm_HandSolder" H 5888 8450 50  0001 C CNN
+F 2 "OTTO_Footprints_Lib:CP_EIA-3216-18_Kemet-A_Pad1.58x1.35mm_HandSolder" H 5888 8450 50  0001 C CNN
 F 3 "https://datasheet.lcsc.com/szlcsc/C7171.pdf" H 5850 8600 50  0001 C CNN
 F 4 "" H 5850 8600 50  0001 C CNN "UnitCost(USD)"
@@
 	1    0    0    -1
 $EndComp
+$Comp
+L Device:CP C?
+U 1 1 5DF0ABC4
+P 7950 4650
+AR Path="/5C4320DF/5DB999B7/5DF0ABC4" Ref="C?"  Part="1"
+AR Path="/5C4320DF/5DF0ABC4" Ref="C?"  Part="1"
+AR Path="/5C4408C6/5DF0ABC4" Ref="C258"  Part="1"
+F 0 "C258" V 7695 4650 50  0000 C CNN
+F 1 "220uF" V 7786 4650 50  0000 C CNN
+F 2 "OTTO_Footprints_Lib:CP_Elec_6.3x4.5" H 7988 4500 50  0001 C CNN
+F 3 "https://datasheet.lcsc.com/szlcsc/C250096.pdf" H 7950 4650 50  0001 C CNN
+F 4 "" H 7950 4650 50  0001 C CNN "UnitCost(USD)"
+F 5 "OVZ221M0JTR-0604" V 8100 4650 50  0000 C CNN "MPN"
+F 6 "" H 7950 4650 50  0001 C CNN "Manufacturer"
+F 7 "EXT" H 7950 4650 50  0001 C CNN "JLCASM"
+F 8 "C250096" H 7950 4650 50  0001 C CNN "LCSC PN"
+	1    7950 4650
+	0    -1   1    0
+$EndComp
 $EndSCHEMATC

Commit message: Hardware v0.2.0 as ordered
Parts:
- U207: LCSC PN C323837 -> C41511
Changed lines of the file:
@@
 F 6 "" H 6800 2750 12700 0001 C CNN "Manufacturer"
 F 7 "EXT" H 6800 2750 50  0001 C CNN "JLCASM"
-F 8 "C323837" H 6800 2750 50  0001 C CNN "LCSC PN"
+F 8 "C41511" H 6800 2750 50  0001 C CNN "LCSC PN"
 	1    6800 2750
 	1    0    0    -1
