File: KiCad/OTTOdiy_SMD.sch (KiCad schematic (older format))
At the start: 19 parts, among them J201 RASPBERRY PI 3 A+

Commit message: roll in changes from Bastian
Parts:
- R?: value 10k -> 2.2k
Changed lines of the file:
@@
 Wire Wire Line
 	3550 3050 3450 3050
-$Comp
-L Mechanical:MountingHole_Pad H212
-U 1 1 5CA1B5B7
-P 800 6700
-F 0 "H212" H 900 6751 50  0000 L CNN
-F 1 "MountingHole_Pad" H 900 6660 50  0000 L CNN
-F 2 "MountingHole:MountingHole_2.7mm_Pad_Via" H 800 6700 50  0001 C CNN
-F 3 "~" H 800 6700 50  0001 C CNN
-	1    800  6700
-	1    0    0    -1
-$EndComp
 Wire Wire Line
 	5150 2850 5250 2850
@@
 F1 "AUDIO.sch" 50
 $EndSheet
-$Comp
-L power:GND #PWR0206
-U 1 1 5C6C4424
-P 800 6850
-F 0 "#PWR0206" H 800 6600 50  0001 C CNN
-F 1 "GND" H 805 6677 50  0000 C CNN
-F 2 "" H 800 6850 50  0001 C CNN
-F 3 "" H 800 6850 50  0001 C CNN
-	1    800  6850
-	1    0    0    -1
-$EndComp
 $Comp
 L Mechanical:MountingHole H201
@@
 $EndComp
 $Comp
-L power:GND #PWR0203
-U 1 1 5DFC7588
-P 1850 6850
-F 0 "#PWR0203" H 1850 6600 50  0001 C CNN
-F 1 "GND" H 1855 6677 50  0000 C CNN
-F 2 "" H 1850 6850 50  0001 C CNN
-F 3 "" H 1850 6850 50  0001 C CNN
-	1    1850 6850
-	1    0    0    -1
-$EndComp
-$Comp
 L Mechanical:MountingHole_Pad H215
 U 1 1 5DFC860B
@@
 $EndComp
 $Comp
-L power:GND #PWR0205
-U 1 1 5DFC8611
-P 1850 7450
-F 0 "#PWR0205" H 1850 7200 50  0001 C CNN
-F 1 "GND" H 1855 7277 50  0000 C CNN
-F 2 "" H 1850 7450 50  0001 C CNN
-F 3 "" H 1850 7450 50  0001 C CNN
-	1    1850 7450
-	1    0    0    -1
-$EndComp
-$Comp
 L Mechanical:MountingHole H207
 U 1 1 5DDBF7EF
@@
 F 3 "~" H 2850 6050 50  0001 C CNN
 	1    2850 6050
-	1    0    0    -1
-$EndComp
-$Comp
-L Mechanical:MountingHole_Pad H214
-U 1 1 5E868395
-P 2850 6700
-F 0 "H214" H 2950 6751 50  0000 L CNN
-F 1 "MountingHole_Pad" H 2950 6660 50  0000 L CNN
-F 2 "MountingHole:MountingHole_2.7mm_Pad_Via" H 2850 6700 50  0001 C CNN
-F 3 "~" H 2850 6700 50  0001 C CNN
-	1    2850 6700
-	1    0    0    -1
-$EndComp
-$Comp
-L power:GND #PWR0204
-U 1 1 5E86839B
-P 2850 6850
-F 0 "#PWR0204" H 2850 6600 50  0001 C CNN
-F 1 "GND" H 2855 6677 50  0000 C CNN
-F 2 "" H 2850 6850 50  0001 C CNN
-F 3 "" H 2850 6850 50  0001 C CNN
-	1    2850 6850
 	1    0    0    -1
 $EndComp
@@
 NoConn ~ 5150 3750
 NoConn ~ 5150 3850
-Wire Wire Line
-	800  6800 800  6850
-Wire Wire Line
-	1850 6800 1850 6850
-Wire Wire Line
-	2850 6800 2850 6850
-Wire Wire Line
-	1850 7400 1850 7450
 $Comp
 L Device:R R?
@@
 P 5750 2750
 F 0 "R?" V 5543 2750 50  0000 C CNN
-F 1 "10k" V 5634 2750 50  0000 C CNN
+F 1 "2.2k" V 5634 2750 50  0000 C CNN
 F 2 "" V 5680 2750 50  0001 C CNN
 F 3 "~" H 5750 2750 50  0001 C CNN
@@
 Wire Wire Line
 	5900 2750 6100 2750
+Wire Wire Line
+	1850 6800 1850 6850
+$Comp
+L power:GND #PWR0203
+U 1 1 5DFC7588
+P 1850 6850
+F 0 "#PWR0203" H 1850 6600 50  0001 C CNN
+F 1 "GND" H 1855 6677 50  0000 C CNN
+F 2 "" H 1850 6850 50  0001 C CNN
+F 3 "" H 1850 6850 50  0001 C CNN
+	1    1850 6850
+	1    0    0    -1
+$EndComp
+Wire Wire Line
+	1850 7400 1850 7450
+$Comp
+L power:GND #PWR0205
+U 1 1 5DFC8611
+P 1850 7450
+F 0 "#PWR0205" H 1850 7200 50  0001 C CNN
+F 1 "GND" H 1855 7277 50  0000 C CNN
+F 2 "" H 1850 7450 50  0001 C CNN
+F 3 "" H 1850 7450 50  0001 C CNN
+	1    1850 7450
+	1    0    0    -1
+$EndComp
+$Comp
+L power:GND #PWR0206
+U 1 1 5C6C4424
+P 800 6850
+F 0 "#PWR0206" H 800 6600 50  0001 C CNN
+F 1 "GND" H 805 6677 50  0000 C CNN
+F 2 "" H 800 6850 50  0001 C CNN
+F 3 "" H 800 6850 50  0001 C CNN
+	1    800  6850
+	1    0    0    -1
+$EndComp
+Wire Wire Line
+	800  6800 800  6850
+Wire Wire Line
+	2850 6800 2850 6850
+$Comp
+L power:GND #PWR0204
+U 1 1 5E86839B
+P 2850 6850
+F 0 "#PWR0204" H 2850 6600 50  0001 C CNN
+F 1 "GND" H 2855 6677 50  0000 C CNN
+F 2 "" H 2850 6850 50  0001 C CNN
+F 3 "" H 2850 6850 50  0001 C CNN
+	1    2850 6850
+	1    0    0    -1
+$EndComp
+$Comp
+L Mechanical:MountingHole_Pad H214
+U 1 1 5E868395
+P 2850 6700
+F 0 "H214" H 2950 6751 50  0000 L CNN
+F 1 "MountingHole_Pad" H 2950 6660 50  0000 L CNN
+F 2 "MountingHole:MountingHole_2.7mm_Pad_Via" H 2850 6700 50  0001 C CNN
+F 3 "~" H 2850 6700 50  0001 C CNN
+	1    2850 6700
+	1    0    0    -1
+$EndComp
+$Comp
+L Mechanical:MountingHole_Pad H212
+U 1 1 5CA1B5B7
+P 800 6700
+F 0 "H212" H 900 6751 50  0000 L CNN
+F 1 "MountingHole_Pad" H 900 6660 50  0000 L CNN
+F 2 "MountingHole:MountingHole_2.7mm_Pad_Via" H 800 6700 50  0001 C CNN
+F 3 "~" H 800 6700 50  0001 C CNN
+	1    800  6700
+	1    0    0    -1
+$EndComp
 $EndSCHEMATC

Commit message: added power switching and extra pulls for programming lines
Parts:
- added R? (x2): 1k, symbol Device:R
- R?: value 2.2k -> 1k
Connections:
- net labels added: +5V_PI
- net labels removed: +5V_MAIN
- wire segments 51 -> 53
Changed lines of the file:
@@
-EESchema Schematic File Version 4
+EESchema Schematic File Version 5
 EELAYER 30 0
 EELAYER END
-$Descr A4 11693 8268
+$Descr A3 16535 11693
 encoding utf-8
 Sheet 1 7
@@
 Comment3 ""
 Comment4 ""
+Comment5 ""
+Comment6 ""
+Comment7 ""
+Comment8 ""
+Comment9 ""
 $EndDescr
 $Sheet
@@
 +3V3_RASPI
 Text GLabel 3450 1650 0    50   Input ~ 0
-+5V_MAIN
++5V_PI
 Wire Wire Line
 	3650 1250 3650 1150
@@
 	1    0    0    -1
 $EndComp
-Wire Wire Line
-	3450 3450 3550 3450
-Wire Wire Line
-	3450 3550 3550 3550
 $Sheet
 S 700  750  650  600
@@
 Text GLabel 6100 2750 2    50   Output ~ 0
 ICP_RST
-Text GLabel 3450 3450 0    50   Output ~ 0
+Text GLabel 2650 3450 0    50   Output ~ 0
 ICP_SWDIO
-Text GLabel 3450 3550 0    50   Output ~ 0
+Text GLabel 2650 3550 0    50   Output ~ 0
 ICP_SWCLK
 Text GLabel 3450 3250 0    50   BiDi ~ 0
@@
 P 5750 2750
 F 0 "R?" V 5543 2750 50  0000 C CNN
-F 1 "2.2k" V 5634 2750 50  0000 C CNN
+F 1 "1k" V 5634 2750 50  0000 C CNN
 F 2 "" V 5680 2750 50  0001 C CNN
 F 3 "~" H 5750 2750 50  0001 C CNN
@@
 	1    0    0    -1
 $EndComp
+$Comp
+L Device:R R?
+U 1 1 5E17B63D
+P 3100 3550
+F 0 "R?" V 3150 3750 50  0000 C CNN
+F 1 "1k" V 3150 3350 50  0000 C CNN
+F 2 "" V 3030 3550 50  0001 C CNN
+F 3 "~" H 3100 3550 50  0001 C CNN
+	1    3100 3550
+	0    -1   -1   0
+$EndComp
+$Comp
+L Device:R R?
+U 1 1 5E17D8BA
+P 3100 3450
+F 0 "R?" V 3150 3650 50  0000 C CNN
+F 1 "1k" V 3150 3250 50  0000 C CNN
+F 2 "" V 3030 3450 50  0001 C CNN
+F 3 "~" H 3100 3450 50  0001 C CNN
+	1    3100 3450
+	0    -1   -1   0
+$EndComp
+Wire Wire Line
+	3250 3450 3550 3450
+Wire Wire Line
+	3250 3550 3550 3550
+Wire Wire Line
+	2650 3450 2950 3450
+Wire Wire Line
+	2650 3550 2950 3550
 $EndSCHEMATC

Commit message: connected unconnected signals and MIDI to spare MCU UART
Parts:
- gave numbers to parts that had none: 3

Commit message: add all resistor part numbers and create footprint library
Parts:
- removed C201: 10µF, Capacitor_SMD:C_0805_2012Metric_Pad1.15x1.40mm_HandSolder, symbol Device:C
- removed DUMMY201: RASPBERRY PI 3 A+, Spatz:Raspberry Pi A, symbol Connector:Raspberry_Pi_2_3
- H201, H202, H203, H204, H205, H206, H207, H208, H209, H210, H211, H212, H213, H214, H215: AssemblyOption (none) -> DNP; EstimatedCost(USD) (none) -> $0.00
- J201: footprint Connector_Harwin:Harwin_M20-7812045_2x20_P2.54mm_Vertical_SolderHoles -> OTTOdiy_SMD-library:Raspberry_Pi_A_FacingDown_TH; EstimatedCost(USD) (none) -> $3.97; MPN (none) -> M20-7812045; Manufacturer (none) -> Harwin
- R1, R2, R3: footprint (none) -> Resistor_SMD:R_0805_2012Metric_Pad1.15x1.40mm_HandSolder; EstimatedCost(USD) (none) -> $.001763; MPN (none) -> RC0805FR-071KL; Manufacturer (none) -> Yageo
Connections:
- net labels added: PI_PWR_EN
- wire segments 53 -> 51
- no-connect marks 48 -> 7
Other:
- note removed: "Dummy for component alignment"

Commit message: add more part numbers, samtec connector footprint
Parts:
- H201, H202, H203, H204, H205, H206, H207, H208, H209, H210, H211: footprint Spatz:Mounting_Hole_M2.5_Loose_Fit -> OTTO_Footprints_Lib:Mounting_Hole_M2.5_Loose_Fit; MPN (none) -> N/A; Manufacturer (none) -> N/A
- H212, H213, H214, H215: MPN (none) -> N/A; Manufacturer (none) -> N/A
Changed lines of the file:
@@
 F 0 "H201" H 2900 6496 50  0000 L CNN
 F 1 "MountingHole" H 2900 6405 50  0000 L CNN
-F 2 "Spatz:Mounting_Hole_M2.5_Loose_Fit" H 2800 6450 50  0001 C CNN
-F 3 "" H 2800 6450 50  0001 C CNN
+F 2 "OTTO_Footprints_Lib:Mounting_Hole_M2.5_Loose_Fit" H 2800 6450 50  0001 C CNN
+F 3 "N/A" H 2800 6450 50  0001 C CNN
 F 4 "$0.00" H 2800 6450 50  0001 C CNN "EstimatedCost(USD)"
 F 5 "DNP" H 2800 6450 50  0001 C CNN "AssemblyOption"
+F 6 "N/A" H 2800 6450 50  0001 C CNN "MPN"
+F 7 "N/A" H 2800 6450 50  0001 C CNN "Manufacturer"
 	1    2800 6450
 	1    0    0    -1
@@
 F 0 "H204" H 2900 6796 50  0000 L CNN
 F 1 "MountingHole" H 2900 6705 50  0000 L CNN
-F 2 "Spatz:Mounting_Hole_M2.5_Loose_Fit" H 2800 6750 50  0001 C CNN
-F 3 "" H 2800 6750 50  0001 C CNN
+F 2 "OTTO_Footprints_Lib:Mounting_Hole_M2.5_Loose_Fit" H 2800 6750 50  0001 C CNN
+F 3 "N/A" H 2800 6750 50  0001 C CNN
 F 4 "DNP" H 2800 6750 50  0001 C CNN "AssemblyOption"
 F 5 "$0.00" H 2800 6750 50  0001 C CNN "EstimatedCost(USD)"
+F 6 "N/A" H 2800 6750 50  0001 C CNN "MPN"
+F 7 "N/A" H 2800 6750 50  0001 C CNN "Manufacturer"
 	1    2800 6750
 	1    0    0    -1
@@
 F 0 "H202" H 3950 6496 50  0000 L CNN
 F 1 "MountingHole" H 3950 6405 50  0000 L CNN
-F 2 "Spatz:Mounting_Hole_M2.5_Loose_Fit" H 3850 6450 50  0001 C CNN
-F 3 "" H 3850 6450 50  0001 C CNN
+F 2 "OTTO_Footprints_Lib:Mounting_Hole_M2.5_Loose_Fit" H 3850 6450 50  0001 C CNN
+F 3 "N/A" H 3850 6450 50  0001 C CNN
 F 4 "DNP" H 3850 6450 50  0001 C CNN "AssemblyOption"
 F 5 "$0.00" H 3850 6450 50  0001 C CNN "EstimatedCost(USD)"
+F 6 "N/A" H 3850 6450 50  0001 C CNN "MPN"
+F 7 "N/A" H 3850 6450 50  0001 C CNN "Manufacturer"
 	1    3850 6450
 	1    0    0    -1
@@
 F 0 "H205" H 3950 6796 50  0000 L CNN
 F 1 "MountingHole" H 3950 6705 50  0000 L CNN
-F 2 "Spatz:Mounting_Hole_M2.5_Loose_Fit" H 3850 6750 50  0001 C CNN
-F 3 "" H 3850 6750 50  0001 C CNN
+F 2 "OTTO_Footprints_Lib:Mounting_Hole_M2.5_Loose_Fit" H 3850 6750 50  0001 C CNN
+F 3 "N/A" H 3850 6750 50  0001 C CNN
 F 4 "DNP" H 3850 6750 50  0001 C CNN "AssemblyOption"
 F 5 "$0.00" H 3850 6750 50  0001 C CNN "EstimatedCost(USD)"
+F 6 "N/A" H 3850 6750 50  0001 C CNN "MPN"
+F 7 "N/A" H 3850 6750 50  0001 C CNN "Manufacturer"
 	1    3850 6750
 	1    0    0    -1
@@
 F 1 "MountingHole_Pad" H 3950 7660 50  0000 L CNN
 F 2 "MountingHole:MountingHole_2.7mm_Pad_Via" H 3850 7700 50  0001 C CNN
-F 3 "" H 3850 7700 50  0001 C CNN
+F 3 "N/A" H 3850 7700 50  0001 C CNN
 F 4 "DNP" H 3850 7700 50  0001 C CNN "AssemblyOption"
 F 5 "$0.00" H 3850 7700 50  0001 C CNN "EstimatedCost(USD)"
+F 6 "N/A" H 3850 7700 50  0001 C CNN "MPN"
+F 7 "N/A" H 3850 7700 50  0001 C CNN "Manufacturer"
 	1    3850 7700
 	1    0    0    -1
@@
 F 1 "MountingHole_Pad" H 3950 8260 50  0000 L CNN
 F 2 "MountingHole:MountingHole_2.7mm_Pad_Via" H 3850 8300 50  0001 C CNN
-F 3 "" H 3850 8300 50  0001 C CNN
+F 3 "N/A" H 3850 8300 50  0001 C CNN
 F 4 "DNP" H 3850 8300 50  0001 C CNN "AssemblyOption"
 F 5 "$0.00" H 3850 8300 50  0001 C CNN "EstimatedCost(USD)"
+F 6 "N/A" H 3850 8300 50  0001 C CNN "MPN"
+F 7 "N/A" H 3850 8300 50  0001 C CNN "Manufacturer"
 	1    3850 8300
 	1    0    0    -1
@@
 F 0 "H207" H 2900 7096 50  0000 L CNN
 F 1 "MountingHole" H 2900 7005 50  0000 L CNN
-F 2 "Spatz:Mounting_Hole_M2.5_Loose_Fit" H 2800 7050 50  0001 C CNN
-F 3 "" H 2800 7050 50  0001 C CNN
+F 2 "OTTO_Footprints_Lib:Mounting_Hole_M2.5_Loose_Fit" H 2800 7050 50  0001 C CNN
+F 3 "N/A" H 2800 7050 50  0001 C CNN
 F 4 "DNP" H 2800 7050 50  0001 C CNN "AssemblyOption"
 F 5 "$0.00" H 2800 7050 50  0001 C CNN "EstimatedCost(USD)"
+F 6 "N/A" H 2800 7050 50  0001 C CNN "MPN"
+F 7 "N/A" H 2800 7050 50  0001 C CNN "Manufacturer"
 	1    2800 7050
 	1    0    0    -1
@@
 F 0 "H210" H 2900 7396 50  0000 L CNN
 F 1 "MountingHole" H 2900 7305 50  0000 L CNN
-F 2 "Spatz:Mounting_Hole_M2.5_Loose_Fit" H 2800 7350 50  0001 C CNN
-F 3 "" H 2800 7350 50  0001 C CNN
+F 2 "OTTO_Footprints_Lib:Mounting_Hole_M2.5_Loose_Fit" H 2800 7350 50  0001 C CNN
+F 3 "N/A" H 2800 7350 50  0001 C CNN
 F 4 "DNP" H 2800 7350 50  0001 C CNN "AssemblyOption"
 F 5 "$0.00" H 2800 7350 50  0001 C CNN "EstimatedCost(USD)"
+F 6 "N/A" H 2800 7350 50  0001 C CNN "MPN"
+F 7 "N/A" H 2800 7350 50  0001 C CNN "Manufacturer"
 	1    2800 7350
 	1    0    0    -1
@@
 F 0 "H208" H 3950 7096 50  0000 L CNN
 F 1 "MountingHole" H 3950 7005 50  0000 L CNN
-F 2 "Spatz:Mounting_Hole_M2.5_Loose_Fit" H 3850 7050 50  0001 C CNN
-F 3 "" H 3850 7050 50  0001 C CNN
+F 2 "OTTO_Footprints_Lib:Mounting_Hole_M2.5_Loose_Fit" H 3850 7050 50  0001 C CNN
+F 3 "N/A" H 3850 7050 50  0001 C CNN
 F 4 "DNP" H 3850 7050 50  0001 C CNN "AssemblyOption"
 F 5 "$0.00" H 3850 7050 50  0001 C CNN "EstimatedCost(USD)"
+F 6 "N/A" H 3850 7050 50  0001 C CNN "MPN"
+F 7 "N/A" H 3850 7050 50  0001 C CNN "Manufacturer"
 	1    3850 7050
 	1    0    0    -1
@@
 F 0 "H203" H 4950 6496 50  0000 L CNN
 F 1 "MountingHole" H 4950 6405 50  0000 L CNN
-F 2 "Spatz:Mounting_Hole_M2.5_Loose_Fit" H 4850 6450 50  0001 C CNN
-F 3 "" H 4850 6450 50  0001 C CNN
+F 2 "OTTO_Footprints_Lib:Mounting_Hole_M2.5_Loose_Fit" H 4850 6450 50  0001 C CNN
+F 3 "N/A" H 4850 6450 50  0001 C CNN
 F 4 "DNP" H 4850 6450 50  0001 C CNN "AssemblyOption"
 F 5 "$0.00" H 4850 6450 50  0001 C CNN "EstimatedCost(USD)"
+F 6 "N/A" H 4850 6450 50  0001 C CNN "MPN"
+F 7 "N/A" H 4850 6450 50  0001 C CNN "Manufacturer"
 	1    4850 6450
 	1    0    0    -1
@@
 F 0 "H206" H 4950 6796 50  0000 L CNN
 F 1 "MountingHole" H 4950 6705 50  0000 L CNN
-F 2 "Spatz:Mounting_Hole_M2.5_Loose_Fit" H 4850 6750 50  0001 C CNN
-F 3 "" H 4850 6750 50  0001 C CNN
+F 2 "OTTO_Footprints_Lib:Mounting_Hole_M2.5_Loose_Fit" H 4850 6750 50  0001 C CNN
+F 3 "N/A" H 4850 6750 50  0001 C CNN
 F 4 "DNP" H 4850 6750 50  0001 C CNN "AssemblyOption"
 F 5 "$0.00" H 4850 6750 50  0001 C CNN "EstimatedCost(USD)"
+F 6 "N/A" H 4850 6750 50  0001 C CNN "MPN"
+F 7 "N/A" H 4850 6750 50  0001 C CNN "Manufacturer"
 	1    4850 6750
 	1    0    0    -1
@@
 F 0 "H209" H 4950 7096 50  0000 L CNN
 F 1 "MountingHole" H 4950 7005 50  0000 L CNN
-F 2 "Spatz:Mounting_Hole_M2.5_Loose_Fit" H 4850 7050 50  0001 C CNN
-F 3 "" H 4850 7050 50  0001 C CNN
+F 2 "OTTO_Footprints_Lib:Mounting_Hole_M2.5_Loose_Fit" H 4850 7050 50  0001 C CNN
+F 3 "N/A" H 4850 7050 50  0001 C CNN
 F 4 "DNP" H 4850 7050 50  0001 C CNN "AssemblyOption"
 F 5 "$0.00" H 4850 7050 50  0001 C CNN "EstimatedCost(USD)"
+F 6 "N/A" H 4850 7050 50  0001 C CNN "MPN"
+F 7 "N/A" H 4850 7050 50  0001 C CNN "Manufacturer"
 	1    4850 7050
 	1    0    0    -1
@@
 F 1 "MountingHole_Pad" H 4950 7660 50  0000 L CNN
 F 2 "MountingHole:MountingHole_2.7mm_Pad_Via" H 4850 7700 50  0001 C CNN
-F 3 "" H 4850 7700 50  0001 C CNN
+F 3 "N/A" H 4850 7700 50  0001 C CNN
 F 4 "DNP" H 4850 7700 50  0001 C CNN "AssemblyOption"
 F 5 "$0.00" H 4850 7700 50  0001 C CNN "EstimatedCost(USD)"
+F 6 "N/A" H 4850 7700 50  0001 C CNN "MPN"
+F 7 "N/A" H 4850 7700 50  0001 C CNN "Manufacturer"
 	1    4850 7700
 	1    0    0    -1
@@
 F 1 "MountingHole_Pad" H 2900 7660 50  0000 L CNN
 F 2 "MountingHole:MountingHole_2.7mm_Pad_Via" H 2800 7700 50  0001 C CNN
-F 3 "" H 2800 7700 50  0001 C CNN
+F 3 "N/A" H 2800 7700 50  0001 C CNN
 F 4 "DNP" H 2800 7700 50  0001 C CNN "AssemblyOption"
 F 5 "$0.00" H 2800 7700 50  0001 C CNN "EstimatedCost(USD)"
+F 6 "N/A" H 2800 7700 50  0001 C CNN "MPN"
+F 7 "N/A" H 2800 7700 50  0001 C CNN "Manufacturer"
 	1    2800 7700
 	1    0    0    -1
@@
 F 0 "H211" H 3950 7396 50  0000 L CNN
 F 1 "MountingHole" H 3950 7305 50  0000 L CNN
-F 2 "Spatz:Mounting_Hole_M2.5_Loose_Fit" H 3850 7350 50  0001 C CNN
-F 3 "" H 3850 7350 50  0001 C CNN
+F 2 "OTTO_Footprints_Lib:Mounting_Hole_M2.5_Loose_Fit" H 3850 7350 50  0001 C CNN
+F 3 "N/A" H 3850 7350 50  0001 C CNN
 F 4 "DNP" H 3850 7350 50  0001 C CNN "AssemblyOption"
 F 5 "$0.00" H 3850 7350 50  0001 C CNN "EstimatedCost(USD)"
+F 6 "N/A" H 3850 7350 50  0001 C CNN "MPN"
+F 7 "N/A" H 3850 7350 50  0001 C CNN "Manufacturer"
 	1    3850 7350
 	1    0    0    -1

Commit message: add switch and encoder parts. BM Complete. Footprints complete.
Parts:
- J201: footprint OTTOdiy_SMD-library:Raspberry_Pi_A_FacingDown_TH -> OTTO_Footprints_Lib:Raspberry_Pi_A_FacingDown_TH
Changed lines of the file:
@@
 F 0 "J201" H 6350 5650 50  0000 C CNN
 F 1 "RASPBERRY PI 3 A+" H 6350 5550 50  0000 C CNN
-F 2 "OTTOdiy_SMD-library:Raspberry_Pi_A_FacingDown_TH" H 6350 4050 50  0001 C CNN
+F 2 "OTTO_Footprints_Lib:Raspberry_Pi_A_FacingDown_TH" H 6350 4050 50  0001 C CNN
 F 3 "https://www.raspberrypi.org/app/uploads/2018/11/Raspberry_Pi_3A_product_brief.pdf" H 6350 4050 50  0001 C CNN
 F 4 "M20-7812045" H 6350 4050 50  0001 C CNN "MPN"

Commit message: add BOM scripts, fix schematic hierarchy
Parts:
- added TP2, TP3, TP4, TP5, TP6, TP7, TP8, TP9: TestPoint, TestPoint:TestPoint_Keystone_5000-5004_Miniature, symbol Connector:TestPoint
- H201, H202, H203, H204, H205, H206, H207, H208, H209, H210, H211, H212, H213, H214, H215: EstimatedCost(USD) $0.00 -> (none); UnitCost(USD) (none) -> $0.00
- J201: value RASPBERRY PI 3 A+ -> Raspberry Pi Connector; EstimatedCost(USD) $3.97 -> (none); UnitCost(USD) (none) -> $3.97
- R1, R2, R3: EstimatedCost(USD) $.001763 -> (none); UnitCost(USD) (none) -> $.001763
Connections:
- net labels added: BL_PWM, RPI_PWM1_GPIO13
- net labels removed: PWR_BUTTON
- wire segments 51 -> 73
- no-connect marks 7 -> 1
Other:
- note added: "GPIO0-8 are pulled up during boot time.\nGPIO9-27 are pulled down during boot time."
- note added: "Internal pullups/pulldowns:\nICP_RST: u\nSPI_CS_RASPI_DISPLAY: u"
- note removed: "Internal pullups/pulldowns:\nICP_RST: u\nSPI_CS_RASPI_DISPLAY: u\n***Todo: check states of the other connections \nto MCU to prevent different pull states \nduring boot time***"
- note removed: "PWR_BUTTON must be pulled up during the \nboot time of the Raspberry Pi, so it must \nbe connected to GPIO0-8.\nGPIO9-27 are pulled down during boot time."
