File: KiCad/OTTOdiy_SMD.sch (KiCad schematic (older format))
At the start: 35 parts, among them J201 Raspberry Pi Connector

Commit message: Extend board by 1mm to align ports
Parts:
- removed H207, H208, H210, H211: MountingHole, OTTO_Footprints_Lib:Mounting_Hole_M2.5_Loose_Fit, symbol Mechanical:MountingHole
Changed lines of the file:
@@
-$EndComp
-$Comp
-L Mechanical:MountingHole H207
-U 1 1 5DDBF7EF
-P 950 9400
-F 0 "H207" H 1050 9446 50  0000 L CNN
-F 1 "MountingHole" H 1050 9355 50  0000 L CNN
-F 2 "OTTO_Footprints_Lib:Mounting_Hole_M2.5_Loose_Fit" H 950 9400 50  0001 C CNN
-F 3 "N/A" H 950 9400 50  0001 C CNN
-F 4 "DNP" H 950 9400 50  0001 C CNN "AssemblyOption"
-F 5 "$0.00" H 950 9400 50  0001 C CNN "UnitCost(USD)"
-F 6 "N/A" H 950 9400 50  0001 C CNN "MPN"
-F 7 "N/A" H 950 9400 50  0001 C CNN "Manufacturer"
-	1    950  9400
-	1    0    0    -1
-$EndComp
-$Comp
-L Mechanical:MountingHole H210
-U 1 1 5DDBF7F5
-P 950 9700
-F 0 "H210" H 1050 9746 50  0000 L CNN
-F 1 "MountingHole" H 1050 9655 50  0000 L CNN
-F 2 "OTTO_Footprints_Lib:Mounting_Hole_M2.5_Loose_Fit" H 950 9700 50  0001 C CNN
-F 3 "N/A" H 950 9700 50  0001 C CNN
-F 4 "DNP" H 950 9700 50  0001 C CNN "AssemblyOption"
-F 5 "$0.00" H 950 9700 50  0001 C CNN "UnitCost(USD)"
-F 6 "N/A" H 950 9700 50  0001 C CNN "MPN"
-F 7 "N/A" H 950 9700 50  0001 C CNN "Manufacturer"
-	1    950  9700
-	1    0    0    -1
-$EndComp
-$Comp
-L Mechanical:MountingHole H208
-U 1 1 5DDBF7FB
-P 2000 9400
-F 0 "H208" H 2100 9446 50  0000 L CNN
-F 1 "MountingHole" H 2100 9355 50  0000 L CNN
-F 2 "OTTO_Footprints_Lib:Mounting_Hole_M2.5_Loose_Fit" H 2000 9400 50  0001 C CNN
-F 3 "N/A" H 2000 9400 50  0001 C CNN
-F 4 "DNP" H 2000 9400 50  0001 C CNN "AssemblyOption"
-F 5 "$0.00" H 2000 9400 50  0001 C CNN "UnitCost(USD)"
-F 6 "N/A" H 2000 9400 50  0001 C CNN "MPN"
-F 7 "N/A" H 2000 9400 50  0001 C CNN "Manufacturer"
-	1    2000 9400
-	1    0    0    -1
 $EndComp
 $Comp
@@
 Wire Wire Line
 	6200 4150 6850 4150
-$Comp
-L Mechanical:MountingHole H211
-U 1 1 5DDBF801
-P 2000 9700
-F 0 "H211" H 2100 9746 50  0000 L CNN
-F 1 "MountingHole" H 2100 9655 50  0000 L CNN
-F 2 "OTTO_Footprints_Lib:Mounting_Hole_M2.5_Loose_Fit" H 2000 9700 50  0001 C CNN
-F 3 "N/A" H 2000 9700 50  0001 C CNN
-F 4 "DNP" H 2000 9700 50  0001 C CNN "AssemblyOption"
-F 5 "$0.00" H 2000 9700 50  0001 C CNN "UnitCost(USD)"
-F 6 "N/A" H 2000 9700 50  0001 C CNN "MPN"
-F 7 "N/A" H 2000 9700 50  0001 C CNN "Manufacturer"
-	1    2000 9700
-	1    0    0    -1
-$EndComp
 Wire Wire Line
 	7700 3350 8400 3350

Commit message: More JLC part numbers added
Parts:
- FID1, FID10, FID11, FID12, FID2, FID3, FID4, FID5, FID6, FID7, FID8, FID9, H201, H202, H203, H204, H205, H209, H212, H213, H214, H215: Manufacturer N/A -> (none); UnitCost(USD) $0.00 -> N/A
- J201: Manufacturer Harwin -> (none); UnitCost(USD) $3.97 -> Harwin
- R1, R2, R3: JLCASM (none) -> BASIC; LCSC PN (none) -> C17513; MPN RC0805FR-071KL -> 0805W8F1001T5E; Manufacturer Yageo -> (none); UnitCost(USD) $.001763 -> Yageo
- TP2, TP6, TP7, TP8, TP9: JLCASM (none) -> N/A; Manufacturer N/A -> (none); UnitCost(USD) $0.00 -> N/A

Commit message: Selected all LCSC parts. Check of part numbers complete
Parts:
- FID1, FID10, FID11, FID12, FID2, FID3, FID4, FID5, FID6, FID7, FID8, FID9, H201, H202, H203, H204, H205, H209, H212, H213, H214, H215: JLCASM (none) -> N/A; UnitCost(USD) N/A -> (none)
- J201: JLCASM (none) -> N/A; UnitCost(USD) Harwin -> (none)
- R1, R2, R3: UnitCost(USD) Yageo -> (none)
- TP2, TP6, TP7, TP8, TP9: UnitCost(USD) N/A -> (none)

Commit message: Finish selecting jlc parts
Parts:
- added H1, H2, H3: Tooling Hole, OTTO_Footprints_Lib:JLC_TOOLING_HOLE, symbol Mechanical:MountingHole
Changed lines of the file:
@@
 Text Notes 4550 8600 0    100  ~ 20
 Optical Alignment\n
+$Comp
+L Mechanical:MountingHole H1
+U 1 1 5E979C7D
+P 6500 8600
+F 0 "H1" H 6600 8646 50  0000 L CNN
+F 1 "Tooling Hole" H 6600 8555 50  0000 L CNN
+F 2 "OTTO_Footprints_Lib:JLC_TOOLING_HOLE" H 6500 8600 50  0001 C CNN
+F 3 "" H 6500 8600 50  0001 C CNN
+F 4 "DNP" H 6500 8600 50  0001 C CNN "AssemblyOption"
+F 5 "" H 6500 8600 50  0001 C CNN "UnitCost(USD)"
+F 6 "N/A" H 6500 8600 50  0001 C CNN "MPN"
+F 7 "" H 6500 8600 50  0001 C CNN "Manufacturer"
+F 8 "N/A" H 6500 8600 50  0001 C CNN "JLCASM"
+	1    6500 8600
+	1    0    0    -1
+$EndComp
+$Comp
+L Mechanical:MountingHole H2
+U 1 1 5E97B256
+P 6500 8950
+F 0 "H2" H 6600 8996 50  0000 L CNN
+F 1 "Tooling Hole" H 6600 8905 50  0000 L CNN
+F 2 "OTTO_Footprints_Lib:JLC_TOOLING_HOLE" H 6500 8950 50  0001 C CNN
+F 3 "" H 6500 8950 50  0001 C CNN
+F 4 "DNP" H 6500 8950 50  0001 C CNN "AssemblyOption"
+F 5 "" H 6500 8950 50  0001 C CNN "UnitCost(USD)"
+F 6 "N/A" H 6500 8950 50  0001 C CNN "MPN"
+F 7 "" H 6500 8950 50  0001 C CNN "Manufacturer"
+F 8 "N/A" H 6500 8950 50  0001 C CNN "JLCASM"
+	1    6500 8950
+	1    0    0    -1
+$EndComp
+$Comp
+L Mechanical:MountingHole H3
+U 1 1 5E97B7A3
+P 7400 8950
+F 0 "H3" H 7500 8996 50  0000 L CNN
+F 1 "Tooling Hole" H 7500 8905 50  0000 L CNN
+F 2 "OTTO_Footprints_Lib:JLC_TOOLING_HOLE" H 7400 8950 50  0001 C CNN
+F 3 "" H 7400 8950 50  0001 C CNN
+F 4 "DNP" H 7400 8950 50  0001 C CNN "AssemblyOption"
+F 5 "" H 7400 8950 50  0001 C CNN "UnitCost(USD)"
+F 6 "N/A" H 7400 8950 50  0001 C CNN "MPN"
+F 7 "" H 7400 8950 50  0001 C CNN "Manufacturer"
+F 8 "N/A" H 7400 8950 50  0001 C CNN "JLCASM"
+	1    7400 8950
+	1    0    0    -1
+$EndComp
 $EndSCHEMATC

Commit message: Remove LEDs from main board
Other:
- note added: "To prioritize external jtag connection.\n1k is too much, steven will look into suitable values"
Changed lines of the file:
@@
 	1    0    0    -1
 $EndComp
+Text Notes 10200 4250 0    50   ~ 0
+To prioritize external jtag connection.\n1k is too much, steven will look into suitable values
+Wire Notes Line style solid
+	10350 4300 10250 4400
 $EndSCHEMATC

Commit message: Fix jtag resistors
Parts:
- R1, R2, R3: value 1k -> 0
Other:
- note added: "Might be needed to prioritize external jtag connection."
- note removed: "To prioritize external jtag connection.\n1k is too much, steven will look into suitable values"
Changed lines of the file:
@@
 P 10250 4450
 F 0 "R3" V 10200 4250 50  0000 C CNN
-F 1 "1k" V 10200 4650 50  0000 C CNN
+F 1 "0" V 10200 4650 50  0000 C CNN
 F 2 "Resistor_SMD:R_0805_2012Metric_Pad1.15x1.40mm_HandSolder" V 10180 4450 50  0001 C CNN
 F 3 "https://datasheet.lcsc.com/szlcsc/C17513.pdf" H 10250 4450 50  0001 C CNN
@@
 P 7000 4150
 F 0 "R2" V 7050 4350 50  0000 C CNN
-F 1 "1k" V 7050 3950 50  0000 C CNN
+F 1 "0" V 7050 3950 50  0000 C CNN
 F 2 "Resistor_SMD:R_0805_2012Metric_Pad1.15x1.40mm_HandSolder" V 6930 4150 50  0001 C CNN
 F 3 "https://datasheet.lcsc.com/szlcsc/C17513.pdf" H 7000 4150 50  0001 C CNN
@@
 P 10250 4550
 F 0 "R1" V 10300 4750 50  0000 C CNN
-F 1 "1k" V 10300 4350 50  0000 C CNN
+F 1 "0" V 10300 4350 50  0000 C CNN
 F 2 "Resistor_SMD:R_0805_2012Metric_Pad1.15x1.40mm_HandSolder" V 10180 4550 50  0001 C CNN
 F 3 "https://datasheet.lcsc.com/szlcsc/C17513.pdf" H 10250 4550 50  0001 C CNN
@@
 $EndComp
 Text Notes 10200 4250 0    50   ~ 0
-To prioritize external jtag connection.\n1k is too much, steven will look into suitable values
+Might be needed to prioritize external jtag connection.
 Wire Notes Line style solid
 	10350 4300 10250 4400

Commit message: Screen backlight control (+more)
Connections:
- net labels added: RPI_UART_RX, RPI_UART_TX
- net labels removed: MIDI_IN, MIDI_OUT
Changed lines of the file:
@@
 	9600 4250 9400 4250
-Wire Wire Line
-	7700 3850 7800 3850
-Wire Wire Line
-	7800 3950 7700 3950
 Wire Wire Line
 	7700 4350 7800 4350
@@
 	1    0    0    -1
 $EndComp
-Text GLabel 7700 3850 0    50   Output ~ 0
-MIDI_OUT
-Text GLabel 7700 3950 0    50   Input ~ 0
-MIDI_IN
 Text Notes 7950 5700 0    50   ~ 0
 Harwin M20-7912045 connector
@@
 Wire Notes Line style solid
 	10350 4300 10250 4400
+Text GLabel 7700 3850 0    50   Input ~ 0
+RPI_UART_TX
+Text GLabel 7700 3950 0    50   Input ~ 0
+RPI_UART_RX
+Wire Wire Line
+	7700 3950 7800 3950
+Wire Wire Line
+	7800 3850 7700 3850
 $EndSCHEMATC
