File: KiCad/MIDI.sch (KiCad schematic (older format))
At the start: 14 parts, among them U205 74HC14, U206 H11L1

Commit message: add all resistor part numbers and create footprint library
Parts:
- R212, R214: EstimatedCost(USD) (none) -> $.002557; MPN (none) -> RC0805FR-0710RL; Manufacturer (none) -> Yageo
- R213, R215: EstimatedCost(USD) (none) -> $.001685; MPN (none) -> RC0805FR-0733RL; Manufacturer (none) -> Yageo
- R216: EstimatedCost(USD) (none) -> $.004683; MPN (none) -> RC0805FR-07270RL; Manufacturer (none) -> Yageo
- R217: EstimatedCost(USD) (none) -> $.001595; MPN (none) -> RC0805FR-07220RL; Manufacturer (none) -> Yageo
Changed lines of the file:
@@
 F 1 "10" V 4316 2350 50  0000 C CNN
 F 2 "Resistor_SMD:R_0805_2012Metric_Pad1.15x1.40mm_HandSolder" V 4130 2350 50  0001 C CNN
-F 3 "~" H 4200 2350 50  0001 C CNN
+F 3 "https://datasheet.lcsc.com/szlcsc/YAGEO-RC0805FR-0710RL_C96347.pdf" H 4200 2350 50  0001 C CNN
+F 4 "$.002557" H 4200 2350 50  0001 C CNN "EstimatedCost(USD)"
+F 5 "RC0805FR-0710RL" H 4200 2350 50  0001 C CNN "MPN"
+F 6 "Yageo" H 4200 2350 50  0001 C CNN "Manufacturer"
 	1    4200 2350
 	0    1    -1   0
@@
 F 1 "33" V 4400 2550 50  0000 C CNN
 F 2 "Resistor_SMD:R_0805_2012Metric_Pad1.15x1.40mm_HandSolder" V 4130 2550 50  0001 C CNN
-F 3 "~" H 4200 2550 50  0001 C CNN
+F 3 "https://datasheet.lcsc.com/szlcsc/YAGEO-RC0805FR-0733RL_C126353.pdf" H 4200 2550 50  0001 C CNN
+F 4 "$.001685" H 4200 2550 50  0001 C CNN "EstimatedCost(USD)"
+F 5 "RC0805FR-0733RL" H 4200 2550 50  0001 C CNN "MPN"
+F 6 "Yageo" H 4200 2550 50  0001 C CNN "Manufacturer"
 	1    4200 2550
 	0    1    1    0
@@
 F 1 "10" V 4084 3500 50  0000 C CNN
 F 2 "Resistor_SMD:R_0805_2012Metric_Pad1.15x1.40mm_HandSolder" V 4130 3500 50  0001 C CNN
-F 3 "~" H 4200 3500 50  0001 C CNN
+F 3 "https://datasheet.lcsc.com/szlcsc/YAGEO-RC0805FR-0710RL_C96347.pdf" H 4200 3500 50  0001 C CNN
+F 4 "$.002557" H 4200 3500 50  0001 C CNN "EstimatedCost(USD)"
+F 5 "RC0805FR-0710RL" H 4200 3500 50  0001 C CNN "MPN"
+F 6 "Yageo" H 4200 3500 50  0001 C CNN "Manufacturer"
 	1    4200 3500
 	0    1    1    0
@@
 F 1 "33" V 4400 3700 50  0000 C CNN
 F 2 "Resistor_SMD:R_0805_2012Metric_Pad1.15x1.40mm_HandSolder" V 4130 3700 50  0001 C CNN
-F 3 "~" H 4200 3700 50  0001 C CNN
+F 3 "https://datasheet.lcsc.com/szlcsc/YAGEO-RC0805FR-0733RL_C126353.pdf" H 4200 3700 50  0001 C CNN
+F 4 "$.001685" H 4200 3700 50  0001 C CNN "EstimatedCost(USD)"
+F 5 "RC0805FR-0733RL" H 4200 3700 50  0001 C CNN "MPN"
+F 6 "Yageo" H 4200 3700 50  0001 C CNN "Manufacturer"
 	1    4200 3700
 	0    1    1    0
@@
 F 1 "220" V 3784 4650 50  0000 C CNN
 F 2 "Resistor_SMD:R_0805_2012Metric_Pad1.15x1.40mm_HandSolder" V 3830 4650 50  0001 C CNN
-F 3 "~" H 3900 4650 50  0001 C CNN
+F 3 "https://datasheet.lcsc.com/szlcsc/YAGEO-RC0805FR-07220RL_C114519.pdf" H 3900 4650 50  0001 C CNN
+F 4 "$.001595" H 3900 4650 50  0001 C CNN "EstimatedCost(USD)"
+F 5 "RC0805FR-07220RL" H 3900 4650 50  0001 C CNN "MPN"
+F 6 "Yageo" H 3900 4650 50  0001 C CNN "Manufacturer"
 	1    3900 4650
 	0    1    1    0
@@
 F 1 "270" H 5420 4405 50  0000 L CNN
 F 2 "Resistor_SMD:R_0805_2012Metric_Pad1.15x1.40mm_HandSolder" V 5280 4450 50  0001 C CNN
-F 3 "~" H 5350 4450 50  0001 C CNN
+F 3 "https://datasheet.lcsc.com/szlcsc/YAGEO-RC0805FR-07270RL_C137558.pdf" H 5350 4450 50  0001 C CNN
+F 4 "$.004683" H 5350 4450 50  0001 C CNN "EstimatedCost(USD)"
+F 5 "RC0805FR-07270RL" H 5350 4450 50  0001 C CNN "MPN"
+F 6 "Yageo" H 5350 4450 50  0001 C CNN "Manufacturer"
 	1    5350 4450
 	1    0    0    -1

Commit message: added part numbers for capacitors and crystals
Parts:
- C68, C69: footprint Capacitor_SMD:C_0805_2012Metric_Pad1.15x1.40mm_HandSolder_marked -> Capacitor_SMD:C_0805_2012Metric_Pad1.15x1.40mm_HandSolder; EstimatedCost(USD) (none) -> $0.017724; MPN (none) -> CL21B104JBCNNNC; Manufacturer (none) -> Samsung Electro-Mechanics
Changed lines of the file:
@@
 F 0 "C69" V 3187 6850 50  0000 C CNN
 F 1 "100nF" V 3278 6850 50  0000 C CNN
-F 2 "Capacitor_SMD:C_0805_2012Metric_Pad1.15x1.40mm_HandSolder_marked" H 3050 6850 50  0001 C CNN
-F 3 "~" H 3050 6850 50  0001 C CNN
+F 2 "Capacitor_SMD:C_0805_2012Metric_Pad1.15x1.40mm_HandSolder" H 3050 6850 50  0001 C CNN
+F 3 "https://datasheet.lcsc.com/szlcsc/Samsung-Electro-Mechanics-CL21B104JBCNNNC_C62912.pdf" H 3050 6850 50  0001 C CNN
+F 4 "$0.017724" H 3050 6850 12700 0001 C CNN "EstimatedCost(USD)"
+F 5 "CL21B104JBCNNNC" H 3050 6850 12700 0001 C CNN "MPN"
+F 6 "Samsung Electro-Mechanics" H 3050 6850 12700 0001 C CNN "Manufacturer"
 	1    3050 6850
 	0    1    1    0
@@
 F 0 "C68" H 5808 4654 50  0000 R CNN
 F 1 "100nF" H 5808 4745 50  0000 R CNN
-F 2 "Capacitor_SMD:C_0805_2012Metric_Pad1.15x1.40mm_HandSolder_marked" H 5900 4700 50  0001 C CNN
-F 3 "~" H 5900 4700 50  0001 C CNN
+F 2 "Capacitor_SMD:C_0805_2012Metric_Pad1.15x1.40mm_HandSolder" H 5900 4700 50  0001 C CNN
+F 3 "https://datasheet.lcsc.com/szlcsc/Samsung-Electro-Mechanics-CL21B104JBCNNNC_C62912.pdf" H 5900 4700 50  0001 C CNN
+F 4 "$0.017724" H 5900 4700 12700 0001 C CNN "EstimatedCost(USD)"
+F 5 "CL21B104JBCNNNC" H 5900 4700 12700 0001 C CNN "MPN"
+F 6 "Samsung Electro-Mechanics" H 5900 4700 12700 0001 C CNN "Manufacturer"
 	1    5900 4700
 	-1   0    0    1

Commit message: add more part numbers, samtec connector footprint
Parts:
- D206: value 1N4148 -> 1N4148W; footprint Diode_SMD:D_SMA -> Diode_SMD:D_SOD-123; EstimatedCost(USD) (none) -> $0.007483; MPN (none) -> 1N4148W; Manufacturer (none) -> MDD(Microdiode Electronics)
Changed lines of the file:
@@
 P 4250 4700
 F 0 "D206" V 4204 4779 50  0000 L CNN
-F 1 "1N4148" V 4295 4779 50  0000 L CNN
-F 2 "Diode_SMD:D_SMA" H 4250 4700 50  0001 C CNN
-F 3 "~" H 4250 4700 50  0001 C CNN
+F 1 "1N4148W" V 4295 4779 50  0000 L CNN
+F 2 "Diode_SMD:D_SOD-123" H 4250 4700 50  0001 C CNN
+F 3 "https://datasheet.lcsc.com/szlcsc/1903051131_MDD-Jiangsu-Yutai-Elec-1N4148W_C84367.pdf" H 4250 4700 50  0001 C CNN
+F 4 "$0.007483" H 4250 4700 50  0001 C CNN "EstimatedCost(USD)"
+F 5 "1N4148W" H 4250 4700 50  0001 C CNN "MPN"
+F 6 "MDD(Microdiode Electronics)" H 4250 4700 50  0001 C CNN "Manufacturer"
 	1    4250 4700
 	0    1    1    0

Commit message: add switch and encoder parts. BM Complete. Footprints complete.
Parts:
- TRS201, TRS202, TRS203: value PJ-393-7A -> PJ-3930-8A; footprint Spatz:3.5mm_jack_PJ-3930-8A -> OTTO_Footprints_Lib:3.5mm_jack_PJ-3930-8A; EstimatedCost(USD) (none) -> $0.456061; MPN (none) -> PJ-3930-8A; Manufacturer (none) -> Korean Hroparts Elec
- U205: value 74HC14 -> SN74HC14; EstimatedCost(USD) (none) -> $0.124242; MPN (none) -> SN74HC14DR; Manufacturer (none) -> Texas Instruments
- U206: value H11L1 -> H11L1S; footprint Package_DIP:DIP-6_W7.62mm_SMDSocket_SmallPads -> Package_DIP:SMDIP-6_W7.62mm; EstimatedCost(USD) (none) -> $0.359091; MPN (none) -> H11L1S(TA); Manufacturer (none) -> Everlight Elec
Changed lines of the file:
@@
 P 5350 2350
 F 0 "U205" H 5350 2033 50  0000 C CNN
-F 1 "74HC14" H 5350 2124 50  0000 C CNN
+F 1 "SN74HC14" H 5350 2124 50  0000 C CNN
 F 2 "Package_SO:SOIC-14_3.9x8.7mm_P1.27mm" H 5350 2350 50  0001 C CNN
 F 3 "http://www.ti.com/lit/gpn/sn74HC14" H 5350 2350 50  0001 C CNN
+F 4 "$0.124242" H 5350 2350 12700 0001 C CNN "EstimatedCost(USD)"
+F 5 "SN74HC14DR" H 5350 2350 12700 0001 C CNN "MPN"
+F 6 "Texas Instruments" H 5350 2350 12700 0001 C CNN "Manufacturer"
 	4    5350 2350
 	-1   0    0    1
@@
 P 6050 2350
 F 0 "U205" H 6050 2033 50  0000 C CNN
-F 1 "74HC14" H 6050 2124 50  0000 C CNN
+F 1 "SN74HC14" H 6050 2124 50  0000 C CNN
 F 2 "Package_SO:SOIC-14_3.9x8.7mm_P1.27mm" H 6050 2350 50  0001 C CNN
 F 3 "http://www.ti.com/lit/gpn/sn74HC14" H 6050 2350 50  0001 C CNN
+F 4 "$0.124242" H 6050 2350 12700 0001 C CNN "EstimatedCost(USD)"
+F 5 "SN74HC14DR" H 6050 2350 12700 0001 C CNN "MPN"
+F 6 "Texas Instruments" H 6050 2350 12700 0001 C CNN "Manufacturer"
 	5    6050 2350
 	-1   0    0    1
@@
 P 4950 6550
 F 0 "U205" H 4950 6233 50  0000 C CNN
-F 1 "74HC14" H 4950 6324 50  0000 C CNN
+F 1 "SN74HC14" H 4950 6324 50  0000 C CNN
 F 2 "Package_SO:SOIC-14_3.9x8.7mm_P1.27mm" H 4950 6550 50  0001 C CNN
 F 3 "http://www.ti.com/lit/gpn/sn74HC14" H 4950 6550 50  0001 C CNN
+F 4 "$0.124242" H 4950 6550 12700 0001 C CNN "EstimatedCost(USD)"
+F 5 "SN74HC14DR" H 4950 6550 12700 0001 C CNN "MPN"
+F 6 "Texas Instruments" H 4950 6550 12700 0001 C CNN "Manufacturer"
 	6    4950 6550
 	-1   0    0    1
@@
 P 3050 6500
 F 0 "U205" V 3417 6500 50  0000 C CNN
-F 1 "74HC14" V 3326 6500 50  0000 C CNN
+F 1 "SN74HC14" V 3326 6500 50  0000 C CNN
 F 2 "Package_SO:SOIC-14_3.9x8.7mm_P1.27mm" H 3050 6500 50  0001 C CNN
 F 3 "http://www.ti.com/lit/gpn/sn74HC14" H 3050 6500 50  0001 C CNN
+F 4 "$0.124242" H 3050 6500 12700 0001 C CNN "EstimatedCost(USD)"
+F 5 "SN74HC14DR" H 3050 6500 12700 0001 C CNN "MPN"
+F 6 "Texas Instruments" H 3050 6500 12700 0001 C CNN "Manufacturer"
 	7    3050 6500
 	0    -1   -1   0
@@
 P 4950 4700
 F 0 "U206" H 4550 4350 50  0000 L CNN
-F 1 "H11L1" H 4550 4250 50  0000 L CNN
-F 2 "Package_DIP:DIP-6_W7.62mm_SMDSocket_SmallPads" H 4860 4700 50  0001 C CNN
+F 1 "H11L1S" H 4550 4250 50  0000 L CNN
+F 2 "Package_DIP:SMDIP-6_W7.62mm" H 4860 4700 50  0001 C CNN
 F 3 "https://www.fairchildsemi.com/datasheets/H1/H11L1M.pdf" H 4860 4700 50  0001 C CNN
+F 4 "$0.359091" H 4950 4700 12700 0001 C CNN "EstimatedCost(USD)"
+F 5 "H11L1S(TA)" H 4950 4700 12700 0001 C CNN "MPN"
+F 6 "Everlight Elec" H 4950 4700 12700 0001 C CNN "Manufacturer"
 	1    4950 4700
 	1    0    0    -1
@@
 AR Path="/5DF1F84C" Ref="TRS201"  Part="1"
 F 0 "TRS201" H 3357 2975 50  0000 C CNN
-F 1 "PJ-393-7A" H 3357 2884 50  0000 C CNN
-F 2 "Spatz:3.5mm_jack_PJ-3930-8A" H 3400 2350 50  0001 C CNN
-F 3 "" H 3400 2350 50  0001 C CNN
+F 1 "PJ-3930-8A" H 3357 2884 50  0000 C CNN
+F 2 "OTTO_Footprints_Lib:3.5mm_jack_PJ-3930-8A" H 3400 2350 50  0001 C CNN
+F 3 "https://datasheet.lcsc.com/szlcsc/1911181432_Korean-Hroparts-Elec-PJ-3930-8A_C145811.pdf" H 3400 2350 50  0001 C CNN
+F 4 "$0.456061" H 3300 2350 12700 0001 C CNN "EstimatedCost(USD)"
+F 5 "PJ-3930-8A" H 3300 2350 12700 0001 C CNN "MPN"
+F 6 "Korean Hroparts Elec" H 3300 2350 12700 0001 C CNN "Manufacturer"
 	1    3300 2350
 	1    0    0    -1
@@
 AR Path="/5DF278B3" Ref="TRS202"  Part="1"
 F 0 "TRS202" H 3357 4125 50  0000 C CNN
-F 1 "PJ-393-7A" H 3357 4034 50  0000 C CNN
-F 2 "Spatz:3.5mm_jack_PJ-3930-8A" H 3400 3500 50  0001 C CNN
-F 3 "" H 3400 3500 50  0001 C CNN
+F 1 "PJ-3930-8A" H 3357 4034 50  0000 C CNN
+F 2 "OTTO_Footprints_Lib:3.5mm_jack_PJ-3930-8A" H 3400 3500 50  0001 C CNN
+F 3 "https://datasheet.lcsc.com/szlcsc/1911181432_Korean-Hroparts-Elec-PJ-3930-8A_C145811.pdf" H 3400 3500 50  0001 C CNN
+F 4 "$0.456061" H 3300 3500 12700 0001 C CNN "EstimatedCost(USD)"
+F 5 "PJ-3930-8A" H 3300 3500 12700 0001 C CNN "MPN"
+F 6 "Korean Hroparts Elec" H 3300 3500 12700 0001 C CNN "Manufacturer"
 	1    3300 3500
 	1    0    0    -1
@@
 AR Path="/5DF28FAD" Ref="TRS203"  Part="1"
 F 0 "TRS203" H 3357 5275 50  0000 C CNN
-F 1 "PJ-393-7A" H 3357 5184 50  0000 C CNN
-F 2 "Spatz:3.5mm_jack_PJ-3930-8A" H 3400 4650 50  0001 C CNN
-F 3 "" H 3400 4650 50  0001 C CNN
+F 1 "PJ-3930-8A" H 3357 5184 50  0000 C CNN
+F 2 "OTTO_Footprints_Lib:3.5mm_jack_PJ-3930-8A" H 3400 4650 50  0001 C CNN
+F 3 "https://datasheet.lcsc.com/szlcsc/1911181432_Korean-Hroparts-Elec-PJ-3930-8A_C145811.pdf" H 3400 4650 50  0001 C CNN
+F 4 "$0.456061" H 3300 4650 12700 0001 C CNN "EstimatedCost(USD)"
+F 5 "PJ-3930-8A" H 3300 4650 12700 0001 C CNN "MPN"
+F 6 "Korean Hroparts Elec" H 3300 4650 12700 0001 C CNN "Manufacturer"
 	1    3300 4650
 	1    0    0    -1
@@
 P 6050 3500
 F 0 "U205" H 6050 3183 50  0000 C CNN
-F 1 "74HC14" H 6050 3274 50  0000 C CNN
+F 1 "SN74HC14" H 6050 3274 50  0000 C CNN
 F 2 "Package_SO:SOIC-14_3.9x8.7mm_P1.27mm" H 6050 3500 50  0001 C CNN
 F 3 "http://www.ti.com/lit/gpn/sn74HC14" H 6050 3500 50  0001 C CNN
+F 4 "$0.124242" H 6050 3500 12700 0001 C CNN "EstimatedCost(USD)"
+F 5 "SN74HC14DR" H 6050 3500 12700 0001 C CNN "MPN"
+F 6 "Texas Instruments" H 6050 3500 12700 0001 C CNN "Manufacturer"
 	2    6050 3500
 	-1   0    0    1
@@
 P 5350 3500
 F 0 "U205" H 5350 3183 50  0000 C CNN
-F 1 "74HC14" H 5350 3274 50  0000 C CNN
+F 1 "SN74HC14" H 5350 3274 50  0000 C CNN
 F 2 "Package_SO:SOIC-14_3.9x8.7mm_P1.27mm" H 5350 3500 50  0001 C CNN
 F 3 "http://www.ti.com/lit/gpn/sn74HC14" H 5350 3500 50  0001 C CNN
+F 4 "$0.124242" H 5350 3500 12700 0001 C CNN "EstimatedCost(USD)"
+F 5 "SN74HC14DR" H 5350 3500 12700 0001 C CNN "MPN"
+F 6 "Texas Instruments" H 5350 3500 12700 0001 C CNN "Manufacturer"
 	3    5350 3500
 	-1   0    0    1
@@
 P 4950 5950
 F 0 "U205" H 4950 5633 50  0000 C CNN
-F 1 "74HC14" H 4950 5724 50  0000 C CNN
+F 1 "SN74HC14" H 4950 5724 50  0000 C CNN
 F 2 "Package_SO:SOIC-14_3.9x8.7mm_P1.27mm" H 4950 5950 50  0001 C CNN
 F 3 "http://www.ti.com/lit/gpn/sn74HC14" H 4950 5950 50  0001 C CNN
+F 4 "$0.124242" H 4950 5950 12700 0001 C CNN "EstimatedCost(USD)"
+F 5 "SN74HC14DR" H 4950 5950 12700 0001 C CNN "MPN"
+F 6 "Texas Instruments" H 4950 5950 12700 0001 C CNN "Manufacturer"
 	1    4950 5950
 	-1   0    0    1

Commit message: add BOM scripts, fix schematic hierarchy
Parts:
- C68, C69: EstimatedCost(USD) $0.017724 -> (none); UnitCost(USD) (none) -> $0.017724
- D206: EstimatedCost(USD) $0.007483 -> (none); UnitCost(USD) (none) -> $0.007483
- R212, R214: EstimatedCost(USD) $.002557 -> (none); UnitCost(USD) (none) -> $.002557
- R213, R215: EstimatedCost(USD) $.001685 -> (none); UnitCost(USD) (none) -> $.001685
- R216: EstimatedCost(USD) $.004683 -> (none); UnitCost(USD) (none) -> $.004683
- R217: EstimatedCost(USD) $.001595 -> (none); UnitCost(USD) (none) -> $.001595
- TRS201, TRS202, TRS203: EstimatedCost(USD) $0.456061 -> (none); UnitCost(USD) (none) -> $0.456061
- U205: EstimatedCost(USD) $0.124242 -> (none); UnitCost(USD) (none) -> $0.124242
- U206: EstimatedCost(USD) $0.359091 -> (none); UnitCost(USD) (none) -> $0.359091
Changed lines of the file:
@@
-EESchema Schematic File Version 5
+EESchema Schematic File Version 4
 EELAYER 30 0
 EELAYER END
 $Descr A3 16535 11693
 encoding utf-8
-Sheet 6 7
-Title "OTTOdiy - preliminary"
-Date "2019-01-19"
-Rev "0.1"
-Comp "design by Bastian \"Spatz\" Mohing"
-Comment1 "no footprints assigned yet"
+Sheet 7 7
+Title "OTTOdiy"
+Date "2020-01-10"
+Rev "1.0"
+Comp "https://github.com/otto-project"
+Comment1 "Design by Bastian \"Spatz\" Mohing and Steven \"adorbs\" Hang"
 Comment2 ""
 Comment3 ""
 Comment4 ""
-Comment5 ""
-Comment6 ""
-Comment7 ""
-Comment8 ""
-Comment9 ""
 $EndDescr
 $Comp
@@
 F 2 "Resistor_SMD:R_0805_2012Metric_Pad1.15x1.40mm_HandSolder" V 4130 2350 50  0001 C CNN
 F 3 "https://datasheet.lcsc.com/szlcsc/YAGEO-RC0805FR-0710RL_C96347.pdf" H 4200 2350 50  0001 C CNN
-F 4 "$.002557" H 4200 2350 50  0001 C CNN "EstimatedCost(USD)"
+F 4 "$.002557" H 4200 2350 50  0001 C CNN "UnitCost(USD)"
 F 5 "RC0805FR-0710RL" H 4200 2350 50  0001 C CNN "MPN"
 F 6 "Yageo" H 4200 2350 50  0001 C CNN "Manufacturer"
@@
 F 2 "Resistor_SMD:R_0805_2012Metric_Pad1.15x1.40mm_HandSolder" V 4130 2550 50  0001 C CNN
 F 3 "https://datasheet.lcsc.com/szlcsc/YAGEO-RC0805FR-0733RL_C126353.pdf" H 4200 2550 50  0001 C CNN
-F 4 "$.001685" H 4200 2550 50  0001 C CNN "EstimatedCost(USD)"
+F 4 "$.001685" H 4200 2550 50  0001 C CNN "UnitCost(USD)"
 F 5 "RC0805FR-0733RL" H 4200 2550 50  0001 C CNN "MPN"
 F 6 "Yageo" H 4200 2550 50  0001 C CNN "Manufacturer"
@@
 F 2 "Resistor_SMD:R_0805_2012Metric_Pad1.15x1.40mm_HandSolder" V 4130 3500 50  0001 C CNN
 F 3 "https://datasheet.lcsc.com/szlcsc/YAGEO-RC0805FR-0710RL_C96347.pdf" H 4200 3500 50  0001 C CNN
-F 4 "$.002557" H 4200 3500 50  0001 C CNN "EstimatedCost(USD)"
+F 4 "$.002557" H 4200 3500 50  0001 C CNN "UnitCost(USD)"
 F 5 "RC0805FR-0710RL" H 4200 3500 50  0001 C CNN "MPN"
 F 6 "Yageo" H 4200 3500 50  0001 C CNN "Manufacturer"
@@
 F 2 "Resistor_SMD:R_0805_2012Metric_Pad1.15x1.40mm_HandSolder" V 4130 3700 50  0001 C CNN
 F 3 "https://datasheet.lcsc.com/szlcsc/YAGEO-RC0805FR-0733RL_C126353.pdf" H 4200 3700 50  0001 C CNN
-F 4 "$.001685" H 4200 3700 50  0001 C CNN "EstimatedCost(USD)"
+F 4 "$.001685" H 4200 3700 50  0001 C CNN "UnitCost(USD)"
 F 5 "RC0805FR-0733RL" H 4200 3700 50  0001 C CNN "MPN"
 F 6 "Yageo" H 4200 3700 50  0001 C CNN "Manufacturer"
@@
 F 2 "Resistor_SMD:R_0805_2012Metric_Pad1.15x1.40mm_HandSolder" V 3830 4650 50  0001 C CNN
 F 3 "https://datasheet.lcsc.com/szlcsc/YAGEO-RC0805FR-07220RL_C114519.pdf" H 3900 4650 50  0001 C CNN
-F 4 "$.001595" H 3900 4650 50  0001 C CNN "EstimatedCost(USD)"
+F 4 "$.001595" H 3900 4650 50  0001 C CNN "UnitCost(USD)"
 F 5 "RC0805FR-07220RL" H 3900 4650 50  0001 C CNN "MPN"
 F 6 "Yageo" H 3900 4650 50  0001 C CNN "Manufacturer"
@@
 F 2 "Diode_SMD:D_SOD-123" H 4250 4700 50  0001 C CNN
 F 3 "https://datasheet.lcsc.com/szlcsc/1903051131_MDD-Jiangsu-Yutai-Elec-1N4148W_C84367.pdf" H 4250 4700 50  0001 C CNN
-F 4 "$0.007483" H 4250 4700 50  0001 C CNN "EstimatedCost(USD)"
+F 4 "$0.007483" H 4250 4700 50  0001 C CNN "UnitCost(USD)"
 F 5 "1N4148W" H 4250 4700 50  0001 C CNN "MPN"
 F 6 "MDD(Microdiode Electronics)" H 4250 4700 50  0001 C CNN "Manufacturer"
@@
 F 2 "Resistor_SMD:R_0805_2012Metric_Pad1.15x1.40mm_HandSolder" V 5280 4450 50  0001 C CNN
 F 3 "https://datasheet.lcsc.com/szlcsc/YAGEO-RC0805FR-07270RL_C137558.pdf" H 5350 4450 50  0001 C CNN
-F 4 "$.004683" H 5350 4450 50  0001 C CNN "EstimatedCost(USD)"
+F 4 "$.004683" H 5350 4450 50  0001 C CNN "UnitCost(USD)"
 F 5 "RC0805FR-07270RL" H 5350 4450 50  0001 C CNN "MPN"
 F 6 "Yageo" H 5350 4450 50  0001 C CNN "Manufacturer"
@@
 F 2 "Package_SO:SOIC-14_3.9x8.7mm_P1.27mm" H 5350 2350 50  0001 C CNN
 F 3 "http://www.ti.com/lit/gpn/sn74HC14" H 5350 2350 50  0001 C CNN
-F 4 "$0.124242" H 5350 2350 12700 0001 C CNN "EstimatedCost(USD)"
+F 4 "$0.124242" H 5350 2350 12700 0001 C CNN "UnitCost(USD)"
 F 5 "SN74HC14DR" H 5350 2350 12700 0001 C CNN "MPN"
 F 6 "Texas Instruments" H 5350 2350 12700 0001 C CNN "Manufacturer"
@@
 F 2 "Package_SO:SOIC-14_3.9x8.7mm_P1.27mm" H 6050 2350 50  0001 C CNN
 F 3 "http://www.ti.com/lit/gpn/sn74HC14" H 6050 2350 50  0001 C CNN
-F 4 "$0.124242" H 6050 2350 12700 0001 C CNN "EstimatedCost(USD)"
+F 4 "$0.124242" H 6050 2350 12700 0001 C CNN "UnitCost(USD)"
 F 5 "SN74HC14DR" H 6050 2350 12700 0001 C CNN "MPN"
 F 6 "Texas Instruments" H 6050 2350 12700 0001 C CNN "Manufacturer"
@@
 F 2 "Package_SO:SOIC-14_3.9x8.7mm_P1.27mm" H 4950 6550 50  0001 C CNN
 F 3 "http://www.ti.com/lit/gpn/sn74HC14" H 4950 6550 50  0001 C CNN
-F 4 "$0.124242" H 4950 6550 12700 0001 C CNN "EstimatedCost(USD)"
+F 4 "$0.124242" H 4950 6550 12700 0001 C CNN "UnitCost(USD)"
 F 5 "SN74HC14DR" H 4950 6550 12700 0001 C CNN "MPN"
 F 6 "Texas Instruments" H 4950 6550 12700 0001 C CNN "Manufacturer"
@@
 F 2 "Package_SO:SOIC-14_3.9x8.7mm_P1.27mm" H 3050 6500 50  0001 C CNN
 F 3 "http://www.ti.com/lit/gpn/sn74HC14" H 3050 6500 50  0001 C CNN
-F 4 "$0.124242" H 3050 6500 12700 0001 C CNN "EstimatedCost(USD)"
+F 4 "$0.124242" H 3050 6500 12700 0001 C CNN "UnitCost(USD)"
 F 5 "SN74HC14DR" H 3050 6500 12700 0001 C CNN "MPN"
 F 6 "Texas Instruments" H 3050 6500 12700 0001 C CNN "Manufacturer"
@@
 F 2 "Capacitor_SMD:C_0805_2012Metric_Pad1.15x1.40mm_HandSolder" H 3050 6850 50  0001 C CNN
 F 3 "https://datasheet.lcsc.com/szlcsc/Samsung-Electro-Mechanics-CL21B104JBCNNNC_C62912.pdf" H 3050 6850 50  0001 C CNN
-F 4 "$0.017724" H 3050 6850 12700 0001 C CNN "EstimatedCost(USD)"
+F 4 "$0.017724" H 3050 6850 12700 0001 C CNN "UnitCost(USD)"
 F 5 "CL21B104JBCNNNC" H 3050 6850 12700 0001 C CNN "MPN"
 F 6 "Samsung Electro-Mechanics" H 3050 6850 12700 0001 C CNN "Manufacturer"
@@
 F 2 "Package_DIP:SMDIP-6_W7.62mm" H 4860 4700 50  0001 C CNN
 F 3 "https://www.fairchildsemi.com/datasheets/H1/H11L1M.pdf" H 4860 4700 50  0001 C CNN
-F 4 "$0.359091" H 4950 4700 12700 0001 C CNN "EstimatedCost(USD)"
+F 4 "$0.359091" H 4950 4700 12700 0001 C CNN "UnitCost(USD)"
 F 5 "H11L1S(TA)" H 4950 4700 12700 0001 C CNN "MPN"
 F 6 "Everlight Elec" H 4950 4700 12700 0001 C CNN "Manufacturer"
@@
 F 2 "Capacitor_SMD:C_0805_2012Metric_Pad1.15x1.40mm_HandSolder" H 5900 4700 50  0001 C CNN
 F 3 "https://datasheet.lcsc.com/szlcsc/Samsung-Electro-Mechanics-CL21B104JBCNNNC_C62912.pdf" H 5900 4700 50  0001 C CNN
-F 4 "$0.017724" H 5900 4700 12700 0001 C CNN "EstimatedCost(USD)"
+F 4 "$0.017724" H 5900 4700 12700 0001 C CNN "UnitCost(USD)"
 F 5 "CL21B104JBCNNNC" H 5900 4700 12700 0001 C CNN "MPN"
 F 6 "Samsung Electro-Mechanics" H 5900 4700 12700 0001 C CNN "Manufacturer"
@@
 F 2 "OTTO_Footprints_Lib:3.5mm_jack_PJ-3930-8A" H 3400 2350 50  0001 C CNN
 F 3 "https://datasheet.lcsc.com/szlcsc/1911181432_Korean-Hroparts-Elec-PJ-3930-8A_C145811.pdf" H 3400 2350 50  0001 C CNN
-F 4 "$0.456061" H 3300 2350 12700 0001 C CNN "EstimatedCost(USD)"
+F 4 "$0.456061" H 3300 2350 12700 0001 C CNN "UnitCost(USD)"
 F 5 "PJ-3930-8A" H 3300 2350 12700 0001 C CNN "MPN"
 F 6 "Korean Hroparts Elec" H 3300 2350 12700 0001 C CNN "Manufacturer"
@@
 F 2 "OTTO_Footprints_Lib:3.5mm_jack_PJ-3930-8A" H 3400 3500 50  0001 C CNN
 F 3 "https://datasheet.lcsc.com/szlcsc/1911181432_Korean-Hroparts-Elec-PJ-3930-8A_C145811.pdf" H 3400 3500 50  0001 C CNN
-F 4 "$0.456061" H 3300 3500 12700 0001 C CNN "EstimatedCost(USD)"
+F 4 "$0.456061" H 3300 3500 12700 0001 C CNN "UnitCost(USD)"
 F 5 "PJ-3930-8A" H 3300 3500 12700 0001 C CNN "MPN"
 F 6 "Korean Hroparts Elec" H 3300 3500 12700 0001 C CNN "Manufacturer"
@@
 F 2 "OTTO_Footprints_Lib:3.5mm_jack_PJ-3930-8A" H 3400 4650 50  0001 C CNN
 F 3 "https://datasheet.lcsc.com/szlcsc/1911181432_Korean-Hroparts-Elec-PJ-3930-8A_C145811.pdf" H 3400 4650 50  0001 C CNN
-F 4 "$0.456061" H 3300 4650 12700 0001 C CNN "EstimatedCost(USD)"
+F 4 "$0.456061" H 3300 4650 12700 0001 C CNN "UnitCost(USD)"
 F 5 "PJ-3930-8A" H 3300 4650 12700 0001 C CNN "MPN"
 F 6 "Korean Hroparts Elec" H 3300 4650 12700 0001 C CNN "Manufacturer"
@@
 F 2 "Package_SO:SOIC-14_3.9x8.7mm_P1.27mm" H 6050 3500 50  0001 C CNN
 F 3 "http://www.ti.com/lit/gpn/sn74HC14" H 6050 3500 50  0001 C CNN
-F 4 "$0.124242" H 6050 3500 12700 0001 C CNN "EstimatedCost(USD)"
+F 4 "$0.124242" H 6050 3500 12700 0001 C CNN "UnitCost(USD)"
 F 5 "SN74HC14DR" H 6050 3500 12700 0001 C CNN "MPN"
 F 6 "Texas Instruments" H 6050 3500 12700 0001 C CNN "Manufacturer"
@@
 F 2 "Package_SO:SOIC-14_3.9x8.7mm_P1.27mm" H 5350 3500 50  0001 C CNN
 F 3 "http://www.ti.com/lit/gpn/sn74HC14" H 5350 3500 50  0001 C CNN
-F 4 "$0.124242" H 5350 3500 12700 0001 C CNN "EstimatedCost(USD)"
+F 4 "$0.124242" H 5350 3500 12700 0001 C CNN "UnitCost(USD)"
 F 5 "SN74HC14DR" H 5350 3500 12700 0001 C CNN "MPN"
 F 6 "Texas Instruments" H 5350 3500 12700 0001 C CNN "Manufacturer"
@@
 F 2 "Package_SO:SOIC-14_3.9x8.7mm_P1.27mm" H 4950 5950 50  0001 C CNN
 F 3 "http://www.ti.com/lit/gpn/sn74HC14" H 4950 5950 50  0001 C CNN
-F 4 "$0.124242" H 4950 5950 12700 0001 C CNN "EstimatedCost(USD)"
+F 4 "$0.124242" H 4950 5950 12700 0001 C CNN "UnitCost(USD)"
 F 5 "SN74HC14DR" H 4950 5950 12700 0001 C CNN "MPN"
 F 6 "Texas Instruments" H 4950 5950 12700 0001 C CNN "Manufacturer"
