File: KiCad/MIDI.sch (KiCad schematic (older format))
At the start: 14 parts, among them U205 SN74HC14, U206 H11L1S

Commit message: routed audio
Parts:
- added C98: 100nF, Capacitor_SMD:C_0805_2012Metric_Pad1.15x1.40mm_HandSolder, symbol Device:C_Small
Connections:
- wire segments 49 -> 51
- no-connect marks 16 -> 15

Commit message: add analog ground layout
Connections:
- no-connect marks 15 -> 16
Changed lines of the file:
@@
 Wire Wire Line
 	7850 5250 7750 5250
+NoConn ~ 6750 5500
 $EndSCHEMATC

Commit message: More JLC part numbers added
Parts:
- C68, C69, C98: JLCASM (none) -> BASIC; LCSC PN (none) -> C49678; MPN CL21B104JBCNNNC -> CC0805KRX7R9BB104; Manufacturer Samsung Electro-Mechanics -> (none); UnitCost(USD) $0.017724 -> Samsung Electro-Mechanics
- D206: JLCASM (none) -> BASIC; LCSC PN (none) -> C81598; Manufacturer MDD(Microdiode Electronics) -> (none); UnitCost(USD) $0.007483 -> MDD(Microdiode Electronics)
- R212, R214: JLCASM (none) -> BASIC; LCSC PN (none) -> C17415; MPN RC0805FR-0710RL -> 0805W8F100JT5E; Manufacturer Yageo -> (none); UnitCost(USD) $.002557 -> Yageo
- R213, R215: JLCASM (none) -> BASIC; LCSC PN (none) -> C17634; MPN RC0805FR-0733RL -> 0805W8F330JT5E; Manufacturer Yageo -> (none); UnitCost(USD) $.001685 -> Yageo
- R216: JLCASM (none) -> BASIC; LCSC PN (none) -> C17590; MPN RC0805FR-07270RL -> 0805W8F2700T5E; Manufacturer Yageo -> (none); UnitCost(USD) $.004683 -> Yageo
- R217: JLCASM (none) -> BASIC; LCSC PN (none) -> C17557; MPN RC0805FR-07220RL -> 0805W8F2200T5E; Manufacturer Yageo -> (none); UnitCost(USD) $.001595 -> Yageo
- TRS201, TRS202, TRS203: JLCASM (none) -> DNP; LCSC PN (none) -> C145811; Manufacturer Korean Hroparts Elec -> (none); UnitCost(USD) $0.456061 -> Korean Hroparts Elec
- U205: JLCASM (none) -> EXT; LCSC PN (none) -> C6820; Manufacturer Texas Instruments -> (none); UnitCost(USD) $0.124242 -> Texas Instruments
- U206: JLCASM (none) -> EXT; LCSC PN (none) -> C78589; Manufacturer Everlight Elec -> (none); UnitCost(USD) $0.359091 -> Everlight Elec

Commit message: Selected all LCSC parts. Check of part numbers complete
Parts:
- C68, C69, C98: UnitCost(USD) Samsung Electro-Mechanics -> (none)
- D206: UnitCost(USD) MDD(Microdiode Electronics) -> (none)
- R212, R213, R214, R215, R216, R217: UnitCost(USD) Yageo -> (none)
- TRS201, TRS202, TRS203: UnitCost(USD) Korean Hroparts Elec -> (none)
- U205: UnitCost(USD) Texas Instruments -> (none)
- U206: UnitCost(USD) Everlight Elec -> (none)

Commit message: Finish selecting jlc parts
Parts:
- removed U206: H11L1S, Package_DIP:SMDIP-6_W7.62mm, symbol Isolator:H11L1
- added U201: 6N137, Package_DIP:DIP-8_W8.89mm_SMDSocket_LongPads, symbol Isolator:6N137
Connections:
- net labels added: +5V_RASPI
- no-connect marks 16 -> 17
Changed lines of the file:
@@
 Connection ~ 7700 5850
-$Comp
-L power:GND #PWR0229
-U 1 1 5D56D2C7
-P 9450 6100
-F 0 "#PWR0229" H 9450 5850 50  0001 C CNN
-F 1 "GND" V 9455 5972 50  0000 R CNN
-F 2 "" H 9450 6100 50  0001 C CNN
-F 3 "" H 9450 6100 50  0001 C CNN
-	1    9450 6100
-	0    -1   -1   0
-$EndComp
 $Comp
 L Device:R R216
 U 1 1 5C437769
-P 8800 5450
-F 0 "R216" H 8870 5496 50  0000 L CNN
-F 1 "270" H 8870 5405 50  0000 L CNN
-F 2 "Resistor_SMD:R_0805_2012Metric_Pad1.15x1.40mm_HandSolder" V 8730 5450 50  0001 C CNN
-F 3 "https://datasheet.lcsc.com/szlcsc/C17590.pdf" H 8800 5450 50  0001 C CNN
-F 4 "" H 8800 5450 50  0001 C CNN "UnitCost(USD)"
-F 5 "0805W8F2700T5E" H 8800 5450 50  0001 C CNN "MPN"
-F 6 "" H 8800 5450 50  0001 C CNN "Manufacturer"
-F 7 "BASIC" H 8800 5450 50  0001 C CNN "JLCASM"
-F 8 "C17590" H 8800 5450 50  0001 C CNN "LCSC PN"
-	1    8800 5450
+P 9500 5400
+F 0 "R216" H 9570 5446 50  0000 L CNN
+F 1 "270" H 9570 5355 50  0000 L CNN
+F 2 "Resistor_SMD:R_0805_2012Metric_Pad1.15x1.40mm_HandSolder" V 9430 5400 50  0001 C CNN
+F 3 "https://datasheet.lcsc.com/szlcsc/C17590.pdf" H 9500 5400 50  0001 C CNN
+F 4 "" H 9500 5400 50  0001 C CNN "UnitCost(USD)"
+F 5 "0805W8F2700T5E" H 9500 5400 50  0001 C CNN "MPN"
+F 6 "" H 9500 5400 50  0001 C CNN "Manufacturer"
+F 7 "BASIC" H 9500 5400 50  0001 C CNN "JLCASM"
+F 8 "C17590" H 9500 5400 50  0001 C CNN "LCSC PN"
+	1    9500 5400
 	1    0    0    -1
 $EndComp
-Wire Wire Line
-	9450 6100 9350 6100
 Text GLabel 7900 3350 2    50   Input ~ 0
 +3V3_RASPI
 Text GLabel 7900 4500 2    50   Input ~ 0
 +3V3_RASPI
-Text GLabel 9450 5200 2    50   Input ~ 0
+Text GLabel 9700 5200 2    50   Input ~ 0
 +3V3_RASPI
 $Comp
@@
 F 8 "C6820" H 9500 3550 50  0001 C CNN "LCSC PN"
 	5    9500 3550
-	-1   0    0    1
-$EndComp
-$Comp
-L 74xx:74HC14 U205
-U 6 1 5C68F29D
-P 8400 7550
-F 0 "U205" H 8400 7233 50  0000 C CNN
-F 1 "SN74HC14" H 8400 7324 50  0000 C CNN
-F 2 "Package_SO:SOIC-14_3.9x8.7mm_P1.27mm" H 8400 7550 50  0001 C CNN
-F 3 "https://datasheet.lcsc.com/szlcsc/C6820.pdf" H 8400 7550 50  0001 C CNN
-F 4 "" H 8400 7550 12700 0001 C CNN "UnitCost(USD)"
-F 5 "SN74HC14DR" H 8400 7550 12700 0001 C CNN "MPN"
-F 6 "" H 8400 7550 12700 0001 C CNN "Manufacturer"
-F 7 "EXT" H 8400 7550 50  0001 C CNN "JLCASM"
-F 8 "C6820" H 8400 7550 50  0001 C CNN "LCSC PN"
-	6    8400 7550
 	-1   0    0    1
 $EndComp
@@
 	9100 3550 9200 3550
 Wire Wire Line
-	9800 4700 9900 4700
-Wire Wire Line
 	9900 3550 9800 3550
 Wire Wire Line
@@
 Wire Wire Line
 	8500 3550 7800 3550
-$Comp
-L power:GND #PWR0230
-U 1 1 5C6AE681
-P 8800 6950
-F 0 "#PWR0230" H 8800 6700 50  0001 C CNN
-F 1 "GND" V 8805 6822 50  0000 R CNN
-F 2 "" H 8800 6950 50  0001 C CNN
-F 3 "" H 8800 6950 50  0001 C CNN
-	1    8800 6950
-	0    -1   -1   0
-$EndComp
-$Comp
-L power:GND #PWR0232
-U 1 1 5C6AE711
-P 8800 7550
-F 0 "#PWR0232" H 8800 7300 50  0001 C CNN
-F 1 "GND" V 8805 7422 50  0000 R CNN
-F 2 "" H 8800 7550 50  0001 C CNN
-F 3 "" H 8800 7550 50  0001 C CNN
-	1    8800 7550
-	0    -1   -1   0
-$EndComp
-NoConn ~ 8100 6950
-NoConn ~ 8100 7550
-Wire Wire Line
-	8800 6950 8700 6950
-Wire Wire Line
-	8800 7550 8700 7550
-$Comp
-L Isolator:H11L1 U206
-U 1 1 5D2F89A3
-P 8400 5700
-F 0 "U206" H 8000 5350 50  0000 L CNN
-F 1 "H11L1S" H 8000 5250 50  0000 L CNN
-F 2 "Package_DIP:SMDIP-6_W7.62mm" H 8310 5700 50  0001 C CNN
-F 3 "https://datasheet.lcsc.com/szlcsc/C78589.pdf" H 8310 5700 50  0001 C CNN
-F 4 "" H 8400 5700 12700 0001 C CNN "UnitCost(USD)"
-F 5 "H11L1S(TA)" H 8400 5700 12700 0001 C CNN "MPN"
-F 6 "" H 8400 5700 12700 0001 C CNN "Manufacturer"
-F 7 "EXT" H 8400 5700 50  0001 C CNN "JLCASM"
-F 8 "C78589" H 8400 5700 50  0001 C CNN "LCSC PN"
-	1    8400 5700
-	1    0    0    -1
-$EndComp
 $Comp
 L Device:C_Small C?
 U 1 1 5D588BE8
-P 9350 5700
+P 8950 5200
 AR Path="/5C4320DF/5C4AB546/5D588BE8" Ref="C?"  Part="1"
 AR Path="/5C435D84/5D588BE8" Ref="C68"  Part="1"
-F 0 "C68" H 9258 5654 50  0000 R CNN
-F 1 "100nF" H 9258 5745 50  0000 R CNN
-F 2 "Capacitor_SMD:C_0805_2012Metric_Pad1.15x1.40mm_HandSolder" H 9350 5700 50  0001 C CNN
-F 3 "https://datasheet.lcsc.com/szlcsc/C49678.pdf" H 9350 5700 50  0001 C CNN
-F 4 "" H 9350 5700 12700 0001 C CNN "UnitCost(USD)"
-F 5 "CC0805KRX7R9BB104" H 9350 5700 12700 0001 C CNN "MPN"
-F 6 "" H 9350 5700 12700 0001 C CNN "Manufacturer"
-F 7 "C49678" H 9350 5700 50  0001 C CNN "LCSC PN"
-F 8 "BASIC" H 9350 5700 50  0001 C CNN "JLCASM"
-	1    9350 5700
+F 0 "C68" H 8858 5154 50  0000 R CNN
+F 1 "100nF" H 8858 5245 50  0000 R CNN
+F 2 "Capacitor_SMD:C_0805_2012Metric_Pad1.15x1.40mm_HandSolder" H 8950 5200 50  0001 C CNN
+F 3 "https://datasheet.lcsc.com/szlcsc/C49678.pdf" H 8950 5200 50  0001 C CNN
+F 4 "" H 8950 5200 12700 0001 C CNN "UnitCost(USD)"
+F 5 "CC0805KRX7R9BB104" H 8950 5200 12700 0001 C CNN "MPN"
+F 6 "" H 8950 5200 12700 0001 C CNN "Manufacturer"
+F 7 "C49678" H 8950 5200 50  0001 C CNN "LCSC PN"
+F 8 "BASIC" H 8950 5200 50  0001 C CNN "JLCASM"
+	1    8950 5200
 	-1   0    0    1
 $EndComp
-Wire Wire Line
-	8700 5700 8800 5700
-Wire Wire Line
-	8400 6000 8400 6100
-Wire Wire Line
-	8400 5200 8400 5400
-Wire Wire Line
-	8400 5200 8800 5200
-Wire Wire Line
-	8800 5300 8800 5200
-Connection ~ 8800 5200
-Wire Wire Line
-	8800 5200 9350 5200
-Wire Wire Line
-	8800 5600 8800 5700
-Connection ~ 8800 5700
-Wire Wire Line
-	8800 5700 8900 5700
-Wire Wire Line
-	9350 5600 9350 5200
-Connection ~ 9350 5200
-Wire Wire Line
-	9350 5200 9450 5200
-Wire Wire Line
-	9350 5800 9350 6100
-Connection ~ 9350 6100
-Wire Wire Line
-	9350 6100 8400 6100
 $Comp
 L OTTOdiy_SMD-library:AudioJack4_Switch-Connector-Connector TRS?
@@
 Text GLabel 9900 3550 2    50   Input ~ 0
 MIDI_OUT
-Text GLabel 9900 4700 2    50   Output ~ 0
-MIDI_IN
-Text GLabel 8900 5700 2    50   Output ~ 0
-MIDI_IN
 $Comp
 L 74xx:74HC14 U205
@@
 F 8 "C6820" H 8800 4700 50  0001 C CNN "LCSC PN"
 	3    8800 4700
-	-1   0    0    1
-$EndComp
-$Comp
-L 74xx:74HC14 U205
-U 1 1 5C68EFC4
-P 8400 6950
-F 0 "U205" H 8400 6633 50  0000 C CNN
-F 1 "SN74HC14" H 8400 6724 50  0000 C CNN
-F 2 "Package_SO:SOIC-14_3.9x8.7mm_P1.27mm" H 8400 6950 50  0001 C CNN
-F 3 "https://datasheet.lcsc.com/szlcsc/C6820.pdf" H 8400 6950 50  0001 C CNN
-F 4 "" H 8400 6950 12700 0001 C CNN "UnitCost(USD)"
-F 5 "SN74HC14DR" H 8400 6950 12700 0001 C CNN "MPN"
-F 6 "" H 8400 6950 12700 0001 C CNN "Manufacturer"
-F 7 "EXT" H 8400 6950 50  0001 C CNN "JLCASM"
-F 8 "C6820" H 8400 6950 50  0001 C CNN "LCSC PN"
-	1    8400 6950
 	-1   0    0    1
 $EndComp
@@
 	7850 5250 7750 5250
 NoConn ~ 6750 5500
+$Comp
+L Isolator:6N137 U201
+U 1 1 5E817B20
+P 8400 5600
+F 0 "U201" H 8400 6067 50  0000 C CNN
+F 1 "6N137" H 8400 5976 50  0000 C CNN
+F 2 "Package_DIP:DIP-8_W8.89mm_SMDSocket_LongPads" H 8400 5100 50  0001 C CNN
+F 3 "https://docs.broadcom.com/docs/AV02-0940EN" H 7550 6150 50  0001 C CNN
+F 4 "BASIC" H 8400 5600 50  0001 C CNN "JLCASM"
+F 5 "C110020" H 8400 5600 50  0001 C CNN "LCSC PN"
+F 6 "6N137S1(TA)" H 8400 5600 50  0001 C CNN "MPN"
+	1    8400 5600
+	1    0    0    -1
+$EndComp
+Wire Wire Line
+	8700 5400 8750 5400
+Text GLabel 9700 5000 2    50   Input ~ 0
++5V_RASPI
+Wire Wire Line
+	8750 5000 8750 5400
+NoConn ~ 8700 5500
+Wire Wire Line
+	8700 5600 9500 5600
+Connection ~ 9500 5600
+Wire Wire Line
+	9700 5200 9500 5200
+Wire Wire Line
+	9500 5200 9500 5250
+Wire Wire Line
+	9500 5550 9500 5600
+Wire Wire Line
+	8750 5000 8950 5000
+Wire Wire Line
+	8950 5100 8950 5000
+Connection ~ 8950 5000
+Wire Wire Line
+	8950 5000 9700 5000
+Wire Wire Line
+	8800 7550 8700 7550
+Wire Wire Line
+	8800 6950 8700 6950
+NoConn ~ 8100 7550
+NoConn ~ 8100 6950
+$Comp
+L power:GND #PWR0232
+U 1 1 5C6AE711
+P 8800 7550
+F 0 "#PWR0232" H 8800 7300 50  0001 C CNN
+F 1 "GND" V 8805 7422 50  0000 R CNN
+F 2 "" H 8800 7550 50  0001 C CNN
+F 3 "" H 8800 7550 50  0001 C CNN
+	1    8800 7550
+	0    -1   -1   0
+$EndComp
+$Comp
+L power:GND #PWR0230
+U 1 1 5C6AE681
+P 8800 6950
+F 0 "#PWR0230" H 8800 6700 50  0001 C CNN
+F 1 "GND" V 8805 6822 50  0000 R CNN
+F 2 "" H 8800 6950 50  0001 C CNN
+F 3 "" H 8800 6950 50  0001 C CNN
+	1    8800 6950
+	0    -1   -1   0
+$EndComp
+$Comp
+L 74xx:74HC14 U205
+U 6 1 5C68F29D
+P 8400 7550
+F 0 "U205" H 8400 7233 50  0000 C CNN
+F 1 "SN74HC14" H 8400 7324 50  0000 C CNN
+F 2 "Package_SO:SOIC-14_3.9x8.7mm_P1.27mm" H 8400 7550 50  0001 C CNN
+F 3 "https://datasheet.lcsc.com/szlcsc/C6820.pdf" H 8400 7550 50  0001 C CNN
+F 4 "" H 8400 7550 12700 0001 C CNN "UnitCost(USD)"
+F 5 "SN74HC14DR" H 8400 7550 12700 0001 C CNN "MPN"
+F 6 "" H 8400 7550 12700 0001 C CNN "Manufacturer"
+F 7 "EXT" H 8400 7550 50  0001 C CNN "JLCASM"
+F 8 "C6820" H 8400 7550 50  0001 C CNN "LCSC PN"
+	6    8400 7550
+	-1   0    0    1
+$EndComp
+$Comp
+L 74xx:74HC14 U205
+U 1 1 5C68EFC4
+P 8400 6950
+F 0 "U205" H 8400 6633 50  0000 C CNN
+F 1 "SN74HC14" H 8400 6724 50  0000 C CNN
+F 2 "Package_SO:SOIC-14_3.9x8.7mm_P1.27mm" H 8400 6950 50  0001 C CNN
+F 3 "https://datasheet.lcsc.com/szlcsc/C6820.pdf" H 8400 6950 50  0001 C CNN
+F 4 "" H 8400 6950 12700 0001 C CNN "UnitCost(USD)"
+F 5 "SN74HC14DR" H 8400 6950 12700 0001 C CNN "MPN"
+F 6 "" H 8400 6950 12700 0001 C CNN "Manufacturer"
+F 7 "EXT" H 8400 6950 50  0001 C CNN "JLCASM"
+F 8 "C6820" H 8400 6950 50  0001 C CNN "LCSC PN"
+	1    8400 6950
+	-1   0    0    1
+$EndComp
+Wire Wire Line
+	9500 5600 9900 5600
+Wire Wire Line
+	9800 4700 9900 4700
+Text GLabel 9900 4700 2    50   Output ~ 0
+MIDI_IN
+Text GLabel 9900 5600 2    50   Output ~ 0
+MIDI_IN
+Wire Wire Line
+	8950 5800 8950 5300
+Wire Wire Line
+	8700 5800 8950 5800
+$Comp
+L power:GND #PWR0201
+U 1 1 5E9AEA27
+P 8950 5900
+F 0 "#PWR0201" H 8950 5650 50  0001 C CNN
+F 1 "GND" H 8955 5727 50  0000 C CNN
+F 2 "" H 8950 5900 50  0001 C CNN
+F 3 "" H 8950 5900 50  0001 C CNN
+	1    8950 5900
+	1    0    0    -1
+$EndComp
+Wire Wire Line
+	8950 5900 8950 5800
+Connection ~ 8950 5800
 $EndSCHEMATC

Commit message: Fix DAC footprint and other minor issues.
Parts:
- U201: footprint Package_DIP:DIP-8_W8.89mm_SMDSocket_LongPads -> OTTO_Footprints_Lib:DIP-8_W8.89mm_SMDSocket_LongPads
- U205: footprint Package_SO:SOIC-14_3.9x8.7mm_P1.27mm -> OTTO_Footprints_Lib:SOIC-14_3.9x8.7mm_P1.27mm
Changed lines of the file:
@@
 F 0 "U205" H 8800 3233 50  0000 C CNN
 F 1 "SN74HC14" H 8800 3324 50  0000 C CNN
-F 2 "Package_SO:SOIC-14_3.9x8.7mm_P1.27mm" H 8800 3550 50  0001 C CNN
+F 2 "OTTO_Footprints_Lib:SOIC-14_3.9x8.7mm_P1.27mm" H 8800 3550 50  0001 C CNN
 F 3 "https://datasheet.lcsc.com/szlcsc/C6820.pdf" H 8800 3550 50  0001 C CNN
 F 4 "" H 8800 3550 12700 0001 C CNN "UnitCost(USD)"
@@
 F 0 "U205" H 9500 3233 50  0000 C CNN
 F 1 "SN74HC14" H 9500 3324 50  0000 C CNN
-F 2 "Package_SO:SOIC-14_3.9x8.7mm_P1.27mm" H 9500 3550 50  0001 C CNN
+F 2 "OTTO_Footprints_Lib:SOIC-14_3.9x8.7mm_P1.27mm" H 9500 3550 50  0001 C CNN
 F 3 "https://datasheet.lcsc.com/szlcsc/C6820.pdf" H 9500 3550 50  0001 C CNN
 F 4 "" H 9500 3550 12700 0001 C CNN "UnitCost(USD)"
@@
 F 0 "U205" V 6867 7500 50  0000 C CNN
 F 1 "SN74HC14" V 6776 7500 50  0000 C CNN
-F 2 "Package_SO:SOIC-14_3.9x8.7mm_P1.27mm" H 6500 7500 50  0001 C CNN
+F 2 "OTTO_Footprints_Lib:SOIC-14_3.9x8.7mm_P1.27mm" H 6500 7500 50  0001 C CNN
 F 3 "https://datasheet.lcsc.com/szlcsc/C6820.pdf" H 6500 7500 50  0001 C CNN
 F 4 "" H 6500 7500 12700 0001 C CNN "UnitCost(USD)"
@@
 F 0 "U205" H 9500 4383 50  0000 C CNN
 F 1 "SN74HC14" H 9500 4474 50  0000 C CNN
-F 2 "Package_SO:SOIC-14_3.9x8.7mm_P1.27mm" H 9500 4700 50  0001 C CNN
+F 2 "OTTO_Footprints_Lib:SOIC-14_3.9x8.7mm_P1.27mm" H 9500 4700 50  0001 C CNN
 F 3 "https://datasheet.lcsc.com/szlcsc/C6820.pdf" H 9500 4700 50  0001 C CNN
 F 4 "" H 9500 4700 12700 0001 C CNN "UnitCost(USD)"
@@
 F 0 "U205" H 8800 4383 50  0000 C CNN
 F 1 "SN74HC14" H 8800 4474 50  0000 C CNN
-F 2 "Package_SO:SOIC-14_3.9x8.7mm_P1.27mm" H 8800 4700 50  0001 C CNN
+F 2 "OTTO_Footprints_Lib:SOIC-14_3.9x8.7mm_P1.27mm" H 8800 4700 50  0001 C CNN
 F 3 "https://datasheet.lcsc.com/szlcsc/C6820.pdf" H 8800 4700 50  0001 C CNN
 F 4 "" H 8800 4700 12700 0001 C CNN "UnitCost(USD)"
@@
 F 0 "U201" H 8400 6067 50  0000 C CNN
 F 1 "6N137" H 8400 5976 50  0000 C CNN
-F 2 "Package_DIP:DIP-8_W8.89mm_SMDSocket_LongPads" H 8400 5100 50  0001 C CNN
+F 2 "OTTO_Footprints_Lib:DIP-8_W8.89mm_SMDSocket_LongPads" H 8400 5100 50  0001 C CNN
 F 3 "https://docs.broadcom.com/docs/AV02-0940EN" H 7550 6150 50  0001 C CNN
 F 4 "BASIC" H 8400 5600 50  0001 C CNN "JLCASM"
@@
 F 0 "U205" H 8400 7233 50  0000 C CNN
 F 1 "SN74HC14" H 8400 7324 50  0000 C CNN
-F 2 "Package_SO:SOIC-14_3.9x8.7mm_P1.27mm" H 8400 7550 50  0001 C CNN
+F 2 "OTTO_Footprints_Lib:SOIC-14_3.9x8.7mm_P1.27mm" H 8400 7550 50  0001 C CNN
 F 3 "https://datasheet.lcsc.com/szlcsc/C6820.pdf" H 8400 7550 50  0001 C CNN
 F 4 "" H 8400 7550 12700 0001 C CNN "UnitCost(USD)"
@@
 F 0 "U205" H 8400 6633 50  0000 C CNN
 F 1 "SN74HC14" H 8400 6724 50  0000 C CNN
-F 2 "Package_SO:SOIC-14_3.9x8.7mm_P1.27mm" H 8400 6950 50  0001 C CNN
+F 2 "OTTO_Footprints_Lib:SOIC-14_3.9x8.7mm_P1.27mm" H 8400 6950 50  0001 C CNN
 F 3 "https://datasheet.lcsc.com/szlcsc/C6820.pdf" H 8400 6950 50  0001 C CNN
 F 4 "" H 8400 6950 12700 0001 C CNN "UnitCost(USD)"
