File: KiCad/MIDI.sch (KiCad schematic (older format))
At the start: 15 parts, among them U201 6N137, U205 SN74HC14

Commit message: Main board v0.1.0 as ordered
Parts:
- U201: footprint OTTO_Footprints_Lib:DIP-8_W8.89mm_SMDSocket_LongPads -> Package_DIP:DIP-8_W8.89mm_SMDSocket_LongPads
Changed lines of the file:
@@
 F 0 "U201" H 8400 6067 50  0000 C CNN
 F 1 "6N137" H 8400 5976 50  0000 C CNN
-F 2 "OTTO_Footprints_Lib:DIP-8_W8.89mm_SMDSocket_LongPads" H 8400 5100 50  0001 C CNN
+F 2 "Package_DIP:DIP-8_W8.89mm_SMDSocket_LongPads" H 8400 5100 50  0001 C CNN
 F 3 "https://datasheet.lcsc.com/szlcsc/C110020.pdf" H 7550 6150 50  0001 C CNN
 F 4 "BASIC" H 8400 5600 50  0001 C CNN "JLCASM"
