File: KiCad/KEYS+ENCODERS.sch (KiCad schematic (older format))
At the start: 110 parts, among them SW1 ALPS SKHC, SW10 ALPS SKHC, SW11 ALPS SKHC, SW12 ALPS SKHC, SW13 ALPS SKHC, SW14 ALPS SKHC, SW15 ALPS SKHC, SW16 ALPS SKHC, SW17 ALPS SKHC, SW18 ALPS SKHC, SW19 ALPS SKHC, SW2 ALPS SKHC, SW20 ALPS SKHC, SW21 ALPS SKHC, SW22 ALPS SKHC, SW23 ALPS SKHC, SW24 ALPS SKHC, SW25 ALPS SKHC, SW26 ALPS SKHC, SW27 6x6x13mm, SW28 6x6x13mm, SW29 6x6x13mm, SW3 ALPS SKHC, SW30 6x6x13mm, SW31 6x6x13mm, SW32 6x6x13mm, SW33 6x6x13mm, SW34 6x6x13mm, SW35 6x6x13mm, SW36 6x6x13mm, SW37 6x6x13mm, SW38 6x6x13mm, SW39 6x6x13mm, SW4 ALPS SKHC, SW40 6x6x13mm, SW41 6x6x13mm, SW42 6x6x13mm, SW43 6x6x13mm, SW44 6x6x13mm, SW45 6x6x13mm, SW46 6x6x13mm, SW47 6x6x13mm, SW5 ALPS SKHC, SW6 ALPS SKHC, SW7 ALPS SKHC, SW8 ALPS SKHC, SW9 ALPS SKHC

Commit message: roll in changes from Bastian
Connections:
- wire segments 232 -> 239
Changed lines of the file:
@@
 Wire Wire Line
 	9250 4350 8850 4350
-Wire Wire Line
-	8850 4650 8950 4650
-Wire Wire Line
-	9650 4750 9550 4750
 $Comp
 L Device:D_ALT D41
@@
 Wire Wire Line
 	9250 3200 8850 3200
-Wire Wire Line
-	8850 3500 8950 3500
-Wire Wire Line
-	9650 3600 9550 3600
 $Comp
 L Device:D_ALT D33
@@
 Wire Wire Line
 	13050 3200 12650 3200
-Wire Wire Line
-	12650 3500 12750 3500
-Wire Wire Line
-	13450 3600 13350 3600
 $Comp
 L Device:D_ALT D38
@@
 Wire Wire Line
 	12100 3200 11700 3200
-Wire Wire Line
-	11700 3500 11800 3500
-Wire Wire Line
-	12500 3600 12400 3600
 $Comp
 L Device:D_ALT D37
@@
 Wire Wire Line
 	11150 3200 10750 3200
-Wire Wire Line
-	10750 3500 10850 3500
 $Comp
 L Device:D_ALT D36
@@
 Wire Wire Line
 	10200 3200 9800 3200
-Wire Wire Line
-	9800 3500 9900 3500
-Wire Wire Line
-	10600 3600 10500 3600
 $Comp
 L Device:D_ALT D35
@@
 	10200 4350 9800 4350
 Wire Wire Line
-	9800 4650 9900 4650
-Wire Wire Line
-	10600 4750 10500 4750
+	9800 4650 9800 4750
+Wire Wire Line
+	10600 4750 10550 4750
 Wire Wire Line
 	1550 7850 1550 8250
@@
 $EndComp
 Wire Wire Line
-	9650 3200 9650 3600
-Wire Wire Line
 	9650 4350 9650 4750
 Wire Wire Line
@@
 	10600 4350 10600 4750
 Wire Wire Line
-	10600 3200 10600 3600
-Wire Wire Line
 	10600 5450 10600 5850
 $Comp
@@
 	11550 5450 11550 5850
 Wire Wire Line
-	11550 3200 11550 3600
-Wire Wire Line
 	11550 4350 11550 4750
 Wire Wire Line
 	12500 5450 12500 5850
 Wire Wire Line
-	12500 3200 12500 3600
-Wire Wire Line
 	12500 4350 12500 4750
 Wire Wire Line
 	13450 5450 13450 5850
-Wire Wire Line
-	13450 3200 13450 3600
 Wire Wire Line
 	13450 4350 13450 4750
@@
 Text HLabel 15700 8500 0    50   Input ~ 0
 COL_4
-Text HLabel 9550 3850 0    50   Input ~ 0
+Text HLabel 9600 3650 0    50   Input ~ 0
 COL_4
-Text HLabel 9550 4950 0    50   Input ~ 0
+Text HLabel 9600 4750 0    50   Input ~ 0
 COL_4
 Text HLabel 9550 6050 0    50   Input ~ 0
 COL_4
-Text HLabel 8950 3750 2    50   Input ~ 0
+Text HLabel 8900 3650 2    50   Input ~ 0
 ROW_1
-Text HLabel 8950 4850 2    50   Input ~ 0
+Text HLabel 8900 4750 2    50   Input ~ 0
 ROW_2
 Text HLabel 8950 5950 2    50   Input ~ 0
@@
 Text HLabel 15100 3750 2    50   Input ~ 0
 ROW_8
-Text HLabel 10500 3850 0    50   Input ~ 0
+Text HLabel 10550 3650 0    50   Input ~ 0
 COL_5
-Text HLabel 11450 3850 0    50   Input ~ 0
+Text HLabel 11500 3650 0    50   Input ~ 0
 COL_5
-Text HLabel 12400 3850 0    50   Input ~ 0
+Text HLabel 12450 3650 0    50   Input ~ 0
 COL_5
-Text HLabel 13350 3850 0    50   Input ~ 0
+Text HLabel 13400 3650 0    50   Input ~ 0
 COL_5
 Text HLabel 11450 4950 0    50   Input ~ 0
@@
 Text HLabel 12400 4950 0    50   Input ~ 0
 COL_5
-Text HLabel 10500 4950 0    50   Input ~ 0
+Text HLabel 10550 4750 0    50   Input ~ 0
 COL_5
 Text HLabel 14750 4950 0    50   Input ~ 0
@@
 Text HLabel 12750 4850 2    50   Input ~ 0
 ROW_7
-Text HLabel 11800 3750 2    50   Input ~ 0
+Text HLabel 11750 3650 2    50   Input ~ 0
 ROW_6
 Text HLabel 11800 4850 2    50   Input ~ 0
 ROW_5
-Text HLabel 10850 3750 2    50   Input ~ 0
+Text HLabel 10800 3650 2    50   Input ~ 0
 ROW_4
-Text HLabel 9900 4850 2    50   Input ~ 0
+Text HLabel 9850 4750 2    50   Input ~ 0
 ROW_2
 Text HLabel 10850 4850 2    50   Input ~ 0
 ROW_3
-Text HLabel 12750 3750 2    50   Input ~ 0
+Text HLabel 12700 3650 2    50   Input ~ 0
 ROW_8
 Text HLabel 14750 3850 0    50   Input ~ 0
 COL_6
-Text HLabel 9900 3750 2    50   Input ~ 0
+Text HLabel 9850 3650 2    50   Input ~ 0
 ROW_1
 Text HLabel 13350 4950 0    50   Input ~ 0
@@
 Wire Wire Line
 	7400 4200 7500 4200
-Text HLabel 7950 5150 2    50   Input ~ 0
+Text HLabel 7900 5150 2    50   Input ~ 0
 ROW_4
 Wire Wire Line
 	7900 5150 7800 5150
-Text HLabel 4100 5150 2    50   Input ~ 0
+Text HLabel 4050 5150 2    50   Input ~ 0
 ROW_7
 Wire Wire Line
 	7900 4200 7800 4200
-Text HLabel 7950 4200 2    50   Input ~ 0
+Text HLabel 7900 4200 2    50   Input ~ 0
 ROW_2
-Text HLabel 4100 4200 2    50   Input ~ 0
+Text HLabel 4050 4200 2    50   Input ~ 0
 ROW_1
 Wire Wire Line
 	4050 4200 3950 4200
-Wire Wire Line
-	11450 3600 11550 3600
 Wire Wire Line
 	11450 4750 11550 4750
@@
 Text HLabel 2300 7150 2    50   Input ~ 0
 ROW_1
+Wire Wire Line
+	9650 3200 9650 3650
+Wire Wire Line
+	9650 3650 9600 3650
+Wire Wire Line
+	8850 3500 8850 3650
+Wire Wire Line
+	8850 3650 8900 3650
+Wire Wire Line
+	9800 3500 9800 3650
+Wire Wire Line
+	10600 3650 10550 3650
+Wire Wire Line
+	10600 3200 10600 3650
+Wire Wire Line
+	9850 3650 9800 3650
+Wire Wire Line
+	11550 3650 11500 3650
+Wire Wire Line
+	11550 3200 11550 3650
+Wire Wire Line
+	10750 3500 10750 3650
+Wire Wire Line
+	10750 3650 10800 3650
+Wire Wire Line
+	11700 3500 11700 3650
+Wire Wire Line
+	11700 3650 11750 3650
+Wire Wire Line
+	12450 3650 12500 3650
+Wire Wire Line
+	12500 3200 12500 3650
+Wire Wire Line
+	12650 3500 12650 3650
+Wire Wire Line
+	12650 3650 12700 3650
+Wire Wire Line
+	13450 3650 13400 3650
+Wire Wire Line
+	13450 3200 13450 3650
+Wire Wire Line
+	9650 4750 9600 4750
+Wire Wire Line
+	8900 4750 8850 4750
+Wire Wire Line
+	8850 4750 8850 4650
+Wire Wire Line
+	9800 4750 9850 4750
 $EndSCHEMATC

Commit message: added power switching and extra pulls for programming lines
Connections:
- wire segments 239 -> 279

Commit message: added part numbers for capacitors and crystals
Parts:
- C60, C61, C62, C63, C64, C65, C66, C67: footprint Capacitor_SMD:C_0805_2012Metric_Pad1.15x1.40mm_HandSolder_marked -> Capacitor_SMD:C_0805_2012Metric_Pad1.15x1.40mm_HandSolder; EstimatedCost(USD) (none) -> $0.017724; MPN (none) -> CL21B104JBCNNNC; Manufacturer (none) -> Samsung Electro-Mechanics
Changed lines of the file:
@@
 F 0 "C60" H 2642 4046 50  0000 L CNN
 F 1 "100nF" H 2642 3955 50  0000 L CNN
-F 2 "Capacitor_SMD:C_0805_2012Metric_Pad1.15x1.40mm_HandSolder_marked" H 2550 4000 50  0001 C CNN
-F 3 "~" H 2550 4000 50  0001 C CNN
+F 2 "Capacitor_SMD:C_0805_2012Metric_Pad1.15x1.40mm_HandSolder" H 2550 4000 50  0001 C CNN
+F 3 "https://datasheet.lcsc.com/szlcsc/Samsung-Electro-Mechanics-CL21B104JBCNNNC_C62912.pdf" H 2550 4000 50  0001 C CNN
+F 4 "$0.017724" H 2550 4000 12700 0001 C CNN "EstimatedCost(USD)"
+F 5 "CL21B104JBCNNNC" H 2550 4000 12700 0001 C CNN "MPN"
+F 6 "Samsung Electro-Mechanics" H 2550 4000 12700 0001 C CNN "Manufacturer"
 	1    2550 4000
 	1    0    0    -1
@@
 F 0 "C61" H 2642 4246 50  0000 L CNN
 F 1 "100nF" H 2642 4155 50  0000 L CNN
-F 2 "Capacitor_SMD:C_0805_2012Metric_Pad1.15x1.40mm_HandSolder_marked" H 2550 4200 50  0001 C CNN
-F 3 "~" H 2550 4200 50  0001 C CNN
+F 2 "Capacitor_SMD:C_0805_2012Metric_Pad1.15x1.40mm_HandSolder" H 2550 4200 50  0001 C CNN
+F 3 "https://datasheet.lcsc.com/szlcsc/Samsung-Electro-Mechanics-CL21B104JBCNNNC_C62912.pdf" H 2550 4200 50  0001 C CNN
+F 4 "$0.017724" H 2550 4200 12700 0001 C CNN "EstimatedCost(USD)"
+F 5 "CL21B104JBCNNNC" H 2550 4200 12700 0001 C CNN "MPN"
+F 6 "Samsung Electro-Mechanics" H 2550 4200 12700 0001 C CNN "Manufacturer"
 	1    2550 4200
 	1    0    0    -1
@@
 F 0 "C62" H 2642 4996 50  0000 L CNN
 F 1 "100nF" H 2642 4905 50  0000 L CNN
-F 2 "Capacitor_SMD:C_0805_2012Metric_Pad1.15x1.40mm_HandSolder_marked" H 2550 4950 50  0001 C CNN
-F 3 "~" H 2550 4950 50  0001 C CNN
+F 2 "Capacitor_SMD:C_0805_2012Metric_Pad1.15x1.40mm_HandSolder" H 2550 4950 50  0001 C CNN
+F 3 "https://datasheet.lcsc.com/szlcsc/Samsung-Electro-Mechanics-CL21B104JBCNNNC_C62912.pdf" H 2550 4950 50  0001 C CNN
+F 4 "$0.017724" H 2550 4950 12700 0001 C CNN "EstimatedCost(USD)"
+F 5 "CL21B104JBCNNNC" H 2550 4950 12700 0001 C CNN "MPN"
+F 6 "Samsung Electro-Mechanics" H 2550 4950 12700 0001 C CNN "Manufacturer"
 	1    2550 4950
 	1    0    0    -1
@@
 F 0 "C63" H 2642 5196 50  0000 L CNN
 F 1 "100nF" H 2642 5105 50  0000 L CNN
-F 2 "Capacitor_SMD:C_0805_2012Metric_Pad1.15x1.40mm_HandSolder_marked" H 2550 5150 50  0001 C CNN
-F 3 "~" H 2550 5150 50  0001 C CNN
+F 2 "Capacitor_SMD:C_0805_2012Metric_Pad1.15x1.40mm_HandSolder" H 2550 5150 50  0001 C CNN
+F 3 "https://datasheet.lcsc.com/szlcsc/Samsung-Electro-Mechanics-CL21B104JBCNNNC_C62912.pdf" H 2550 5150 50  0001 C CNN
+F 4 "$0.017724" H 2550 5150 12700 0001 C CNN "EstimatedCost(USD)"
+F 5 "CL21B104JBCNNNC" H 2550 5150 12700 0001 C CNN "MPN"
+F 6 "Samsung Electro-Mechanics" H 2550 5150 12700 0001 C CNN "Manufacturer"
 	1    2550 5150
 	1    0    0    -1
@@
 F 0 "C64" H 6492 4046 50  0000 L CNN
 F 1 "100nF" H 6492 3955 50  0000 L CNN
-F 2 "Capacitor_SMD:C_0805_2012Metric_Pad1.15x1.40mm_HandSolder_marked" H 6400 4000 50  0001 C CNN
-F 3 "~" H 6400 4000 50  0001 C CNN
+F 2 "Capacitor_SMD:C_0805_2012Metric_Pad1.15x1.40mm_HandSolder" H 6400 4000 50  0001 C CNN
+F 3 "https://datasheet.lcsc.com/szlcsc/Samsung-Electro-Mechanics-CL21B104JBCNNNC_C62912.pdf" H 6400 4000 50  0001 C CNN
+F 4 "$0.017724" H 6400 4000 12700 0001 C CNN "EstimatedCost(USD)"
+F 5 "CL21B104JBCNNNC" H 6400 4000 12700 0001 C CNN "MPN"
+F 6 "Samsung Electro-Mechanics" H 6400 4000 12700 0001 C CNN "Manufacturer"
 	1    6400 4000
 	1    0    0    -1
@@
 F 0 "C65" H 6492 4246 50  0000 L CNN
 F 1 "100nF" H 6492 4155 50  0000 L CNN
-F 2 "Capacitor_SMD:C_0805_2012Metric_Pad1.15x1.40mm_HandSolder_marked" H 6400 4200 50  0001 C CNN
-F 3 "~" H 6400 4200 50  0001 C CNN
+F 2 "Capacitor_SMD:C_0805_2012Metric_Pad1.15x1.40mm_HandSolder" H 6400 4200 50  0001 C CNN
+F 3 "https://datasheet.lcsc.com/szlcsc/Samsung-Electro-Mechanics-CL21B104JBCNNNC_C62912.pdf" H 6400 4200 50  0001 C CNN
+F 4 "$0.017724" H 6400 4200 12700 0001 C CNN "EstimatedCost(USD)"
+F 5 "CL21B104JBCNNNC" H 6400 4200 12700 0001 C CNN "MPN"
+F 6 "Samsung Electro-Mechanics" H 6400 4200 12700 0001 C CNN "Manufacturer"
 	1    6400 4200
 	1    0    0    -1
@@
 F 0 "C66" H 6492 4996 50  0000 L CNN
 F 1 "100nF" H 6492 4905 50  0000 L CNN
-F 2 "Capacitor_SMD:C_0805_2012Metric_Pad1.15x1.40mm_HandSolder_marked" H 6400 4950 50  0001 C CNN
-F 3 "~" H 6400 4950 50  0001 C CNN
+F 2 "Capacitor_SMD:C_0805_2012Metric_Pad1.15x1.40mm_HandSolder" H 6400 4950 50  0001 C CNN
+F 3 "https://datasheet.lcsc.com/szlcsc/Samsung-Electro-Mechanics-CL21B104JBCNNNC_C62912.pdf" H 6400 4950 50  0001 C CNN
+F 4 "$0.017724" H 6400 4950 12700 0001 C CNN "EstimatedCost(USD)"
+F 5 "CL21B104JBCNNNC" H 6400 4950 12700 0001 C CNN "MPN"
+F 6 "Samsung Electro-Mechanics" H 6400 4950 12700 0001 C CNN "Manufacturer"
 	1    6400 4950
 	1    0    0    -1
@@
 F 0 "C67" H 6492 5196 50  0000 L CNN
 F 1 "100nF" H 6492 5105 50  0000 L CNN
-F 2 "Capacitor_SMD:C_0805_2012Metric_Pad1.15x1.40mm_HandSolder_marked" H 6400 5150 50  0001 C CNN
-F 3 "~" H 6400 5150 50  0001 C CNN
+F 2 "Capacitor_SMD:C_0805_2012Metric_Pad1.15x1.40mm_HandSolder" H 6400 5150 50  0001 C CNN
+F 3 "https://datasheet.lcsc.com/szlcsc/Samsung-Electro-Mechanics-CL21B104JBCNNNC_C62912.pdf" H 6400 5150 50  0001 C CNN
+F 4 "$0.017724" H 6400 5150 12700 0001 C CNN "EstimatedCost(USD)"
+F 5 "CL21B104JBCNNNC" H 6400 5150 12700 0001 C CNN "MPN"
+F 6 "Samsung Electro-Mechanics" H 6400 5150 12700 0001 C CNN "Manufacturer"
 	1    6400 5150
 	1    0    0    -1

Commit message: add more part numbers, samtec connector footprint
Parts:
- D1, D10, D11, D12, D13, D14, D15, D16, D17, D18, D19, D2, D20, D202, D203, D204, D205, D21, D22, D23, D24, D25, D26, D27, D28, D29, D3, D30, D31, D32, D33, D34, D35, D36, D37, D38, D39, D4, D40, D41, D42, D43, D44, D45, D46, D47, D5, D6, D7, D8, D9: value M7 -> SM4007PL; footprint Diode_SMD:D_SMA -> Diode_SMD:D_SOD-123F; EstimatedCost(USD) (none) -> $0.00574; MPN (none) -> SM4007PL; Manufacturer (none) -> MDD(Microdiode Electronics)
- ENC1, ENC2, ENC3, ENC4: footprint Spatz:ALPS EC11 -> OTTO_Footprints_Lib:ALPS_EC11; EstimatedCost(USD) (none) -> $1.910606; MPN (none) -> EC11E18244AU; Manufacturer (none) -> ALPS Electric

Commit message: add switch and encoder parts. BM Complete. Footprints complete.
Parts:
- SW1, SW10, SW11, SW12, SW13, SW14, SW15, SW16, SW17, SW18, SW19, SW2, SW20, SW21, SW22, SW23, SW24, SW25, SW26, SW3, SW4, SW5, SW6, SW7, SW8, SW9: footprint Spatz:6x6mm_Switch_LargeCap -> OTTO_Footprints_Lib:ALPS_SKHC; EstimatedCost(USD) (none) -> $0.143939; MPN (none) -> SKHCBEA010; Manufacturer (none) -> ALPS Electric
- SW27, SW28, SW29, SW30, SW31, SW32, SW33, SW34, SW35, SW36, SW37, SW38, SW39, SW40, SW41, SW42, SW43, SW44, SW45, SW46, SW47: value 6x6x13mm -> 6x6x12.5mm; footprint Spatz:6x6mm_Switch -> OTTO_Footprints_Lib:6x6mm_Switch; EstimatedCost(USD) (none) -> $0.053035; MPN (none) -> K2-6639DP-R4SW-04; Manufacturer (none) -> Korean Hroparts Elec

Commit message: add BOM scripts, fix schematic hierarchy
Parts:
- C60, C61, C62, C63, C64, C65, C66, C67: EstimatedCost(USD) $0.017724 -> (none); UnitCost(USD) (none) -> $0.017724
- D1, D10, D11, D12, D13, D14, D15, D16, D17, D18, D19, D2, D20, D202, D203, D204, D205, D21, D22, D23, D24, D25, D26, D27, D28, D29, D3, D30, D31, D32, D33, D34, D35, D36, D37, D38, D39, D4, D40, D41, D42, D43, D44, D45, D46, D47, D5, D6, D7, D8, D9: EstimatedCost(USD) $0.00574 -> (none); UnitCost(USD) (none) -> $0.00574
- ENC1, ENC2, ENC3, ENC4: EstimatedCost(USD) $1.910606 -> (none); UnitCost(USD) (none) -> $1.910606
- SW1, SW10, SW11, SW12, SW13, SW14, SW15, SW16, SW17, SW18, SW19, SW2, SW20, SW21, SW22, SW23, SW24, SW25, SW26, SW3, SW4, SW5, SW6, SW7, SW8, SW9: EstimatedCost(USD) $0.143939 -> (none); UnitCost(USD) (none) -> $0.143939
- SW27, SW28, SW29, SW30, SW31, SW32, SW33, SW34, SW35, SW36, SW37, SW38, SW39, SW40, SW41, SW42, SW43, SW44, SW45, SW46, SW47: EstimatedCost(USD) $0.053035 -> (none); UnitCost(USD) (none) -> $0.053035

Commit message: Add power switch and other misc nice to haves
Parts:
- SW1, SW10, SW11, SW12, SW13, SW14, SW15, SW16, SW17, SW18, SW19, SW2, SW20, SW21, SW22, SW23, SW24, SW25, SW26, SW3, SW4, SW5, SW6, SW7, SW8, SW9: value ALPS SKHC -> ALPS SKHH OR SKPF; footprint OTTO_Footprints_Lib:ALPS_SKHC -> OTTO_Footprints_Lib:6x6mm_Switch_LargeCap_ALT_SKPF; MPN SKHCBEA010 -> SKHHDTA010; UnitCost(USD) $0.143939 -> $0.168182
- SW27, SW28, SW29, SW30, SW31, SW32, SW33, SW34, SW35, SW36, SW37, SW38, SW39, SW40, SW41, SW42, SW43, SW44, SW45, SW46, SW47: value 6x6x12.5mm -> 6x6x13mm; MPN K2-6639DP-R4SW-04 -> SKHHDTA010; Manufacturer Korean Hroparts Elec -> ALPS Electric; UnitCost(USD) $0.053035 -> $0.168182

Commit message: routed buck boost supply
Parts:
- SW27, SW28, SW29, SW30, SW31, SW32, SW33, SW34, SW35, SW36, SW37, SW38, SW39, SW40, SW41, SW42, SW43, SW44, SW45, SW46, SW47: MPN SKHHDTA010 -> K2-1102DP-S3SW-04; Manufacturer ALPS Electric -> Korean Hroparts Elec; UnitCost(USD) $0.168182 -> $0.043333
