File: KiCad/KEYS+ENCODERS.sch (KiCad schematic (older format))
At the start: 110 parts, among them SW1 ALPS SKHH OR SKPF, SW10 ALPS SKHH OR SKPF, SW11 ALPS SKHH OR SKPF, SW12 ALPS SKHH OR SKPF, SW13 ALPS SKHH OR SKPF, SW14 ALPS SKHH OR SKPF, SW15 ALPS SKHH OR SKPF, SW16 ALPS SKHH OR SKPF, SW17 ALPS SKHH OR SKPF, SW18 ALPS SKHH OR SKPF, SW19 ALPS SKHH OR SKPF, SW2 ALPS SKHH OR SKPF, SW20 ALPS SKHH OR SKPF, SW21 ALPS SKHH OR SKPF, SW22 ALPS SKHH OR SKPF, SW23 ALPS SKHH OR SKPF, SW24 ALPS SKHH OR SKPF, SW25 ALPS SKHH OR SKPF, SW26 ALPS SKHH OR SKPF, SW27 6x6x13mm, SW28 6x6x13mm, SW29 6x6x13mm, SW3 ALPS SKHH OR SKPF, SW30 6x6x13mm, SW31 6x6x13mm, SW32 6x6x13mm, SW33 6x6x13mm, SW34 6x6x13mm, SW35 6x6x13mm, SW36 6x6x13mm, SW37 6x6x13mm, SW38 6x6x13mm, SW39 6x6x13mm, SW4 ALPS SKHH OR SKPF, SW40 6x6x13mm, SW41 6x6x13mm, SW42 6x6x13mm, SW43 6x6x13mm, SW44 6x6x13mm, SW45 6x6x13mm, SW46 6x6x13mm, SW47 6x6x13mm, SW5 ALPS SKHH OR SKPF, SW6 ALPS SKHH OR SKPF, SW7 ALPS SKHH OR SKPF, SW8 ALPS SKHH OR SKPF, SW9 ALPS SKHH OR SKPF

Commit message: key matrix routed (but untidy), added cutout for CPU heatsink
Changed lines of the file:
@@
 Text HLabel 15750 8250 0    50   Input ~ 0
-COL_4
-Text HLabel 9600 5850 0    50   Input ~ 0
 COL_4
 Text HLabel 10550 5850 0    50   Input ~ 0
@@
 Text HLabel 11500 5850 0    50   Input ~ 0
 COL_4
+Text HLabel 13400 5850 0    50   Input ~ 0
+COL_4
 Text HLabel 12450 5850 0    50   Input ~ 0
 COL_4
-Text HLabel 13400 5850 0    50   Input ~ 0
+Text HLabel 9600 5850 0    50   Input ~ 0
 COL_4
 Text HLabel 14800 5850 0    50   Input ~ 0
 COL_5
-Text HLabel 15750 5850 0    50   Input ~ 0
+Text HLabel 13400 3650 0    50   Input ~ 0
 COL_5
-Text HLabel 14800 4750 0    50   Input ~ 0
+Text HLabel 13400 4750 0    50   Input ~ 0
 COL_5
 Text HLabel 15750 4750 0    50   Input ~ 0
+COL_5
+Text HLabel 15750 5850 0    50   Input ~ 0
 COL_5
 Text HLabel 14800 3650 0    50   Input ~ 0
@@
 Text HLabel 15750 3650 0    50   Input ~ 0
 COL_5
-Text HLabel 13400 4750 0    50   Input ~ 0
+Text HLabel 14800 4750 0    50   Input ~ 0
 COL_5
-Text HLabel 13400 3650 0    50   Input ~ 0
-COL_5
-Text HLabel 12450 3650 0    50   Input ~ 0
+Text HLabel 9600 3650 0    50   Input ~ 0
+COL_6
+Text HLabel 9600 4750 0    50   Input ~ 0
+COL_6
+Text HLabel 11500 4750 0    50   Input ~ 0
 COL_6
 Text HLabel 12450 4750 0    50   Input ~ 0
 COL_6
-Text HLabel 11500 4750 0    50   Input ~ 0
+Text HLabel 12450 3650 0    50   Input ~ 0
+COL_6
+Text HLabel 10550 3650 0    50   Input ~ 0
 COL_6
 Text HLabel 11500 3650 0    50   Input ~ 0
 COL_6
-Text HLabel 10550 3650 0    50   Input ~ 0
-COL_6
 Text HLabel 10550 4750 0    50   Input ~ 0
-COL_6
-Text HLabel 9600 3650 0    50   Input ~ 0
-COL_6
-Text HLabel 9600 4750 0    50   Input ~ 0
 COL_6
 Text HLabel 800  8250 2    50   Input ~ 0
@@
 Text HLabel 15050 8250 2    50   Input ~ 0
 ROW_3
-Text HLabel 8900 5850 2    50   Input ~ 0
+Text HLabel 9850 5850 2    50   Input ~ 0
 ROW_4
-Text HLabel 9850 5850 2    50   Input ~ 0
+Text HLabel 10800 5850 2    50   Input ~ 0
 ROW_5
-Text HLabel 10800 5850 2    50   Input ~ 0
+Text HLabel 12700 5850 2    50   Input ~ 0
 ROW_6
 Text HLabel 11750 5850 2    50   Input ~ 0
 ROW_7
-Text HLabel 12700 5850 2    50   Input ~ 0
+Text HLabel 8900 5850 2    50   Input ~ 0
 ROW_8
 Text HLabel 14100 5850 2    50   Input ~ 0
 ROW_1
-Text HLabel 15050 5850 2    50   Input ~ 0
+Text HLabel 12700 3650 2    50   Input ~ 0
 ROW_2
-Text HLabel 14100 4750 2    50   Input ~ 0
+Text HLabel 12700 4750 2    50   Input ~ 0
 ROW_3
 Text HLabel 15050 4750 2    50   Input ~ 0
 ROW_4
+Text HLabel 15050 5850 2    50   Input ~ 0
+ROW_5
 Text HLabel 14100 3650 2    50   Input ~ 0
+ROW_6
+Text HLabel 14100 4750 2    50   Input ~ 0
+ROW_7
+Text HLabel 15050 3650 2    50   Input ~ 0
+ROW_8
+Text HLabel 10800 3650 2    50   Input ~ 0
+ROW_1
+Text HLabel 11750 3650 2    50   Input ~ 0
+ROW_2
+Text HLabel 11750 4750 2    50   Input ~ 0
+ROW_3
+Text HLabel 8900 3650 2    50   Input ~ 0
+ROW_4
+Text HLabel 9850 4750 2    50   Input ~ 0
 ROW_5
-Text HLabel 15050 3650 2    50   Input ~ 0
-ROW_6
-Text HLabel 12700 3650 2    50   Input ~ 0
-ROW_7
-Text HLabel 12700 4750 2    50   Input ~ 0
-ROW_8
-Text HLabel 8900 3650 2    50   Input ~ 0
-ROW_1
 Text HLabel 9850 3650 2    50   Input ~ 0
-ROW_2
-Text HLabel 10800 3650 2    50   Input ~ 0
-ROW_3
-Text HLabel 11750 3650 2    50   Input ~ 0
-ROW_4
-Text HLabel 8900 4750 2    50   Input ~ 0
-ROW_5
-Text HLabel 9850 4750 2    50   Input ~ 0
 ROW_6
 Text HLabel 10800 4750 2    50   Input ~ 0
 ROW_7
-Text HLabel 11750 4750 2    50   Input ~ 0
+Text HLabel 8900 4750 2    50   Input ~ 0
 ROW_8
 $EndSCHEMATC

Commit message: Add and route 7 extra buttons/LEDs
Parts:
- added D58, D59, D60, D61, D62, D63, D64: SM4007PL, Diode_SMD:D_SOD-123F, symbol Device:D_ALT
- added SW50, SW51, SW52, SW53, SW54, SW55, SW56: 6x6x13mm, OTTO_Footprints_Lib:6x6mm_Switch, symbol Switch:SW_Push
Connections:
- net labels added: COL_8
- wire segments 279 -> 314

Commit message: Added 3d models for encoders and switches
Parts:
- ENC1, ENC2, ENC3, ENC4: value ALPS EC11E18244AU -> ALPS EC11E183440C
Changed lines of the file:
@@
 AR Path="/5C4320DF/5C971830/5C6BBEC5" Ref="ENC1"  Part="1"
 F 0 "ENC1" H 3250 4467 50  0000 C CNN
-F 1 "ALPS EC11E18244AU " H 3250 4376 50  0000 C CNN
+F 1 "ALPS EC11E183440C" H 3250 4376 50  0000 C CNN
 F 2 "OTTO_Footprints_Lib:ALPS_EC11" H 3100 4260 50  0001 C CNN
 F 3 "https://datasheet.lcsc.com/szlcsc/1809200034_ALPS-Electric-EC11E18244AU_C202365.pdf" H 3250 4360 50  0001 C CNN
@@
 AR Path="/5C4320DF/5C971830/5C6BBEED" Ref="ENC2"  Part="1"
 F 0 "ENC2" H 3250 5417 50  0000 C CNN
-F 1 "ALPS EC11E18244AU " H 3250 5326 50  0000 C CNN
+F 1 "ALPS EC11E183440C" H 3250 5326 50  0000 C CNN
 F 2 "OTTO_Footprints_Lib:ALPS_EC11" H 3100 5210 50  0001 C CNN
 F 3 "https://datasheet.lcsc.com/szlcsc/1809200034_ALPS-Electric-EC11E18244AU_C202365.pdf" H 3250 5310 50  0001 C CNN
@@
 AR Path="/5C4320DF/5C971830/5C6BBF14" Ref="ENC3"  Part="1"
 F 0 "ENC3" H 7100 4467 50  0000 C CNN
-F 1 "ALPS EC11E18244AU " H 7100 4376 50  0000 C CNN
+F 1 "ALPS EC11E183440C" H 7100 4376 50  0000 C CNN
 F 2 "OTTO_Footprints_Lib:ALPS_EC11" H 6950 4260 50  0001 C CNN
 F 3 "https://datasheet.lcsc.com/szlcsc/1809200034_ALPS-Electric-EC11E18244AU_C202365.pdf" H 7100 4360 50  0001 C CNN
@@
 AR Path="/5C4320DF/5C971830/5C6BBF3A" Ref="ENC4"  Part="1"
 F 0 "ENC4" H 7100 5417 50  0000 C CNN
-F 1 "ALPS EC11E18244AU " H 7100 5326 50  0000 C CNN
+F 1 "ALPS EC11E183440C" H 7100 5326 50  0000 C CNN
 F 2 "OTTO_Footprints_Lib:ALPS_EC11" H 6950 5210 50  0001 C CNN
 F 3 "https://datasheet.lcsc.com/szlcsc/1809200034_ALPS-Electric-EC11E18244AU_C202365.pdf" H 7100 5310 50  0001 C CNN

Commit message: More JLC part numbers added
Parts:
- C60, C61, C62, C63, C64, C65, C66, C67: JLCASM (none) -> BASIC; LCSC PN (none) -> C49678; MPN CL21B104JBCNNNC -> CC0805KRX7R9BB104; Manufacturer Samsung Electro-Mechanics -> (none); UnitCost(USD) $0.017724 -> Samsung Electro-Mechanics
- D1, D10, D11, D12, D13, D14, D15, D16, D17, D18, D19, D2, D20, D202, D203, D204, D205, D21, D22, D23, D24, D25, D26, D27, D28, D29, D3, D30, D31, D32, D33, D34, D35, D36, D37, D38, D39, D4, D40, D41, D42, D43, D44, D45, D46, D47, D5, D58, D59, D6, D60, D61, D62, D63, D64, D7, D8, D9: JLCASM (none) -> BASIC; LCSC PN (none) -> C64898; Manufacturer MDD(Microdiode Electronics) -> (none); UnitCost(USD) $0.00574 -> MDD(Microdiode Electronics)
- ENC1, ENC2, ENC3, ENC4: JLCASM (none) -> DNP; LCSC PN (none) -> C202365; Manufacturer ALPS Electric -> (none); UnitCost(USD) $1.910606 -> ALPS Electric
- SW1, SW10, SW11, SW12, SW13, SW14, SW15, SW16, SW17, SW18, SW19, SW2, SW20, SW21, SW22, SW23, SW24, SW25, SW26, SW3, SW4, SW5, SW6, SW7, SW8, SW9: JLCASM (none) -> DNP; LCSC PN (none) -> C202419; MPN SKHHDTA010 -> SKHHDGA010; Manufacturer ALPS Electric -> (none); UnitCost(USD) $0.168182 -> ALPS Electric
- SW27, SW28, SW29, SW30, SW31, SW32, SW33, SW34, SW35, SW36, SW37, SW38, SW39, SW40, SW41, SW42, SW43, SW44, SW45, SW46, SW47, SW50, SW51, SW52, SW53, SW54, SW55, SW56: JLCASM (none) -> DNP; LCSC PN (none) -> C136674; Manufacturer Korean Hroparts Elec -> (none); UnitCost(USD) $0.043333 -> Korean Hroparts Elec

Commit message: Selected all LCSC parts. Check of part numbers complete
Parts:
- C60, C61, C62, C63, C64, C65, C66, C67: UnitCost(USD) Samsung Electro-Mechanics -> (none)
- D1, D10, D11, D12, D13, D14, D15, D16, D17, D18, D19, D2, D20, D202, D203, D204, D205, D21, D22, D23, D24, D25, D26, D27, D28, D29, D3, D30, D31, D32, D33, D34, D35, D36, D37, D38, D39, D4, D40, D41, D42, D43, D44, D45, D46, D47, D5, D58, D59, D6, D60, D61, D62, D63, D64, D7, D8, D9: UnitCost(USD) MDD(Microdiode Electronics) -> (none)
- ENC1, ENC2, ENC3, ENC4: LCSC PN C202365 -> C370986; MPN EC11E18244AU -> EC11E183440C; UnitCost(USD) ALPS Electric -> (none)
- SW1, SW10, SW11, SW12, SW13, SW14, SW15, SW16, SW17, SW18, SW19, SW2, SW20, SW21, SW22, SW23, SW24, SW25, SW26, SW3, SW4, SW5, SW6, SW7, SW8, SW9: UnitCost(USD) ALPS Electric -> (none)
- SW27, SW28, SW29, SW30, SW31, SW32, SW33, SW34, SW35, SW36, SW37, SW38, SW39, SW40, SW41, SW42, SW43, SW44, SW45, SW46, SW47, SW50, SW51, SW52, SW53, SW54, SW55, SW56: UnitCost(USD) Korean Hroparts Elec -> (none)

Commit message: Route SKHC switches
Parts:
- SW1, SW10, SW11, SW12, SW13, SW14, SW15, SW16, SW17, SW18, SW19, SW2, SW20, SW21, SW22, SW23, SW24, SW25, SW26, SW3, SW4, SW5, SW6, SW7, SW8, SW9: value ALPS SKHH OR SKPF -> ALPS SKHC; footprint OTTO_Footprints_Lib:6x6mm_Switch_LargeCap_ALT_SKPF -> OTTO_Footprints_Lib:ALPS_SKHC

Commit message: Remove LEDs from main board
Parts:
- SW1, SW10, SW11, SW12, SW13, SW14, SW15, SW16, SW17, SW18, SW19, SW2, SW20, SW21, SW22, SW23, SW24, SW25, SW26, SW3, SW4, SW5, SW6, SW7, SW8, SW9: value ALPS SKHC -> ALPS SKHH OR SKPF; footprint OTTO_Footprints_Lib:ALPS_SKHC -> OTTO_Footprints_Lib:6x6mm_Switch_LargeCap_ALT_SKPF
