File: KiCad/KEYS+ENCODERS.sch (KiCad schematic (older format))
At the start: 124 parts, among them SW1 ALPS SKHC, SW10 ALPS SKHC, SW11 ALPS SKHC, SW12 ALPS SKHC, SW13 ALPS SKHC, SW14 ALPS SKHC, SW15 ALPS SKHC, SW16 ALPS SKHC, SW17 ALPS SKHC, SW18 ALPS SKHC, SW19 ALPS SKHC, SW2 ALPS SKHC, SW20 ALPS SKHC, SW21 ALPS SKHC, SW22 ALPS SKHC, SW23 ALPS SKHC, SW24 ALPS SKHC, SW25 ALPS SKHC, SW26 ALPS SKHC, SW27 6x6x13mm, SW28 6x6x13mm, SW29 6x6x13mm, SW3 ALPS SKHC, SW30 6x6x13mm, SW31 6x6x13mm, SW32 6x6x13mm, SW33 6x6x13mm, SW34 6x6x13mm, SW35 6x6x13mm, SW36 6x6x13mm, SW37 6x6x13mm, SW38 6x6x13mm, SW39 6x6x13mm, SW4 ALPS SKHC, SW40 6x6x13mm, SW41 6x6x13mm, SW42 6x6x13mm, SW43 6x6x13mm, SW44 6x6x13mm, SW45 6x6x13mm, SW46 6x6x13mm, SW47 6x6x13mm, SW5 ALPS SKHC, SW50 6x6x13mm, SW51 6x6x13mm, SW52 6x6x13mm, SW53 6x6x13mm, SW54 6x6x13mm, SW55 6x6x13mm, SW56 6x6x13mm, SW6 ALPS SKHC, SW7 ALPS SKHC, SW8 ALPS SKHC, SW9 ALPS SKHC

Commit message: 3d models
Parts:
- SW1, SW10, SW11, SW12, SW13, SW14, SW15, SW16, SW2, SW3, SW4, SW5, SW6, SW7, SW8, SW9: footprint OTTO_Footprints_Lib:ALPS_SKHC -> OTTO_Footprints_Lib:ALPS_SKHC_white
- SW17, SW18, SW19, SW20, SW21, SW22, SW23, SW24, SW25, SW26: footprint OTTO_Footprints_Lib:ALPS_SKHC -> OTTO_Footprints_Lib:ALPS_SKHC_black
Changed lines of the file:
@@
 $Descr A3 16535 11693
 encoding utf-8
-Sheet 6 7
+Sheet 5 7
 Title "OTTO beta"
 Date "2020-05-25"
@@
 F 0 "SW17" H 2800 6935 50  0000 C CNN
 F 1 "ALPS SKHC" H 2800 6844 50  0000 C CNN
-F 2 "OTTO_Footprints_Lib:ALPS_SKHC" H 2800 6850 50  0001 C CNN
+F 2 "OTTO_Footprints_Lib:ALPS_SKHC_black" H 2800 6850 50  0001 C CNN
 F 3 "https://datasheet.lcsc.com/szlcsc/C202419.pdf" H 2800 6850 50  0001 C CNN
 F 4 "" H 2800 6650 12700 0001 C CNN "UnitCost(USD)"
@@
 F 0 "SW1" H 1350 8135 50  0000 C CNN
 F 1 "ALPS SKHC" H 1350 8044 50  0000 C CNN
-F 2 "OTTO_Footprints_Lib:ALPS_SKHC" H 1350 8050 50  0001 C CNN
+F 2 "OTTO_Footprints_Lib:ALPS_SKHC_white" H 1350 8050 50  0001 C CNN
 F 3 "https://datasheet.lcsc.com/szlcsc/C202419.pdf" H 1350 8050 50  0001 C CNN
 F 4 "" H 1350 7850 12700 0001 C CNN "UnitCost(USD)"
@@
 F 0 "SW18" H 3750 6935 50  0000 C CNN
 F 1 "ALPS SKHC" H 3750 6844 50  0000 C CNN
-F 2 "OTTO_Footprints_Lib:ALPS_SKHC" H 3750 6850 50  0001 C CNN
+F 2 "OTTO_Footprints_Lib:ALPS_SKHC_black" H 3750 6850 50  0001 C CNN
 F 3 "https://datasheet.lcsc.com/szlcsc/C202419.pdf" H 3750 6850 50  0001 C CNN
 F 4 "" H 3750 6650 12700 0001 C CNN "UnitCost(USD)"
@@
 F 0 "SW19" H 5650 6935 50  0000 C CNN
 F 1 "ALPS SKHC" H 5650 6844 50  0000 C CNN
-F 2 "OTTO_Footprints_Lib:ALPS_SKHC" H 5650 6850 50  0001 C CNN
+F 2 "OTTO_Footprints_Lib:ALPS_SKHC_black" H 5650 6850 50  0001 C CNN
 F 3 "https://datasheet.lcsc.com/szlcsc/C202419.pdf" H 5650 6850 50  0001 C CNN
 F 4 "" H 5650 6650 12700 0001 C CNN "UnitCost(USD)"
@@
 F 0 "SW20" H 6600 6935 50  0000 C CNN
 F 1 "ALPS SKHC" H 6600 6844 50  0000 C CNN
-F 2 "OTTO_Footprints_Lib:ALPS_SKHC" H 6600 6850 50  0001 C CNN
+F 2 "OTTO_Footprints_Lib:ALPS_SKHC_black" H 6600 6850 50  0001 C CNN
 F 3 "https://datasheet.lcsc.com/szlcsc/C202419.pdf" H 6600 6850 50  0001 C CNN
 F 4 "" H 6600 6650 12700 0001 C CNN "UnitCost(USD)"
@@
 F 0 "SW21" H 7550 6935 50  0000 C CNN
 F 1 "ALPS SKHC" H 7550 6844 50  0000 C CNN
-F 2 "OTTO_Footprints_Lib:ALPS_SKHC" H 7550 6850 50  0001 C CNN
+F 2 "OTTO_Footprints_Lib:ALPS_SKHC_black" H 7550 6850 50  0001 C CNN
 F 3 "https://datasheet.lcsc.com/szlcsc/C202419.pdf" H 7550 6850 50  0001 C CNN
 F 4 "" H 7550 6650 12700 0001 C CNN "UnitCost(USD)"
@@
 F 0 "SW2" H 2300 8135 50  0000 C CNN
 F 1 "ALPS SKHC" H 2300 8044 50  0000 C CNN
-F 2 "OTTO_Footprints_Lib:ALPS_SKHC" H 2300 8050 50  0001 C CNN
+F 2 "OTTO_Footprints_Lib:ALPS_SKHC_white" H 2300 8050 50  0001 C CNN
 F 3 "https://datasheet.lcsc.com/szlcsc/C202419.pdf" H 2300 8050 50  0001 C CNN
 F 4 "" H 2300 7850 12700 0001 C CNN "UnitCost(USD)"
@@
 F 0 "SW22" H 9450 6935 50  0000 C CNN
 F 1 "ALPS SKHC" H 9450 6844 50  0000 C CNN
-F 2 "OTTO_Footprints_Lib:ALPS_SKHC" H 9450 6850 50  0001 C CNN
+F 2 "OTTO_Footprints_Lib:ALPS_SKHC_black" H 9450 6850 50  0001 C CNN
 F 3 "https://datasheet.lcsc.com/szlcsc/C202419.pdf" H 9450 6850 50  0001 C CNN
 F 4 "" H 9450 6650 12700 0001 C CNN "UnitCost(USD)"
@@
 F 0 "SW23" H 10400 6935 50  0000 C CNN
 F 1 "ALPS SKHC" H 10400 6844 50  0000 C CNN
-F 2 "OTTO_Footprints_Lib:ALPS_SKHC" H 10400 6850 50  0001 C CNN
+F 2 "OTTO_Footprints_Lib:ALPS_SKHC_black" H 10400 6850 50  0001 C CNN
 F 3 "https://datasheet.lcsc.com/szlcsc/C202419.pdf" H 10400 6850 50  0001 C CNN
 F 4 "" H 10400 6650 12700 0001 C CNN "UnitCost(USD)"
@@
 F 0 "SW24" H 12300 6935 50  0000 C CNN
 F 1 "ALPS SKHC" H 12300 6844 50  0000 C CNN
-F 2 "OTTO_Footprints_Lib:ALPS_SKHC" H 12300 6850 50  0001 C CNN
+F 2 "OTTO_Footprints_Lib:ALPS_SKHC_black" H 12300 6850 50  0001 C CNN
 F 3 "https://datasheet.lcsc.com/szlcsc/C202419.pdf" H 12300 6850 50  0001 C CNN
 F 4 "" H 12300 6650 12700 0001 C CNN "UnitCost(USD)"
@@
 F 0 "SW25" H 13250 6935 50  0000 C CNN
 F 1 "ALPS SKHC" H 13250 6844 50  0000 C CNN
-F 2 "OTTO_Footprints_Lib:ALPS_SKHC" H 13250 6850 50  0001 C CNN
+F 2 "OTTO_Footprints_Lib:ALPS_SKHC_black" H 13250 6850 50  0001 C CNN
 F 3 "https://datasheet.lcsc.com/szlcsc/C202419.pdf" H 13250 6850 50  0001 C CNN
 F 4 "" H 13250 6650 12700 0001 C CNN "UnitCost(USD)"
@@
 F 0 "SW26" H 14200 6935 50  0000 C CNN
 F 1 "ALPS SKHC" H 14200 6844 50  0000 C CNN
-F 2 "OTTO_Footprints_Lib:ALPS_SKHC" H 14200 6850 50  0001 C CNN
+F 2 "OTTO_Footprints_Lib:ALPS_SKHC_black" H 14200 6850 50  0001 C CNN
 F 3 "https://datasheet.lcsc.com/szlcsc/C202419.pdf" H 14200 6850 50  0001 C CNN
 F 4 "" H 14200 6650 12700 0001 C CNN "UnitCost(USD)"
@@
 F 0 "SW3" H 3250 8135 50  0000 C CNN
 F 1 "ALPS SKHC" H 3250 8044 50  0000 C CNN
-F 2 "OTTO_Footprints_Lib:ALPS_SKHC" H 3250 8050 50  0001 C CNN
+F 2 "OTTO_Footprints_Lib:ALPS_SKHC_white" H 3250 8050 50  0001 C CNN
 F 3 "https://datasheet.lcsc.com/szlcsc/C202419.pdf" H 3250 8050 50  0001 C CNN
 F 4 "" H 3250 7850 12700 0001 C CNN "UnitCost(USD)"
@@
 F 0 "SW4" H 4200 8135 50  0000 C CNN
 F 1 "ALPS SKHC" H 4200 8044 50  0000 C CNN
-F 2 "OTTO_Footprints_Lib:ALPS_SKHC" H 4200 8050 50  0001 C CNN
+F 2 "OTTO_Footprints_Lib:ALPS_SKHC_white" H 4200 8050 50  0001 C CNN
 F 3 "https://datasheet.lcsc.com/szlcsc/C202419.pdf" H 4200 8050 50  0001 C CNN
 F 4 "" H 4200 7850 12700 0001 C CNN "UnitCost(USD)"
@@
 F 0 "SW5" H 5150 8135 50  0000 C CNN
 F 1 "ALPS SKHC" H 5150 8044 50  0000 C CNN
-F 2 "OTTO_Footprints_Lib:ALPS_SKHC" H 5150 8050 50  0001 C CNN
+F 2 "OTTO_Footprints_Lib:ALPS_SKHC_white" H 5150 8050 50  0001 C CNN
 F 3 "https://datasheet.lcsc.com/szlcsc/C202419.pdf" H 5150 8050 50  0001 C CNN
 F 4 "" H 5150 7850 12700 0001 C CNN "UnitCost(USD)"
@@
 F 0 "SW6" H 6100 8135 50  0000 C CNN
 F 1 "ALPS SKHC" H 6100 8044 50  0000 C CNN
-F 2 "OTTO_Footprints_Lib:ALPS_SKHC" H 6100 8050 50  0001 C CNN
+F 2 "OTTO_Footprints_Lib:ALPS_SKHC_white" H 6100 8050 50  0001 C CNN
 F 3 "https://datasheet.lcsc.com/szlcsc/C202419.pdf" H 6100 8050 50  0001 C CNN
 F 4 "" H 6100 7850 12700 0001 C CNN "UnitCost(USD)"
@@
 F 0 "SW7" H 7050 8135 50  0000 C CNN
 F 1 "ALPS SKHC" H 7050 8044 50  0000 C CNN
-F 2 "OTTO_Footprints_Lib:ALPS_SKHC" H 7050 8050 50  0001 C CNN
+F 2 "OTTO_Footprints_Lib:ALPS_SKHC_white" H 7050 8050 50  0001 C CNN
 F 3 "https://datasheet.lcsc.com/szlcsc/C202419.pdf" H 7050 8050 50  0001 C CNN
 F 4 "" H 7050 7850 12700 0001 C CNN "UnitCost(USD)"
@@
 F 0 "SW8" H 8000 8135 50  0000 C CNN
 F 1 "ALPS SKHC" H 8000 8044 50  0000 C CNN
-F 2 "OTTO_Footprints_Lib:ALPS_SKHC" H 8000 8050 50  0001 C CNN
+F 2 "OTTO_Footprints_Lib:ALPS_SKHC_white" H 8000 8050 50  0001 C CNN
 F 3 "https://datasheet.lcsc.com/szlcsc/C202419.pdf" H 8000 8050 50  0001 C CNN
 F 4 "" H 8000 7850 12700 0001 C CNN "UnitCost(USD)"
@@
 F 0 "SW9" H 8950 8135 50  0000 C CNN
 F 1 "ALPS SKHC" H 8950 8044 50  0000 C CNN
-F 2 "OTTO_Footprints_Lib:ALPS_SKHC" H 8950 8050 50  0001 C CNN
+F 2 "OTTO_Footprints_Lib:ALPS_SKHC_white" H 8950 8050 50  0001 C CNN
 F 3 "https://datasheet.lcsc.com/szlcsc/C202419.pdf" H 8950 8050 50  0001 C CNN
 F 4 "" H 8950 7850 12700 0001 C CNN "UnitCost(USD)"
@@
 F 0 "SW10" H 9900 8135 50  0000 C CNN
 F 1 "ALPS SKHC" H 9900 8044 50  0000 C CNN
-F 2 "OTTO_Footprints_Lib:ALPS_SKHC" H 9900 8050 50  0001 C CNN
+F 2 "OTTO_Footprints_Lib:ALPS_SKHC_white" H 9900 8050 50  0001 C CNN
 F 3 "https://datasheet.lcsc.com/szlcsc/C202419.pdf" H 9900 8050 50  0001 C CNN
 F 4 "" H 9900 7850 12700 0001 C CNN "UnitCost(USD)"
@@
 F 0 "SW11" H 10850 8135 50  0000 C CNN
 F 1 "ALPS SKHC" H 10850 8044 50  0000 C CNN
-F 2 "OTTO_Footprints_Lib:ALPS_SKHC" H 10850 8050 50  0001 C CNN
+F 2 "OTTO_Footprints_Lib:ALPS_SKHC_white" H 10850 8050 50  0001 C CNN
 F 3 "https://datasheet.lcsc.com/szlcsc/C202419.pdf" H 10850 8050 50  0001 C CNN
 F 4 "" H 10850 7850 12700 0001 C CNN "UnitCost(USD)"
@@
 F 0 "SW12" H 11800 8135 50  0000 C CNN
 F 1 "ALPS SKHC" H 11800 8044 50  0000 C CNN
-F 2 "OTTO_Footprints_Lib:ALPS_SKHC" H 11800 8050 50  0001 C CNN
+F 2 "OTTO_Footprints_Lib:ALPS_SKHC_white" H 11800 8050 50  0001 C CNN
 F 3 "https://datasheet.lcsc.com/szlcsc/C202419.pdf" H 11800 8050 50  0001 C CNN
 F 4 "" H 11800 7850 12700 0001 C CNN "UnitCost(USD)"
@@
 F 0 "SW13" H 12750 8135 50  0000 C CNN
 F 1 "ALPS SKHC" H 12750 8044 50  0000 C CNN
-F 2 "OTTO_Footprints_Lib:ALPS_SKHC" H 12750 8050 50  0001 C CNN
+F 2 "OTTO_Footprints_Lib:ALPS_SKHC_white" H 12750 8050 50  0001 C CNN
 F 3 "https://datasheet.lcsc.com/szlcsc/C202419.pdf" H 12750 8050 50  0001 C CNN
 F 4 "" H 12750 7850 12700 0001 C CNN "UnitCost(USD)"
@@
 F 0 "SW14" H 13700 8135 50  0000 C CNN
 F 1 "ALPS SKHC" H 13700 8044 50  0000 C CNN
-F 2 "OTTO_Footprints_Lib:ALPS_SKHC" H 13700 8050 50  0001 C CNN
+F 2 "OTTO_Footprints_Lib:ALPS_SKHC_white" H 13700 8050 50  0001 C CNN
 F 3 "https://datasheet.lcsc.com/szlcsc/C202419.pdf" H 13700 8050 50  0001 C CNN
 F 4 "" H 13700 7850 12700 0001 C CNN "UnitCost(USD)"
@@
 F 0 "SW15" H 14650 8135 50  0000 C CNN
 F 1 "ALPS SKHC" H 14650 8044 50  0000 C CNN
-F 2 "OTTO_Footprints_Lib:ALPS_SKHC" H 14650 8050 50  0001 C CNN
+F 2 "OTTO_Footprints_Lib:ALPS_SKHC_white" H 14650 8050 50  0001 C CNN
 F 3 "https://datasheet.lcsc.com/szlcsc/C202419.pdf" H 14650 8050 50  0001 C CNN
 F 4 "" H 14650 7850 12700 0001 C CNN "UnitCost(USD)"
@@
 F 0 "SW16" H 15600 8135 50  0000 C CNN
 F 1 "ALPS SKHC" H 15600 8044 50  0000 C CNN
-F 2 "OTTO_Footprints_Lib:ALPS_SKHC" H 15600 8050 50  0001 C CNN
+F 2 "OTTO_Footprints_Lib:ALPS_SKHC_white" H 15600 8050 50  0001 C CNN
 F 3 "https://datasheet.lcsc.com/szlcsc/C202419.pdf" H 15600 8050 50  0001 C CNN
 F 4 "" H 15600 7850 12700 0001 C CNN "UnitCost(USD)"

Commit message: Add HEX spacers and fix AUX LED pinouts
Parts:
- SW1, SW10, SW11, SW12, SW13, SW14, SW15, SW16, SW17, SW18, SW19, SW2, SW20, SW21, SW22, SW23, SW24, SW25, SW26, SW3, SW4, SW5, SW6, SW7, SW8, SW9: LCSC PN C202419 -> C139753; MPN SKHHDGA010 -> SKHCBGA010
