File: KiCad/LEDS.sch (KiCad schematic (older format))
At the start: 99 parts, among them U203 74HC125D

Commit message: added power switching and extra pulls for programming lines
Parts:
- removed C57: 100nF, Capacitor_SMD:C_0805_2012Metric_Pad1.15x1.40mm_HandSolder_marked, symbol Device:C
- removed JP201: SolderJumper_3_Open, Jumper:SolderJumper-3_P2.0mm_Open_TrianglePad1.0x1.5mm, symbol Jumper:SolderJumper_3_Open
- removed U203: 74HC125D, Package_SO:SOIC-14_3.9x8.7mm_P1.27mm, symbol 74xx:74LS125
- added C?: 100nF, Capacitor_SMD:C_0805_2012Metric_Pad1.15x1.40mm_HandSolder_marked, symbol Device:C
- added C?: 47uF, Capacitor_SMD:C_0805_2012Metric_Pad1.15x1.40mm_HandSolder_marked, symbol Device:C
- added C?: 10nF, Capacitor_SMD:C_0805_2012Metric_Pad1.15x1.40mm_HandSolder_marked, symbol Device:C
- added R? (x2): 100k, symbol Device:R
- added R?: 0, symbol Device:R
- added TP?: TestPoint, symbol Connector:TestPoint
- added U?: TPS22918_SOT23-6_A, Package_TO_SOT_SMD:SOT-23-6, symbol OTTOdiy_SMD-library:TPS22918_SOT23-6_A
- added U?: SN74LV1T125_SOT-23_A, Package_TO_SOT_SMD:SOT-23-5_HandSoldering, symbol OTTOdiy_SMD-library:SN74LV1T125_SOT-23_A
Connections:
- net labels added: +3V3_MCU, +5V_LEDS, +5V_REG, LED_PWR_EN, SPI_MOSI_MCU_5V
- net labels removed: +5V_MAIN
- wire segments 291 -> 376
- no-connect marks 3 -> 0
Other:
- note removed: "LEDs are connected to the MCU via SPI as there's \na library that uses SPI for the timing of the LED data."

Commit message: connected unconnected signals and MIDI to spare MCU UART
Parts:
- gave numbers to parts that had none: 10
Changed lines of the file:
@@
 	4850 2400 5250 2400
 $Comp
-L Device:R R?
+L Device:R R11
 U 1 1 5E2E14CF
 P 3800 5650
-F 0 "R?" H 3870 5696 50  0000 L CNN
+F 0 "R11" H 3870 5696 50  0000 L CNN
 F 1 "100k" H 3870 5605 50  0000 L CNN
 F 2 "" V 3730 5650 50  0001 C CNN
@@
 $EndComp
 $Comp
-L power:GND #PWR?
+L power:GND #PWR0109
 U 1 1 5E2E1B34
 P 3800 5950
-F 0 "#PWR?" H 3800 5700 50  0001 C CNN
+F 0 "#PWR0109" H 3800 5700 50  0001 C CNN
 F 1 "GND" H 3805 5777 50  0000 C CNN
 F 2 "" H 3800 5950 50  0001 C CNN
@@
 	5250 3000 5950 3000
 $Comp
-L OTTOdiy_SMD-library:TPS22918_SOT23-6_A U?
+L OTTOdiy_SMD-library:TPS22918_SOT23-6_A U2
 U 1 1 5E0B982C
 P 3200 1850
-F 0 "U?" H 3200 2216 50  0000 C CNN
+F 0 "U2" H 3200 2216 50  0000 C CNN
 F 1 "TPS22918_SOT23-6_A" H 3200 2125 50  0000 C CNN
 F 2 "Package_TO_SOT_SMD:SOT-23-6" H 3200 2350 50  0001 C CNN
@@
 $EndComp
 $Comp
-L OTTOdiy_SMD-library:SN74LV1T125_SOT-23_A U?
+L OTTOdiy_SMD-library:SN74LV1T125_SOT-23_A U1
 U 1 1 5E0C47FE
 P 2350 5300
-F 0 "U?" H 2100 5600 60  0000 L CNN
+F 0 "U1" H 2100 5600 60  0000 L CNN
 F 1 "SN74LV1T125_SOT-23_A" H 2500 5100 60  0000 L CNN
 F 2 "Package_TO_SOT_SMD:SOT-23-5_HandSoldering" H 2550 5500 60  0001 L CNN
@@
 $EndComp
 $Comp
-L Device:C C?
+L Device:C C78
 U 1 1 5E0C5D75
 P 2650 4550
-F 0 "C?" H 2765 4596 50  0000 L CNN
+F 0 "C78" H 2765 4596 50  0000 L CNN
 F 1 "100nF" H 2765 4505 50  0000 L CNN
 F 2 "Capacitor_SMD:C_0805_2012Metric_Pad1.15x1.40mm_HandSolder_marked" H 2688 4400 50  0001 C CNN
@@
 SPI_MOSI_MCU_5V
 $Comp
-L power:GND #PWR?
+L power:GND #PWR0110
 U 1 1 5E0CC3A4
 P 2350 5800
-F 0 "#PWR?" H 2350 5550 50  0001 C CNN
+F 0 "#PWR0110" H 2350 5550 50  0001 C CNN
 F 1 "GND" H 2355 5627 50  0000 C CNN
 F 2 "" H 2350 5800 50  0001 C CNN
@@
 	2350 4250 2350 5000
 $Comp
-L power:GND #PWR?
+L power:GND #PWR0111
 U 1 1 5E0CCF85
 P 2650 4800
-F 0 "#PWR?" H 2650 4550 50  0001 C CNN
+F 0 "#PWR0111" H 2650 4550 50  0001 C CNN
 F 1 "GND" H 2655 4627 50  0000 C CNN
 F 2 "" H 2650 4800 50  0001 C CNN
@@
 	1700 5200 1900 5200
 $Comp
-L Device:R R?
+L Device:R R9
 U 1 1 5E0D106C
 P 1900 4750
-F 0 "R?" H 1970 4796 50  0000 L CNN
+F 0 "R9" H 1970 4796 50  0000 L CNN
 F 1 "100k" H 1970 4705 50  0000 L CNN
 F 2 "" V 1830 4750 50  0001 C CNN
@@
 	1900 5200 2050 5200
 $Comp
-L Connector:TestPoint TP?
+L Connector:TestPoint TP1
 U 1 1 5E0D1862
 P 12550 7850
-F 0 "TP?" V 12505 8038 50  0000 L CNN
+F 0 "TP1" V 12505 8038 50  0000 L CNN
 F 1 "TestPoint" V 12595 8038 50  0000 L CNN
 F 2 "" H 12750 7850 50  0001 C CNN
@@
 	1600 1750 1750 1750
 $Comp
-L Device:C C?
+L Device:C C76
 U 1 1 5E0D93C1
 P 1750 2100
-F 0 "C?" H 1865 2146 50  0000 L CNN
+F 0 "C76" H 1865 2146 50  0000 L CNN
 F 1 "47uF" H 1865 2055 50  0000 L CNN
 F 2 "Capacitor_SMD:C_0805_2012Metric_Pad1.15x1.40mm_HandSolder_marked" H 1788 1950 50  0001 C CNN
@@
 	1750 1750 2800 1750
 $Comp
-L power:GND #PWR?
+L power:GND #PWR0112
 U 1 1 5E0DA22E
 P 1750 2450
-F 0 "#PWR?" H 1750 2200 50  0001 C CNN
+F 0 "#PWR0112" H 1750 2200 50  0001 C CNN
 F 1 "GND" H 1755 2277 50  0000 C CNN
 F 2 "" H 1750 2450 50  0001 C CNN
@@
 +5V_LEDS
 $Comp
-L Device:C C?
+L Device:C C77
 U 1 1 5E0DB8E2
 P 2250 2100
-F 0 "C?" H 2365 2146 50  0000 L CNN
+F 0 "C77" H 2365 2146 50  0000 L CNN
 F 1 "10nF" H 2365 2055 50  0000 L CNN
 F 2 "Capacitor_SMD:C_0805_2012Metric_Pad1.15x1.40mm_HandSolder_marked" H 2288 1950 50  0001 C CNN
@@
 	2250 1850 2800 1850
 $Comp
-L power:GND #PWR?
+L power:GND #PWR0113
 U 1 1 5E0DCD0C
 P 2250 2450
-F 0 "#PWR?" H 2250 2200 50  0001 C CNN
+F 0 "#PWR0113" H 2250 2200 50  0001 C CNN
 F 1 "GND" H 2255 2277 50  0000 C CNN
 F 2 "" H 2250 2450 50  0001 C CNN
@@
 	2800 1950 2650 1950
 $Comp
-L Device:R R?
+L Device:R R10
 U 1 1 5E0DD0E7
 P 2650 3050
-F 0 "R?" H 2720 3096 50  0000 L CNN
+F 0 "R10" H 2720 3096 50  0000 L CNN
 F 1 "100k" H 2720 3005 50  0000 L CNN
 F 2 "" V 2580 3050 50  0001 C CNN
@@
 	2650 2800 2650 2900
 $Comp
-L power:GND #PWR?
+L power:GND #PWR0114
 U 1 1 5E0DF9C6
 P 2650 3300
-F 0 "#PWR?" H 2650 3050 50  0001 C CNN
+F 0 "#PWR0114" H 2650 3050 50  0001 C CNN
 F 1 "GND" H 2655 3127 50  0000 C CNN
 F 2 "" H 2650 3300 50  0001 C CNN
@@
 	2650 3200 2650 3300
 $Comp
-L power:GND #PWR?
+L power:GND #PWR0115
 U 1 1 5E0DFD2F
 P 3200 2350
-F 0 "#PWR?" H 3200 2100 50  0001 C CNN
+F 0 "#PWR0115" H 3200 2100 50  0001 C CNN
 F 1 "GND" H 3205 2177 50  0000 C CNN
 F 2 "" H 3200 2350 50  0001 C CNN
@@
 	3200 2150 3200 2350
 $Comp
-L Device:R R?
+L Device:R R12
 U 1 1 5E0E015C
 P 3950 2050
-F 0 "R?" V 3744 2050 50  0000 C CNN
+F 0 "R12" V 3744 2050 50  0000 C CNN
 F 1 "0" V 3835 2050 50  0000 C CNN
 F 2 "" V 3880 2050 50  0001 C CNN

Commit message: add all resistor part numbers and create footprint library
Parts:
- LED1, LED10, LED11, LED12, LED13, LED14, LED15, LED16, LED17, LED18, LED19, LED2, LED20, LED21, LED22, LED23, LED24, LED25, LED26, LED27, LED28, LED29, LED3, LED30, LED31, LED32, LED33, LED34, LED35, LED36, LED37, LED38, LED39, LED4, LED40, LED41, LED42, LED43, LED44, LED45, LED46, LED47, LED5, LED6, LED7, LED8, LED9: value WS2812D-F5 -> WS2812B-Mini; footprint Spatz:LED_D5.0mm-4 -> OTTO_Footprints_Lib:LED3535; EstimatedCost(USD) (none) -> $.107155; MPN (none) -> WS2812B-Mini; Manufacturer (none) -> Worldsemi
- R10, R11, R9: footprint (none) -> Resistor_SMD:R_0805_2012Metric_Pad1.15x1.40mm_HandSolder; EstimatedCost(USD) (none) -> $.00169; MPN (none) -> RC0805FR-07100KL; Manufacturer (none) -> Yageo
- R12: footprint (none) -> Resistor_SMD:R_0805_2012Metric_Pad1.15x1.40mm_HandSolder; EstimatedCost(USD) (none) -> $.001203; MPN (none) -> RC0805JR-070RL; Manufacturer (none) -> Yageo
- R208: EstimatedCost(USD) (none) -> $.001752; MPN (none) -> RC0805FR-07100RL; Manufacturer (none) -> Yageo
- U1: Manufacturer (none) -> Texas Instruments

Commit message: added part numbers for capacitors and crystals
Parts:
- C1, C10, C11, C12, C13, C14, C15, C16, C17, C18, C19, C2, C20, C21, C22, C23, C24, C25, C26, C27, C28, C29, C3, C30, C31, C32, C33, C34, C35, C36, C37, C38, C39, C4, C40, C41, C42, C43, C44, C45, C46, C47, C5, C6, C7, C78, C8, C9: footprint Capacitor_SMD:C_0805_2012Metric_Pad1.15x1.40mm_HandSolder_marked -> Capacitor_SMD:C_0805_2012Metric_Pad1.15x1.40mm_HandSolder; EstimatedCost(USD) (none) -> $0.017724; MPN (none) -> CL21B104JBCNNNC; Manufacturer (none) -> Samsung Electro-Mechanics
- C76: footprint Capacitor_SMD:C_0805_2012Metric_Pad1.15x1.40mm_HandSolder_marked -> Capacitor_SMD:C_1206_3216Metric_Pad1.42x1.75mm_HandSolder; EstimatedCost(USD) (none) -> $0.390909; MPN (none) -> GRM31CR61E476ME44L; Manufacturer (none) -> Murata Electronics
- C77: footprint Capacitor_SMD:C_0805_2012Metric_Pad1.15x1.40mm_HandSolder_marked -> Capacitor_SMD:C_0805_2012Metric_Pad1.15x1.40mm_HandSolder; EstimatedCost(USD) (none) -> $0.007546; MPN (none) -> CL21B103KBCNNNC; Manufacturer (none) -> Samsung Electro-Mechanics
- LED1, LED10, LED11, LED12, LED13, LED14, LED15, LED16, LED17, LED18, LED19, LED2, LED20, LED21, LED22, LED23, LED24, LED25, LED26, LED27, LED28, LED29, LED3, LED30, LED31, LED32, LED33, LED34, LED35, LED36, LED37, LED38, LED39, LED4, LED40, LED41, LED42, LED43, LED44, LED45, LED46, LED47, LED5, LED6, LED7, LED8, LED9: value WS2812B-Mini -> WS2812D-5; footprint OTTO_Footprints_Lib:LED3535 -> OTTO_Footprints_Lib:LED_D5.0mm-4; EstimatedCost(USD) $.107155 -> $0.10303; MPN WS2812B-Mini -> WS2812D-F5

Commit message: add switch and encoder parts. BM Complete. Footprints complete.
Parts:
- TP1: footprint (none) -> TestPoint:TestPoint_Keystone_5000-5004_Miniature; AssemblyOption (none) -> DNP; EstimatedCost(USD) (none) -> $0.00; MPN (none) -> N/A; Manufacturer (none) -> N/A
- U1: EstimatedCost(USD) (none) -> $0.45
- U2: EstimatedCost(USD) (none) -> $0.228788; MPN (none) -> TPS22918DBVR; Manufacturer (none) -> Texas Instruments
Changed lines of the file:
@@
 F 2 "Package_TO_SOT_SMD:SOT-23-6" H 3200 2350 50  0001 C CNN
 F 3 "http://www.ti.com/lit/ds/symlink/tps22918.pdf" H 3250 1150 50  0001 C CNN
+F 4 "$0.228788" H 3200 1850 12700 0001 C CNN "EstimatedCost(USD)"
+F 5 "TPS22918DBVR" H 3200 1850 12700 0001 C CNN "MPN"
+F 6 "Texas Instruments" H 3200 1850 12700 0001 C CNN "Manufacturer"
 	1    3200 1850
 	1    0    0    -1
@@
 F 4 "SN74LV1T125DBVR " H 2550 5800 60  0001 L CNN "MPN"
 F 5 "Texas Instruments" H 2350 5300 50  0001 C CNN "Manufacturer"
+F 6 "$0.45" H 2350 5300 12700 0001 C CNN "EstimatedCost(USD)"
 	1    2350 5300
 	1    0    0    -1
@@
 F 0 "TP1" V 12505 8038 50  0000 L CNN
 F 1 "TestPoint" V 12595 8038 50  0000 L CNN
-F 2 "" H 12750 7850 50  0001 C CNN
-F 3 "~" H 12750 7850 50  0001 C CNN
+F 2 "TestPoint:TestPoint_Keystone_5000-5004_Miniature" H 12750 7850 50  0001 C CNN
+F 3 "N/A" H 12750 7850 50  0001 C CNN
+F 4 "DNP" H 12550 7850 12700 0001 C CNN "AssemblyOption"
+F 5 "$0.00" H 12550 7850 12700 0001 C CNN "EstimatedCost(USD)"
+F 6 "N/A" H 12550 7850 12700 0001 C CNN "MPN"
+F 7 "N/A" H 12550 7850 12700 0001 C CNN "Manufacturer"
 	1    12550 7850
 	0    1    1    0

Commit message: add BOM scripts, fix schematic hierarchy
Parts:
- removed C76: 47uF, Capacitor_SMD:C_1206_3216Metric_Pad1.42x1.75mm_HandSolder, symbol Device:C
- removed C77: 10nF, Capacitor_SMD:C_0805_2012Metric_Pad1.15x1.40mm_HandSolder, symbol Device:C
- removed R10: 100k, Resistor_SMD:R_0805_2012Metric_Pad1.15x1.40mm_HandSolder, symbol Device:R
- removed R12: 0, Resistor_SMD:R_0805_2012Metric_Pad1.15x1.40mm_HandSolder, symbol Device:R
- removed U2: TPS22918_SOT23-6_A, Package_TO_SOT_SMD:SOT-23-6, symbol OTTOdiy_SMD-library:TPS22918_SOT23-6_A
- C1, C10, C11, C12, C13, C14, C15, C16, C17, C18, C19, C2, C20, C21, C22, C23, C24, C25, C26, C27, C28, C29, C3, C30, C31, C32, C33, C34, C35, C36, C37, C38, C39, C4, C40, C41, C42, C43, C44, C45, C46, C47, C5, C6, C7, C78, C8, C9: EstimatedCost(USD) $0.017724 -> (none); UnitCost(USD) (none) -> $0.017724
- LED1, LED10, LED11, LED12, LED13, LED14, LED15, LED16, LED17, LED18, LED19, LED2, LED20, LED21, LED22, LED23, LED24, LED25, LED26, LED27, LED28, LED29, LED3, LED30, LED31, LED32, LED33, LED34, LED35, LED36, LED37, LED38, LED39, LED4, LED40, LED41, LED42, LED43, LED44, LED45, LED46, LED47, LED5, LED6, LED7, LED8, LED9: EstimatedCost(USD) $0.10303 -> (none); UnitCost(USD) (none) -> $0.10303
- R11, R9: EstimatedCost(USD) $.00169 -> (none); UnitCost(USD) (none) -> $.00169
- R208: EstimatedCost(USD) $.001752 -> (none); UnitCost(USD) (none) -> $.001752
- TP1: EstimatedCost(USD) $0.00 -> (none); UnitCost(USD) (none) -> $0.00
- U1: EstimatedCost(USD) $0.45 -> (none); UnitCost(USD) (none) -> $0.45
Connections:
- net labels removed: +5V_MCU, +5V_REG, LED_PWR_EN
- wire segments 376 -> 356

Commit message: routed buck boost supply
Parts:
- removed TP1: TestPoint, TestPoint:TestPoint_Keystone_5000-5004_Miniature, symbol Connector:TestPoint
- added R27: 100, Resistor_SMD:R_0805_2012Metric_Pad1.15x1.40mm_HandSolder, symbol Device:R
Connections:
- wire segments 356 -> 360
