File: KiCad/LEDS.sch (KiCad schematic (older format))
At the start: 100 parts, among them U1 SN74LV1T125_SOT-23_A

Commit message: Add and route 7 extra buttons/LEDs
Parts:
- added C100, C101, C102, C103, C104, C105, C99: 100nF, Capacitor_SMD:C_0805_2012Metric_Pad1.15x1.40mm_HandSolder, symbol Device:C_Small
- added LED48, LED49, LED50, LED51, LED52, LED53, LED54: WS2812D-5, OTTO_Footprints_Lib:LED_D5.0mm-4, symbol OTTOdiy_SMD-library:NeoPixel_THT-LED
Connections:
- net labels added: LED_CONN3
- wire segments 360 -> 410

Commit message: More JLC part numbers added
Parts:
- removed R9: 100k, Resistor_SMD:R_0805_2012Metric_Pad1.15x1.40mm_HandSolder, symbol Device:R
- C1, C10, C100, C101, C102, C103, C104, C105, C11, C12, C13, C14, C15, C16, C17, C18, C19, C2, C20, C21, C22, C23, C24, C25, C26, C27, C28, C29, C3, C30, C31, C32, C33, C34, C35, C36, C37, C38, C39, C4, C40, C41, C42, C43, C44, C45, C46, C47, C5, C6, C7, C78, C8, C9, C99: JLCASM (none) -> BASIC; LCSC PN (none) -> C49678; MPN CL21B104JBCNNNC -> CC0805KRX7R9BB104; Manufacturer Samsung Electro-Mechanics -> (none); UnitCost(USD) $0.017724 -> Samsung Electro-Mechanics
- LED1, LED10, LED11, LED12, LED13, LED14, LED15, LED16, LED17, LED18, LED19, LED2, LED20, LED21, LED22, LED23, LED24, LED25, LED26, LED27, LED28, LED29, LED3, LED30, LED31, LED32, LED33, LED34, LED35, LED36, LED37, LED38, LED39, LED4, LED40, LED41, LED42, LED43, LED44, LED45, LED46, LED47, LED48, LED49, LED5, LED50, LED51, LED52, LED53, LED54, LED6, LED7, LED8, LED9: JLCASM (none) -> DNP; LCSC PN (none) -> C190565; Manufacturer Worldsemi -> (none); UnitCost(USD) $0.10303 -> Worldsemi
- R11: JLCASM (none) -> BASIC; LCSC PN (none) -> C17407; MPN RC0805FR-07100KL -> 0805W8F1003T5E; Manufacturer Yageo -> (none); UnitCost(USD) $.00169 -> Yageo
- R208: JLCASM (none) -> BASIC; LCSC PN (none) -> C17408; MPN RC0805FR-07100RL -> 0805W8F1000T5E; Manufacturer Yageo -> (none); UnitCost(USD) $.001752 -> Yageo
- R27: AssemblyOption DNP -> (none); JLCASM (none) -> BASIC; LCSC PN (none) -> C17408; MPN RC0805FR-07100RL -> 0805W8F1000T5E; Manufacturer Yageo -> (none); UnitCost(USD) $.001752 -> Yageo
- U1: value SN74LV1T125_SOT-23_A -> SN74LV1T34_SOT-23_A; symbol OTTOdiy_SMD-library:SN74LV1T125_SOT-23_A -> OTTOdiy_SMD-library:SN74LV1T34_SOT-23_A; JLCASM (none) -> EXT; LCSC PN (none) -> C100024; MPN SN74LV1T125DBVR -> SN74LV1T34DBVR; Manufacturer Texas Instruments -> (none); UnitCost(USD) $0.45 -> Texas Instruments
Connections:
- net labels removed: +3V3_MCU, SPI_CS_MCU_LED
- wire segments 410 -> 405

Commit message: Selected all LCSC parts. Check of part numbers complete
Parts:
- C1, C10, C100, C101, C102, C103, C104, C105, C11, C12, C13, C14, C15, C16, C17, C18, C19, C2, C20, C21, C22, C23, C24, C25, C26, C27, C28, C29, C3, C30, C31, C32, C33, C34, C35, C36, C37, C38, C39, C4, C40, C41, C42, C43, C44, C45, C46, C47, C5, C6, C7, C78, C8, C9, C99: UnitCost(USD) Samsung Electro-Mechanics -> (none)
- LED1, LED10, LED11, LED12, LED13, LED14, LED15, LED16, LED17, LED18, LED19, LED2, LED20, LED21, LED22, LED23, LED24, LED25, LED26, LED27, LED28, LED29, LED3, LED30, LED31, LED32, LED33, LED34, LED35, LED36, LED37, LED38, LED39, LED4, LED40, LED41, LED42, LED43, LED44, LED45, LED46, LED47, LED48, LED49, LED5, LED50, LED51, LED52, LED53, LED54, LED6, LED7, LED8, LED9: UnitCost(USD) Worldsemi -> (none)
- R11, R208, R27: UnitCost(USD) Yageo -> (none)
- U1: UnitCost(USD) Texas Instruments -> (none)

Commit message: Finish selecting jlc parts
Parts:
- U1: JLCASM EXT -> EXTDNP
Changed lines of the file:
@@
 F 5 "" H 3050 5300 50  0001 C CNN "Manufacturer"
 F 6 "" H 3050 5300 12700 0001 C CNN "UnitCost(USD)"
-F 7 "EXT" H 3050 5300 50  0001 C CNN "JLCASM"
+F 7 "EXTDNP" H 3050 5300 50  0001 C CNN "JLCASM"
 F 8 "C100024" H 3050 5300 50  0001 C CNN "LCSC PN"
 	1    3050 5300

Commit message: Remove LEDs from main board
Parts:
- removed C1, C10, C100, C101, C102, C103, C104, C105, C11, C12, C13, C14, C15, C16, C17, C18, C19, C2, C20, C21, C22, C23, C24, C25, C26, C27, C28, C29, C3, C30, C31, C32, C33, C34, C35, C36, C37, C38, C39, C4, C40, C41, C42, C43, C44, C45, C46, C47, C5, C6, C7, C8, C9, C99: 100nF, Capacitor_SMD:C_0805_2012Metric_Pad1.15x1.40mm_HandSolder, symbol Device:C_Small
- removed C78: 100nF, Capacitor_SMD:C_0805_2012Metric_Pad1.15x1.40mm_HandSolder, symbol Device:C
- removed LED1, LED10, LED11, LED12, LED13, LED14, LED15, LED16, LED17, LED18, LED19, LED2, LED20, LED21, LED22, LED23, LED24, LED25, LED26, LED27, LED28, LED29, LED3, LED30, LED31, LED32, LED33, LED34, LED35, LED36, LED37, LED38, LED39, LED4, LED40, LED41, LED42, LED43, LED44, LED45, LED46, LED47, LED48, LED49, LED5, LED50, LED51, LED52, LED53, LED54, LED6, LED7, LED8, LED9: WS2812D-5, OTTO_Footprints_Lib:LED_D5.0mm-4, symbol OTTOdiy_SMD-library:NeoPixel_THT-LED
- removed R11: 100k, Resistor_SMD:R_0805_2012Metric_Pad1.15x1.40mm_HandSolder, symbol Device:R
- removed R208, R27: 100, Resistor_SMD:R_0805_2012Metric_Pad1.15x1.40mm_HandSolder, symbol Device:R
- removed U1: SN74LV1T34_SOT-23_A, Package_TO_SOT_SMD:SOT-23-5_HandSoldering, symbol OTTOdiy_SMD-library:SN74LV1T34_SOT-23_A
Connections:
- net labels removed: LED_CONN1, LED_CONN2, LED_CONN3, LED_IN, LED_OUT, SPI_MOSI_MCU_5V
- wire segments 405 -> 5

Commit message: 3d models
Connections:
- net labels removed: +5V_LEDS, GND, SPI_MOSI_MCU
- wire segments 5 -> 0
Changed lines of the file:
@@
 Comment4 ""
 $EndDescr
-Text HLabel 2400 5400 0    50   Input ~ 0
-SPI_MOSI_MCU
-Text GLabel 2900 4250 0    50   Input ~ 0
-+5V_LEDS
-$Comp
-L power:GND #PWR0110
-U 1 1 5E0CC3A4
-P 3050 5800
-F 0 "#PWR0110" H 3050 5550 50  0001 C CNN
-F 1 "GND" H 3055 5627 50  0000 C CNN
-F 2 "" H 3050 5800 50  0001 C CNN
-F 3 "" H 3050 5800 50  0001 C CNN
-	1    3050 5800
-	1    0    0    -1
-$EndComp
-Wire Wire Line
-	3050 5600 3050 5800
-Wire Wire Line
-	3350 4250 3350 4400
-Wire Wire Line
-	2400 5400 2750 5400
 $Bitmap
 Pos 15400 10300
@@
 EndData
 $EndBitmap
-Wire Wire Line
-	6300 10350 8800 10350
-Wire Wire Line
-	2900 4250 3350 4250
 $EndSCHEMATC
