File: KiCad/OTTOdiy_SMD.kicad_pcb (KiCad board)
At the start: 4 copper layers, 297 x 91 mm, 419 parts, among them CN201 1x4 MALE Molex PicoBlade, CN202 1x4 MALE Molex PicoBlade, J1 Conn_ARM_JTAG_SWD_10, J2 Conn_02x04, J201 Raspberry Pi Connector, J202 Conn_02x04, J203 Conn_02x05, J204 Conn_02x05, J205 Conn_02x04, J206 Conn_02x06, J207 Conn_02x03, Q1 AO4485, SW1 ALPS SKHH OR SKPF, SW10 ALPS SKHH OR SKPF, SW11 ALPS SKHH OR SKPF, SW12 ALPS SKHH OR SKPF, SW13 ALPS SKHH OR SKPF, SW14 ALPS SKHH OR SKPF, SW15 ALPS SKHH OR SKPF, SW16 ALPS SKHH OR SKPF, SW17 ALPS SKHH OR SKPF, SW18 ALPS SKHH OR SKPF, SW19 ALPS SKHH OR SKPF, SW2 ALPS SKHH OR SKPF, SW20 ALPS SKHH OR SKPF, SW201 6x6x5mm, SW202 SW_DIP_x02, SW203 6x6x5.85mm (RA), SW21 ALPS SKHH OR SKPF, SW22 ALPS SKHH OR SKPF, SW23 ALPS SKHH OR SKPF, SW24 ALPS SKHH OR SKPF, SW25 ALPS SKHH OR SKPF, SW26 ALPS SKHH OR SKPF, SW27 6x6x13mm, SW28 6x6x13mm, SW29 6x6x13mm, SW3 ALPS SKHH OR SKPF, SW30 6x6x13mm, SW31 6x6x13mm, SW32 6x6x13mm, SW33 6x6x13mm, SW34 6x6x13mm, SW35 6x6x13mm, SW36 6x6x13mm, SW37 6x6x13mm, SW38 6x6x13mm, SW39 6x6x13mm, SW4 ALPS SKHH OR SKPF, SW40 6x6x13mm, SW41 6x6x13mm, SW42 6x6x13mm, SW43 6x6x13mm, SW44 6x6x13mm, SW45 6x6x13mm, SW46 6x6x13mm, SW47 6x6x13mm, SW48 SW_DIP_x02, SW49 SW_SP3T (DP3T Parallel), SW5 ALPS SKHH OR SKPF, SW6 ALPS SKHH OR SKPF, SW7 ALPS SKHH OR SKPF, SW8 ALPS SKHH OR SKPF, SW9 ALPS SKHH OR SKPF, U1 SN74LV1T125_SOT-23_A, U2 TPS22918_SOT23-6_A, U202 STM32F407VGTx, U204 USB6B1, U205 SN74HC14, U206 H11L1S, U207 WM8731, U208 TPS79533, U3 LTC3112_TSSOP20_A, U4 TLV62568_SOT-23-5_A, U5 TPS22918_SOT23-6_A, Y201 8MHz, Y202 32.768kHz, Y203 12.288MHz

Commit message: routed 3v3 and power switches
Parts:
- added D57: RED LED, LED_SMD:LED_0805_2012Metric_Pad1.15x1.40mm_HandSolder, B.Cu at (273.3, 95.2)
- added R28: 330, Resistor_SMD:R_0805_2012Metric_Pad1.15x1.40mm_HandSolder, B.Cu at (278.0, 95.2)
- C76, C77, C79, C81, C84, C86, C87, C88, C93, J1, L2, R10, R12, R16, R17, R18, R19, SW49, U2, U4, U5: moved to B.Cu
- PHOTO201: value VAL** -> ALS-PDIC243-3B
- USB201: value VAL** -> USB_B
- moved U2 206.7 mm to (52.1, 173.2), turned to 270 degrees
- moved R12 200.0 mm to (54.1, 176.3)
- moved R18 197.7 mm to (53.4, 164.6), turned to 180 degrees
- moved C88 196.1 mm to (49.7, 158.8)
- moved C77 193.1 mm to (55.0, 173.3), turned to 90 degrees
- moved R19 186.2 mm to (50.6, 165.4), turned to 270 degrees
- moved L2 185.7 mm to (46.0, 163.6), turned to 90 degrees
- moved R10 183.2 mm to (56.9, 173.3), turned to 270 degrees
- moved C86 181.1 mm to (53.4, 158.8), turned to 180 degrees
- moved U4 176.3 mm to (53.4, 161.7)
- moved C93 175.9 mm to (53.4, 166.4), turned to 180 degrees
- moved C76 159.5 mm to (50.6, 170.1)
- moved C81 154.0 mm to (116.9, 173.6), turned to 180 degrees
- moved C79 150.8 mm to (116.9, 180.8), turned to 180 degrees
- moved C87 150.2 mm to (116.0, 160.3), turned to 270 degrees
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Connections:
- net /MCU/PERIPHERALS/SW1 renamed /MCU/PERIPHERALS/5V_SW1
- net /MCU/PERIPHERALS/SW2 renamed /MCU/PERIPHERALS/5V_SW2
- net Net-(D48-Pad1) renamed /MCU/PERIPHERALS/BARL
- net Net-(L2-Pad1) renamed /MCU/PERIPHERALS/3V3_SW
- U202 pad 44: (no net) -> Net-(R28-Pad1)
Routing:
- net GND: track 42.8 -> 66.2 mm, vias 16 -> 37
- net /MCU/DC_IN: track 6.43 -> 27.7 mm, vias 4 -> 8
- net /MCU/+5V_USB: track 36.9 -> 55.8 mm
- net +5V_REG: track 3.65 -> 21.5 mm, vias 5 -> 17
- net /MCU/BATT_IN: track 5.52 -> 18.2 mm
- net /MCU/PERIPHERALS/3V3_SW: track 0.00 -> 7.46 mm
- net Net-(C93-Pad2): track 0.00 -> 6.95 mm
- net /MCU/BRIGHTNESS: track 0.00 -> 6.35 mm
- net Net-(LED4-Pad1): track 14.2 -> 20.5 mm
- net PI_PWR_EN: track 0.00 -> 5.62 mm
- net /MCU/LED_PWR_EN: track 0.00 -> 5.44 mm
- net Net-(R17-Pad2): track 0.00 -> 4.39 mm
- net Net-(R12-Pad2): track 0.00 -> 4.31 mm
- net +5V_RASPI: track 6.24 -> 9.64 mm, vias 0 -> 4
- net +3V3_MCU: track 32.5 -> 35.5 mm, vias 0 -> 5
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- added copper zone on B.Cu, net +3V3_MCU
- added copper zone on B.Cu, net +5V_RASPI
- added copper zone on F.Cu, net /MCU/DC_IN
- added copper zone on B.Cu, net /MCU/PERIPHERALS/3V3_SW
- added copper zone on B.Cu, net /MCU/PERIPHERALS/BARL
- added copper zone on In2.Cu, net GND
- removed copper zone on F.Cu, net /MCU/BARREL_IN
