File: KicadAUXBoard/OTTO_AUX_SMD.kicad_pcb (KiCad board)
At the start: 2 copper layers, 288.5 x 95 mm, 212 parts, among them J1 Conn_02x05_Odd_Even, J1_KD028QVFMA17 Conn_02x25_Counter_Clockwise, J2 Conn_02x05_Odd_Even, Q1 AO3400A, SW1 ALPS SKHC, SW10 ALPS SKHC, SW11 ALPS SKHC, SW12 ALPS SKHC, SW13 ALPS SKHC, SW14 ALPS SKHC, SW15 ALPS SKHC, SW16 ALPS SKHC, SW17 ALPS SKHC, SW18 ALPS SKHC, SW19 ALPS SKHC, SW2 ALPS SKHC, SW20 ALPS SKHC, SW21 ALPS SKHC, SW22 ALPS SKHC, SW23 ALPS SKHC, SW24 ALPS SKHC, SW25 ALPS SKHC, SW26 ALPS SKHC, SW27 6x6x13mm, SW28 6x6x13mm, SW29 6x6x13mm, SW3 ALPS SKHC, SW30 6x6x13mm, SW31 6x6x13mm, SW32 6x6x13mm, SW33 6x6x13mm, SW34 6x6x13mm, SW35 6x6x13mm, SW36 6x6x13mm, SW37 6x6x13mm, SW38 6x6x13mm, SW39 6x6x13mm, SW4 ALPS SKHC, SW40 6x6x13mm, SW41 6x6x13mm, SW42 6x6x13mm, SW43 6x6x13mm, SW44 6x6x13mm, SW45 6x6x13mm, SW46 6x6x13mm, SW47 6x6x13mm, SW5 ALPS SKHC, SW50 6x6x13mm, SW51 6x6x13mm, SW52 6x6x13mm, SW53 6x6x13mm, SW54 6x6x13mm, SW55 6x6x13mm, SW56 6x6x13mm, SW6 ALPS SKHC, SW7 ALPS SKHC, SW8 ALPS SKHC, SW9 ALPS SKHC, U1 SN74LV1T34_SOT-23_A, U2 TPS22918_SOT23-6_A

Commit message: Add HEX spacers and fix AUX LED pinouts
Parts:
- removed DISPLAY1: 2.8 Inch IPS Display, SPI Interface, OTTO_Footprints_Lib:2.8_INCH_IPS_DISPLAY
- removed FID1, FID7: Fiducial, Fiducial:Fiducial_1mm_Mask2mm
- removed H213: MountingHole_Pad, MountingHole:MountingHole_2.7mm_Pad_Via
- removed J1_KD028QVFMA17: Conn_02x25_Counter_Clockwise, OTTO_Footprints_Lib:F0501-B-50-20T-R
- added G***: otto_logo, OTTO_Footprints_Lib:otto_logo_small, F.Cu at (46.6, 18.5)
- added H3: MountingHole_Pad, OTTO_Footprints_Lib:MountingHoleHole, F.Cu at (35.2, 87.0)
- added H4: MountingHole_Pad, OTTO_Footprints_Lib:MountingHoleHole, F.Cu at (287.2, 87.0)
- added J1_KD028QVFMA017: Conn_02x25_Counter_Clockwise, OTTO_Footprints_Lib:F0501-B-50-20T-R, F.Cu at (145.3, 39.9)
- H1: renamed from H212; footprint MountingHole:MountingHole_2.7mm_Pad_Via -> OTTO_Footprints_Lib:MountingHoleHole
- H2: renamed from H214; footprint MountingHole:MountingHole_2.7mm_Pad_Via -> OTTO_Footprints_Lib:MountingHoleHole
- H5: renamed from H215; footprint MountingHole:MountingHole_2.7mm_Pad_Via -> OTTO_Footprints_Lib:MountingHoleHole
- moved H2 231.1 mm to (276.3, 27.6)
- moved H5 220.0 mm to (161.2, 87.6)
- moved H1 139.6 mm to (30.5, 22.4)
- moved H202 66.0 mm to (161.2, 80.6)
- moved FID12 17.7 mm to (287.2, 93.7)
- moved FID6 17.7 mm to (287.2, 93.7)
- moved H201 15.3 mm to (20.9, 80.0)
- moved H204 15.1 mm to (301.5, 80.6)
- moved C46 7.10 mm to (287.8, 28.7), turned to 315 degrees
- moved H203 3.03 mm to (20.9, 19.1)
- moved R11 1.06 mm to (44.7, 71.9)
- turned LED34 to 45 degrees
- turned LED35 to 45 degrees
- turned LED36 to 45 degrees
- turned LED37 to 45 degrees
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- renumbered H1 to H101, H2 to H102, H3 to H103, H203 to H202, H204 to H203, H202 to H204
Connections:
- LED1 pad 1: Net-(LED1-Pad1) -> +5V_LEDS
- LED1 pad 2: +5V_LEDS -> Net-(LED1-Pad2)
- LED10 pad 1: Net-(LED10-Pad1) -> +5V_LEDS
- LED10 pad 2: +5V_LEDS -> Net-(LED10-Pad2)
- LED11 pad 1: Net-(LED11-Pad1) -> +5V_LEDS
- LED11 pad 2: +5V_LEDS -> Net-(LED11-Pad2)
- LED11 pad 4: Net-(LED10-Pad1) -> Net-(LED10-Pad2)
- LED12 pad 1: Net-(LED12-Pad1) -> +5V_LEDS
- LED12 pad 2: +5V_LEDS -> Net-(LED12-Pad2)
- LED12 pad 4: Net-(LED11-Pad1) -> Net-(LED11-Pad2)
- LED13 pad 1: Net-(LED13-Pad1) -> +5V_LEDS
- LED13 pad 2: +5V_LEDS -> Net-(LED13-Pad2)
- LED13 pad 4: Net-(LED12-Pad1) -> Net-(LED12-Pad2)
- LED14 pad 1: Net-(LED14-Pad1) -> +5V_LEDS
- LED14 pad 2: +5V_LEDS -> Net-(LED14-Pad2)
- LED14 pad 4: Net-(LED13-Pad1) -> Net-(LED13-Pad2)
- LED15 pad 1: Net-(LED15-Pad1) -> +5V_LEDS
- LED15 pad 2: +5V_LEDS -> Net-(LED15-Pad2)
- LED15 pad 4: Net-(LED14-Pad1) -> Net-(LED14-Pad2)
- LED16 pad 1: /LEDs/LED_CONN2 -> +5V_LEDS
- LED16 pad 2: +5V_LEDS -> /LEDs/LED_CONN2
- LED16 pad 4: Net-(LED15-Pad1) -> Net-(LED15-Pad2)
- LED17 pad 1: Net-(LED17-Pad1) -> +5V_LEDS
- LED17 pad 2: +5V_LEDS -> Net-(LED17-Pad2)
- LED18 pad 1: Net-(LED18-Pad1) -> +5V_LEDS
- LED18 pad 2: +5V_LEDS -> Net-(LED18-Pad2)
- LED18 pad 4: Net-(LED17-Pad1) -> Net-(LED17-Pad2)
- LED19 pad 1: Net-(LED19-Pad1) -> +5V_LEDS
- LED19 pad 2: +5V_LEDS -> Net-(LED19-Pad2)
- LED19 pad 4: Net-(LED18-Pad1) -> Net-(LED18-Pad2)
- LED2 pad 1: Net-(LED2-Pad1) -> +5V_LEDS
- LED2 pad 2: +5V_LEDS -> Net-(LED2-Pad2)
- LED2 pad 4: Net-(LED1-Pad1) -> Net-(LED1-Pad2)
- LED20 pad 1: Net-(LED20-Pad1) -> +5V_LEDS
- LED20 pad 2: +5V_LEDS -> Net-(LED20-Pad2)
- LED20 pad 4: Net-(LED19-Pad1) -> Net-(LED19-Pad2)
- LED21 pad 1: Net-(LED21-Pad1) -> +5V_LEDS
- LED21 pad 2: +5V_LEDS -> Net-(LED21-Pad2)
- LED21 pad 4: Net-(LED20-Pad1) -> Net-(LED20-Pad2)
- LED22 pad 1: Net-(LED22-Pad1) -> +5V_LEDS
- LED22 pad 2: +5V_LEDS -> Net-(LED22-Pad2)
- LED22 pad 4: Net-(LED21-Pad1) -> Net-(LED21-Pad2)
- LED23 pad 1: Net-(LED23-Pad1) -> +5V_LEDS
- LED23 pad 2: +5V_LEDS -> Net-(LED23-Pad2)
- LED23 pad 4: Net-(LED22-Pad1) -> Net-(LED22-Pad2)
- LED24 pad 1: Net-(LED24-Pad1) -> +5V_LEDS
- LED24 pad 2: +5V_LEDS -> Net-(LED24-Pad2)
- LED24 pad 4: Net-(LED23-Pad1) -> Net-(LED23-Pad2)
- LED25 pad 1: Net-(LED25-Pad1) -> +5V_LEDS
- LED25 pad 2: +5V_LEDS -> Net-(LED25-Pad2)
- LED25 pad 4: Net-(LED24-Pad1) -> Net-(LED24-Pad2)
- LED26 pad 1: /LEDs/LED_CONN1 -> +5V_LEDS
- LED26 pad 2: +5V_LEDS -> /LEDs/LED_CONN1
- LED26 pad 4: Net-(LED25-Pad1) -> Net-(LED25-Pad2)
- LED27 pad 1: Net-(LED27-Pad1) -> +5V_LEDS
- LED27 pad 2: +5V_LEDS -> Net-(LED27-Pad2)
- LED28 pad 1: Net-(LED28-Pad1) -> +5V_LEDS
- LED28 pad 2: +5V_LEDS -> Net-(LED28-Pad2)
- LED28 pad 4: Net-(LED27-Pad1) -> Net-(LED27-Pad2)
- LED29 pad 1: Net-(LED29-Pad1) -> +5V_LEDS
- LED29 pad 2: +5V_LEDS -> Net-(LED29-Pad2)
- LED29 pad 4: Net-(LED28-Pad1) -> Net-(LED28-Pad2)
- LED3 pad 1: Net-(LED3-Pad1) -> +5V_LEDS
- LED3 pad 2: +5V_LEDS -> Net-(LED3-Pad2)
- LED3 pad 4: Net-(LED2-Pad1) -> Net-(LED2-Pad2)
- LED30 pad 1: Net-(LED30-Pad1) -> +5V_LEDS
- LED30 pad 2: +5V_LEDS -> Net-(LED30-Pad2)
- LED30 pad 4: Net-(LED29-Pad1) -> Net-(LED29-Pad2)
- LED31 pad 1: Net-(LED31-Pad1) -> +5V_LEDS
- LED31 pad 2: +5V_LEDS -> Net-(LED31-Pad2)
- LED31 pad 4: Net-(LED30-Pad1) -> Net-(LED30-Pad2)
- LED32 pad 1: Net-(LED32-Pad1) -> +5V_LEDS
- LED32 pad 2: +5V_LEDS -> Net-(LED32-Pad2)
- LED32 pad 4: Net-(LED31-Pad1) -> Net-(LED31-Pad2)
- LED33 pad 1: Net-(LED33-Pad1) -> +5V_LEDS
- LED33 pad 2: +5V_LEDS -> Net-(LED33-Pad2)
- LED33 pad 4: Net-(LED32-Pad1) -> Net-(LED32-Pad2)
- LED34 pad 1: Net-(LED34-Pad1) -> +5V_LEDS
- LED34 pad 2: +5V_LEDS -> Net-(LED34-Pad2)
- LED35 pad 1: Net-(LED34-Pad4) -> +5V_LEDS
- LED35 pad 2: +5V_LEDS -> Net-(LED34-Pad4)
- LED36 pad 1: Net-(LED35-Pad4) -> +5V_LEDS
- LED36 pad 2: +5V_LEDS -> Net-(LED35-Pad4)
- LED37 pad 1: Net-(LED36-Pad4) -> +5V_LEDS
- LED37 pad 2: +5V_LEDS -> Net-(LED36-Pad4)
- LED38 pad 1: Net-(LED37-Pad4) -> +5V_LEDS
- LED38 pad 2: +5V_LEDS -> Net-(LED37-Pad4)
- LED39 pad 1: Net-(LED38-Pad4) -> +5V_LEDS
- LED39 pad 2: +5V_LEDS -> Net-(LED38-Pad4)
- LED4 pad 1: Net-(LED4-Pad1) -> +5V_LEDS
- LED4 pad 2: +5V_LEDS -> Net-(LED4-Pad2)
- LED4 pad 4: Net-(LED3-Pad1) -> Net-(LED3-Pad2)
- LED40 pad 1: Net-(LED39-Pad4) -> +5V_LEDS
- LED40 pad 2: +5V_LEDS -> Net-(LED39-Pad4)
- LED40 pad 4: Net-(LED33-Pad1) -> Net-(LED33-Pad2)
- LED41 pad 1: Net-(LED41-Pad1) -> +5V_LEDS
- LED41 pad 2: +5V_LEDS -> Net-(LED41-Pad2)
- LED41 pad 4: Net-(LED34-Pad1) -> Net-(LED34-Pad2)
- LED42 pad 1: Net-(LED42-Pad1) -> +5V_LEDS
- LED42 pad 2: +5V_LEDS -> Net-(LED42-Pad2)
- LED42 pad 4: Net-(LED41-Pad1) -> Net-(LED41-Pad2)
- LED43 pad 1: Net-(LED43-Pad1) -> +5V_LEDS
- LED43 pad 2: +5V_LEDS -> Net-(LED43-Pad2)
- LED43 pad 4: Net-(LED42-Pad1) -> Net-(LED42-Pad2)
- LED44 pad 1: Net-(LED44-Pad1) -> +5V_LEDS
- LED44 pad 2: +5V_LEDS -> Net-(LED44-Pad2)
- LED44 pad 4: Net-(LED43-Pad1) -> Net-(LED43-Pad2)
- LED45 pad 1: Net-(LED45-Pad1) -> +5V_LEDS
- LED45 pad 2: +5V_LEDS -> Net-(LED45-Pad2)
- LED45 pad 4: Net-(LED44-Pad1) -> Net-(LED44-Pad2)
- LED46 pad 1: Net-(LED46-Pad1) -> +5V_LEDS
- LED46 pad 2: +5V_LEDS -> Net-(LED46-Pad2)
- LED46 pad 4: Net-(LED45-Pad1) -> Net-(LED45-Pad2)
- LED47 pad 1: /LEDs/LED_CONN3 -> +5V_LEDS
- LED47 pad 2: +5V_LEDS -> /LEDs/LED_CONN3
- LED47 pad 4: Net-(LED46-Pad1) -> Net-(LED46-Pad2)
- LED48 pad 1: Net-(LED48-Pad1) -> +5V_LEDS
- LED48 pad 2: +5V_LEDS -> Net-(LED48-Pad2)
- LED49 pad 1: Net-(LED49-Pad1) -> +5V_LEDS
- LED49 pad 2: +5V_LEDS -> Net-(LED49-Pad2)
- LED49 pad 4: Net-(LED48-Pad1) -> Net-(LED48-Pad2)
- LED5 pad 1: Net-(LED5-Pad1) -> +5V_LEDS
- LED5 pad 2: +5V_LEDS -> Net-(LED5-Pad2)
- LED5 pad 4: Net-(LED4-Pad1) -> Net-(LED4-Pad2)
- LED50 pad 1: Net-(LED50-Pad1) -> +5V_LEDS
- LED50 pad 2: +5V_LEDS -> Net-(LED50-Pad2)
- LED50 pad 4: Net-(LED49-Pad1) -> Net-(LED49-Pad2)
- LED51 pad 1: Net-(LED51-Pad1) -> +5V_LEDS
- LED51 pad 2: +5V_LEDS -> Net-(LED51-Pad2)
- LED51 pad 4: Net-(LED50-Pad1) -> Net-(LED50-Pad2)
- LED52 pad 1: Net-(LED52-Pad1) -> +5V_LEDS
- LED52 pad 2: +5V_LEDS -> Net-(LED52-Pad2)
- LED52 pad 4: Net-(LED51-Pad1) -> Net-(LED51-Pad2)
- LED53 pad 1: Net-(LED53-Pad1) -> +5V_LEDS
- LED53 pad 2: +5V_LEDS -> Net-(LED53-Pad2)
- LED53 pad 4: Net-(LED52-Pad1) -> Net-(LED52-Pad2)
- LED54 pad 1: (no net) -> +5V_LEDS
- LED54 pad 2: +5V_LEDS -> (no net)
- LED54 pad 4: Net-(LED53-Pad1) -> Net-(LED53-Pad2)
- LED6 pad 1: Net-(LED6-Pad1) -> +5V_LEDS
- LED6 pad 2: +5V_LEDS -> Net-(LED6-Pad2)
- LED6 pad 4: Net-(LED5-Pad1) -> Net-(LED5-Pad2)
- LED7 pad 1: Net-(LED7-Pad1) -> +5V_LEDS
- LED7 pad 2: +5V_LEDS -> Net-(LED7-Pad2)
- LED7 pad 4: Net-(LED6-Pad1) -> Net-(LED6-Pad2)
- LED8 pad 1: Net-(LED8-Pad1) -> +5V_LEDS
- LED8 pad 2: +5V_LEDS -> Net-(LED8-Pad2)
- LED8 pad 4: Net-(LED7-Pad1) -> Net-(LED7-Pad2)
- LED9 pad 1: Net-(LED10-Pad4) -> +5V_LEDS
- LED9 pad 2: +5V_LEDS -> Net-(LED10-Pad4)
- LED9 pad 4: Net-(LED8-Pad1) -> Net-(LED8-Pad2)
Routing:
- net +5V_LEDS: track 324.6 -> 1370.7 mm
- net Net-(LED21-Pad1): track 37.7 -> 0.00 mm
- net Net-(LED23-Pad1): track 37.4 -> 0.00 mm
- net Net-(LED23-Pad2): track 0.00 -> 33.6 mm
- net Net-(LED21-Pad2): track 0.00 -> 32.4 mm
- net Net-(LED18-Pad2): track 0.00 -> 32.4 mm
- net Net-(LED18-Pad1): track 31.1 -> 0.00 mm
- net Net-(LED52-Pad2): track 0.00 -> 19.2 mm
- net Net-(LED45-Pad2): track 0.00 -> 19.2 mm
- net Net-(LED31-Pad2): track 0.00 -> 19.2 mm
- net Net-(LED31-Pad1): track 16.0 -> 0.00 mm
- net Net-(LED52-Pad1): track 16.0 -> 0.00 mm
- net Net-(LED45-Pad1): track 16.0 -> 0.00 mm
- net Net-(LED1-Pad2): track 0.00 -> 15.8 mm
- net Net-(LED15-Pad2): track 0.00 -> 15.3 mm
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- removed copper zone on B.Cu, net +5V_LEDS
Other:
- outline, holes or cut-outs redrawn
- board text added: "BLUE"
- board text added: "GREEN"
- board text added: "RED"
- board text added: "To access the SD card, unscrew H1-H5 The two-board assembly can then be lifted out of the case"
- board text added: "YELLOW"

Commit message: v0.1.0 as ordered
Parts:
- LED1, LED10, LED11, LED12, LED13, LED14, LED15, LED16, LED17, LED18, LED19, LED2, LED20, LED21, LED22, LED23, LED24, LED25, LED26, LED27, LED28, LED29, LED3, LED30, LED31, LED32, LED33, LED34, LED35, LED36, LED37, LED38, LED39, LED4, LED40, LED41, LED42, LED43, LED44, LED45, LED46, LED47, LED48, LED49, LED5, LED50, LED51, LED52, LED53, LED54, LED6, LED7, LED8, LED9: value WS2812D-5 -> WS2812B
- Q1: footprint Package_TO_SOT_SMD:SOT-23 -> OTTO_Footprints_Lib:SOT-23
- U1: footprint Package_TO_SOT_SMD:SOT-23-5_HandSoldering -> OTTO_Footprints_Lib:SOT-23-5_HandSoldering
- turned Q1 to 180 degrees
- turned U1 to 270 degrees
- renumbered J1_KD028QVFMA017 to J1_KD028QVFMA17
