File: KicadFrontPanel/OTTO_FrontPanel_SMD.kicad_pcb (KiCad board)
At the start: 2 copper layers, 291.5 x 98.4 mm, 65 parts, among them SW1 ALPS SKHC, SW10 ALPS SKHC, SW11 ALPS SKHC, SW12 ALPS SKHC, SW13 ALPS SKHC, SW14 ALPS SKHC, SW15 ALPS SKHC, SW16 ALPS SKHC, SW17 ALPS SKHC, SW18 ALPS SKHC, SW19 ALPS SKHC, SW2 ALPS SKHC, SW20 ALPS SKHC, SW21 ALPS SKHC, SW22 ALPS SKHC, SW23 ALPS SKHC, SW24 ALPS SKHC, SW25 ALPS SKHC, SW26 ALPS SKHC, SW3 ALPS SKHC, SW32 6x6x13mm, SW33 6x6x13mm, SW38 6x6x13mm, SW4 ALPS SKHC, SW5 ALPS SKHC, SW6 ALPS SKHC, SW7 ALPS SKHC, SW8 ALPS SKHC, SW9 ALPS SKHC

Commit message: Cutouts for mounting frontplate
Added cutouts to AUX board.
Frontplate is now the correct size under the following assumptions:
- 2mm space on left/right side of inner boards to box
- 5 mm space as above on the front side. This is mainly to allow for insertion (the power switch sticks out)
- no space on the back side
Parts:
- added REF**: RightAngle_Small, OTTO_Footprints_Lib:RightAngle_Small, B.Cu at (35.0, 110.1)
- added REF**: RightAngle_Small, OTTO_Footprints_Lib:RightAngle_Small, B.Cu at (106.9, 110.1)
- added REF**: RightAngle_Small, OTTO_Footprints_Lib:RightAngle_Small, B.Cu at (209.4, 10.1)
- added REF**: RightAngle_Small, OTTO_Footprints_Lib:RightAngle_Small, B.Cu at (289.6, 10.1)
- added REF**: RightAngle_Large, OTTO_Footprints_Lib:RightAngle_Large, B.Cu at (50.6, 10.1)
- added REF**: RightAngle_Small, OTTO_Footprints_Lib:RightAngle_Small, B.Cu at (215.4, 110.1)
- added REF**: RightAngle_Small, OTTO_Footprints_Lib:RightAngle_Small, B.Cu at (287.4, 110.1)
- added REF**: RightAngle_Large, OTTO_Footprints_Lib:RightAngle_Large, B.Cu at (114.0, 10.1)
Other:
- board size 291.5 x 98.4 mm -> 294.5 x 102 mm

Commit message: Frontplate changes
Changed icon placement and updated synth, loop, sequencer icons.
Changed dimensions and added mounting brackets to the frontplate.
Parts:
- added ?: MountingHole_2.7mm_M2.5, MountingHole:MountingHole_2.7mm_M2.5, F.Cu at (161.2, 80.6)
- G***: footprint OTTO_Icons_Lib:icons_grid -> OTTO_Icons_Lib:icons_grid_v2
- moved REF** 0.80 mm to (209.4, 9.32)
- moved REF** 0.80 mm to (289.6, 9.32)
- moved REF** 0.80 mm to (50.6, 9.32)
- moved REF** 0.80 mm to (114.0, 9.32)
- moved REF** 0.50 mm to (35.0, 109.6)
- moved REF** 0.50 mm to (106.9, 109.6)
- moved REF** 0.50 mm to (215.4, 109.6)
- moved REF** 0.50 mm to (287.4, 109.6)
Other:
- board size 294.5 x 102 mm -> 294.5 x 102.3 mm

Commit message: Add bracket step files
Parts:
- removed ?: MountingHole_2.7mm_M2.5, MountingHole:MountingHole_2.7mm_M2.5
- removed the REF** at (35.0, 109.6)
- removed the REF** at (106.9, 109.6)
- removed the REF** at (209.4, 9.32)
- removed the REF** at (289.6, 9.32)
- removed the REF** at (50.6, 9.32)
- removed the REF** at (215.4, 109.6)
- removed the REF** at (287.4, 109.6)
- removed the REF** at (114.0, 9.32)
- G***: footprint OTTO_Icons_Lib:icons_grid_v2 -> OTTO_Icons_Lib:icons_grid
Other:
- board size 294.5 x 102.3 mm -> 291.5 x 98.4 mm
