File: KiCad/FrontPanel/OTTO-Beta-Front.kicad_pcb (KiCad board)
At the start: 2 copper layers, 294.5 x 102.3 mm, 71 parts, among them SW1 ALPS SKHC, SW10 ALPS SKHC, SW11 ALPS SKHC, SW12 ALPS SKHC, SW13 ALPS SKHC, SW14 ALPS SKHC, SW15 ALPS SKHC, SW16 ALPS SKHC, SW17 ALPS SKHC, SW18 ALPS SKHC, SW19 ALPS SKHC, SW2 ALPS SKHC, SW20 ALPS SKHC, SW21 ALPS SKHC, SW22 ALPS SKHC, SW23 ALPS SKHC, SW24 ALPS SKHC, SW25 ALPS SKHC, SW26 ALPS SKHC, SW3 ALPS SKHC, SW32 6x6x13mm, SW33 6x6x13mm, SW38 6x6x13mm, SW4 ALPS SKHC, SW5 ALPS SKHC, SW6 ALPS SKHC, SW7 ALPS SKHC, SW8 ALPS SKHC, SW9 ALPS SKHC

Commit message: Front Panel v0.3.0
Other:
- outline, holes or cut-outs redrawn
- board text added: "12-24V DC"
- board text added: "OFF"
- board text added: "ON"
- board text added: "OTTO FRONT v0.3.0"
- board text added: "PHONES"
- board text added: "USB-A"
- board text added: "USB-B"
- board text removed: "HEADPHONES"
- board text removed: "USB"
- board text removed: "v0.3.0 - COPPER"

Commit message: Rearranged front plate icons
Parts:
- G***: footprint OTTO_Icons_Lib:icons_grid_v3 -> OTTO_Icons_Lib:icons_grid_v4
